Commit message: Used scaling principle to get dynamics working for sdf
Former-commit-id: 1b4adcb1a3a012e2516e2c1b22edd9021edb6681 [formerly ceafb9f3e26ec634ef57ff2ba7d2f4182900ed36]
Former-commit-id: a2fe313560f1b4190d81abe279bcef804c640dd7

File: src/soccer_description/models/soccerbot_kinematic/model.urdf (robot description, URDF)
Before this commit: robot soccerbot_noarms, 21 links, 20 joints
Links:
- link head: mass 1 -> 123.765
- link left_ankle: mass 1 -> 457.117
- link left_bicep: mass 1 -> 119.410
- link left_calve: mass 1 -> 110.154
- link left_foot: mass 1 -> 28.542
- link left_forearm: mass 1 -> 41.632
- link left_hip_front: mass 1 -> 136.507
- link left_hip_side: mass 1 -> 8.737
- link left_thigh: mass 1 -> 19.605
- link neck: mass 1 -> 70.031
- link right_ankle: mass 1 -> 457.117
- link right_bicep: mass 1 -> 119.410
- link right_calve: mass 1 -> 110.154
- link right_foot: mass 1 -> 28.542
- link right_forearm: mass 1 -> 41.632
- link right_hip_front: mass 1 -> 136.507
- link right_hip_side: mass 1 -> 8.737
- link right_thigh: mass 1 -> 19.605
- link torso: mass 1.140687 -> 1140.687
Joints:
- joint neck_head: axis 0  0  1 -> 1  0  0
- joint torso_neck: axis 1  0  0 -> 0  1  0
