Commit message: Commit
Former-commit-id: a05318960deb76fca67fa06a4d8d61507c7934ee [formerly f0d38da76a16d8686636f83f6e5aa024ec34ae43]
Former-commit-id: d6be247ed9582bec4f1385229ccf4d381c396ccb

File: src/soccer_description/models/soccerbot v3/model.urdf (robot description, URDF)
Before this commit: robot soccerbot_noarms, 22 links, 21 joints
Links:
- link head: geometry collision box size=0.094 0.09596 0.0712; visual mesh filename=package://soccer_description/meshes/soccerbot v3/Head.stl scale=0.001 0.001 0.001
- link left_ankle: geometry collision box size=0.090769 0.0506 0.042; visual mesh filename=package://soccer_description/meshes/soccerbot v3/Left Ankle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 scale=0.001 0.001 0.001
- link left_bicep: geometry collision box size=0.04 0.103 0.045; visual mesh filename=package://soccer_description/meshes/soccerbot v3/Left Bicep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 scale=0.001 0.001 0.001
- link left_calve: geometry collision box size=0.031883 0.105683 0.048; visual mesh filename=package://soccer_description/meshes/soccerbot v3/Left Calve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 scale=0.001 0.001 0.001
- link left_foot: geometry collision box size=0.09 0.03674 0.07; visual mesh filename=package://soccer_description/meshes/soccerbot v3/Left Foot.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 scale=0.001 0.001 0.001
- link left_forearm: geometry collision box size=0.035 0.124 0.049; visual mesh filename=package://soccer_description/meshes/soccerbot v3/Left Forea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 scale=0.001 0.001 0.001
- link left_hip_front: geometry collision box size=0.083747 0.0506 0.04885; visual mesh filename=package://soccer_description/meshes/soccerbot v3/Left Hip F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 scale=0.001 0.001 0.001
- link left_hip_side: geometry collision box size=0.022 0.039 0.0475; visual mesh filename=package://soccer_description/meshes/soccerbot v3/Left Hip S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 scale=0.001 0.001 0.001
- link left_thigh: geometry collision box size=0.022 0.111 0.048; visual mesh filename=package://soccer_description/meshes/soccerbot v3/Left Thigh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 scale=0.001 0.001 0.001
- link neck: geometry collision box size=0.0523 0.033 0.022; visual mesh filename=package://soccer_description/meshes/soccerbot v3/Neck.stl scale=0.001 0.001 0.001
- link right_ankle: geometry collision box size=0.090769 0.0506 0.042; visual mesh filename=package://soccer_description/meshes/soccerbot v3/Right Ankl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 scale=0.001 0.001 0.001
- link right_bicep: geometry collision box size=0.04 0.103 0.045; visual mesh filename=package://soccer_description/meshes/soccerbot v3/Right Bice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 scale=0.001 0.001 0.001
- link right_calve: geometry collision box size=0.031883 0.105683 0.048; visual mesh filename=package://soccer_description/meshes/soccerbot v3/Right Calv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 scale=0.001 0.001 0.001
- link right_foot: geometry collision box size=0.09 0.03674 0.07; visual mesh filename=package://soccer_description/meshes/soccerbot v3/Right foot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 scale=0.001 0.001 0.001
- link right_forearm: geometry collision box size=0.035 0.124 0.049; visual mesh filename=package://soccer_description/meshes/soccerbot v3/Right Fore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 scale=0.001 0.001 0.001
- link right_hip_front: geometry collision box size=0.083747 0.0506 0.04885; visual mesh filename=package://soccer_description/meshes/soccerbot v3/Right Hip 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 scale=0.001 0.001 0.001
- link right_hip_side: geometry collision box size=0.022 0.039 0.0475; visual mesh filename=package://soccer_description/meshes/soccerbot v3/Right Hip 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 scale=0.001 0.001 0.001
- link right_thigh: geometry collision box size=0.022 0.111 0.048; visual mesh filename=package://soccer_description/meshes/soccerbot v3/Right Thig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 scale=0.001 0.001 0.001
- link torso: geometry collision box size=0.152 0.1 0.145; visual mesh filename=package://soccer_description/meshes/soccerbot v3/Torso.stl scale=0.001 0.001 0.001
