Commit message: Simulation working
Former-commit-id: 6b6d7919dd21ba178b53b5fba50d2215c656bbe9 [formerly b3b7a2e7e229240f07cd7f156e1c9f464743c5cc]
Former-commit-id: 53e0ab3bda044e4111d00e461e9ec127ec5698d2

File: src/soccer_description/models/soccerbot/model.urdf (robot description, URDF)
Before this commit: robot soccerbot, 20 links, 19 joints
Links:
- added link base_link
- link head: geometry collision box size=0.094 0.09596 0.0712; visual mesh filename=package://soccer_description/meshes/Head.stl scale=0.001 0.001 0.001
- link left_ankle: geometry collision box size=0.090769 0.0506 0.042; visual mesh filename=package://soccer_description/meshes/Left Ankle.stl scale=0.001 0.001 0.001
- link left_bicep: geometry collision box size=0.04 0.103 0.045; visual mesh filename=package://soccer_description/meshes/Left Bicep.stl scale=0.001 0.001 0.001
- link left_calve: geometry collision box size=0.031883 0.105683 0.048; visual mesh filename=package://soccer_description/meshes/Left Calve.stl scale=0.001 0.001 0.001
- link left_foot: geometry collision box size=0.09 0.03674 0.07; visual mesh filename=package://soccer_description/meshes/Left Foot.stl scale=0.001 0.001 0.001
- link left_forearm: geometry collision box size=0.035 0.124 0.049; visual mesh filename=package://soccer_description/meshes/Left Forearm.stl scale=0.001 0.001 0.001
- link left_hip_front: geometry collision box size=0.083747 0.0506 0.04885; visual mesh filename=package://soccer_description/meshes/Left Hip Front.stl scale=0.001 0.001 0.001
- link left_hip_side: geometry collision box size=0.022 0.039 0.0475; visual mesh filename=package://soccer_description/meshes/Left Hip Side.stl scale=0.001 0.001 0.001
- link left_thigh: geometry collision box size=0.022 0.111 0.048; visual mesh filename=package://soccer_description/meshes/Left Thigh.stl scale=0.001 0.001 0.001
- link neck: geometry collision box size=0.0523 0.033 0.022; visual mesh filename=package://soccer_description/meshes/Neck.stl scale=0.001 0.001 0.001
- link right_ankle: geometry collision box size=0.090769 0.0506 0.042; visual mesh filename=package://soccer_description/meshes/Right Ankle.stl scale=0.001 0.001 0.001
- link right_bicep: geometry collision box size=0.04 0.103 0.045; visual mesh filename=package://soccer_description/meshes/Right Bicep.stl scale=0.001 0.001 0.001
- link right_calve: geometry collision box size=0.031883 0.105683 0.048; visual mesh filename=package://soccer_description/meshes/Right Calve.stl scale=0.001 0.001 0.001
- link right_foot: geometry collision box size=0.09 0.03674 0.07; visual mesh filename=package://soccer_description/meshes/Right foot.stl scale=0.001 0.001 0.001
- link right_forearm: geometry collision box size=0.035 0.124 0.049; visual mesh filename=package://soccer_description/meshes/Right Forearm.stl scale=0.001 0.001 0.001
- link right_hip_front: geometry collision box size=0.083747 0.0506 0.04885; visual mesh filename=package://soccer_description/meshes/Right Hip Front.stl scale=0.001 0.001 0.001
- link right_hip_side: geometry collision box size=0.022 0.039 0.0475; visual mesh filename=package://soccer_description/meshes/Right Hip Side.stl scale=0.001 0.001 0.001
- link right_thigh: geometry collision box size=0.022 0.111 0.048; visual mesh filename=package://soccer_description/meshes/Right Thigh.stl scale=0.001 0.001 0.001
- link torso: geometry collision box size=0.152 0.1 0.145; visual mesh filename=package://soccer_description/meshes/Torso.stl scale=0.001 0.001 0.001
Joints:
- added joint base_link_torso: type fixed, parent base_link, child torso, origin xyz=0 0 0 rpy=0  0 0, axis 1  0  0
- joint head_camera: origin xyz=0      0.0699  0.1 rpy=2.35619 -1.57079  2.35619 -> xyz=0      0.0699  0.07 rpy=2.35619 -1.57079  2.35619
- joint left_ankle_foot: axis 1  0  0 -> 1 0 0; limit lower=-1.79769e+308 upper=1.79769e+308 effort=-1.0 velocity=-1.0 -> lower=-1.79769e+308 upper=1.79769e+308 effort=30.0 velocity=1.0
- joint left_bicep_forearm: limit lower=-1.79769e+308 upper=1.79769e+308 effort=-1.0 velocity=-1.0 -> lower=-1.79769e+308 upper=1.79769e+308 effort=30.0 velocity=1.0
- joint left_calve_ankle: axis 0.00000000e+00   1.00000000e+00   6.00000000e-05 -> 0 0 1; limit lower=-1.79769e+308 upper=1.79769e+308 effort=-1.0 velocity=-1.0 -> lower=-1.79769e+308 upper=1.79769e+308 effort=30.0 velocity=1.0
- joint left_hip_front_thigh: axis 1  0  0 -> 0  0  1; limit lower=-1.79769e+308 upper=1.79769e+308 effort=-1.0 velocity=-1.0 -> lower=-1.79769e+308 upper=1.79769e+308 effort=30.0 velocity=1.0
- joint left_hip_side_hip_front: axis 0  1  0 -> 1  0  0; limit lower=-1.79769e+308 upper=1.79769e+308 effort=-1.0 velocity=-1.0 -> lower=-1.79769e+308 upper=1.79769e+308 effort=30.0 velocity=1.0
- joint left_thigh_calve: axis 0  1  0 -> 0  0  1; limit lower=-1.79769e+308 upper=1.79769e+308 effort=-1.0 velocity=-1.0 -> lower=-1.79769e+308 upper=1.79769e+308 effort=30.0 velocity=1.0
- joint neck_head: limit lower=-1.79769e+308 upper=1.79769e+308 effort=-1.0 velocity=-1.0 -> lower=-1.79769e+308 upper=1.79769e+308 effort=30.0 velocity=1.0
- joint right_ankle_foot: axis 1  0  0 -> 1 0 0; limit lower=-1.79769e+308 upper=1.79769e+308 effort=-1.0 velocity=-1.0 -> lower=-1.79769e+308 upper=1.79769e+308 effort=30.0 velocity=1.0
- joint right_bicep_forearm: limit lower=-1.79769e+308 upper=1.79769e+308 effort=-1.0 velocity=-1.0 -> lower=-1.79769e+308 upper=1.79769e+308 effort=30.0 velocity=1.0
- joint right_calve_ankle: axis 0.00000000e+00   1.00000000e+00   6.00000000e-05 -> 0 0 1; limit lower=-1.79769e+308 upper=1.79769e+308 effort=-1.0 velocity=-1.0 -> lower=-1.79769e+308 upper=1.79769e+308 effort=30.0 velocity=1.0
- joint right_hip_front_thigh: axis 0  1  0 -> 0  0  1; limit lower=-1.79769e+308 upper=1.79769e+308 effort=-1.0 velocity=-1.0 -> lower=-1.79769e+308 upper=1.79769e+308 effort=30.0 velocity=1.0
- joint right_hip_side_hip_front: limit lower=-1.79769e+308 upper=1.79769e+308 effort=-1.0 velocity=-1.0 -> lower=-1.79769e+308 upper=1.79769e+308 effort=30.0 velocity=1.0
- joint right_thigh_calve: axis 0  1  0 -> 0  0  1; limit lower=-1.79769e+308 upper=1.79769e+308 effort=-1.0 velocity=-1.0 -> lower=-1.79769e+308 upper=1.79769e+308 effort=30.0 velocity=1.0
- joint torso_left_bicep: limit lower=-1.79769e+308 upper=1.79769e+308 effort=-1.0 velocity=-1.0 -> lower=-1.79769e+308 upper=1.79769e+308 effort=30.0 velocity=1.0
- joint torso_left_hip_side: limit lower=-1.79769e+308 upper=1.79769e+308 effort=-1.0 velocity=-1.0 -> lower=-1.79769e+308 upper=1.79769e+308 effort=30.0 velocity=1.0
- joint torso_neck: limit lower=-1.79769e+308 upper=1.79769e+308 effort=-1.0 velocity=-1.0 -> lower=-1.79769e+308 upper=1.79769e+308 effort=30.0 velocity=1.0
- joint torso_right_bicep: axis 0  1  0 -> 0  0  1; limit lower=-1.79769e+308 upper=1.79769e+308 effort=-1.0 velocity=-1.0 -> lower=-1.79769e+308 upper=1.79769e+308 effort=30.0 velocity=1.0
- joint torso_right_hip_side: limit lower=-1.79769e+308 upper=1.79769e+308 effort=-1.0 velocity=-1.0 -> lower=-1.79769e+308 upper=1.79769e+308 effort=30.0 velocity=1.0

File: src/soccer_description/models/soccerbot_noarms/model.urdf (robot description, URDF)
Before this commit: robot soccerbot_noarms, 16 links, 15 joints
Links:
- added link base_link
- link head: geometry collision box size=0.094 0.09596 0.0712; visual mesh filename=package://soccer_description/meshes/Head.stl scale=0.001 0.001 0.001
- link left_ankle: geometry collision box size=0.090769 0.0506 0.042; visual mesh filename=package://soccer_description/meshes/Left Ankle.stl scale=0.001 0.001 0.001
- link left_calve: geometry collision box size=0.031883 0.105683 0.048; visual mesh filename=package://soccer_description/meshes/Left Calve.stl scale=0.001 0.001 0.001
- link left_foot: geometry collision box size=0.09 0.03674 0.07; visual mesh filename=package://soccer_description/meshes/Left Foot.stl scale=0.001 0.001 0.001
- link left_hip_front: geometry collision box size=0.083747 0.0506 0.04885; visual mesh filename=package://soccer_description/meshes/Left Hip Front.stl scale=0.001 0.001 0.001
- link left_hip_side: geometry collision box size=0.022 0.039 0.0475; visual mesh filename=package://soccer_description/meshes/Left Hip Side.stl scale=0.001 0.001 0.001
- link left_thigh: geometry collision box size=0.022 0.111 0.048; visual mesh filename=package://soccer_description/meshes/Left Thigh.stl scale=0.001 0.001 0.001
- link neck: geometry collision box size=0.0523 0.033 0.022; visual mesh filename=package://soccer_description/meshes/Neck.stl scale=0.001 0.001 0.001
- link right_ankle: geometry collision box size=0.090769 0.0506 0.042; visual mesh filename=package://soccer_description/meshes/Right Ankle.stl scale=0.001 0.001 0.001
- link right_calve: geometry collision box size=0.031883 0.105683 0.048; visual mesh filename=package://soccer_description/meshes/Right Calve.stl scale=0.001 0.001 0.001
- link right_foot: geometry collision box size=0.09 0.03674 0.07; visual mesh filename=package://soccer_description/meshes/Right foot.stl scale=0.001 0.001 0.001
- link right_hip_front: geometry collision box size=0.083747 0.0506 0.04885; visual mesh filename=package://soccer_description/meshes/Right Hip Front.stl scale=0.001 0.001 0.001
- link right_hip_side: geometry collision box size=0.022 0.039 0.0475; visual mesh filename=package://soccer_description/meshes/Right Hip Side.stl scale=0.001 0.001 0.001
- link right_thigh: geometry collision box size=0.022 0.111 0.048; visual mesh filename=package://soccer_description/meshes/Right Thigh.stl scale=0.001 0.001 0.001
- link torso: geometry collision box size=0.152 0.1 0.145; visual mesh filename=package://soccer_description/meshes/Torso.stl scale=0.001 0.001 0.001
Joints:
- added joint base_link_torso: type fixed, parent base_link, child torso, origin xyz=0 0 0 rpy=0  0 0, axis 1  0  0
- joint left_ankle_foot: axis 1  0  0 -> 1 0 0; limit lower=-1.79769e+308 upper=1.79769e+308 effort=-1.0 velocity=-1.0 -> lower=-1.79769e+308 upper=1.79769e+308 effort=30.0 velocity=1.0
- joint left_calve_ankle: axis 0.00000000e+00   1.00000000e+00   6.00000000e-05 -> 0 0 1; limit lower=-1.79769e+308 upper=1.79769e+308 effort=-1.0 velocity=-1.0 -> lower=-1.79769e+308 upper=1.79769e+308 effort=30.0 velocity=1.0
- joint left_hip_front_thigh: axis 1  0  0 -> 0  0  1; limit lower=-1.79769e+308 upper=1.79769e+308 effort=-1.0 velocity=-1.0 -> lower=-1.79769e+308 upper=1.79769e+308 effort=30.0 velocity=1.0
- joint left_hip_side_hip_front: axis 0  1  0 -> 1  0  0; limit lower=-1.79769e+308 upper=1.79769e+308 effort=-1.0 velocity=-1.0 -> lower=-1.79769e+308 upper=1.79769e+308 effort=30.0 velocity=1.0
- joint left_thigh_calve: axis 0  1  0 -> 0  0  1; limit lower=-1.79769e+308 upper=1.79769e+308 effort=-1.0 velocity=-1.0 -> lower=-1.79769e+308 upper=1.79769e+308 effort=30.0 velocity=1.0
- joint neck_head: limit lower=-1.79769e+308 upper=1.79769e+308 effort=-1.0 velocity=-1.0 -> lower=-1.79769e+308 upper=1.79769e+308 effort=30.0 velocity=1.0
- joint right_ankle_foot: axis 1  0  0 -> 1 0 0; limit lower=-1.79769e+308 upper=1.79769e+308 effort=-1.0 velocity=-1.0 -> lower=-1.79769e+308 upper=1.79769e+308 effort=30.0 velocity=1.0
- joint right_calve_ankle: axis 0.00000000e+00   1.00000000e+00   6.00000000e-05 -> 0 0 1; limit lower=-1.79769e+308 upper=1.79769e+308 effort=-1.0 velocity=-1.0 -> lower=-1.79769e+308 upper=1.79769e+308 effort=30.0 velocity=1.0
- joint right_hip_front_thigh: axis 0  1  0 -> 0  0  1; limit lower=-1.79769e+308 upper=1.79769e+308 effort=-1.0 velocity=-1.0 -> lower=-1.79769e+308 upper=1.79769e+308 effort=30.0 velocity=1.0
- joint right_hip_side_hip_front: limit lower=-1.79769e+308 upper=1.79769e+308 effort=-1.0 velocity=-1.0 -> lower=-1.79769e+308 upper=1.79769e+308 effort=30.0 velocity=1.0
- joint right_thigh_calve: axis 0  1  0 -> 0  0  1; limit lower=-1.79769e+308 upper=1.79769e+308 effort=-1.0 velocity=-1.0 -> lower=-1.79769e+308 upper=1.79769e+308 effort=30.0 velocity=1.0
- joint torso_left_hip_side: limit lower=-1.79769e+308 upper=1.79769e+308 effort=-1.0 velocity=-1.0 -> lower=-1.79769e+308 upper=1.79769e+308 effort=30.0 velocity=1.0
- joint torso_neck: limit lower=-1.79769e+308 upper=1.79769e+308 effort=-1.0 velocity=-1.0 -> lower=-1.79769e+308 upper=1.79769e+308 effort=30.0 velocity=1.0
- joint torso_right_hip_side: limit lower=-1.79769e+308 upper=1.79769e+308 effort=-1.0 velocity=-1.0 -> lower=-1.79769e+308 upper=1.79769e+308 effort=30.0 velocity=1.0

Commit message: Updates
Former-commit-id: a9abd8eafebccb82132cfa9d81f8421636362af7 [formerly 15f6d6538e1c55496a67e723d584921fb6db03df]
Former-commit-id: 7239b3f839ba97bd0eb1a4d4bebdd63a7459f179

File: src/soccer_description/models/soccerbot/model.urdf (robot description, URDF)
Before this commit: robot soccerbot_noarms, 21 links, 20 joints
Joints:
- joint left_bicep_forearm: axis 0 -1  0 -> 0 0 1
- joint right_bicep_forearm: axis 0  1  0 -> 0 0 1
- joint torso_left_bicep: axis 0 -1  0 -> 0 0 1

Commit message: Changes
Former-commit-id: 9511d18afb3130324c861e6c5171b4617fcca7f9 [formerly 1c11bffaf3af81876013350cb5feac1529e913c0]
Former-commit-id: 3a1c00a72c75d00bd1ecb83036afb0a61dbc87b2

File: src/soccer_description/models/soccerbot/model.urdf (robot description, URDF)
Before this commit: robot soccerbot_noarms, 21 links, 20 joints
Links:
- link torso: mass 1 -> 1.140687

Commit message: Fixed some angles
Former-commit-id: c34ccc5e4cb05a9371b8498cc219f57abb0cf4f8 [formerly 0dc84276c394165a8fded8c88f5def375f329b1c]
Former-commit-id: ff4a7ec69d9a5d890f85e78d8fe7a2dad845c984

File: src/soccer_description/models/soccerbot/model.urdf (robot description, URDF)
Before this commit: robot soccerbot_noarms, 21 links, 20 joints
Links:
- added link world
Joints:
- added joint world_base_link: type fixed, parent world, child base_link, origin xyz=0 0 0 rpy=0  0 0, axis 1  0  0
- joint left_ankle_foot: limit lower=-1.79769e+308 upper=1.79769e+308 effort=30.0 velocity=1.0 -> lower=-1.79769e+308 upper=1.79769e+308 effort=31000.0 velocity=1.0
- joint left_bicep_forearm: limit lower=-1.79769e+308 upper=1.79769e+308 effort=30.0 velocity=1.0 -> lower=-1.79769e+308 upper=1.79769e+308 effort=15000.0 velocity=1.0
- joint left_calve_ankle: limit lower=-1.79769e+308 upper=1.79769e+308 effort=30.0 velocity=1.0 -> lower=-1.79769e+308 upper=1.79769e+308 effort=31000.0 velocity=1.0
- joint left_hip_front_thigh: limit lower=-1.79769e+308 upper=1.79769e+308 effort=30.0 velocity=1.0 -> lower=-1.79769e+308 upper=1.79769e+308 effort=31000.0 velocity=1.0
- joint left_hip_side_hip_front: limit lower=-1.79769e+308 upper=1.79769e+308 effort=30.0 velocity=1.0 -> lower=-1.79769e+308 upper=1.79769e+308 effort=31000.0 velocity=1.0
- joint left_thigh_calve: limit lower=-1.79769e+308 upper=1.79769e+308 effort=30.0 velocity=1.0 -> lower=-1.79769e+308 upper=1.79769e+308 effort=31000.0 velocity=1.0
- joint neck_head: limit lower=-1.79769e+308 upper=1.79769e+308 effort=30.0 velocity=1.0 -> lower=-1.79769e+308 upper=1.79769e+308 effort=15000.0 velocity=1.0
- joint right_ankle_foot: limit lower=-1.79769e+308 upper=1.79769e+308 effort=30.0 velocity=1.0 -> lower=-1.79769e+308 upper=1.79769e+308 effort=31000.0 velocity=1.0
- joint right_bicep_forearm: limit lower=-1.79769e+308 upper=1.79769e+308 effort=30.0 velocity=1.0 -> lower=-1.79769e+308 upper=1.79769e+308 effort=15000.0 velocity=1.0
- joint right_calve_ankle: limit lower=-1.79769e+308 upper=1.79769e+308 effort=30.0 velocity=1.0 -> lower=-1.79769e+308 upper=1.79769e+308 effort=31000.0 velocity=1.0
- joint right_hip_front_thigh: limit lower=-1.79769e+308 upper=1.79769e+308 effort=30.0 velocity=1.0 -> lower=-1.79769e+308 upper=1.79769e+308 effort=31000.0 velocity=1.0
- joint right_hip_side_hip_front: limit lower=-1.79769e+308 upper=1.79769e+308 effort=30.0 velocity=1.0 -> lower=-1.79769e+308 upper=1.79769e+308 effort=31000.0 velocity=1.0
- joint right_thigh_calve: limit lower=-1.79769e+308 upper=1.79769e+308 effort=30.0 velocity=1.0 -> lower=-1.79769e+308 upper=1.79769e+308 effort=31000.0 velocity=1.0
- joint torso_left_bicep: limit lower=-1.79769e+308 upper=1.79769e+308 effort=30.0 velocity=1.0 -> lower=-1.79769e+308 upper=1.79769e+308 effort=15000.0 velocity=1.0
- joint torso_left_hip_side: axis 1  0  0 -> 0  1  0; limit lower=-1.79769e+308 upper=1.79769e+308 effort=30.0 velocity=1.0 -> lower=-1.79769e+308 upper=1.79769e+308 effort=31000.0 velocity=1.0
- joint torso_neck: limit lower=-1.79769e+308 upper=1.79769e+308 effort=30.0 velocity=1.0 -> lower=-1.79769e+308 upper=1.79769e+308 effort=15000.0 velocity=1.0
- joint torso_right_bicep: limit lower=-1.79769e+308 upper=1.79769e+308 effort=30.0 velocity=1.0 -> lower=-1.79769e+308 upper=1.79769e+308 effort=15000.0 velocity=1.0
- joint torso_right_hip_side: axis 1  0  0 -> 0  1  0; limit lower=-1.79769e+308 upper=1.79769e+308 effort=30.0 velocity=1.0 -> lower=-1.79769e+308 upper=1.79769e+308 effort=31000.0 velocity=1.0

Commit message: Added tylers comm
Former-commit-id: 3c869653c4e5b340ed8dade241bcfc1abb5bbd12 [formerly 552cd63d15af503f60cc380e6f56cfec14118ab4]
Former-commit-id: 9e403339490ccbdc22b00439b3f9290b9d8c8387

File: src/soccer_description/models/soccerbot/model.urdf (robot description, URDF)
Before this commit: robot soccerbot_noarms, 22 links, 21 joints
Joints:
- joint left_ankle_foot: axis 1 0 0 -> -1 0 0
- joint left_hip_side_hip_front: axis 1  0  0 -> -1  0  0
- joint right_ankle_foot: axis 1 0 0 -> -1 0 0
- joint right_hip_side_hip_front: axis 1  0  0 -> -1  0  0
- joint torso_left_hip_side: axis 0  1  0 -> 0  -1  0
- joint torso_right_hip_side: axis 0  1  0 -> 0  -1  0

Commit message: Commit

File: src/soccer_description/models/soccerbot/model.urdf (robot description, URDF)
Before this commit: robot soccerbot_noarms, 22 links, 21 joints
Links:
- link head: geometry collision box size=0.094 0.09596 0.0712; visual mesh filename=package://soccer_description/meshes/soccerbot v4/Head.stl scale=0.001 0.001 0.001
- link left_ankle: geometry collision box size=0.090769 0.0506 0.042; visual mesh filename=package://soccer_description/meshes/soccerbot v4/Left Ankle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 scale=0.001 0.001 0.001
- link left_bicep: geometry collision box size=0.04 0.103 0.045; visual mesh filename=package://soccer_description/meshes/soccerbot v4/Left Bicep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 scale=0.001 0.001 0.001
- link left_calve: geometry collision box size=0.031883 0.105683 0.048; visual mesh filename=package://soccer_description/meshes/soccerbot v4/Left Calve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 scale=0.001 0.001 0.001
- link left_foot: geometry collision box size=0.09 0.03674 0.07; visual mesh filename=package://soccer_description/meshes/soccerbot v4/Left Foot.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 scale=0.001 0.001 0.001
- link left_forearm: geometry collision box size=0.035 0.124 0.049; visual mesh filename=package://soccer_description/meshes/soccerbot v4/Left Forea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 scale=0.001 0.001 0.001
- link left_hip_front: geometry collision box size=0.083747 0.0506 0.04885; visual mesh filename=package://soccer_description/meshes/soccerbot v4/Left Hip F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 scale=0.001 0.001 0.001
- link left_hip_side: geometry collision box size=0.022 0.039 0.0475; visual mesh filename=package://soccer_description/meshes/soccerbot v4/Left Hip S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 scale=0.001 0.001 0.001
- link left_thigh: geometry collision box size=0.022 0.111 0.048; visual mesh filename=package://soccer_description/meshes/soccerbot v4/Left Thigh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 scale=0.001 0.001 0.001
- link neck: geometry collision box size=0.0523 0.033 0.022; visual mesh filename=package://soccer_description/meshes/soccerbot v4/Neck.stl scale=0.001 0.001 0.001
- link right_ankle: geometry collision box size=0.090769 0.0506 0.042; visual mesh filename=package://soccer_description/meshes/soccerbot v4/Right Ankl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 scale=0.001 0.001 0.001
- link right_bicep: geometry collision box size=0.04 0.103 0.045; visual mesh filename=package://soccer_description/meshes/soccerbot v4/Right Bice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 scale=0.001 0.001 0.001
- link right_calve: geometry collision box size=0.031883 0.105683 0.048; visual mesh filename=package://soccer_description/meshes/soccerbot v4/Right Calv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 scale=0.001 0.001 0.001
- link right_foot: geometry collision box size=0.09 0.03674 0.07; visual mesh filename=package://soccer_description/meshes/soccerbot v4/Right foot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 scale=0.001 0.001 0.001
- link right_forearm: geometry collision box size=0.035 0.124 0.049; visual mesh filename=package://soccer_description/meshes/soccerbot v4/Right Fore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 scale=0.001 0.001 0.001
- link right_hip_front: geometry collision box size=0.083747 0.0506 0.04885; visual mesh filename=package://soccer_description/meshes/soccerbot v4/Right Hip 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 scale=0.001 0.001 0.001
- link right_hip_side: geometry collision box size=0.022 0.039 0.0475; visual mesh filename=package://soccer_description/meshes/soccerbot v4/Right Hip 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 scale=0.001 0.001 0.001
- link right_thigh: geometry collision box size=0.022 0.111 0.048; visual mesh filename=package://soccer_description/meshes/soccerbot v4/Right Thig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 scale=0.001 0.001 0.001
- link torso: geometry collision box size=0.152 0.1 0.145; visual mesh filename=package://soccer_description/meshes/soccerbot v4/Torso.stl scale=0.001 0.001 0.001
