Commit message: Updated modeL
Former-commit-id: 5b4196fda3ede9160b0e7f0a78a2deb44e97507d [formerly 03a8c0d1611e99e361a13bc08fe9247ba25d57ac]
Former-commit-id: b9186d4c8c85e8bb18054480ca957a989d34da04

File: src/soccer_description/models/soccerbot/model.urdf (robot description, URDF)
Before this commit: robot soccerbot_noarms, 22 links, 21 joints
Links:
- link right_foot: geometry collision box size=0.09 0.03674 0.07; visual mesh filename=package://soccer_description/meshes/soccerbot v4/Right Foot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 scale=0.001 0.001 0.001
- link torso: geometry collision box size=0.152 0.145 0.130; visual mesh filename=package://soccer_description/meshes/soccerbot v4/Torso.stl scale=0.001 0.001 0.001
Joints:
- joint base_link_torso: axis 1  0  0 -> 1 0 0; origin xyz=0 0 0 rpy=0  0 0 -> xyz=0 0 0.3536 rpy=0 0 0
- joint head_camera: origin xyz=0      0.0699  0.07 rpy=2.35619 -1.57079  2.35619 -> xyz=0      0.0699  0.07 rpy=2.35619 -1.57079 2.35619
- joint left_ankle_foot: origin xyz=0  0  0 rpy=0  0  0 -> xyz=0 0 0 rpy=0 0 0
- joint left_bicep_forearm: origin xyz=0   -0.08  0 rpy=0  0  0 -> xyz=0 -0.08 0 rpy=0 0 0
- joint left_calve_ankle: origin xyz=0     -0.0827  0 rpy=-6.00000000e-05   0.00000000e+00   0.00000000e+00 -> xyz=0 -0.0827 0 rpy=0 0 0
- joint left_hip_front_thigh: origin xyz=0  0  0 rpy=1.00000000e-05   0.00000000e+00   0.00000000e+00 -> xyz=0 0 0 rpy=0 0 0
- joint left_hip_side_hip_front: origin xyz=0  0  0 rpy=-2.3562  -1.57079  2.35619 -> xyz=0 0 0 rpy=0 0 0
- joint left_thigh_calve: origin xyz=0      -0.08897  0 rpy=-1.00000000e-05   0.00000000e+00   0.00000000e+00 -> xyz=0 -0.09290  0 rpy=0 0 0
- joint neck_head: axis 1  0  0 -> 1 0 0; origin xyz=0     0.022  0 rpy=1.00000000e-05   1.00000000e-05   0.00000000e+00 -> xyz=0 0.022 0 rpy=0 0 0
- joint right_ankle_foot: origin xyz=0  0  0 rpy=0  0  0 -> xyz=0 0 0 rpy=0 0 0
- joint right_bicep_forearm: origin xyz=0   -0.08  0 rpy=0  0  0 -> xyz=0 -0.08 0 rpy=0 0 0
- joint right_calve_ankle: origin xyz=0     -0.0827  0 rpy=-6.00000000e-05   0.00000000e+00   0.00000000e+00 -> xyz=0 -0.0827 0 rpy=0 0 0
- joint right_hip_front_thigh: axis 0  0  1 -> 0 0 1; origin xyz=0  0  0 rpy=1.00000000e-05   0.00000000e+00   0.00000000e+00 -> xyz=0 0 0 rpy=0 0 0
- joint right_hip_side_hip_front: axis -1  0  0 -> -1 0 0; origin xyz=0  0  0 rpy=-2.3562  -1.57079  2.35619 -> xyz=0 0 0 rpy=0 0 0
- joint right_thigh_calve: axis 0  0  1 -> 0 0 1; origin xyz=0      -0.08897  0 rpy=-1.00000000e-05   0.00000000e+00   0.00000000e+00 -> xyz=0 -0.0929 0 rpy=0 0 0
- joint torso_left_bicep: origin xyz=0      -0.076    0.34767 rpy=1.5708  0      0 -> xyz=0 -0.0775 0 rpy=1.5708 0 0
- joint torso_left_hip_side: origin xyz=0      -0.03149  0.197 rpy=1.5708  0      1.5708 -> xyz=0.0135 -0.035 -0.156 rpy=1.5708 0 1.5708
- joint torso_neck: origin xyz=0       0       0.37391 rpy=1.57079  0       1.57079 -> xyz=0.024 0 0.08275 rpy=1.57079 0 1.57079
- joint torso_right_bicep: origin xyz=0       0.076    0.34767 rpy=1.5708  0      0 -> xyz=0 0.0775 0 rpy=1.5708 0 0
- joint torso_right_hip_side: origin xyz=0       0.03149  0.197 rpy=1.5708  0      1.5708 -> xyz=0.0135 0.035 -0.156 rpy=1.5708 0 1.5708

Commit message: Fixed colliders
Former-commit-id: f4542d55e98c9263510c0efaaa37f62fc3c5c56c [formerly fc1a14055d3a5089735d073ed858da03027a4edc]
Former-commit-id: b2d3f8dc3794a9e5e61bfe202f611306918322c3

File: src/soccer_description/models/soccerbot/model.urdf (robot description, URDF)
Before this commit: robot soccerbot_noarms, 22 links, 21 joints
Links:
- link head: geometry collision box size=0.094 0.0779 0.0712; visual mesh filename=package://soccer_description/meshes/soccerbot v4/Head.stl scale=0.001 0.001 0.001
Joints:
- joint torso_left_bicep: origin xyz=0 -0.0775 0 rpy=1.5708 0 0 -> xyz=0 -0.0725 0 rpy=1.5708 0 0
- joint torso_neck: origin xyz=0.024 0 0.08275 rpy=1.57079 0 1.57079 -> xyz=0.024 0 0.05875 rpy=1.57079 0 1.57079
- joint torso_right_bicep: origin xyz=0 0.0775 0 rpy=1.5708 0 0 -> xyz=0 0.0725 0 rpy=1.5708 0 0

Commit message: Fixed all inertia problems
Former-commit-id: 32af48dbb286c0240f9691036dc6f9fb6c774d99 [formerly 1d0138b85d9ada114948ef3b67ac9c86e99e53c2]
Former-commit-id: 6e640023aa01beb31c070c984bf987cf0a14b8e4

File: src/soccer_description/models/soccerbot/model.urdf (robot description, URDF)
Before this commit: robot soccerbot_noarms, 22 links, 21 joints
Links:
- link head: mass 123.765 -> 282.919
- link left_ankle: mass 457.117 -> 153.186
- link left_bicep: mass 119.410 -> 203.882
- link left_calve: mass 110.154 -> 86.598
- link left_foot: mass 28.542 -> 23.216
- link left_hip_front: mass 136.507 -> 153.238
- link left_hip_side: mass 8.737 -> 9.364
- link left_thigh: mass 19.605 -> 21.438
- link right_ankle: mass 457.117 -> 153.238
- link right_bicep: mass 119.410 -> 203.882
- link right_calve: mass 110.154 -> 86.598
- link right_foot: mass 28.542 -> 23.216
- link right_hip_front: mass 136.507 -> 153.238
- link right_hip_side: mass 8.737 -> 9.364
- link right_thigh: mass 19.605 -> 21.438
- link torso: mass 1140.687 -> 1219.727

Commit message: Added IMU sensor to soccerbot
Former-commit-id: 91dfcd944e1da656413c5e42569bcc91f2908668 [formerly 732ffba5bf6f8d16e7b20dfbc1d766098a7aa873]
Former-commit-id: f4145fedea5cb8f69a241c12490a4d2b482329bb

File: src/soccer_description/models/soccerbot/model.urdf (robot description, URDF)
Before this commit: robot soccerbot_noarms, 22 links, 21 joints
Links:
- removed link world
- added link imu
- link camera: mass 1 -> None
Joints:
- removed joint world_base_link
- added joint torso_imu: type fixed, parent torso, child imu, origin xyz=-0.3095 -0.562  0.001286 rpy=0 0 0, axis 0  0  0, limit lower=0 upper=0 effort=0 velocity=0
- joint head_camera: origin xyz=0      0.0699  0.07 rpy=2.35619 -1.57079 2.35619 -> xyz=0 0.0699  0.07 rpy=0 -1.5708 1.5708
- joint left_ankle_foot: axis -1 0 0 -> 0 0 -1
- joint left_calve_ankle: axis 0 0 1 -> -1 0 0
- joint left_hip_front_thigh: axis 0  0  1 -> -1 0 0
- joint left_hip_side_hip_front: axis -1  0  0 -> 0 0 -1
- joint left_thigh_calve: axis 0  0  1 -> -1 0 0
- joint right_ankle_foot: axis -1 0 0 -> 0 0 -1
- joint right_calve_ankle: axis 0 0 1 -> -1 0 0
- joint right_hip_front_thigh: axis 0 0 1 -> -1 0 0
- joint right_hip_side_hip_front: axis -1 0 0 -> 0 0 -1
- joint right_thigh_calve: axis 0 0 1 -> -1 0 0
- joint torso_left_bicep: origin xyz=0 -0.0725 0 rpy=1.5708 0 0 -> xyz=0.0157 -0.0725 0 rpy=1.5708 0 0
- joint torso_right_bicep: origin xyz=0 0.0725 0 rpy=1.5708 0 0 -> xyz=0.0157 0.0725 0 rpy=1.5708 0 0

Commit message: Done
Former-commit-id: b01bb3f5d7d664f26147dafe87fb7902bcd89620 [formerly b4138f82ddda3e9ac38c11aea395b7a9fcdf8c69]
Former-commit-id: 959d883272d2472253f63a285a398754a525e910

File: src/soccer_description/models/soccerbot/model.urdf (robot description, URDF)
Before this commit: robot soccerbot_noarms, 22 links, 21 joints
Links:
- link left_forearm: geometry collision box size=0.035 0.204 0.049; visual mesh filename=package://soccer_description/meshes/soccerbot v4/Left Forea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 scale=0.001 0.001 0.001
- link right_forearm: geometry collision box size=0.035 0.204 0.049; visual mesh filename=package://soccer_description/meshes/soccerbot v4/Right Fore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 scale=0.001 0.001 0.001
Joints:
- joint head_camera: origin xyz=0 0.0699  0.07 rpy=0 -1.5708 1.5708 -> xyz=0 0.0699  0.07 rpy=0 -1.5708 -1.5708

Commit message: Lots of updates
Former-commit-id: c7ff9bafc18c2f654268884c3e6ce5d9c0e4da4a [formerly 5a3e3d87458d0c71e4a38d45f61f70946d083a3f]
Former-commit-id: f3672215c290f0d693aea64425a7ff32dd71889c

File: src/soccer_description/models/soccerbot/model.urdf (robot description, URDF)
Before this commit: robot soccerbot_noarms, 22 links, 21 joints
Joints:
- joint torso_imu: origin xyz=-0.3095 -0.562  0.001286 rpy=0 0 0 -> xyz=-0.03095 -0.0562  0.001286 rpy=0 0 0; parent torso -> base_link

Commit message: Removed all Icon files
Former-commit-id: 32d3768471f7b2346ebbddd57021ee7d55a8deac [formerly e5d511dce8ee80ce8d343129baaba2962c3b0b8d]
Former-commit-id: 0e80978eec1d75cbf20db76e07c70b3eec02dfd2

File: src/soccer_description/models/soccerbot/model.urdf (robot description, URDF)
Before this commit: robot soccerbot_noarms, 22 links, 21 joints
Joints:
- joint torso_imu: parent base_link -> torso

Commit message: Added things
Former-commit-id: 0aae1ee3ca4b05f65ac23508be2a6bb8b494dbeb [formerly da5019254ec9dba772c789b49286e17fa3972a7c]
Former-commit-id: 554bd4ee467ad9b3e24e2ca9ea99ab5066b91e6f

File: src/soccer_description/models/soccerbot/model.urdf (robot description, URDF)
Before this commit: robot soccerbot_noarms, 22 links, 21 joints
Joints:
- joint torso_imu: origin xyz=-0.3095 -0.562  0.001286 rpy=0 0 0 -> xyz=-0.03095 -0.0562  0.001286 rpy=0 0 0
