Commit message: Fixed all problems
Former-commit-id: 8ad9b81f6d2cc57e3b610d9d7307535b579e736f [formerly 68e0ed4c430758c4c3dedb1b7242e4a87f3f180a]
Former-commit-id: 8c4c29b1f3f826840c8f5b4a125d5810b8fd0ffd

File: omnibot/omnibot_description/models/omnibot/model.xacro (robot description, xacro)
@@ -1,4 +1,6 @@
 <?xml version='1.0'?>
 <robot name="omnibot" xmlns:xacro="http://www.ros.org/wiki/xacro">
+    <xacro:property name="PI" value="3.1415926535897931"/>
+    <xacro:include filename="$(find omnibot_description)/models/omnibot/model.gazebo" />
     <!-- Joint to keep the robot up in midair -->
     <link name="world"/>
@@ -6,5 +8,5 @@
         <parent link="world"/>
         <child link="base_link"/>
-        <origin rpy="0 0 0" xyz="0 0 0"/>
+        <origin rpy="0 0 0" xyz="0 0 1"/>
         <axis xyz="1 0 0"/>
     </joint>
@@ -12,24 +14,36 @@
     <link name="base_link"/>
     <link name="body">
-        <origin rpy="0 0 0" xyz="0 0 0"/>
+        <inertial>
+            <mass value="10"/>
+            <origin rpy="0 0 0" xyz="0 0 0.20"/>
+            <inertia ixx="0.198" ixy="0" ixz="0" iyy="0.198" iyz="0" izz="0.13"/>
+        </inertial>
+        <collision name='collision'>
+            <origin rpy="0 0 0" xyz="0 0 0.22"/>
+            <geometry>
+                <box size="0.25 0.25 0.40"/>
+            </geometry>
+        </collision>
         <visual name="visual">
+            <origin rpy="0 0 0" xyz="0 0 0"/>
             <geometry>
                 <mesh filename="package://omnibot_description/meshes/bodycentre2v6.stl" scale="0.001 0.001 0.001"/>
             </geometry>
         </visual>
-        <collision name='collision'>
-            <geometry>
-                <mesh filename="package://omnibot_description/meshes/bodycentre2v6.stl" scale="0.001 0.001 0.001"/>
-            </geometry>
-        </collision>
     </link>
     <link name="left_front_wheel">
-        <collision name="collision">
+        <inertial>
+            <mass value="1"/>
+            <origin rpy="0 1.57 0" xyz="0 0 0"/>
+            <inertia ixx="0.075" ixy="0" ixz="0" iyy="0.075" iyz="0" izz="0.3"/>
+        </inertial>
+        <collision name='collision'>
+            <origin rpy="0 1.57 0" xyz="0 0 0"/>
             <geometry>
-                <mesh filename="package://omnibot_description/meshes/wheelCentrev1.stl" scale="0.001 0.001 0.001"/>
+                <cylinder radius="0.05" length="0.03" />
             </geometry>
         </collision>
         <visual name="visual">
-            <origin rpy="0 0 0.785398" xyz="-0.15 -0.15 0"/>
+            <origin rpy="0 0 0" xyz="0 0 0"/>
             <geometry>
                 <mesh filename="package://omnibot_description/meshes/wheelCentrev1.stl" scale="0.001 0.001 0.001"/>
@@ -38,11 +52,17 @@
     </link>
     <link name="left_back_wheel">
-        <collision name="collision">
+        <inertial>
+            <mass value="1"/>
+            <origin rpy="0 1.57 0" xyz="0 0 0"/>
+            <inertia ixx="0.075" ixy="0" ixz="0" iyy="0.075" iyz="0" izz="0.3"/>
+        </inertial>
+        <collision name='collision'>
+            <origin rpy="0 1.57 0" xyz="0 0 0"/>
             <geometry>
-                <mesh filename="package://omnibot_description/meshes/wheelCentrev1.stl" scale="0.001 0.001 0.001"/>
+                <cylinder radius="0.05" length="0.03" />
             </geometry>
         </collision>
         <visual name="visual">
-            <origin rpy="0 0 2.35619" xyz="0.15 -0.15 0"/>
+            <origin rpy="0  0 0" xyz="0 0 0"/>
             <geometry>
                 <mesh filename="package://omnibot_description/meshes/wheelCentrev1.stl" scale="0.001 0.001 0.001"/>
@@ -51,11 +71,17 @@
     </link>
     <link name="right_front_wheel">
-        <collision name="collision">
+        <inertial>
+            <mass value="1"/>
+            <origin rpy="0 1.57 0" xyz="0 0 0"/>
+            <inertia ixx="0.075" ixy="0" ixz="0" iyy="0.075" iyz="0" izz="0.3"/>
+        </inertial>
+        <collision name='collision'>
+            <origin rpy="0 1.57 0" xyz="0 0 0"/>
             <geometry>
-                <mesh filename="package://omnibot_description/meshes/wheelCentrev1.stl" scale="0.001 0.001 0.001"/>
+                <cylinder radius="0.05" length="0.03" />
             </geometry>
         </collision>
         <visual name="visual">
-            <origin rpy="0 0 3.92699" xyz="0.15 0.15 0"/>
+            <origin rpy="0 0 0" xyz="0 0 0"/>
             <geometry>
                 <mesh filename="package://omnibot_description/meshes/wheelCentrev1.stl" scale="0.001 0.001 0.001"/>
@@ -64,11 +90,17 @@
     </link>
     <link name="right_back_wheel">
-        <collision name="collision">
+        <inertial>
+            <mass value="1"/>
+            <origin rpy="0 1.57 0" xyz="0 0 0"/>
+            <inertia ixx="0.075" ixy="0" ixz="0" iyy="0.075" iyz="0" izz="0.3"/>
+        </inertial>
+        <collision name='collision'>
+            <origin rpy="0 1.57 0" xyz="0 0 0"/>
             <geometry>
-                <mesh filename="package://omnibot_description/meshes/wheelCentrev1.stl" scale="0.001 0.001 0.001"/>
+                <cylinder radius="0.05" length="0.03" />
             </geometry>
         </collision>
         <visual name="visual">
-            <origin rpy="0 0 5.49779" xyz="-0.15 0.15 0"/>
+            <origin rpy="0 0 0" xyz="0 0 0"/>
             <geometry>
                 <mesh filename="package://omnibot_description/meshes/wheelCentrev1.stl" scale="0.001 0.001 0.001"/>
@@ -81,5 +113,5 @@
         <parent link="base_link"/>
         <child link="body"/>
-        <origin rpy="0  0 0" xyz="0 0 0"/>
+        <origin rpy="0 0 0" xyz="0 0 0"/>
         <axis xyz="1 0 0"/>
     </joint>
@@ -87,33 +119,33 @@
         <child link="left_front_wheel"/>
         <parent link="body"/>
-        <origin rpy="0 0 0" xyz="0 0 0"/>
+        <origin rpy="0 0 0.785398" xyz="-0.15 -0.15 0"/>
         <axis xyz="1 0 0"/>
-        <limit effort="0" lower="0" upper="0" velocity="0"/>
+        <limit effort="100"  lower="-1e10" upper="1e10" velocity="5"/>
     </joint>
     <joint type="revolute" name="right_front_wheel_hinge">
         <child link="right_front_wheel"/>
         <parent link="body"/>
-        <origin rpy="0 0 0" xyz="0 0 0"/>
+        <origin rpy="0 0 3.92699" xyz="0.15 0.15 0"/>
         <axis xyz="1 0 0"/>
-        <limit effort="0" lower="0" upper="0" velocity="0"/>
+        <limit effort="100"  lower="-1e10" upper="1e10" velocity="5"/>
     </joint>
     <joint type="revolute" name="left_back_wheel_hinge">
         <child link="left_back_wheel"/>
         <parent link="body"/>
-        <origin rpy="0  0 0" xyz="0 0 0"/>
+        <origin rpy="0 0 2.35619" xyz="0.15 -0.15 0"/>
         <axis xyz="1 0 0"/>
-        <limit effort="0" lower="0" upper="0" velocity="0"/>
+        <limit effort="100"  lower="-1e10" upper="1e10" velocity="5"/>
     </joint>
     <joint type="revolute" name="right_back_wheel_hinge">
         <child link="right_back_wheel"/>
         <parent link="body"/>
-        <origin rpy="0 0 0" xyz="0 0 0"/>
+        <origin rpy="0 0 5.49779" xyz="-0.15 0.15 0"/>
         <axis xyz="1 0 0"/>
-        <limit effort="0" lower="0" upper="0" velocity="0"/>
+        <limit effort="100"  lower="-1e10" upper="1e10" velocity="5"/>
     </joint>
     <joint name="camera_joint" type="fixed">
-        <origin rpy="0 0 0" xyz="0 0 1"/> <!-- fixme -->
-        <parent>body</parent>
-        <child>camera_link</child>
+        <parent link="base_link" />
+        <child link="camera" />
+        <origin rpy="0 0 1.57" xyz="0 0.12 0.45"/>
     </joint>
     <!-- Transmission -->
@@ -133,5 +165,5 @@
             <hardwareInterface>hardware_interface/EffortJointInterface</hardwareInterface>
         </joint>
-        <actuator name="motor1">
+        <actuator name="motor2">
             <hardwareInterface>hardware_interface/EffortJointInterface</hardwareInterface>
             <mechanicalReduction>1</mechanicalReduction>
@@ -143,5 +175,5 @@
             <hardwareInterface>hardware_interface/EffortJointInterface</hardwareInterface>
         </joint>
-        <actuator name="motor1">
+        <actuator name="motor3">
             <hardwareInterface>hardware_interface/EffortJointInterface</hardwareInterface>
             <mechanicalReduction>1</mechanicalReduction>
@@ -153,5 +185,5 @@
             <hardwareInterface>hardware_interface/EffortJointInterface</hardwareInterface>
         </joint>
-        <actuator name="motor1">
+        <actuator name="motor4">
             <hardwareInterface>hardware_interface/EffortJointInterface</hardwareInterface>
             <mechanicalReduction>1</mechanicalReduction>

Commit message: Tuned a little bit, but still jittering, ok for now
Former-commit-id: 019b5321871ef1d33a69f219cd72b917f56a6acf [formerly 8e8d83e99af436fda283bf03c1381f11ddb482c6]
Former-commit-id: 064537e2331f26ba5de6ac4d6fdd1f84af4aae83

File: omnibot/omnibot_description/models/omnibot/model.xacro (robot description, xacro)
@@ -4,11 +4,11 @@
     <xacro:include filename="$(find omnibot_description)/models/omnibot/model.gazebo" />
     <!-- Joint to keep the robot up in midair -->
-    <link name="world"/>
-    <joint name="world_base_link" type="fixed">
-        <parent link="world"/>
-        <child link="base_link"/>
-        <origin rpy="0 0 0" xyz="0 0 1"/>
-        <axis xyz="1 0 0"/>
-    </joint>
+    <!--<link name="world"/>-->
+    <!--<joint name="world_base_link" type="fixed">-->
+        <!--<parent link="world"/>-->
+        <!--<child link="base_link"/>-->
+        <!--<origin rpy="0 0 0" xyz="0 0 1"/>-->
+        <!--<axis xyz="1 0 0"/>-->
+    <!--</joint>-->
     <!-- Links -->
     <link name="base_link"/>
@@ -121,5 +121,6 @@
         <origin rpy="0 0 0.785398" xyz="-0.15 -0.15 0"/>
         <axis xyz="1 0 0"/>
-        <limit effort="100"  lower="-1e10" upper="1e10" velocity="5"/>
+        <dynamics damping="0.0" friction="30.0" />
+        <limit effort="100"  lower="-1e10" upper="1e10" velocity="1"/>
     </joint>
     <joint type="revolute" name="right_front_wheel_hinge">
@@ -128,5 +129,6 @@
         <origin rpy="0 0 3.92699" xyz="0.15 0.15 0"/>
         <axis xyz="1 0 0"/>
-        <limit effort="100"  lower="-1e10" upper="1e10" velocity="5"/>
+        <dynamics damping="0.0" friction="30.0" />
+        <limit effort="100"  lower="-1e10" upper="1e10" velocity="1"/>
     </joint>
     <joint type="revolute" name="left_back_wheel_hinge">
@@ -135,5 +137,6 @@
         <origin rpy="0 0 2.35619" xyz="0.15 -0.15 0"/>
         <axis xyz="1 0 0"/>
-        <limit effort="100"  lower="-1e10" upper="1e10" velocity="5"/>
+        <dynamics damping="0.0" friction="30.0" />
+        <limit effort="100"  lower="-1e10" upper="1e10" velocity="1"/>
     </joint>
     <joint type="revolute" name="right_back_wheel_hinge">
@@ -142,5 +145,6 @@
         <origin rpy="0 0 5.49779" xyz="-0.15 0.15 0"/>
         <axis xyz="1 0 0"/>
-        <limit effort="100"  lower="-1e10" upper="1e10" velocity="5"/>
+        <dynamics damping="0.0" friction="30.0" />
+        <limit effort="100"  lower="-1e10" upper="1e10" velocity="1"/>
     </joint>
     <joint name="camera_joint" type="fixed">

Commit message: Temp Commit
Former-commit-id: 8a24f582384bc20562213a0330ef9d43f1fc2ff1 [formerly 34f63e7fc3fa54d540057a90523f47a9b0119b28]
Former-commit-id: bf2741a5ef288df1fd612065adc88601074df285

File: omnibot/omnibot_description/models/omnibot/model.xacro (robot description, xacro)
@@ -15,5 +15,5 @@
     <link name="body">
         <inertial>
-            <mass value="10"/>
+            <mass value="8"/>
             <origin rpy="0 0 0" xyz="0 0 0.20"/>
             <inertia ixx="0.198" ixy="0" ixz="0" iyy="0.198" iyz="0" izz="0.13"/>
@@ -28,5 +28,5 @@
             <origin rpy="0 0 0" xyz="0 0 0"/>
             <geometry>
-                <mesh filename="package://omnibot_description/meshes/bodycentre2v6.stl" scale="0.001 0.001 0.001"/>
+                <mesh filename="package://omnibot_description/meshes/body.stl" scale="0.001 0.001 0.001"/>
             </geometry>
         </visual>
@@ -34,5 +34,5 @@
     <link name="left_front_wheel">
         <inertial>
-            <mass value="1"/>
+            <mass value="0.5"/>
             <origin rpy="0 1.57 0" xyz="0 0 0"/>
             <inertia ixx="0.075" ixy="0" ixz="0" iyy="0.075" iyz="0" izz="0.3"/>
@@ -45,7 +45,7 @@
         </collision>
         <visual name="visual">
-            <origin rpy="0 0 0" xyz="0 0 0"/>
+            <origin rpy="0 0 0" xyz="0.05 0 0"/>
             <geometry>
-                <mesh filename="package://omnibot_description/meshes/wheelCentrev1.stl" scale="0.001 0.001 0.001"/>
+                <mesh filename="package://omnibot_description/meshes/wheel.stl" scale="0.001 0.001 0.001"/>
             </geometry>
         </visual>
@@ -53,5 +53,5 @@
     <link name="left_back_wheel">
         <inertial>
-            <mass value="1"/>
+            <mass value="0.5"/>
             <origin rpy="0 1.57 0" xyz="0 0 0"/>
             <inertia ixx="0.075" ixy="0" ixz="0" iyy="0.075" iyz="0" izz="0.3"/>
@@ -64,7 +64,7 @@
         </collision>
         <visual name="visual">
-            <origin rpy="0  0 0" xyz="0 0 0"/>
+            <origin rpy="0  0 0" xyz="0.05 0 0"/>
             <geometry>
-                <mesh filename="package://omnibot_description/meshes/wheelCentrev1.stl" scale="0.001 0.001 0.001"/>
+                <mesh filename="package://omnibot_description/meshes/wheel.stl" scale="0.001 0.001 0.001"/>
             </geometry>
         </visual>
@@ -72,5 +72,5 @@
     <link name="right_front_wheel">
         <inertial>
-            <mass value="1"/>
+            <mass value="0.5"/>
             <origin rpy="0 1.57 0" xyz="0 0 0"/>
             <inertia ixx="0.075" ixy="0" ixz="0" iyy="0.075" iyz="0" izz="0.3"/>
@@ -83,7 +83,7 @@
         </collision>
         <visual name="visual">
-            <origin rpy="0 0 0" xyz="0 0 0"/>
+            <origin rpy="0 0 0" xyz="0.05 0 0"/>
             <geometry>
-                <mesh filename="package://omnibot_description/meshes/wheelCentrev1.stl" scale="0.001 0.001 0.001"/>
+                <mesh filename="package://omnibot_description/meshes/wheel.stl" scale="0.001 0.001 0.001"/>
             </geometry>
         </visual>
@@ -91,5 +91,5 @@
     <link name="right_back_wheel">
         <inertial>
-            <mass value="1"/>
+            <mass value="0.5"/>
             <origin rpy="0 1.57 0" xyz="0 0 0"/>
             <inertia ixx="0.075" ixy="0" ixz="0" iyy="0.075" iyz="0" izz="0.3"/>
@@ -102,7 +102,7 @@
         </collision>
         <visual name="visual">
-            <origin rpy="0 0 0" xyz="0 0 0"/>
+            <origin rpy="0 0 0" xyz="0.05 0 0"/>
             <geometry>
-                <mesh filename="package://omnibot_description/meshes/wheelCentrev1.stl" scale="0.001 0.001 0.001"/>
+                <mesh filename="package://omnibot_description/meshes/wheel.stl" scale="0.001 0.001 0.001"/>
             </geometry>
         </visual>
@@ -121,5 +121,5 @@
         <origin rpy="0 0 0.785398" xyz="-0.15 -0.15 0"/>
         <axis xyz="1 0 0"/>
-        <dynamics damping="0.0" friction="30.0" />
+        <dynamics damping="0.0" friction="40.0" />
         <limit effort="100"  lower="-1e10" upper="1e10" velocity="1"/>
     </joint>
@@ -129,5 +129,5 @@
         <origin rpy="0 0 3.92699" xyz="0.15 0.15 0"/>
         <axis xyz="1 0 0"/>
-        <dynamics damping="0.0" friction="30.0" />
+        <dynamics damping="0.0" friction="40.0" />
         <limit effort="100"  lower="-1e10" upper="1e10" velocity="1"/>
     </joint>
@@ -137,5 +137,5 @@
         <origin rpy="0 0 2.35619" xyz="0.15 -0.15 0"/>
         <axis xyz="1 0 0"/>
-        <dynamics damping="0.0" friction="30.0" />
+        <dynamics damping="0.0" friction="40.0" />
         <limit effort="100"  lower="-1e10" upper="1e10" velocity="1"/>
     </joint>
@@ -145,5 +145,5 @@
         <origin rpy="0 0 5.49779" xyz="-0.15 0.15 0"/>
         <axis xyz="1 0 0"/>
-        <dynamics damping="0.0" friction="30.0" />
+        <dynamics damping="0.0" friction="40.0" />
         <limit effort="100"  lower="-1e10" upper="1e10" velocity="1"/>
     </joint>

Commit message: Added teleop, drive
Former-commit-id: 40cb201be0974d0d3d0a1e1cfdc1cdd131c99e42 [formerly f6f0d89f823554e7b3951088e3a0c8fad061bedd]
Former-commit-id: b79be7c41727e4411eb016617782479f2de50a8b

File: omnibot/omnibot_description/models/omnibot/model.xacro (robot description, xacro)
@@ -4,11 +4,11 @@
     <xacro:include filename="$(find omnibot_description)/models/omnibot/model.gazebo" />
     <!-- Joint to keep the robot up in midair -->
-    <!--<link name="world"/>-->
-    <!--<joint name="world_base_link" type="fixed">-->
-        <!--<parent link="world"/>-->
-        <!--<child link="base_link"/>-->
-        <!--<origin rpy="0 0 0" xyz="0 0 1"/>-->
-        <!--<axis xyz="1 0 0"/>-->
-    <!--</joint>-->
+    <link name="world"/>
+    <joint name="world_base_link" type="fixed">
+        <parent link="world"/>
+        <child link="base_link"/>
+        <origin rpy="0 0 0" xyz="0 0 1"/>
+        <axis xyz="1 0 0"/>
+    </joint>
     <!-- Links -->
     <link name="base_link"/>
@@ -16,5 +16,5 @@
         <inertial>
             <mass value="8"/>
-            <origin rpy="0 0 0" xyz="0 0 0.20"/>
+            <origin rpy="0 0 0" xyz="0 0 0"/>
             <inertia ixx="0.198" ixy="0" ixz="0" iyy="0.198" iyz="0" izz="0.13"/>
         </inertial>
@@ -34,5 +34,5 @@
     <link name="left_front_wheel">
         <inertial>
-            <mass value="0.5"/>
+            <mass value="1"/>
             <origin rpy="0 1.57 0" xyz="0 0 0"/>
             <inertia ixx="0.075" ixy="0" ixz="0" iyy="0.075" iyz="0" izz="0.3"/>
@@ -53,5 +53,5 @@
     <link name="left_back_wheel">
         <inertial>
-            <mass value="0.5"/>
+            <mass value="1"/>
             <origin rpy="0 1.57 0" xyz="0 0 0"/>
             <inertia ixx="0.075" ixy="0" ixz="0" iyy="0.075" iyz="0" izz="0.3"/>
@@ -72,5 +72,5 @@
     <link name="right_front_wheel">
         <inertial>
-            <mass value="0.5"/>
+            <mass value="1"/>
             <origin rpy="0 1.57 0" xyz="0 0 0"/>
             <inertia ixx="0.075" ixy="0" ixz="0" iyy="0.075" iyz="0" izz="0.3"/>
@@ -91,5 +91,5 @@
     <link name="right_back_wheel">
         <inertial>
-            <mass value="0.5"/>
+            <mass value="1"/>
             <origin rpy="0 1.57 0" xyz="0 0 0"/>
             <inertia ixx="0.075" ixy="0" ixz="0" iyy="0.075" iyz="0" izz="0.3"/>
@@ -116,11 +116,11 @@
         <axis xyz="1 0 0"/>
     </joint>
-    <joint type="revolute" name="left_front_wheel_hinge">
-        <child link="left_front_wheel"/>
+    <joint type="revolute" name="left_back_wheel_hinge">
+        <child link="left_back_wheel"/>
         <parent link="body"/>
         <origin rpy="0 0 0.785398" xyz="-0.15 -0.15 0"/>
-        <axis xyz="1 0 0"/>
-        <dynamics damping="0.0" friction="40.0" />
-        <limit effort="100"  lower="-1e10" upper="1e10" velocity="1"/>
+        <axis xyz="-1 0 0"/>
+        <dynamics damping="0.0" friction="10.0" />
+        <limit effort="1000"  lower="-1e10" upper="1e10" velocity="5"/>
     </joint>
     <joint type="revolute" name="right_front_wheel_hinge">
@@ -129,22 +129,22 @@
         <origin rpy="0 0 3.92699" xyz="0.15 0.15 0"/>
         <axis xyz="1 0 0"/>
-        <dynamics damping="0.0" friction="40.0" />
-        <limit effort="100"  lower="-1e10" upper="1e10" velocity="1"/>
-    </joint>
-    <joint type="revolute" name="left_back_wheel_hinge">
-        <child link="left_back_wheel"/>
-        <parent link="body"/>
-        <origin rpy="0 0 2.35619" xyz="0.15 -0.15 0"/>
-        <axis xyz="1 0 0"/>
-        <dynamics damping="0.0" friction="40.0" />
-        <limit effort="100"  lower="-1e10" upper="1e10" velocity="1"/>
+        <dynamics damping="0.0" friction="10.0" />
+        <limit effort="1000"  lower="-1e10" upper="1e10" velocity="5"/>
     </joint>
     <joint type="revolute" name="right_back_wheel_hinge">
         <child link="right_back_wheel"/>
         <parent link="body"/>
+        <origin rpy="0 0 2.35619" xyz="0.15 -0.15 0"/>
+        <axis xyz="1 0 0"/>
+        <dynamics damping="0.0" friction="10.0" />
+        <limit effort="1000"  lower="-1e10" upper="1e10" velocity="5"/>
+    </joint>
+    <joint type="revolute" name="left_front_wheel_hinge">
+        <child link="left_front_wheel"/>
+        <parent link="body"/>
         <origin rpy="0 0 5.49779" xyz="-0.15 0.15 0"/>
-        <axis xyz="1 0 0"/>
-        <dynamics damping="0.0" friction="40.0" />
-        <limit effort="100"  lower="-1e10" upper="1e10" velocity="1"/>
+        <axis xyz="-1 0 0"/>
+        <dynamics damping="0.0" friction="10.0" />
+        <limit effort="1000"  lower="-1e10" upper="1e10" velocity="5"/>
     </joint>
     <joint name="camera_joint" type="fixed">

Commit message: First commit

File: omnibot/omnibot_description/models/omnibot/model.xacro (robot description, xacro)
@@ -3,12 +3,4 @@
     <xacro:property name="PI" value="3.1415926535897931"/>
     <xacro:include filename="$(find omnibot_description)/models/omnibot/model.gazebo" />
-    <!-- Joint to keep the robot up in midair -->
-    <link name="world"/>
-    <joint name="world_base_link" type="fixed">
-        <parent link="world"/>
-        <child link="base_link"/>
-        <origin rpy="0 0 0" xyz="0 0 1"/>
-        <axis xyz="1 0 0"/>
-    </joint>
     <!-- Links -->
     <link name="base_link"/>

Commit message: Fixed
Former-commit-id: c89d4b566a2dc4e9acd4052147ff8e90b8951abb [formerly f3ac6132655a18068b44599e484d04a71b17eaa9]
Former-commit-id: 9ad1cfa8090a389d7500922c2551f63e12ec36ec

File: omnibot/omnibot_description/models/omnibot/model.xacro (robot description, xacro)
@@ -4,11 +4,11 @@
     <xacro:include filename="$(find omnibot_description)/models/omnibot/model.gazebo" />
     <!-- Joint to keep the robot up in midair -->
-    <link name="world"/>
-    <joint name="world_base_link" type="fixed">
-        <parent link="world"/>
-        <child link="base_link"/>
-        <origin rpy="0 0 0" xyz="0 0 1"/>
-        <axis xyz="1 0 0"/>
-    </joint>
+    <!--<link name="world"/>-->
+    <!--<joint name="world_base_link" type="fixed">-->
+        <!--<parent link="world"/>-->
+        <!--<child link="base_link"/>-->
+        <!--<origin rpy="0 0 0" xyz="0 0 1"/>-->
+        <!--<axis xyz="1 0 0"/>-->
+    <!--</joint>-->
     <!-- Links -->
     <link name="base_link"/>
