Commit message: Convetions fixed

File: soccer_description/models/head.xacro (robot description, xacro)
@@ -45,5 +45,5 @@
             </visual>
         </link>
-        <joint name="${origin}_neck" type="revolute">
+        <joint name="head_motor_0" type="revolute">
             <parent link="${origin}"/>
             <child link="neck"/>
@@ -53,5 +53,5 @@
             <limit effort="${AX12_TORQUE}" lower="-${PI/2}" upper="${PI/2}" velocity="${AX12_VELOCITY}"/>
         </joint>
-        <joint name="neck_head" type="revolute">
+        <joint name="head_motor_1" type="revolute">
             <parent link="neck"/>
             <child link="head"/>
@@ -71,10 +71,10 @@
             </actuator>
         </transmission>
-        <transmission name="neck_head">
+        <transmission name="head_motor_1">
             <type>transmission_interface/SimpleTransmission</type>
-            <joint name="neck_head">
+            <joint name="head_motor_1">
                 <hardwareInterface>hardware_interface/EffortJointInterface</hardwareInterface>
             </joint>
-            <actuator name="neck_head">
+            <actuator name="head_motor_1">
                 <hardwareInterface>hardware_interface/EffortJointInterface</hardwareInterface>
                 <mechanicalReduction>1</mechanicalReduction>

File: soccer_description/models/leg.xacro (robot description, xacro)
@@ -134,5 +134,5 @@
             </visual>
         </link>
-        <joint name="torso_${name}_hip_side" type="revolute">
+        <joint name="${name}_leg_motor_0" type="revolute">
             <parent link="torso"/>
             <child link="${name}_hip_side"/>
@@ -142,5 +142,5 @@
             <limit effort="${MX28_TORQUE}" lower="-1.309" upper="0.524" velocity="${MX28_VELOCITY}"/>
         </joint>
-        <joint name="${name}_hip_side_hip_front" type="revolute">
+        <joint name="${name}_leg_motor_1" type="revolute">
             <parent link="${name}_hip_side"/>
             <child link="${name}_hip_front"/>
@@ -155,5 +155,5 @@
             </xacro:if>
         </joint>
-        <joint name="${name}_hip_front_thigh" type="revolute">
+        <joint name="${name}_leg_motor_2" type="revolute">
             <parent link="${name}_hip_front"/>
             <child link="${name}_thigh"/>
@@ -163,5 +163,5 @@
             <limit effort="${MX28_TORQUE}" lower="-${PI/4}" upper="${PI*3/4}" velocity="${MX28_VELOCITY}"/>
         </joint>
-        <joint name="${name}_thigh_calve" type="revolute">
+        <joint name="${name}_leg_motor_3" type="revolute">
             <parent link="${name}_thigh"/>
             <child link="${name}_calve"/>
@@ -171,5 +171,5 @@
             <limit effort="${MX28_TORQUE}" lower="-2.793" upper="0" velocity="${MX28_VELOCITY}"/>
         </joint>
-        <joint name="${name}_calve_ankle" type="revolute">
+        <joint name="${name}_leg_motor_4" type="revolute">
             <parent link="${name}_calve"/>
             <child link="${name}_ankle"/>
@@ -179,5 +179,5 @@
             <limit effort="${MX28_TORQUE}" lower="-${PI/4}" upper="${PI/2}" velocity="${MX28_VELOCITY}"/>
         </joint>
-        <joint name="${name}_ankle_foot" type="revolute">
+        <joint name="${name}_leg_motor_5" type="revolute">
             <parent link="${name}_ankle"/>
             <child link="${name}_foot"/>
@@ -187,60 +187,60 @@
             <limit effort="${MX28_TORQUE}" lower="-${PI/4}" upper="${PI/4}" velocity="${MX28_VELOCITY}"/>
         </joint>
-        <transmission name="torso_${name}_hip_side">
-            <type>transmission_interface/SimpleTransmission</type>
-            <joint name="torso_${name}_hip_side">
-                <hardwareInterface>hardware_interface/EffortJointInterface</hardwareInterface>
-            </joint>
-            <actuator name="torso_${name}_hip_side_motor">
-                <hardwareInterface>hardware_interface/EffortJointInterface</hardwareInterface>
-                <mechanicalReduction>1</mechanicalReduction>
-            </actuator>
-        </transmission>
-        <transmission name="${name}_hip_side_hip_front">
-            <type>transmission_interface/SimpleTransmission</type>
-            <joint name="${name}_hip_side_hip_front">
-                <hardwareInterface>hardware_interface/EffortJointInterface</hardwareInterface>
-            </joint>
-            <actuator name="${name}_hip_side_hip_front_motor">
-                <hardwareInterface>hardware_interface/EffortJointInterface</hardwareInterface>
-                <mechanicalReduction>1</mechanicalReduction>
-            </actuator>
-        </transmission>
-        <transmission name="${name}_hip_front_thigh">
-            <type>transmission_interface/SimpleTransmission</type>
-            <joint name="${name}_hip_front_thigh">
-                <hardwareInterface>hardware_interface/EffortJointInterface</hardwareInterface>
-            </joint>
-            <actuator name="${name}_hip_front_thigh_motor">
-                <hardwareInterface>hardware_interface/EffortJointInterface</hardwareInterface>
-                <mechanicalReduction>1</mechanicalReduction>
-            </actuator>
-        </transmission>
-        <transmission name="${name}_thigh_calve">
-            <type>transmission_interface/SimpleTransmission</type>
-            <joint name="${name}_thigh_calve">
-                <hardwareInterface>hardware_interface/EffortJointInterface</hardwareInterface>
-            </joint>
-            <actuator name="${name}_thigh_calve_motor">
-                <hardwareInterface>hardware_interface/EffortJointInterface</hardwareInterface>
-                <mechanicalReduction>1</mechanicalReduction>
-            </actuator>
-        </transmission>
-        <transmission name="${name}_calve_ankle">
-            <type>transmission_interface/SimpleTransmission</type>
-            <joint name="${name}_calve_ankle">
-                <hardwareInterface>hardware_interface/EffortJointInterface</hardwareInterface>
-            </joint>
-            <actuator name="${name}_calve_ankle_motor">
-                <hardwareInterface>hardware_interface/EffortJointInterface</hardwareInterface>
-                <mechanicalReduction>1</mechanicalReduction>
-            </actuator>
-        </transmission>
-        <transmission name="${name}_ankle_foot">
-            <type>transmission_interface/SimpleTransmission</type>
-            <joint name="${name}_ankle_foot">
-                <hardwareInterface>hardware_interface/EffortJointInterface</hardwareInterface>
-            </joint>
-            <actuator name="${name}_ankle_foot_motor">
+        <transmission name="${name}_leg_motor_0">
+            <type>transmission_interface/SimpleTransmission</type>
+            <joint name="${name}_leg_motor_0">
+                <hardwareInterface>hardware_interface/EffortJointInterface</hardwareInterface>
+            </joint>
+            <actuator name="${name}_leg_motor_0">
+                <hardwareInterface>hardware_interface/EffortJointInterface</hardwareInterface>
+                <mechanicalReduction>1</mechanicalReduction>
+            </actuator>
+        </transmission>
+        <transmission name="${name}_leg_motor_1">
+            <type>transmission_interface/SimpleTransmission</type>
+            <joint name="${name}_leg_motor_1">
+                <hardwareInterface>hardware_interface/EffortJointInterface</hardwareInterface>
+            </joint>
+            <actuator name="${name}_leg_motor_1">
+                <hardwareInterface>hardware_interface/EffortJointInterface</hardwareInterface>
+                <mechanicalReduction>1</mechanicalReduction>
+            </actuator>
+        </transmission>
+        <transmission name="${name}_leg_motor_2">
+            <type>transmission_interface/SimpleTransmission</type>
+            <joint name="${name}_leg_motor_2">
+                <hardwareInterface>hardware_interface/EffortJointInterface</hardwareInterface>
+            </joint>
+            <actuator name="${name}_leg_motor_2">
+                <hardwareInterface>hardware_interface/EffortJointInterface</hardwareInterface>
+                <mechanicalReduction>1</mechanicalReduction>
+            </actuator>
+        </transmission>
+        <transmission name="${name}_leg_motor_3">
+            <type>transmission_interface/SimpleTransmission</type>
+            <joint name="${name}_leg_motor_3">
+                <hardwareInterface>hardware_interface/EffortJointInterface</hardwareInterface>
+            </joint>
+            <actuator name="${name}_leg_motor_3">
+                <hardwareInterface>hardware_interface/EffortJointInterface</hardwareInterface>
+                <mechanicalReduction>1</mechanicalReduction>
+            </actuator>
+        </transmission>
+        <transmission name="${name}_leg_motor_4">
+            <type>transmission_interface/SimpleTransmission</type>
+            <joint name="${name}_leg_motor_4">
+                <hardwareInterface>hardware_interface/EffortJointInterface</hardwareInterface>
+            </joint>
+            <actuator name="${name}_leg_motor_4">
+                <hardwareInterface>hardware_interface/EffortJointInterface</hardwareInterface>
+                <mechanicalReduction>1</mechanicalReduction>
+            </actuator>
+        </transmission>
+        <transmission name="${name}_leg_motor_5">
+            <type>transmission_interface/SimpleTransmission</type>
+            <joint name="${name}_leg_motor_5">
+                <hardwareInterface>hardware_interface/EffortJointInterface</hardwareInterface>
+            </joint>
+            <actuator name="${name}_leg_motor_5">
                 <hardwareInterface>hardware_interface/EffortJointInterface</hardwareInterface>
                 <mechanicalReduction>1</mechanicalReduction>

File: soccer_description/models/soccerbot_stl.urdf (robot description, URDF)
Before this commit: robot soccerbot, 21 links, 20 joints
Joints:
- removed joint left_ankle_foot
- removed joint left_bicep_forearm
- removed joint left_calve_ankle
- removed joint left_hip_front_thigh
- removed joint left_hip_side_hip_front
- removed joint left_thigh_calve
- removed joint neck_head
- removed joint right_ankle_foot
- removed joint right_bicep_forearm
- removed joint right_calve_ankle
- removed joint right_hip_front_thigh
- removed joint right_hip_side_hip_front
- removed joint right_thigh_calve
- removed joint torso_left_bicep
- removed joint torso_left_hip_side
- removed joint torso_neck
- removed joint torso_right_bicep
- removed joint torso_right_hip_side
- added joint head_motor_0: type revolute, parent torso, child neck, origin xyz=0.024 0 0.05875 rpy=0 0 0, axis 0 0 1, limit lower=-1.57079632679 upper=1.57079632679 effort=1.5 velocity=1
- added joint head_motor_1: type revolute, parent neck, child head, origin xyz=0 0 0.024 rpy=0 0 0, axis 0 1 0, limit lower=-2.35619449019 upper=2.35619449019 effort=1.5 velocity=1
- added joint left_arm_motor_0: type revolute, parent torso, child left_bicep, origin xyz=-0.0157 -0.0725 0 rpy=0 0 0, axis 0 -1 0, limit lower=-1.57079632679 upper=3.92699081699 effort=1.5 velocity=1
- added joint left_arm_motor_1: type revolute, parent left_bicep, child left_forearm, origin xyz=0 0 -0.10 rpy=0 0 0, axis 0 -1 0, limit lower=0 upper=3.14159265359 effort=1.5 velocity=1
- added joint left_leg_motor_0: type revolute, parent torso, child left_hip_side, origin xyz=0.0135 -0.035 -0.156 rpy=0 0 0, axis 0 0 1, limit lower=-1.309 upper=0.524 effort=2.5 velocity=1
- added joint left_leg_motor_1: type revolute, parent left_hip_side, child left_hip_front, origin xyz=0 0 0 rpy=0 0 0, axis -1 0 0, limit lower=-1.57079632679 upper=0.785398163397 effort=2.5 velocity=1
- added joint left_leg_motor_2: type revolute, parent left_hip_front, child left_thigh, origin xyz=0 0 0 rpy=0 0 0, axis 0 -1 0, limit lower=-0.785398163397 upper=2.35619449019 effort=2.5 velocity=1
- added joint left_leg_motor_3: type revolute, parent left_thigh, child left_calve, origin xyz=0 0 -0.09290 rpy=0 0 0, axis 0 -1 0, limit lower=-2.793 upper=0 effort=2.5 velocity=1
- added joint left_leg_motor_4: type revolute, parent left_calve, child left_ankle, origin xyz=0 0 -0.0827 rpy=0 0 0, axis 0 -1 0, limit lower=-0.785398163397 upper=1.57079632679 effort=2.5 velocity=1
- added joint left_leg_motor_5: type revolute, parent left_ankle, child left_foot, origin xyz=0 0 0 rpy=0 0 0, axis -1 0 0, limit lower=-0.785398163397 upper=0.785398163397 effort=2.5 velocity=1
- added joint right_arm_motor_0: type revolute, parent torso, child right_bicep, origin xyz=-0.0157 0.0725 0 rpy=0 0 0, axis 0 -1 0, limit lower=-1.57079632679 upper=3.92699081699 effort=1.5 velocity=1
- added joint right_arm_motor_1: type revolute, parent right_bicep, child right_forearm, origin xyz=0 0 -0.10 rpy=0 0 0, axis 0 -1 0, limit lower=0 upper=3.14159265359 effort=1.5 velocity=1
- added joint right_leg_motor_0: type revolute, parent torso, child right_hip_side, origin xyz=0.0135 0.035 -0.156 rpy=0 0 0, axis 0 0 -1, limit lower=-1.309 upper=0.524 effort=2.5 velocity=1
- added joint right_leg_motor_1: type revolute, parent right_hip_side, child right_hip_front, origin xyz=0 0 0 rpy=0 0 0, axis -1 0 0, limit lower=-0.785398163397 upper=1.57079632679 effort=2.5 velocity=1
- added joint right_leg_motor_2: type revolute, parent right_hip_front, child right_thigh, origin xyz=0 0 0 rpy=0 0 0, axis 0 -1 0, limit lower=-0.785398163397 upper=2.35619449019 effort=2.5 velocity=1
- added joint right_leg_motor_3: type revolute, parent right_thigh, child right_calve, origin xyz=0 0 -0.09290 rpy=0 0 0, axis 0 -1 0, limit lower=-2.793 upper=0 effort=2.5 velocity=1
- added joint right_leg_motor_4: type revolute, parent right_calve, child right_ankle, origin xyz=0 0 -0.0827 rpy=0 0 0, axis 0 -1 0, limit lower=-0.785398163397 upper=1.57079632679 effort=2.5 velocity=1
- added joint right_leg_motor_5: type revolute, parent right_ankle, child right_foot, origin xyz=0 0 0 rpy=0 0 0, axis -1 0 0, limit lower=-0.785398163397 upper=0.785398163397 effort=2.5 velocity=1

Commit message: bad commit message name
Former-commit-id: 0193aae67363285a0ed6475e0b7b4d7cc79e7ab2 [formerly f01c4a3a055f35b94dde1d6c22d68fdd73a7d9c2]
Former-commit-id: 61d4e57e9d008a5c8f015b64b15b1aa0906ef930

File: soccer_description/models/head.xacro (robot description, xacro)
@@ -61,10 +61,10 @@
             <limit effort="${AX12_TORQUE}" lower="-${PI*3/4}" upper="${PI*3/4}" velocity="${AX12_VELOCITY}"/>
         </joint>
-        <transmission name="${origin}_neck">
+        <transmission name="head_motor_0">
             <type>transmission_interface/SimpleTransmission</type>
-            <joint name="${origin}_neck">
+            <joint name="head_motor_0">
                 <hardwareInterface>hardware_interface/EffortJointInterface</hardwareInterface>
             </joint>
-            <actuator name="${origin}_neck">
+            <actuator name="head_motor_0">
                 <hardwareInterface>hardware_interface/EffortJointInterface</hardwareInterface>
                 <mechanicalReduction>1</mechanicalReduction>

Commit message: estimate the bounding box location through visual inspection in gazebo, update box size
Former-commit-id: 1fedbc8acaada1f9fb0b682cb8df149337a4580a [formerly 2e99033f3893f0228be88c142a388aad1e17f831]
Former-commit-id: d06cfde69289c3dbbd347a2d80c5e63cff188729

File: soccer_description/models/head.xacro (robot description, xacro)
@@ -32,7 +32,7 @@
             </inertial>
             <collision name="collision">
-                <origin rpy="0  0  0" xyz="0.01735 0 0.01995"/>
+                <origin rpy="0  0  0" xyz="-0.013 0 0.025"/>
                 <geometry>
-                    <box size="0.0712 0.094 0.0839"/>
+                    <box size="0.0712 0.094 0.0779"/>
                 </geometry>
             </collision>
