Commit message: Start
Former-commit-id: 773b3176a9a5c28f6d88726c01c549334a8d2671 [formerly 71434a1737e7c6797e562a5c8ce8e2efc4f76267]
Former-commit-id: fcd40565d6da2e71e2fb969850b304725745305d

File: soccer_description/models/soccerbot_stand.xacro (robot description, xacro)
@@ -3,15 +3,51 @@
     <xacro:include filename="$(find soccer_description)/models/soccerbot.xacro" />
     <!-- Base Link -->
+    <xacro:macro name="foot_support" params="name">
+        <link name="${name}_foot_support">
+            <collision>
+                <origin xyz="0 0 0" rpy="0 0 0"/>
+                <geometry>
+                    <box size="0.40 0.40 0.02"/>
+                </geometry>
+            </collision>
+            <visual>
+                <origin xyz="0 0 0" rpy="0 0 0"/>
+                <geometry>
+                    <box size="0.40 0.40 0.02"/>
+                </geometry>
+                <material name="orange"/>
+            </visual>
+            <inertial>
+                <origin xyz="0 0 0.1" rpy="0 0 0"/>
+                <mass value="1e-3"/>
+                <inertia
+                        ixx="1e-6" ixy="0.0" ixz="0.0"
+                        iyy="1e-6" iyz="0.0"
+                        izz="1e-6"/>
+            </inertial>
+        </link>
+        <gazebo reference="${name}_foot">
+            <material>Gazebo/GreyTransparent</material>
+        </gazebo>
+        <joint name="${name}_foot_support_link" type="fixed">
+            <parent link="${name}_foot"/>
+            <child link="${name}_foot_support"/>
+            <origin rpy="0 0 0" xyz="0 0 ${-0.01474 + 0.01}"/>
+            <axis xyz="1 0 0"/>
+        </joint>
+    </xacro:macro>
+    <foot_support name="left" />
+    <foot_support name="right" />
     <link name="body_support">
         <collision>
-            <origin xyz="0 0 0.1" rpy="0 0 0"/>
+            <origin xyz="0 0 0" rpy="0 0 0"/>
             <geometry>
-                <box size="1 1 0.14"/>
+                <box size="0.20 0.20 0.1"/>
             </geometry>
         </collision>
         <visual>
-            <origin xyz="0 0 0.1" rpy="0 0 0"/>
+            <origin xyz="0 0 0" rpy="0 0 0"/>
             <geometry>
-                <box size="1 1 0.14"/>
+                <box size="0.420 0.40 0.1"/>
             </geometry>
             <material name="orange"/>
@@ -27,7 +63,7 @@
     </link>
     <joint name="body_support_footprint" type="fixed">
-        <parent link="body_support"/>
-        <child link="base_footprint"/>
-        <origin rpy="0 0 0" xyz="0 0 0"/>
+        <parent link="base_footprint"/>
+        <child link="body_support"/>
+        <origin rpy="0 0 0" xyz="0 0 0.09"/>
         <axis xyz="1 0 0"/>
     </joint>

Commit message: I work all the time
Former-commit-id: d0cde1494d36debe1c10fe71f661cdc0a837ea8c [formerly 898590dd815045d98971d9047a6c8342ca472a47]
Former-commit-id: 233c365a43b1210685af651f9713a1e0370e4516

File: soccer_description/models/soccerbot_stand.xacro (robot description, xacro)
@@ -8,5 +8,5 @@
                 <origin xyz="0 0 0" rpy="0 0 0"/>
                 <geometry>
-                    <box size="0.40 0.40 0.02"/>
+                    <cylinder radius="0.2" length="0.05" />
                 </geometry>
             </collision>
@@ -14,5 +14,6 @@
                 <origin xyz="0 0 0" rpy="0 0 0"/>
                 <geometry>
-                    <box size="0.40 0.40 0.02"/>
+                    <cylinder radius="0.2" length="0.05" />
+<!--                    <box size="0.20 0.20 0.05"/>-->
                 </geometry>
                 <material name="orange"/>
@@ -20,9 +21,9 @@
             <inertial>
                 <origin xyz="0 0 0.1" rpy="0 0 0"/>
-                <mass value="1e-3"/>
+                <mass value="0.2"/>
                 <inertia
-                        ixx="1e-6" ixy="0.0" ixz="0.0"
-                        iyy="1e-6" iyz="0.0"
-                        izz="1e-6"/>
+                        ixx="1e-4" ixy="0.0" ixz="0.0"
+                        iyy="1e-4" iyz="0.0"
+                        izz="1e-4"/>
             </inertial>
         </link>
@@ -33,5 +34,5 @@
             <parent link="${name}_foot"/>
             <child link="${name}_foot_support"/>
-            <origin rpy="0 0 0" xyz="0 0 ${-0.01474 + 0.01}"/>
+            <origin rpy="0 0 0" xyz="0 0 ${-0.01474 + 0.025}"/>
             <axis xyz="1 0 0"/>
         </joint>
@@ -39,37 +40,37 @@
     <foot_support name="left" />
     <foot_support name="right" />
-    <link name="body_support">
-        <collision>
-            <origin xyz="0 0 0" rpy="0 0 0"/>
-            <geometry>
-                <box size="0.20 0.20 0.1"/>
-            </geometry>
-        </collision>
-        <visual>
-            <origin xyz="0 0 0" rpy="0 0 0"/>
-            <geometry>
-                <box size="0.420 0.40 0.1"/>
-            </geometry>
-            <material name="orange"/>
-        </visual>
-        <inertial>
-            <origin xyz="0 0 0.1" rpy="0 0 0"/>
-            <mass value="1e-3"/>
-            <inertia
-                    ixx="1e-6" ixy="0.0" ixz="0.0"
-                    iyy="1e-6" iyz="0.0"
-                    izz="1e-6"/>
-        </inertial>
-    </link>
-    <joint name="body_support_footprint" type="fixed">
-        <parent link="base_footprint"/>
-        <child link="body_support"/>
-        <origin rpy="0 0 0" xyz="0 0 0.09"/>
-        <axis xyz="1 0 0"/>
-    </joint>
-    <gazebo reference="body_support">
-        <material>Gazebo/GreyTransparent</material>
-        <mu1>0.0</mu1>
-        <mu2>0.0</mu2>
-    </gazebo>
+<!--    <link name="body_support">-->
+<!--        <collision>-->
+<!--            <origin xyz="0 0 0" rpy="0 0 0"/>-->
+<!--            <geometry>-->
+<!--                <box size="0.20 0.20 0.1"/>-->
+<!--            </geometry>-->
+<!--        </collision>-->
+<!--        <visual>-->
+<!--            <origin xyz="0 0 0" rpy="0 0 0"/>-->
+<!--            <geometry>-->
+<!--                <box size="0.420 0.40 0.1"/>-->
+<!--            </geometry>-->
+<!--            <material name="orange"/>-->
+<!--        </visual>-->
+<!--        <inertial>-->
+<!--            <origin xyz="0 0 0.1" rpy="0 0 0"/>-->
+<!--            <mass value="1e-3"/>-->
+<!--            <inertia-->
+<!--                    ixx="1e-6" ixy="0.0" ixz="0.0"-->
+<!--                    iyy="1e-6" iyz="0.0"-->
+<!--                    izz="1e-6"/>-->
+<!--        </inertial>-->
+<!--    </link>-->
+<!--    <joint name="body_support_footprint" type="fixed">-->
+<!--        <parent link="base_footprint"/>-->
+<!--        <child link="body_support"/>-->
+<!--        <origin rpy="0 0 0" xyz="0 0 0.09"/>-->
+<!--        <axis xyz="1 0 0"/>-->
+<!--    </joint>-->
+<!--    <gazebo reference="body_support">-->
+<!--        <material>Gazebo/GreyTransparent</material>-->
+<!--        <mu1>0.0</mu1>-->
+<!--        <mu2>0.0</mu2>-->
+<!--    </gazebo>-->
 </robot>

Commit message: Fix
Former-commit-id: 3fdfc551d8e5d52d872a800e3a53cf0f552d4278 [formerly 60600fb826c06362182ebff00f3031e87ac45f7c]
Former-commit-id: 7d2aa5b8de94fab975ecb61576435c9cadef132d

File: soccer_description/models/soccerbot_stand.xacro (robot description, xacro)
@@ -40,37 +40,37 @@
     <foot_support name="left" />
     <foot_support name="right" />
-<!--    <link name="body_support">-->
-<!--        <collision>-->
-<!--            <origin xyz="0 0 0" rpy="0 0 0"/>-->
-<!--            <geometry>-->
-<!--                <box size="0.20 0.20 0.1"/>-->
-<!--            </geometry>-->
-<!--        </collision>-->
-<!--        <visual>-->
-<!--            <origin xyz="0 0 0" rpy="0 0 0"/>-->
-<!--            <geometry>-->
-<!--                <box size="0.420 0.40 0.1"/>-->
-<!--            </geometry>-->
-<!--            <material name="orange"/>-->
-<!--        </visual>-->
-<!--        <inertial>-->
-<!--            <origin xyz="0 0 0.1" rpy="0 0 0"/>-->
-<!--            <mass value="1e-3"/>-->
-<!--            <inertia-->
-<!--                    ixx="1e-6" ixy="0.0" ixz="0.0"-->
-<!--                    iyy="1e-6" iyz="0.0"-->
-<!--                    izz="1e-6"/>-->
-<!--        </inertial>-->
-<!--    </link>-->
-<!--    <joint name="body_support_footprint" type="fixed">-->
-<!--        <parent link="base_footprint"/>-->
-<!--        <child link="body_support"/>-->
-<!--        <origin rpy="0 0 0" xyz="0 0 0.09"/>-->
-<!--        <axis xyz="1 0 0"/>-->
-<!--    </joint>-->
-<!--    <gazebo reference="body_support">-->
-<!--        <material>Gazebo/GreyTransparent</material>-->
-<!--        <mu1>0.0</mu1>-->
-<!--        <mu2>0.0</mu2>-->
-<!--    </gazebo>-->
+    <link name="body_support">
+        <collision>
+            <origin xyz="0 0 0" rpy="0 0 0"/>
+            <geometry>
+                <box size="0.20 0.20 0.1"/>
+            </geometry>
+        </collision>
+        <visual>
+            <origin xyz="0 0 0" rpy="0 0 0"/>
+            <geometry>
+                <box size="0.420 0.40 0.1"/>
+            </geometry>
+            <material name="orange"/>
+        </visual>
+        <inertial>
+            <origin xyz="0 0 0.1" rpy="0 0 0"/>
+            <mass value="1e-3"/>
+            <inertia
+                    ixx="1e-6" ixy="0.0" ixz="0.0"
+                    iyy="1e-6" iyz="0.0"
+                    izz="1e-6"/>
+        </inertial>
+    </link>
+    <joint name="body_support_footprint" type="fixed">
+        <parent link="base_footprint"/>
+        <child link="body_support"/>
+        <origin rpy="0 0 0" xyz="0 0 0.09"/>
+        <axis xyz="1 0 0"/>
+    </joint>
+    <gazebo reference="body_support">
+        <material>Gazebo/GreyTransparent</material>
+        <mu1>0.0</mu1>
+        <mu2>0.0</mu2>
+    </gazebo>
 </robot>
