Commit message: Fixed computer off centered bug
Former-commit-id: 7a7ce1b71be8dfc35975c12fa3c9edd81711bf4b [formerly 6966d6a55b7533863c4c561f292902e30807bf2e]
Former-commit-id: 4169e81e3d9eabd9a768a1344ffc85b9f1dc1818

File: soccer_description/models/soccerbot.xacro (robot description, xacro)
@@ -5,4 +5,11 @@
     <soccerbot />
     <link name="base_link" />
+    <link name="world" />
+    <joint name="base_link_map" type="fixed">
+        <parent link="world"/>
+        <child link="base_link"/>
+        <origin rpy="0 0 0" xyz="0 0 0"/>
+        <axis xyz="1 0 0"/>
+    </joint>
     <joint name="base_link_torso" type="fixed">
         <parent link="base_link"/>

Commit message: Stuffs
Former-commit-id: 6998fe938b1f4dc3ae96923d1c8d4fd07b213772 [formerly 900b37b6f6ee2368e7e357d60cbcfdcbab007f04]
Former-commit-id: 435ba595b17cefe682e69d66eef442137e7b301a

File: soccer_description/models/soccerbot.xacro (robot description, xacro)
@@ -1,8 +1,44 @@
 <?xml version="1.0" ?>
 <robot name="soccerbot" xmlns:xacro="http://www.ros.org/wiki/xacro">
+    <xacro:arg name="robot_name" default="/" />
+    <xacro:arg name="MODEL_TYPE" default="dae" />
+    <xacro:arg name="FILE_PATH" default="package://soccer_description" />
+    <xacro:property name="FILE_PATH" value="$(arg FILE_PATH)"/>
+    <xacro:property name="MODEL_TYPE" value="$(arg MODEL_TYPE)"/>
     <xacro:include filename="$(find soccer_description)/models/parameters.xacro" />
-    <xacro:include filename="$(find soccer_description)/models/robot.xacro" />
-    <soccerbot />
+    <xacro:include filename="$(find soccer_description)/models/arm.xacro" />
+    <xacro:include filename="$(find soccer_description)/models/leg.xacro" />
+    <xacro:include filename="$(find soccer_description)/models/head.xacro" />
+    <xacro:include filename="$(find soccer_description)/models/front_camera.xacro" />
+    <xacro:include filename="$(find soccer_description)/models/imu.xacro" />
     <link name="base_footprint" />
+    <link name="torso">
+        <inertial>
+            <mass value="1.529"/>
+            <origin rpy="0 0 0" xyz="0.0082498 -0.0017440 -0.0522479"/>
+            <inertia ixx="4.323e-3" ixy="5.549e-6" ixz="3.960e-5"
+                     iyy="5.198e-3" iyz="-1.509e-5"
+                     izz="3.567e-3"/>
+        </inertial>
+        <collision name="collision">
+            <origin rpy="0 0 0" xyz="0 0 -0.052"/>
+            <geometry>
+                <box size="0.130 0.145 0.152"/>
+            </geometry>
+        </collision>
+        <visual name="visual">
+            <origin rpy="0 0 0" xyz="0 0 0"/>
+            <geometry>
+                <mesh filename="${FILE_PATH}/meshes/torso.${MODEL_TYPE}" scale="1 1 1"/>
+            </geometry>
+        </visual>
+    </link>
+    <arm name="left" origin="torso" direction="1" />
+    <arm name="right" origin="torso" direction="-1" />
+    <leg name="left" origin="torso" direction="1" />
+    <leg name="right" origin="torso" direction="-1" />
+    <head origin="torso" />
+    <imu origin="torso" />
+    <front_camera origin="head" />
     <joint name="base_footprint_torso" type="fixed">
         <parent link="base_footprint"/>
@@ -11,4 +47,16 @@
         <axis xyz="1 0 0"/>
     </joint>
+    <gazebo>
+        <plugin name="gazebo_ros_control" filename="libgazebo_ros_control.so">
+            <robotNamespace>$(arg robot_name)</robotNamespace>
+            <robotSimType>gazebo_ros_control/DefaultRobotHWSim</robotSimType>
+        </plugin>
+    </gazebo>
+    <gazebo reference="torso">
+        <kp>${JOINT_KP}</kp>
+        <kd>${JOINT_KD}</kd>
+        <mu1>${JOINT_MU1}</mu1>
+        <mu2>${JOINT_MU2}</mu2>
+    </gazebo>
     <gazebo reference="base_footprint">
         <kp>${JOINT_KP}</kp>

Commit message: Fixed matlab difference
Former-commit-id: 1b262e52e5a4f1fa45ee5d4350c220ece02e31e9 [formerly 503d25d4e88489abdae1cf5eeb494e7a6db39401]
Former-commit-id: 76572b2d3dc7212a7723da3ab08a8b1df08634ab

File: soccer_description/models/soccerbot.xacro (robot description, xacro)
@@ -2,6 +2,7 @@
 <robot name="soccerbot" xmlns:xacro="http://www.ros.org/wiki/xacro">
     <xacro:arg name="robot_name" default="/" />
-    <xacro:arg name="MODEL_TYPE" default="dae" />
-    <xacro:arg name="FILE_PATH" default="package://soccer_description" />
+    <xacro:arg name="MODEL_TYPE" default="stl" />
+    <xacro:arg name="FILE_PATH" default="../soccer_description" />
+    <xacro:arg name="has_base_footprint" default="false" />
     <xacro:property name="FILE_PATH" value="$(arg FILE_PATH)"/>
     <xacro:property name="MODEL_TYPE" value="$(arg MODEL_TYPE)"/>
@@ -12,5 +13,4 @@
     <xacro:include filename="$(find soccer_description)/models/front_camera.xacro" />
     <xacro:include filename="$(find soccer_description)/models/imu.xacro" />
-    <link name="base_footprint" />
     <link name="torso">
         <inertial>
@@ -41,10 +41,19 @@
     <imu origin="torso" />
     <front_camera origin="head" />
-    <joint name="base_footprint_torso" type="fixed">
-        <parent link="base_footprint"/>
-        <child link="torso"/>
-        <origin rpy="0 0 0" xyz="0 0 0.3536"/>
-        <axis xyz="1 0 0"/>
-    </joint>
+    <xacro:if value="$(arg has_base_footprint)">
+        <link name="base_footprint" />
+        <joint name="base_footprint_torso" type="fixed">
+            <parent link="base_footprint"/>
+            <child link="torso"/>
+            <origin rpy="0 0 0" xyz="0 0 0.3536"/>
+            <axis xyz="1 0 0"/>
+        </joint>
+        <gazebo reference="base_footprint">
+            <kp>${JOINT_KP}</kp>
+            <kd>${JOINT_KD}</kd>
+            <mu1>${JOINT_MU1}</mu1>
+            <mu2>${JOINT_MU2}</mu2>
+        </gazebo>
+    </xacro:if>
     <gazebo>
         <plugin name="gazebo_ros_control" filename="libgazebo_ros_control.so">
@@ -59,9 +68,3 @@
         <mu2>${JOINT_MU2}</mu2>
     </gazebo>
-    <gazebo reference="base_footprint">
-        <kp>${JOINT_KP}</kp>
-        <kd>${JOINT_KD}</kd>
-        <mu1>${JOINT_MU1}</mu1>
-        <mu2>${JOINT_MU2}</mu2>
-    </gazebo>
 </robot>

Commit message: Fixed stuff
Former-commit-id: a4d524621bb8afd23d1318bef8eb200089ba1823 [formerly aedd73ef40c914dc92424dc1b2c4071ae064e85e]
Former-commit-id: 9be2db8aac326f6b3a8800daa2d0b5f57f4b03d1

File: soccer_description/models/soccerbot.xacro (robot description, xacro)
@@ -2,9 +2,9 @@
 <robot name="soccerbot" xmlns:xacro="http://www.ros.org/wiki/xacro">
     <xacro:arg name="robot_name" default="/" />
-    <xacro:arg name="MODEL_TYPE" default="stl" />
-    <xacro:arg name="FILE_PATH" default="../soccer_description" />
+    <xacro:arg name="model_type" default="stl" />
+    <xacro:arg name="file_path" default="../soccer_description" />
     <xacro:arg name="has_base_footprint" default="false" />
-    <xacro:property name="FILE_PATH" value="$(arg FILE_PATH)"/>
-    <xacro:property name="MODEL_TYPE" value="$(arg MODEL_TYPE)"/>
+    <xacro:property name="FILE_PATH" value="$(arg file_path)"/>
+    <xacro:property name="MODEL_TYPE" value="$(arg model_type)"/>
     <xacro:include filename="$(find soccer_description)/models/parameters.xacro" />
     <xacro:include filename="$(find soccer_description)/models/arm.xacro" />

Commit message: Start
Former-commit-id: 3187801847c3fd0655420361ce9a7f5cd6c7205c [formerly 3432f5e20b4c68459c60491a1fe6e8ad08d8e88f]
Former-commit-id: ed4302daf74743daa7fb8ef692d5708880cc6279

File: soccer_description/models/soccerbot.xacro (robot description, xacro)
@@ -2,5 +2,5 @@
 <robot name="soccerbot" xmlns:xacro="http://www.ros.org/wiki/xacro">
     <xacro:arg name="robot_name" default="/" />
-    <xacro:arg name="model_type" default="stl" />
+    <xacro:arg name="model_type" default="dae" />
     <xacro:arg name="file_path" default="../soccer_description" />
     <xacro:arg name="has_base_footprint" default="false" />

File: soccer_description/models/soccerbot_stl.urdf (robot description, URDF)
Before this commit: robot soccerbot, 21 links, 20 joints
Links:
- link head: geometry collision box size=0.0712 0.094 0.0779; visual mesh filename=../soccer_description/meshes/head.dae scale=1 1 1
- link left_ankle: geometry collision box size=0.090769 0.042 0.0506; visual mesh filename=../soccer_description/meshes/left_ankle.dae scale=1 1 1
- link left_bicep: geometry collision box size=0.04 0.04776 0.123; visual mesh filename=../soccer_description/meshes/left_bicep.dae scale=1 1 1
- link left_calve: geometry collision box size=0.031883 0.048 0.105683; visual mesh filename=../soccer_description/meshes/left_calve.dae scale=1 1 1
- link left_foot: geometry collision box size=0.09 0.07 0.03674; visual mesh filename=../soccer_description/meshes/left_foot.dae scale=1 1 1
- link left_forearm: geometry collision box size=0.035 0.049 0.144; visual mesh filename=../soccer_description/meshes/left_forearm.dae scale=1 1 1
- link left_hip_front: geometry collision box size=0.083747 0.04885 0.0506; visual mesh filename=../soccer_description/meshes/left_hip_front.dae scale=1 1 1
- link left_hip_side: geometry collision box size=0.0485 0.022 0.0039; visual mesh filename=../soccer_description/meshes/left_hip_side.dae scale=1 1 1
- link left_thigh: geometry collision box size=0.022 0.048 0.111; visual mesh filename=../soccer_description/meshes/left_thigh.dae scale=1 1 1
- link neck: geometry collision box size=0.022 0.0523 0.033; visual mesh filename=../soccer_description/meshes/neck.dae scale=1 1 1
- link right_ankle: geometry collision box size=0.090769 0.042 0.0506; visual mesh filename=../soccer_description/meshes/right_ankle.dae scale=1 1 1
- link right_bicep: geometry collision box size=0.04 0.04776 0.123; visual mesh filename=../soccer_description/meshes/right_bicep.dae scale=1 1 1
- link right_calve: geometry collision box size=0.031883 0.048 0.105683; visual mesh filename=../soccer_description/meshes/right_calve.dae scale=1 1 1
- link right_foot: geometry collision box size=0.09 0.07 0.03674; visual mesh filename=../soccer_description/meshes/right_foot.dae scale=1 1 1
- link right_forearm: geometry collision box size=0.035 0.049 0.144; visual mesh filename=../soccer_description/meshes/right_forearm.dae scale=1 1 1
- link right_hip_front: geometry collision box size=0.083747 0.04885 0.0506; visual mesh filename=../soccer_description/meshes/right_hip_front.dae scale=1 1 1
- link right_hip_side: geometry collision box size=0.0485 0.022 0.0039; visual mesh filename=../soccer_description/meshes/right_hip_side.dae scale=1 1 1
- link right_thigh: geometry collision box size=0.022 0.048 0.111; visual mesh filename=../soccer_description/meshes/right_thigh.dae scale=1 1 1
- link torso: geometry collision box size=0.130 0.145 0.152; visual mesh filename=../soccer_description/meshes/torso.dae scale=1 1 1
