Commit message: shift camera back, guess the amount based on visual inspection
Former-commit-id: e920aa68aad4582afd6be3883bc14d2ac4f01e16 [formerly 4d1e56aa06d1629473326395ec8b43f4d71ab09d]
Former-commit-id: 5d49440a59ed971c9c0062cab264cdb77a2cc614

File: soccer_description/models/front_camera.xacro (robot description, xacro)
@@ -5,5 +5,5 @@
             <parent link="head"/>
             <child link="camera"/>
-            <origin rpy="0 0 0" xyz="0.05295 0.00145 0.04740"/>
+            <origin rpy="0 0 0" xyz="0.015 0.00145 0.04740"/>
             <axis xyz="0  0  0"/>
             <dynamics damping="${JOINT_DAMPING}" friction="${JOINT_FRICTION}" />

Commit message: updated stl
Former-commit-id: b87aacfd909222d4e2c71a37f14969607383c3a6 [formerly 339fec3c7fa1682df5f48c705fa0e6acbdf1810e]
Former-commit-id: 57ece1e3572b6b0f09737d419bc08859cad4eef9

File: soccer_description/models/front_camera.xacro (robot description, xacro)
@@ -1,5 +1,13 @@
 <robot name="soccerbot" xmlns:xacro="http://www.ros.org/wiki/xacro">
     <xacro:macro name="front_camera" params="origin">
-        <link name="camera" />
+        <link name="camera" >
+            <inertial>
+                <mass value="0.01"/>
+                <origin rpy="0  0  0" xyz="0 0 0"/>
+                <inertia ixx="1e-9" ixy="0" ixz="0"
+                         iyy="1e-9" iyz="0"
+                         izz="1e-9"/>
+            </inertial>
+        </link>
         <joint name="${origin}_camera" type="fixed">
             <parent link="head"/>
@@ -10,6 +18,4 @@
             <limit effort="0" lower="0" upper="0" velocity="0"/>
         </joint>
-        rotation 0.707105 -0.000001 0.707108 3.141591
-        rotation 1.0 0.0 0.0 3.141591
         <gazebo reference="camera">
             <sensor type="camera" name="main_camera" >

File: soccer_description/models/imu.xacro (robot description, xacro)
@@ -1,5 +1,13 @@
 <robot name="soccerbot" xmlns:xacro="http://www.ros.org/wiki/xacro">
     <xacro:macro name="imu" params="origin">
-        <link name="imu_link" />
+        <link name="imu_link" >
+            <inertial>
+                <mass value="0.01"/>
+                <origin rpy="0  0  0" xyz="0 0 0"/>
+                <inertia ixx="1e-9" ixy="0" ixz="0"
+                         iyy="1e-9" iyz="0"
+                         izz="1e-9"/>
+            </inertial>
+        </link>
         <joint name="${origin}_imu" type="fixed">
             <parent link="${origin}"/>

File: soccer_description/models/soccerbot_stl.urdf (robot description, URDF)
Before this commit: robot soccerbot, 21 links, 20 joints
Links:
- link camera: mass None -> 0.01
- link imu_link: mass None -> 0.01
