Commit message: Fixed conventions

File: soccer_description/models/leg.xacro (robot description, xacro)
@@ -146,5 +146,5 @@
             <child link="${name}_hip_front"/>
             <origin rpy="0 0 0" xyz="0 0 0"/>
-            <axis xyz="-1 0 0"/>
+            <axis xyz="${direction} 0 0"/>
             <dynamics damping="${JOINT_DAMPING}" friction="${JOINT_FRICTION}" />
             <xacro:if value="${direction == 1}">

File: soccer_description/models/soccerbot_stl.urdf (robot description, URDF)
Before this commit: robot soccerbot, 21 links, 20 joints
Joints:
- joint left_leg_motor_1: axis -1 0 0 -> 1 0 0

Commit message: Done

File: soccer_description/models/leg.xacro (robot description, xacro)
@@ -148,10 +148,5 @@
             <axis xyz="${direction} 0 0"/>
             <dynamics damping="${JOINT_DAMPING}" friction="${JOINT_FRICTION}" />
-            <xacro:if value="${direction == 1}">
-             <limit effort="${MX28_TORQUE}" lower="-${PI/4}" upper="${PI/2}" velocity="${MX28_VELOCITY}"/>
-            </xacro:if>
-            <xacro:if value="${direction == -1}">
-            <limit effort="${MX28_TORQUE}" lower="-${PI/2}" upper="${PI/4}" velocity="${MX28_VELOCITY}"/>
-            </xacro:if>
+            <limit effort="${MX28_TORQUE}" lower="-${PI/4}" upper="${PI/2}" velocity="${MX28_VELOCITY}"/>
         </joint>
         <joint name="${name}_leg_motor_2" type="revolute">
@@ -183,5 +178,5 @@
             <child link="${name}_foot"/>
             <origin rpy="0 0 0" xyz="0 0 0"/>
-            <axis xyz="-1 0 0"/>
+            <axis xyz="${direction} 0 0"/>
             <dynamics damping="${JOINT_DAMPING}" friction="${JOINT_FRICTION}" />
             <limit effort="${MX28_TORQUE}" lower="-${PI/4}" upper="${PI/4}" velocity="${MX28_VELOCITY}"/>

File: soccer_description/models/soccerbot_stl.urdf (robot description, URDF)
Before this commit: robot soccerbot, 21 links, 20 joints
Joints:
- joint left_leg_motor_5: axis -1 0 0 -> 1 0 0
- joint right_leg_motor_1: limit lower=-1.57079632679 upper=0.785398163397 effort=2.5 velocity=1 -> lower=-0.785398163397 upper=1.57079632679 effort=2.5 velocity=1

Commit message: Dc walking (#72)
* Fixed slx

* Manual inverse kinematics done

* Finished making path for robot

* Add all

* add stf

* added path for foot

* accounting for first step left

* Temp

* Accomplished enough today

* Missing robot path

* Main and geometry

* Forgot robot

* Working

* Fixed inverse kinematics, fucking pain in the pass

* Added simply motor publisher node

* Added simple control node for ros

* Fixed ikine yet again. Added more realistic hip trajectories

* Added media test

* Made faster stronger and better

* Sure

* Convetions fixed

* current file changes

* Temp

* Walks

* Speed

* Added simply motor publisher node

* Added simply motor publisher node

* System

* used wrong transform names, now head rotates and stops when sees ball

* Fixed direction

* fix convention

* Fixed conventions

* add comments for conventions

* coding conventions...

* fix the ankle positive direction convention

* Done

* Ltatest

* Commit


Former-commit-id: bbced040a7abd600b47214eb368a380825f9f5f2 [formerly 0e25ca7090a84501817d1a2a096ae18534ecca26]
Former-commit-id: 79bf23e7cdf63403dc42f58ad4924c0c168c1ad2

File: soccer_description/models/leg.xacro (robot description, xacro)
@@ -146,12 +146,7 @@
             <child link="${name}_hip_front"/>
             <origin rpy="0 0 0" xyz="0 0 0"/>
-            <axis xyz="-1 0 0"/>
-            <dynamics damping="${JOINT_DAMPING}" friction="${JOINT_FRICTION}" />
-            <xacro:if value="${direction == 1}">
-             <limit effort="${MX28_TORQUE}" lower="-${PI/4}" upper="${PI/2}" velocity="${MX28_VELOCITY}"/>
-            </xacro:if>
-            <xacro:if value="${direction == -1}">
-            <limit effort="${MX28_TORQUE}" lower="-${PI/2}" upper="${PI/4}" velocity="${MX28_VELOCITY}"/>
-            </xacro:if>
+            <axis xyz="${direction} 0 0"/>
+            <dynamics damping="${JOINT_DAMPING}" friction="${JOINT_FRICTION}" />
+            <limit effort="${MX28_TORQUE}" lower="-${PI/4}" upper="${PI/2}" velocity="${MX28_VELOCITY}"/>
         </joint>
         <joint name="${name}_leg_motor_2" type="revolute">
@@ -183,5 +178,5 @@
             <child link="${name}_foot"/>
             <origin rpy="0 0 0" xyz="0 0 0"/>
-            <axis xyz="-1 0 0"/>
+            <axis xyz="${direction} 0 0"/>
             <dynamics damping="${JOINT_DAMPING}" friction="${JOINT_FRICTION}" />
             <limit effort="${MX28_TORQUE}" lower="-${PI/4}" upper="${PI/4}" velocity="${MX28_VELOCITY}"/>

File: soccer_description/models/soccerbot_stl.urdf (robot description, URDF)
Before this commit: robot soccerbot, 21 links, 20 joints
Joints:
- joint left_leg_motor_1: axis -1 0 0 -> 1 0 0
- joint left_leg_motor_5: axis -1 0 0 -> 1 0 0
- joint right_leg_motor_1: limit lower=-1.57079632679 upper=0.785398163397 effort=2.5 velocity=1 -> lower=-0.785398163397 upper=1.57079632679 effort=2.5 velocity=1

Commit message: Fixed knee joint
Former-commit-id: 4d553a3c89587bd3f32a896840f7693a676216cd [formerly 3e4427dd4002b8b876ab72a4d96b1dd344879153]
Former-commit-id: 6d329ef0e60ffd5c9f598012681cb92b193f98af

File: soccer_description/models/leg.xacro (robot description, xacro)
@@ -161,5 +161,5 @@
             <parent link="${name}_thigh"/>
             <child link="${name}_calve"/>
-            <origin rpy="0 0 0" xyz="0 0 -0.09290"/>
+            <origin rpy="0 0 0" xyz="0 0 -0.0890"/>
             <axis xyz="0 -1 0"/>
             <dynamics damping="${JOINT_DAMPING}" friction="${JOINT_FRICTION}" />

File: soccer_description/models/soccerbot_stl.urdf (robot description, URDF)
Before this commit: robot soccerbot, 21 links, 20 joints
Joints:
- joint left_leg_motor_3: origin xyz=0 0 -0.09290 rpy=0 0 0 -> xyz=0 0 -0.0890 rpy=0 0 0
- joint right_leg_motor_3: origin xyz=0 0 -0.09290 rpy=0 0 0 -> xyz=0 0 -0.0890 rpy=0 0 0
