Commit message: First commit

File: soccer_description/models/arm.xacro (robot description, xacro)
@@ -18,5 +18,5 @@
                     <origin rpy="0  0  0" xyz="0  0  0"/>
                     <geometry>
-                        <mesh filename="package://soccer_description/meshes/${name}_bicep.dae" scale="1 1 1"/>
+                        <mesh filename="${FILE_PATH}meshes/${name}_bicep.${MODEL_TYPE}" scale="1 1 1"/>
                     </geometry>
                     <material name="black" />
@@ -40,5 +40,5 @@
                     <origin rpy="0  0  0" xyz="0  0  0"/>
                     <geometry>
-                        <mesh filename="package://soccer_description/meshes/${name}_forearm.dae" scale="1 1 1"/>
+                        <mesh filename="${FILE_PATH}meshes/${name}_forearm.${MODEL_TYPE}" scale="1 1 1"/>
                     </geometry>
                     <material name="black" />

File: soccer_description/models/head.xacro (robot description, xacro)
@@ -18,5 +18,5 @@
                 <origin rpy="0  0  0" xyz="0  0  0"/>
                 <geometry>
-                    <mesh filename="package://soccer_description/meshes/neck.dae" scale="1 1 1"/>
+                    <mesh filename="${FILE_PATH}meshes/neck.${MODEL_TYPE}" scale="1 1 1"/>
                 </geometry>
                 <material name="black" />
@@ -40,5 +40,5 @@
                 <origin rpy="0  0  0" xyz="0  0  0"/>
                 <geometry>
-                    <mesh filename="package://soccer_description/meshes/head.dae" scale="1 1 1"/>
+                    <mesh filename="${FILE_PATH}meshes/head.${MODEL_TYPE}" scale="1 1 1"/>
                 </geometry>
                 <material name="black" />

File: soccer_description/models/leg.xacro (robot description, xacro)
@@ -18,5 +18,5 @@
                 <origin rpy="0  0  0" xyz="0  0  0"/>
                 <geometry>
-                    <mesh filename="package://soccer_description/meshes/${name}_hip_side.dae" scale="1 1 1"/>
+                    <mesh filename="${FILE_PATH}meshes/${name}_hip_side.${MODEL_TYPE}" scale="1 1 1"/>
                 </geometry>
                 <material name="black" />
@@ -40,5 +40,5 @@
                 <origin rpy="0  0  0" xyz="0  0  0"/>
                 <geometry>
-                    <mesh filename="package://soccer_description/meshes/${name}_hip_front.dae" scale="1 1 1"/>
+                    <mesh filename="${FILE_PATH}meshes/${name}_hip_front.${MODEL_TYPE}" scale="1 1 1"/>
                 </geometry>
                 <material name="black" />
@@ -62,5 +62,5 @@
                 <origin rpy="0  0  0" xyz="0  0  0"/>
                 <geometry>
-                    <mesh filename="package://soccer_description/meshes/${name}_thigh.dae" scale="1 1 1"/>
+                    <mesh filename="${FILE_PATH}meshes/${name}_thigh.${MODEL_TYPE}" scale="1 1 1"/>
                 </geometry>
                 <material name="black" />
@@ -84,5 +84,5 @@
                 <origin rpy="0 0 0" xyz="0 0 -0.0827"/>
                 <geometry>
-                    <mesh filename="package://soccer_description/meshes/${name}_calve.dae" scale="1 1 1"/>
+                    <mesh filename="${FILE_PATH}meshes/${name}_calve.${MODEL_TYPE}" scale="1 1 1"/>
                 </geometry>
                 <material name="black" />
@@ -106,5 +106,5 @@
                 <origin rpy="0 0 0" xyz="0  0  0"/>
                 <geometry>
-                    <mesh filename="package://soccer_description/meshes/${name}_ankle.dae" scale="1 1 1"/>
+                    <mesh filename="${FILE_PATH}meshes/${name}_ankle.${MODEL_TYPE}" scale="1 1 1"/>
                 </geometry>
                 <material name="black" />
@@ -129,5 +129,5 @@
                 <origin rpy="0  0  0" xyz="0  0  0"/>
                 <geometry>
-                    <mesh filename="package://soccer_description/meshes/${name}_foot.dae" scale="1 1 1"/>
+                    <mesh filename="${FILE_PATH}meshes/${name}_foot.${MODEL_TYPE}" scale="1 1 1"/>
                 </geometry>
                 <material name="black" />

File: soccer_description/models/soccerbot.xacro (robot description, xacro)
@@ -2,62 +2,5 @@
 <robot name="soccerbot" xmlns:xacro="http://www.ros.org/wiki/xacro">
     <xacro:include filename="$(find soccer_description)/models/parameters.xacro" />
-    <xacro:include filename="$(find soccer_description)/models/arm.xacro" />
-    <xacro:include filename="$(find soccer_description)/models/leg.xacro" />
-    <xacro:include filename="$(find soccer_description)/models/head.xacro" />
-    <xacro:include filename="front_camera.xacro" />
-    <xacro:include filename="$(find soccer_description)/models/imu.xacro" />
-    <link name="base_link" />
-    <link name="torso">
-        <inertial>
-            <mass value="1529.201"/>
-            <origin rpy="0 0 0" xyz="0.0082498 -0.0017440 -0.0522479"/>
-            <inertia ixx="4.323" ixy="0.006" ixz="0.040"
-                     iyy="5.198" iyz="-0.015"
-                     izz="3.567"/>
-        </inertial>
-        <collision name="collision">
-            <origin rpy="0 0 0" xyz="0 0 -0.052"/>
-            <geometry>
-                <box size="0.130 0.145 0.152"/>
-            </geometry>
-        </collision>
-        <visual name="visual">
-            <origin rpy="0 0 0" xyz="0 0 0"/>
-            <geometry>
-                <mesh filename="package://soccer_description/meshes/torso.dae" scale="1 1 1"/>
-            </geometry>
-        </visual>
-    </link>
-    <!-- Joints -->
-    <joint name="base_link_torso" type="fixed">
-        <parent link="base_link"/>
-        <child link="torso"/>
-        <origin rpy="0 0 0" xyz="0 0 0.3536"/>
-        <axis xyz="1 0 0"/>
-    </joint>
-    <arm name="right" origin="torso" direction="1" />
-    <arm name="left" origin="torso" direction="-1" />
-    <leg name="right" origin="torso" direction="1" />
-    <leg name="left" origin="torso" direction="-1" />
-    <head origin="torso" />
-    <imu origin="torso" />
-    <front_camera origin="head" />
-    <gazebo>
-        <plugin name="gazebo_ros_control" filename="libgazebo_ros_control.so">
-            <robotNamespace>/</robotNamespace>
-            <robotSimType>gazebo_ros_control/DefaultRobotHWSim</robotSimType>
-        </plugin>
-    </gazebo>
-    <gazebo reference="base_link">
-        <kp>${JOINT_KP}</kp>
-        <kd>${JOINT_KD}</kd>
-        <mu1>${JOINT_MU1}</mu1>
-        <mu2>${JOINT_MU2}</mu2>
-    </gazebo>
-    <gazebo reference="torso">
-        <kp>${JOINT_KP}</kp>
-        <kd>${JOINT_KD}</kd>
-        <mu1>${JOINT_MU1}</mu1>
-        <mu2>${JOINT_MU2}</mu2>
-    </gazebo>
+    <xacro:include filename="$(find soccer_description)/models/robot.xacro" />
+    <soccerbot />
 </robot>

Commit message: Auto build urdf

File: soccer_description/models/arm.xacro (robot description, xacro)
@@ -18,5 +18,5 @@
                     <origin rpy="0  0  0" xyz="0  0  0"/>
                     <geometry>
-                        <mesh filename="${FILE_PATH}meshes/${name}_bicep.${MODEL_TYPE}" scale="1 1 1"/>
+                        <mesh filename="${FILE_PATH}/meshes/${name}_bicep.${MODEL_TYPE}" scale="1 1 1"/>
                     </geometry>
                     <material name="black" />
@@ -40,5 +40,5 @@
                     <origin rpy="0  0  0" xyz="0  0  0"/>
                     <geometry>
-                        <mesh filename="${FILE_PATH}meshes/${name}_forearm.${MODEL_TYPE}" scale="1 1 1"/>
+                        <mesh filename="${FILE_PATH}/meshes/${name}_forearm.${MODEL_TYPE}" scale="1 1 1"/>
                     </geometry>
                     <material name="black" />

File: soccer_description/models/head.xacro (robot description, xacro)
@@ -18,5 +18,5 @@
                 <origin rpy="0  0  0" xyz="0  0  0"/>
                 <geometry>
-                    <mesh filename="${FILE_PATH}meshes/neck.${MODEL_TYPE}" scale="1 1 1"/>
+                    <mesh filename="${FILE_PATH}/meshes/neck.${MODEL_TYPE}" scale="1 1 1"/>
                 </geometry>
                 <material name="black" />
@@ -40,5 +40,5 @@
                 <origin rpy="0  0  0" xyz="0  0  0"/>
                 <geometry>
-                    <mesh filename="${FILE_PATH}meshes/head.${MODEL_TYPE}" scale="1 1 1"/>
+                    <mesh filename="${FILE_PATH}/meshes/head.${MODEL_TYPE}" scale="1 1 1"/>
                 </geometry>
                 <material name="black" />

File: soccer_description/models/leg.xacro (robot description, xacro)
@@ -18,5 +18,5 @@
                 <origin rpy="0  0  0" xyz="0  0  0"/>
                 <geometry>
-                    <mesh filename="${FILE_PATH}meshes/${name}_hip_side.${MODEL_TYPE}" scale="1 1 1"/>
+                    <mesh filename="${FILE_PATH}/meshes/${name}_hip_side.${MODEL_TYPE}" scale="1 1 1"/>
                 </geometry>
                 <material name="black" />
@@ -40,5 +40,5 @@
                 <origin rpy="0  0  0" xyz="0  0  0"/>
                 <geometry>
-                    <mesh filename="${FILE_PATH}meshes/${name}_hip_front.${MODEL_TYPE}" scale="1 1 1"/>
+                    <mesh filename="${FILE_PATH}/meshes/${name}_hip_front.${MODEL_TYPE}" scale="1 1 1"/>
                 </geometry>
                 <material name="black" />
@@ -62,5 +62,5 @@
                 <origin rpy="0  0  0" xyz="0  0  0"/>
                 <geometry>
-                    <mesh filename="${FILE_PATH}meshes/${name}_thigh.${MODEL_TYPE}" scale="1 1 1"/>
+                    <mesh filename="${FILE_PATH}/meshes/${name}_thigh.${MODEL_TYPE}" scale="1 1 1"/>
                 </geometry>
                 <material name="black" />
@@ -84,5 +84,5 @@
                 <origin rpy="0 0 0" xyz="0 0 -0.0827"/>
                 <geometry>
-                    <mesh filename="${FILE_PATH}meshes/${name}_calve.${MODEL_TYPE}" scale="1 1 1"/>
+                    <mesh filename="${FILE_PATH}/meshes/${name}_calve.${MODEL_TYPE}" scale="1 1 1"/>
                 </geometry>
                 <material name="black" />
@@ -106,5 +106,5 @@
                 <origin rpy="0 0 0" xyz="0  0  0"/>
                 <geometry>
-                    <mesh filename="${FILE_PATH}meshes/${name}_ankle.${MODEL_TYPE}" scale="1 1 1"/>
+                    <mesh filename="${FILE_PATH}/meshes/${name}_ankle.${MODEL_TYPE}" scale="1 1 1"/>
                 </geometry>
                 <material name="black" />
@@ -129,5 +129,5 @@
                 <origin rpy="0  0  0" xyz="0  0  0"/>
                 <geometry>
-                    <mesh filename="${FILE_PATH}meshes/${name}_foot.${MODEL_TYPE}" scale="1 1 1"/>
+                    <mesh filename="${FILE_PATH}/meshes/${name}_foot.${MODEL_TYPE}" scale="1 1 1"/>
                 </geometry>
                 <material name="black" />

File: soccer_description/models/robot.xacro (robot description, xacro)
@@ -1,5 +1,5 @@
 <?xml version="1.0" ?>
 <robot name="soccerbot" xmlns:xacro="http://www.ros.org/wiki/xacro">
-    <xacro:macro name="soccerbot" params="FILE_PATH:=${FILE_PATH} MODEL_TYPE:=dae" >
+    <xacro:macro name="soccerbot" params="FILE_PATH:=package://soccer_description MODEL_TYPE:=dae" >
         <xacro:include filename="$(find soccer_description)/models/arm.xacro" />
         <xacro:include filename="$(find soccer_description)/models/leg.xacro" />
@@ -25,5 +25,5 @@
                 <origin rpy="0 0 0" xyz="0 0 0"/>
                 <geometry>
-                    <mesh filename="${FILE_PATH}meshes/torso.${MODEL_TYPE}" scale="1 1 1"/>
+                    <mesh filename="${FILE_PATH}/meshes/torso.${MODEL_TYPE}" scale="1 1 1"/>
                 </geometry>
             </visual>

File: soccer_description/models/soccerbot_stl.xacro (robot description, xacro)
@@ -3,4 +3,4 @@
     <xacro:include filename="$(find soccer_description)/models/parameters.xacro" />
     <xacro:include filename="$(find soccer_description)/models/robot.xacro" />
-    <soccerbot FILE_PATH="../soccer_description/" MODEL_TYPE="stl" />
+    <soccerbot FILE_PATH="../soccer_description" MODEL_TYPE="stl" />
 </robot>
