Commit message: Simulink Model (#45)
* First commit

* Auto build urdf

* Cleans up gazebo faster

* Cleans up gazebo faster

* Cleanup

* Cleaning up

* Cleanup cmake

* Cleaning up


Former-commit-id: 3cc341b9f035ce7ab9c104f5ea70e76d3acf6a94 [formerly baa48e0f13643972acb5428ebf75cfb83ca45d42]
Former-commit-id: 04b257c2775ff5800dc33641606dcadcfb72a63c

File: soccer_description/models/arm.xacro (robot description, xacro)
@@ -3,9 +3,9 @@
             <link name="${name}_bicep">
                 <inertial>
-                    <mass value="213.5130"/>
+                    <mass value="0.213e-3"/>
                     <origin rpy="0  0  0" xyz="0.000 ${direction * 0.02579} -0.04955"/>
-                    <inertia ixx="0.282" ixy="0.000" ixz="${direction * 0.000}"
-                             iyy="0.274" iyz="${direction * 0.012}"
-                             izz="0.024" />
+                    <inertia ixx="2.824e-4" ixy="0.000" ixz="${direction * 0.000}"
+                             iyy="2.744e-4" iyz="${direction * 1.165e-5}"
+                             izz="2.433e-5" />
                 </inertial>
                 <collision name="collision">
@@ -18,5 +18,5 @@
                     <origin rpy="0  0  0" xyz="0  0  0"/>
                     <geometry>
-                        <mesh filename="package://soccer_description/meshes/${name}_bicep.dae" scale="1 1 1"/>
+                        <mesh filename="${FILE_PATH}/meshes/${name}_bicep.${MODEL_TYPE}" scale="1 1 1"/>
                     </geometry>
                     <material name="black" />
@@ -25,9 +25,9 @@
             <link name="${name}_forearm">
                 <inertial>
-                    <mass value="45.7"/>
+                    <mass value="45.7e-3"/>
                     <origin rpy="0  0  0" xyz="0 0.0245 -0.0546097" />
-                    <inertia ixx="0.113" ixy="0.000" ixz="${direction * 0.001}"
-                             iyy="0.107" iyz="${direction * 0.000}"
-                             izz="0.012" />
+                    <inertia ixx="0.113e-3" ixy="0.000" ixz="${direction * 0.001e-3}"
+                             iyy="0.107e-3" iyz="${direction * 0.000}"
+                             izz="0.012e-3" />
                 </inertial>
                 <collision name="collision">
@@ -40,5 +40,5 @@
                     <origin rpy="0  0  0" xyz="0  0  0"/>
                     <geometry>
-                        <mesh filename="package://soccer_description/meshes/${name}_forearm.dae" scale="1 1 1"/>
+                        <mesh filename="${FILE_PATH}/meshes/${name}_forearm.${MODEL_TYPE}" scale="1 1 1"/>
                     </geometry>
                     <material name="black" />

File: soccer_description/models/head.xacro (robot description, xacro)
@@ -3,9 +3,9 @@
         <link name="neck">
             <inertial>
-                <mass value="11.294"/>
+                <mass value="0.011294"/>
                 <origin rpy="0  0  0" xyz="0 -0.0006476 0.0092453"/>
-                <inertia ixx="0.005" ixy="0" ixz="0"
-                         iyy="0.001" iyz="0"
-                         izz="0.005"/>
+                <inertia ixx="5.489e-6" ixy="0" ixz="0"
+                         iyy="1.433e-6" iyz="0"
+                         izz="4.955e-6"/>
             </inertial>
             <collision name="collision">
@@ -18,5 +18,5 @@
                 <origin rpy="0  0  0" xyz="0  0  0"/>
                 <geometry>
-                    <mesh filename="package://soccer_description/meshes/neck.dae" scale="1 1 1"/>
+                    <mesh filename="${FILE_PATH}/meshes/neck.${MODEL_TYPE}" scale="1 1 1"/>
                 </geometry>
                 <material name="black" />
@@ -25,9 +25,9 @@
         <link name="head">
             <inertial>
-                <mass value="282.919"/>
+                <mass value="0.282"/>
                 <origin rpy="0  0  0" xyz="0.0237166 0.0018096 0.0255966"/>
-                <inertia ixx="0.206" ixy="0.001" ixz="-0.057"
-                         iyy="0.206" iyz="0.003"
-                         izz="0.160"/>
+                <inertia ixx="2.06e-4" ixy="1.06e-6" ixz="-5.73e-5"
+                         iyy="2.057e-4" iyz="2.534e-6"
+                         izz="1.603e-4"/>
             </inertial>
             <collision name="collision">
@@ -40,5 +40,5 @@
                 <origin rpy="0  0  0" xyz="0  0  0"/>
                 <geometry>
-                    <mesh filename="package://soccer_description/meshes/head.dae" scale="1 1 1"/>
+                    <mesh filename="${FILE_PATH}/meshes/head.${MODEL_TYPE}" scale="1 1 1"/>
                 </geometry>
                 <material name="black" />
@@ -51,5 +51,5 @@
             <axis xyz="0 0 1"/>
             <dynamics damping="${JOINT_DAMPING}" friction="${JOINT_FRICTION}" />
-            <limit effort="${AX12_TORQUE}" lower="-${PI/2}" upper="${PI/2}" velocity="${MX28_VELOCITY}"/>
+            <limit effort="${AX12_TORQUE}" lower="-${PI/2}" upper="${PI/2}" velocity="${AX12_VELOCITY}"/>
         </joint>
         <joint name="neck_head" type="revolute">
@@ -59,5 +59,5 @@
             <axis xyz="0 1 0"/>
             <dynamics damping="${JOINT_DAMPING}" friction="${JOINT_FRICTION}" />
-            <limit effort="${AX12_TORQUE}" lower="-${PI*3/4}" upper="${PI*3/4}" velocity="${MX28_VELOCITY}"/>
+            <limit effort="${AX12_TORQUE}" lower="-${PI*3/4}" upper="${PI*3/4}" velocity="${AX12_VELOCITY}"/>
         </joint>
         <transmission name="${origin}_neck">

File: soccer_description/models/leg.xacro (robot description, xacro)
@@ -3,9 +3,9 @@
         <link name="${name}_hip_side">
             <inertial>
-                <mass value="9.364"/>
+                <mass value="9.364e-3"/>
                 <origin rpy="0  0  0" xyz="0.0003695 0.0000 0.01689"/>
-                <inertia ixx="0.002" ixy="0.000" ixz="0.000"
-                         iyy="0.005" iyz="0.000"
-                         izz="0.004"/>
+                <inertia ixx="0.002e-3" ixy="0.000" ixz="0.000"
+                         iyy="0.005e-3" iyz="0.000"
+                         izz="0.004e-3"/>
             </inertial>
             <collision name="collision">
@@ -18,5 +18,5 @@
                 <origin rpy="0  0  0" xyz="0  0  0"/>
                 <geometry>
-                    <mesh filename="package://soccer_description/meshes/${name}_hip_side.dae" scale="1 1 1"/>
+                    <mesh filename="${FILE_PATH}/meshes/${name}_hip_side.${MODEL_TYPE}" scale="1 1 1"/>
                 </geometry>
                 <material name="black" />
@@ -25,9 +25,9 @@
         <link name="${name}_hip_front">
             <inertial>
-                <mass value="153.186"/>
+                <mass value="153.186e-3"/>
                 <origin rpy="0 0 0" xyz="-0.02093 0 -0.011313"/>
-                <inertia ixx="0.041" ixy="0.000" ixz="-0.002"
-                         iyy="0.118" iyz="0.000"
-                         izz="0.106"/>
+                <inertia ixx="0.041e-3" ixy="0.000" ixz="-0.002e-3"
+                         iyy="0.118e-3" iyz="0.000"
+                         izz="0.106e-3"/>
             </inertial>
             <collision name="collision">
@@ -40,5 +40,5 @@
                 <origin rpy="0  0  0" xyz="0  0  0"/>
                 <geometry>
-                    <mesh filename="package://soccer_description/meshes/${name}_hip_front.dae" scale="1 1 1"/>
+                    <mesh filename="${FILE_PATH}/meshes/${name}_hip_front.${MODEL_TYPE}" scale="1 1 1"/>
                 </geometry>
                 <material name="black" />
@@ -47,9 +47,9 @@
         <link name="${name}_thigh">
             <inertial>
-                <mass value="21.438"/>
+                <mass value="21.438e-3"/>
                 <origin rpy="0 0 0" xyz="0.0019422 ${direction * 0.0001419} -0.0469409"/>
-                <inertia ixx="0.025" ixy="${direction * 0.002}" ixz="0.000"
-                         iyy="0.016" iyz="0.000"
-                         izz="0.010"/>
+                <inertia ixx="0.025e-3" ixy="${direction * 0.002e-3}" ixz="0.000"
+                         iyy="0.016e-3" iyz="0.000"
+                         izz="0.010e-3"/>
             </inertial>
             <collision name="collision">
@@ -62,5 +62,5 @@
                 <origin rpy="0  0  0" xyz="0  0  0"/>
                 <geometry>
-                    <mesh filename="package://soccer_description/meshes/${name}_thigh.dae" scale="1 1 1"/>
+                    <mesh filename="${FILE_PATH}/meshes/${name}_thigh.${MODEL_TYPE}" scale="1 1 1"/>
                 </geometry>
                 <material name="black" />
@@ -69,9 +69,9 @@
         <link name="${name}_calve">
             <inertial>
-                <mass value="86.547"/>
-                <origin rpy="0  0  0" xyz="0 ${direction * -0.0003259} -0.0150123"/>
-                <inertia ixx="0.054" ixy="0.000" ixz="0.000"
-                         iyy="0.046" iyz="-0.001"
-                         izz="0.019"/>
+                <mass value="86.547e-3"/>
+                <origin rpy="0  0  0" xyz="0 ${direction * -0.0003259e-3} -0.0150123e-3"/>
+                <inertia ixx="0.054e-3" ixy="0.000" ixz="0.000"
+                         iyy="0.046e-3" iyz="-0.001e-3"
+                         izz="0.019e-3"/>
             </inertial>
             <collision name="collision">
@@ -84,5 +84,5 @@
                 <origin rpy="0 0 0" xyz="0 0 -0.0827"/>
                 <geometry>
-                    <mesh filename="package://soccer_description/meshes/${name}_calve.dae" scale="1 1 1"/>
+                    <mesh filename="${FILE_PATH}/meshes/${name}_calve.${MODEL_TYPE}" scale="1 1 1"/>
                 </geometry>
                 <material name="black" />
@@ -91,9 +91,9 @@
         <link name="${name}_ankle">
             <inertial>
-                <mass value="153.186"/>
-                <origin rpy="0 0 0" xyz="-0.020939 0.000 0.011313"/>
-                <inertia ixx="0.041" ixy="0.000" ixz="0.002"
-                         iyy="0.118" iyz="0.000"
-                         izz="0.106"/>
+                <mass value="153.186e-3"/>
+                <origin rpy="0 0 0" xyz="-0.020939e-3 0.000 0.011313e-3"/>
+                <inertia ixx="0.041e-3" ixy="0.000" ixz="0.002e-3"
+                         iyy="0.118e-3" iyz="0.000"
+                         izz="0.106e-3"/>
             </inertial>
             <collision name="collision">
@@ -106,5 +106,5 @@
                 <origin rpy="0 0 0" xyz="0  0  0"/>
                 <geometry>
-                    <mesh filename="package://soccer_description/meshes/${name}_ankle.dae" scale="1 1 1"/>
+                    <mesh filename="${FILE_PATH}/meshes/${name}_ankle.${MODEL_TYPE}" scale="1 1 1"/>
                 </geometry>
                 <material name="black" />
@@ -113,9 +113,9 @@
         <link name="${name}_foot">
             <inertial>
-                <mass value="23.216"/>
+                <mass value="23.216e-3"/>
                 <origin rpy="0 0 0" xyz="-0.020939 0.0 0.011313"/>
-                <inertia ixx="0.006" ixy="0.000" ixz="0.000"
-                         iyy="0.018" iyz="0.000"
-                         izz="0.022"/>
+                <inertia ixx="0.006e-3" ixy="0.000" ixz="0.000"
+                         iyy="0.018e-3" iyz="0.000"
+                         izz="0.022e-3"/>
             </inertial>
             <collision name="collision">
@@ -129,5 +129,5 @@
                 <origin rpy="0  0  0" xyz="0  0  0"/>
                 <geometry>
-                    <mesh filename="package://soccer_description/meshes/${name}_foot.dae" scale="1 1 1"/>
+                    <mesh filename="${FILE_PATH}/meshes/${name}_foot.${MODEL_TYPE}" scale="1 1 1"/>
                 </geometry>
                 <material name="black" />

File: soccer_description/models/parameters.xacro (robot description, xacro)
@@ -1,15 +1,15 @@
 <robot name="soccerbot" xmlns:xacro="http://www.ros.org/wiki/xacro">
     <xacro:property name="PI" value="3.1415926535897931"/>
-    <xacro:property name="JOINT_KP" value="1000000.0"/>
-    <xacro:property name="JOINT_KD" value="1.0"/>
-    <xacro:property name="JOINT_MU1" value="0.8"/>
-    <xacro:property name="JOINT_MU2" value="0.8"/>
-    <xacro:property name="FOREARM_MU1" value="1000"/>
-    <xacro:property name="FOREARM_MU2" value="500"/>
-    <xacro:property name="JOINT_FRICTION" value="2000"/>
-    <xacro:property name="JOINT_DAMPING" value="0.0"/>
-    <xacro:property name="MX28_TORQUE" value="31000"/>
-    <xacro:property name="MX28_VELOCITY" value="0.0"/>
-    <xacro:property name="AX12_TORQUE" value="15000"/>
-    <xacro:property name="AX12_VELOCITY" value="0.0"/>
+    <xacro:property name="JOINT_KP" value="1e15"/>
+    <xacro:property name="JOINT_KD" value="1e13"/>
+    <xacro:property name="JOINT_MU1" value="0.2"/>
+    <xacro:property name="JOINT_MU2" value="0.2"/>
+    <xacro:property name="FOREARM_MU1" value="0.2"/>
+    <xacro:property name="FOREARM_MU2" value="0.2"/>
+    <xacro:property name="JOINT_FRICTION" value="0.05"/>
+    <xacro:property name="JOINT_DAMPING" value="0.02"/>
+    <xacro:property name="MX28_TORQUE" value="2.5"/>
+    <xacro:property name="MX28_VELOCITY" value="1"/>
+    <xacro:property name="AX12_TORQUE" value="1.5"/>
+    <xacro:property name="AX12_VELOCITY" value="1"/>
 </robot>

File: soccer_description/models/soccerbot.xacro (robot description, xacro)
@@ -2,32 +2,7 @@
 <robot name="soccerbot" xmlns:xacro="http://www.ros.org/wiki/xacro">
     <xacro:include filename="$(find soccer_description)/models/parameters.xacro" />
-    <xacro:include filename="$(find soccer_description)/models/arm.xacro" />
-    <xacro:include filename="$(find soccer_description)/models/leg.xacro" />
-    <xacro:include filename="$(find soccer_description)/models/head.xacro" />
-    <xacro:include filename="front_camera.xacro" />
-    <xacro:include filename="$(find soccer_description)/models/imu.xacro" />
+    <xacro:include filename="$(find soccer_description)/models/robot.xacro" />
+    <soccerbot />
     <link name="base_link" />
-    <link name="torso">
-        <inertial>
-            <mass value="1529.201"/>
-            <origin rpy="0 0 0" xyz="0.0082498 -0.0017440 -0.0522479"/>
-            <inertia ixx="4.323" ixy="0.006" ixz="0.040"
-                     iyy="5.198" iyz="-0.015"
-                     izz="3.567"/>
-        </inertial>
-        <collision name="collision">
-            <origin rpy="0 0 0" xyz="0 0 -0.052"/>
-            <geometry>
-                <box size="0.130 0.145 0.152"/>
-            </geometry>
-        </collision>
-        <visual name="visual">
-            <origin rpy="0 0 0" xyz="0 0 0"/>
-            <geometry>
-                <mesh filename="package://soccer_description/meshes/torso.dae" scale="1 1 1"/>
-            </geometry>
-        </visual>
-    </link>
-    <!-- Joints -->
     <joint name="base_link_torso" type="fixed">
         <parent link="base_link"/>
@@ -36,17 +11,4 @@
         <axis xyz="1 0 0"/>
     </joint>
-    <arm name="right" origin="torso" direction="1" />
-    <arm name="left" origin="torso" direction="-1" />
-    <leg name="right" origin="torso" direction="1" />
-    <leg name="left" origin="torso" direction="-1" />
-    <head origin="torso" />
-    <imu origin="torso" />
-    <front_camera origin="head" />
-    <gazebo>
-        <plugin name="gazebo_ros_control" filename="libgazebo_ros_control.so">
-            <robotNamespace>/</robotNamespace>
-            <robotSimType>gazebo_ros_control/DefaultRobotHWSim</robotSimType>
-        </plugin>
-    </gazebo>
     <gazebo reference="base_link">
         <kp>${JOINT_KP}</kp>
@@ -55,9 +17,3 @@
         <mu2>${JOINT_MU2}</mu2>
     </gazebo>
-    <gazebo reference="torso">
-        <kp>${JOINT_KP}</kp>
-        <kd>${JOINT_KD}</kd>
-        <mu1>${JOINT_MU1}</mu1>
-        <mu2>${JOINT_MU2}</mu2>
-    </gazebo>
 </robot>
