Commit message: Change all transforms to add support multi-robot.Added multi-robot functionality. Tuned localization to have multiple field lines. Can localize up to 3 robots and have 2 with darknet turned on
Former-commit-id: ca7e6ced67ef34ee522a0ccd58e40e69667b0d8b [formerly 891ac9929c61227a5f8d3d543dcddf4320bb06a6]
Former-commit-id: 34289cd58f84bb6905460abe8f6b80d30970d062

File: soccer_description/models/arm.xacro (robot description, xacro)
@@ -1,5 +1,5 @@
     <robot name="soccerbot" xmlns:xacro="http://www.ros.org/wiki/xacro">
         <xacro:macro name="arm" params="name origin direction">
-            <link name="${name}_bicep">
+            <link name="$(arg tf_prefix)/${name}_bicep">
                 <inertial>
                     <mass value="0.213e-3"/>
@@ -23,5 +23,5 @@
                 </visual>
             </link>
-            <link name="${name}_forearm">
+            <link name="$(arg tf_prefix)/${name}_forearm">
                 <inertial>
                     <mass value="45.7e-3"/>
@@ -47,5 +47,5 @@
             <joint name="${name}_arm_motor_0" type="revolute">
                 <parent link="${origin}"/>
-                <child link="${name}_bicep"/>
+                <child link="$(arg tf_prefix)/${name}_bicep"/>
                 <origin rpy="0 0 0" xyz="-0.0157 ${direction * 0.0725} 0"/>
                 <axis xyz="0 -1 0"/>
@@ -54,6 +54,6 @@
             </joint>
             <joint name="${name}_arm_motor_1" type="revolute">
-                <parent link="${name}_bicep"/>
-                <child link="${name}_forearm"/>
+                <parent link="$(arg tf_prefix)/${name}_bicep"/>
+                <child link="$(arg tf_prefix)/${name}_forearm"/>
                 <origin rpy="0 0 0" xyz="0 0 -0.10"/>
                 <axis xyz="0 -1 0"/>
@@ -61,5 +61,5 @@
                 <limit effort="${AX12_TORQUE}" lower="0" upper="${PI}" velocity="${AX12_VELOCITY}"/>
             </joint>
-            <gazebo reference="${name}_forearm">
+            <gazebo reference="$(arg tf_prefix)/${name}_forearm">
                 <mu1>${FOREARM_MU1}</mu1>
                 <mu2>${FOREARM_MU2}</mu2>
@@ -85,5 +85,5 @@
                 </actuator>
             </transmission>
-            <gazebo reference="${name}_bicep">
+            <gazebo reference="$(arg tf_prefix)/${name}_bicep">
                 <kp>${JOINT_KP}</kp>
                 <kd>${JOINT_KD}</kd>
@@ -91,5 +91,5 @@
                 <mu2>${JOINT_MU2}</mu2>
             </gazebo>
-            <gazebo reference="${name}_forearm">
+            <gazebo reference="$(arg tf_prefix)/${name}_forearm">
                 <kp>${JOINT_KP}</kp>
                 <kd>${JOINT_KD}</kd>

File: soccer_description/models/front_camera.xacro (robot description, xacro)
@@ -1,5 +1,5 @@
 <robot name="soccerbot" xmlns:xacro="http://www.ros.org/wiki/xacro">
     <xacro:macro name="front_camera" params="origin">
-        <link name="camera" >
+        <link name="$(arg tf_prefix)/camera" >
             <inertial>
                 <mass value="0.01"/>
@@ -11,6 +11,6 @@
         </link>
         <joint name="${origin}_camera" type="fixed">
-            <parent link="head"/>
-            <child link="camera"/>
+            <parent link="$(arg tf_prefix)/head"/>
+            <child link="$(arg tf_prefix)/camera"/>
             <origin rpy="0 0 0" xyz="0.015 0.00145 0.04740"/>
             <axis xyz="0  0  0"/>
@@ -18,5 +18,5 @@
             <limit effort="0" lower="0" upper="0" velocity="0"/>
         </joint>
-        <gazebo reference="camera">
+        <gazebo reference="$(arg tf_prefix)/camera">
             <sensor type="camera" name="main_camera" >
                 <always_on>1</always_on>
@@ -56,5 +56,5 @@
             </sensor>
         </gazebo>
-        <gazebo reference="camera">
+        <gazebo reference="$(arg tf_prefix)/camera">
             <kp>${JOINT_KP}</kp>
             <kd>${JOINT_KD}</kd>

File: soccer_description/models/head.xacro (robot description, xacro)
@@ -1,5 +1,5 @@
 <robot name="soccerbot" xmlns:xacro="http://www.ros.org/wiki/xacro">
     <xacro:macro name="head" params="origin">
-        <link name="neck">
+        <link name="$(arg tf_prefix)/neck">
             <inertial>
                 <mass value="0.011294"/>
@@ -23,5 +23,5 @@
             </visual>
         </link>
-        <link name="head">
+        <link name="$(arg tf_prefix)/head">
             <inertial>
                 <mass value="0.282"/>
@@ -47,5 +47,5 @@
         <joint name="head_motor_0" type="revolute">
             <parent link="${origin}"/>
-            <child link="neck"/>
+            <child link="$(arg tf_prefix)/neck"/>
             <origin rpy="0 0 0" xyz="0.024 0 0.05875"/>
             <axis xyz="0 0 1"/>
@@ -54,6 +54,6 @@
         </joint>
         <joint name="head_motor_1" type="revolute">
-            <parent link="neck"/>
-            <child link="head"/>
+            <parent link="$(arg tf_prefix)/neck"/>
+            <child link="$(arg tf_prefix)/head"/>
             <origin rpy="0 0 0" xyz="0 0 0.024"/>
             <axis xyz="0 1 0"/>
@@ -81,5 +81,5 @@
             </actuator>
         </transmission>
-        <gazebo reference="neck">
+        <gazebo reference="$(arg tf_prefix)/neck">
             <kp>${JOINT_KP}</kp>
             <kd>${JOINT_KD}</kd>
@@ -87,5 +87,5 @@
             <mu2>${JOINT_MU2}</mu2>
         </gazebo>
-        <gazebo reference="head">
+        <gazebo reference="$(arg tf_prefix)/head">
             <kp>${JOINT_KP}</kp>
             <kd>${JOINT_KD}</kd>

File: soccer_description/models/imu.xacro (robot description, xacro)
@@ -1,5 +1,5 @@
 <robot name="soccerbot" xmlns:xacro="http://www.ros.org/wiki/xacro">
     <xacro:macro name="imu" params="origin">
-        <link name="imu_link" >
+        <link name="$(arg tf_prefix)/imu_link" >
             <inertial>
                 <mass value="0.01"/>
@@ -12,9 +12,9 @@
         <joint name="${origin}_imu" type="fixed">
             <parent link="${origin}"/>
-            <child link="imu_link"/>
+            <child link="$(arg tf_prefix)/imu_link"/>
             <origin rpy="0 0 0" xyz="0.1 0 0.0075"/>
             <axis xyz="0 0 0"/>
         </joint>
-        <gazebo reference="imu_link">
+        <gazebo reference="$(arg tf_prefix)/imu_link">
             <gravity>true</gravity>
             <sensor name="imu_sensor" type="imu">
@@ -35,5 +35,5 @@
             </sensor>
         </gazebo>
-        <gazebo reference="imu_link">
+        <gazebo reference="$(arg tf_prefix)/imu_link">
             <kp>${JOINT_KP}</kp>
             <kd>${JOINT_KD}</kd>

File: soccer_description/models/leg.xacro (robot description, xacro)
@@ -1,5 +1,5 @@
 <robot name="soccerbot" xmlns:xacro="http://www.ros.org/wiki/xacro">
     <xacro:macro name="leg" params="name origin direction">
-        <link name="${name}_hip_side">
+        <link name="$(arg tf_prefix)/${name}_hip_side">
             <inertial>
                 <mass value="9.364e-3"/>
@@ -23,5 +23,5 @@
             </visual>
         </link>
-        <link name="${name}_hip_front">
+        <link name="$(arg tf_prefix)/${name}_hip_front">
             <inertial>
                 <mass value="153.186e-3"/>
@@ -45,5 +45,5 @@
             </visual>
         </link>
-        <link name="${name}_thigh">
+        <link name="$(arg tf_prefix)/${name}_thigh">
             <inertial>
                 <mass value="21.438e-3"/>
@@ -67,5 +67,5 @@
             </visual>
         </link>
-        <link name="${name}_calve">
+        <link name="$(arg tf_prefix)/${name}_calve">
             <inertial>
                 <mass value="86.547e-3"/>
@@ -89,5 +89,5 @@
             </visual>
         </link>
-        <link name="${name}_ankle">
+        <link name="$(arg tf_prefix)/${name}_ankle">
             <inertial>
                 <mass value="153.186e-3"/>
@@ -111,5 +111,5 @@
             </visual>
         </link>
-        <link name="${name}_foot">
+        <link name="$(arg tf_prefix)/${name}_foot">
             <inertial>
                 <mass value="23.216e-3"/>
@@ -135,6 +135,6 @@
         </link>
         <joint name="${name}_leg_motor_0" type="revolute">
-            <parent link="torso"/>
-            <child link="${name}_hip_side"/>
+            <parent link="$(arg tf_prefix)/torso"/>
+            <child link="$(arg tf_prefix)/${name}_hip_side"/>
             <origin rpy="0 0 0" xyz="0.0135 ${direction * 0.035} -0.156"/>
             <axis xyz="0 0 ${direction * -1}"/>
@@ -143,6 +143,6 @@
         </joint>
         <joint name="${name}_leg_motor_1" type="revolute">
-            <parent link="${name}_hip_side"/>
-            <child link="${name}_hip_front"/>
+            <parent link="$(arg tf_prefix)/${name}_hip_side"/>
+            <child link="$(arg tf_prefix)/${name}_hip_front"/>
             <origin rpy="0 0 0" xyz="0 0 0"/>
             <axis xyz="${direction} 0 0"/>
@@ -151,6 +151,6 @@
         </joint>
         <joint name="${name}_leg_motor_2" type="revolute">
-            <parent link="${name}_hip_front"/>
-            <child link="${name}_thigh"/>
+            <parent link="$(arg tf_prefix)/${name}_hip_front"/>
+            <child link="$(arg tf_prefix)/${name}_thigh"/>
             <origin rpy="0 0 0" xyz="0 0 0"/>
             <axis xyz="0 -1 0"/>
@@ -159,6 +159,6 @@
         </joint>
         <joint name="${name}_leg_motor_3" type="revolute">
-            <parent link="${name}_thigh"/>
-            <child link="${name}_calve"/>
+            <parent link="$(arg tf_prefix)/${name}_thigh"/>
+            <child link="$(arg tf_prefix)/${name}_calve"/>
             <origin rpy="0 0 0" xyz="0 0 -0.0890"/>
             <axis xyz="0 -1 0"/>
@@ -167,6 +167,6 @@
         </joint>
         <joint name="${name}_leg_motor_4" type="revolute">
-            <parent link="${name}_calve"/>
-            <child link="${name}_ankle"/>
+            <parent link="$(arg tf_prefix)/${name}_calve"/>
+            <child link="$(arg tf_prefix)/${name}_ankle"/>
             <origin rpy="0 0 0" xyz="0 0 -0.0827"/>
             <axis xyz="0 -1 0"/>
@@ -175,6 +175,6 @@
         </joint>
         <joint name="${name}_leg_motor_5" type="revolute">
-            <parent link="${name}_ankle"/>
-            <child link="${name}_foot"/>
+            <parent link="$(arg tf_prefix)/${name}_ankle"/>
+            <child link="$(arg tf_prefix)/${name}_foot"/>
             <origin rpy="0 0 0" xyz="0 0 0"/>
             <axis xyz="${direction} 0 0"/>
@@ -242,35 +242,35 @@
             </actuator>
         </transmission>
-        <gazebo reference="${name}_hip_side">
-            <kp>${JOINT_KP}</kp>
-            <kd>${JOINT_KD}</kd>
-            <mu1>${JOINT_MU1}</mu1>
-            <mu2>${JOINT_MU2}</mu2>
-        </gazebo>
-        <gazebo reference="${name}_hip_front">
-            <kp>${JOINT_KP}</kp>
-            <kd>${JOINT_KD}</kd>
-            <mu1>${JOINT_MU1}</mu1>
-            <mu2>${JOINT_MU2}</mu2>
-        </gazebo>
-        <gazebo reference="${name}_thigh">
-            <kp>${JOINT_KP}</kp>
-            <kd>${JOINT_KD}</kd>
-            <mu1>${JOINT_MU1}</mu1>
-            <mu2>${JOINT_MU2}</mu2>
-        </gazebo>
-        <gazebo reference="${name}_calve">
-            <kp>${JOINT_KP}</kp>
-            <kd>${JOINT_KD}</kd>
-            <mu1>${JOINT_MU1}</mu1>
-            <mu2>${JOINT_MU2}</mu2>
-        </gazebo>
-        <gazebo reference="${name}_ankle">
-            <kp>${JOINT_KP}</kp>
-            <kd>${JOINT_KD}</kd>
-            <mu1>${JOINT_MU1}</mu1>
-            <mu2>${JOINT_MU2}</mu2>
-        </gazebo>
-        <gazebo reference="${name}_foot">
+        <gazebo reference="$(arg tf_prefix)/${name}_hip_side">
+            <kp>${JOINT_KP}</kp>
+            <kd>${JOINT_KD}</kd>
+            <mu1>${JOINT_MU1}</mu1>
+            <mu2>${JOINT_MU2}</mu2>
+        </gazebo>
+        <gazebo reference="$(arg tf_prefix)/${name}_hip_front">
+            <kp>${JOINT_KP}</kp>
+            <kd>${JOINT_KD}</kd>
+            <mu1>${JOINT_MU1}</mu1>
+            <mu2>${JOINT_MU2}</mu2>
+        </gazebo>
+        <gazebo reference="$(arg tf_prefix)/${name}_thigh">
+            <kp>${JOINT_KP}</kp>
+            <kd>${JOINT_KD}</kd>
+            <mu1>${JOINT_MU1}</mu1>
+            <mu2>${JOINT_MU2}</mu2>
+        </gazebo>
+        <gazebo reference="$(arg tf_prefix)/${name}_calve">
+            <kp>${JOINT_KP}</kp>
+            <kd>${JOINT_KD}</kd>
+            <mu1>${JOINT_MU1}</mu1>
+            <mu2>${JOINT_MU2}</mu2>
+        </gazebo>
+        <gazebo reference="$(arg tf_prefix)/${name}_ankle">
+            <kp>${JOINT_KP}</kp>
+            <kd>${JOINT_KD}</kd>
+            <mu1>${JOINT_MU1}</mu1>
+            <mu2>${JOINT_MU2}</mu2>
+        </gazebo>
+        <gazebo reference="$(arg tf_prefix)/${name}_foot">
             <mu1>${FOREARM_MU1}</mu1>
             <mu2>${FOREARM_MU2}</mu2>

File: soccer_description/models/soccerbot.xacro (robot description, xacro)
@@ -5,4 +5,5 @@
     <xacro:arg name="file_path" default="../soccer_description" />
     <xacro:arg name="has_base_footprint" default="false" />
+    <xacro:arg name="tf_prefix" default="" />
     <xacro:property name="FILE_PATH" value="$(arg file_path)"/>
     <xacro:property name="MODEL_TYPE" value="$(arg model_type)"/>
@@ -13,5 +14,5 @@
     <xacro:include filename="$(find soccer_description)/models/front_camera.xacro" />
     <xacro:include filename="$(find soccer_description)/models/imu.xacro" />
-    <link name="torso">
+    <link name="$(arg tf_prefix)/torso">
         <inertial>
             <mass value="1.529"/>
@@ -34,20 +35,20 @@
         </visual>
     </link>
-    <xacro:arm name="left" origin="torso" direction="1" />
-    <xacro:arm name="right" origin="torso" direction="-1" />
-    <xacro:leg name="left" origin="torso" direction="1" />
-    <xacro:leg name="right" origin="torso" direction="-1" />
-    <xacro:head origin="torso" />
-    <xacro:imu origin="torso" />
-    <xacro:front_camera origin="head" />
+    <xacro:arm name="left" origin="$(arg tf_prefix)/torso" direction="1" />
+    <xacro:arm name="right" origin="$(arg tf_prefix)/torso" direction="-1" />
+    <xacro:leg name="left" origin="$(arg tf_prefix)/torso" direction="1" />
+    <xacro:leg name="right" origin="$(arg tf_prefix)/torso" direction="-1" />
+    <xacro:head origin="$(arg tf_prefix)/torso" />
+    <xacro:imu origin="$(arg tf_prefix)/torso" />
+    <xacro:front_camera origin="$(arg tf_prefix)/head" />
     <xacro:if value="$(arg has_base_footprint)">
-        <link name="base_footprint" />
+        <link name="$(arg tf_prefix)/base_footprint" />
         <joint name="base_footprint_torso" type="fixed">
-            <parent link="base_footprint"/>
-            <child link="torso"/>
+            <parent link="$(arg tf_prefix)/base_footprint"/>
+            <child link="$(arg tf_prefix)/torso"/>
             <origin rpy="0 0 0" xyz="0 0 0.3536"/>
             <axis xyz="1 0 0"/>
         </joint>
-        <gazebo reference="base_footprint">
+        <gazebo reference="$(arg tf_prefix)/base_footprint">
             <kp>${JOINT_KP}</kp>
             <kd>${JOINT_KD}</kd>
@@ -72,5 +73,5 @@
         </plugin>
     </gazebo>
-    <gazebo reference="torso">
+    <gazebo reference="$(arg tf_prefix)/torso">
         <kp>${JOINT_KP}</kp>
         <kd>${JOINT_KD}</kd>

File: soccer_description/models/soccerbot_stl.urdf (robot description, URDF)
Before this commit: robot soccerbot, 21 links, 20 joints
Links:
- removed link camera
- removed link head
- removed link imu_link
- removed link left_ankle
- removed link left_bicep
- removed link left_calve
- removed link left_foot
- removed link left_forearm
- removed link left_hip_front
- removed link left_hip_side
- removed link left_thigh
- removed link neck
- removed link right_ankle
- removed link right_bicep
- removed link right_calve
- removed link right_foot
- removed link right_forearm
- removed link right_hip_front
- removed link right_hip_side
- removed link right_thigh
- removed link torso
- added link /camera, mass 0.01
- added link /head, mass 0.282; collision box size=0.0712 0.094 0.0779; visual mesh filename=../soccer_description/meshes/head.dae scale=1 1 1
- added link /imu_link, mass 0.01
- added link /left_ankle, mass 153.186e-3; collision box size=0.090769 0.042 0.0506; visual mesh filename=../soccer_description/meshes/left_ankle.dae scale=1 1 1
- added link /left_bicep, mass 0.213e-3; collision box size=0.04 0.04776 0.123; visual mesh filename=../soccer_description/meshes/left_bicep.dae scale=1 1 1
- added link /left_calve, mass 86.547e-3; collision box size=0.031883 0.048 0.105683; visual mesh filename=../soccer_description/meshes/left_calve.dae scale=1 1 1
- added link /left_foot, mass 23.216e-3; collision box size=0.09 0.07 0.03674; visual mesh filename=../soccer_description/meshes/left_foot.dae scale=1 1 1
- added link /left_forearm, mass 45.7e-3; collision box size=0.035 0.049 0.144; visual mesh filename=../soccer_description/meshes/left_forearm.dae scale=1 1 1
- added link /left_hip_front, mass 153.186e-3; collision box size=0.083747 0.04885 0.0506; visual mesh filename=../soccer_description/meshes/left_hip_front.dae scale=1 1 1
- added link /left_hip_side, mass 9.364e-3; collision box size=0.0485 0.022 0.0039; visual mesh filename=../soccer_description/meshes/left_hip_side.dae scale=1 1 1
- added link /left_thigh, mass 21.438e-3; collision box size=0.022 0.048 0.111; visual mesh filename=../soccer_description/meshes/left_thigh.dae scale=1 1 1
- added link /neck, mass 0.011294; collision box size=0.022 0.0523 0.033; visual mesh filename=../soccer_description/meshes/neck.dae scale=1 1 1
- added link /right_ankle, mass 153.186e-3; collision box size=0.090769 0.042 0.0506; visual mesh filename=../soccer_description/meshes/right_ankle.dae scale=1 1 1
- added link /right_bicep, mass 0.213e-3; collision box size=0.04 0.04776 0.123; visual mesh filename=../soccer_description/meshes/right_bicep.dae scale=1 1 1
- added link /right_calve, mass 86.547e-3; collision box size=0.031883 0.048 0.105683; visual mesh filename=../soccer_description/meshes/right_calve.dae scale=1 1 1
- added link /right_foot, mass 23.216e-3; collision box size=0.09 0.07 0.03674; visual mesh filename=../soccer_description/meshes/right_foot.dae scale=1 1 1
- added link /right_forearm, mass 45.7e-3; collision box size=0.035 0.049 0.144; visual mesh filename=../soccer_description/meshes/right_forearm.dae scale=1 1 1
- added link /right_hip_front, mass 153.186e-3; collision box size=0.083747 0.04885 0.0506; visual mesh filename=../soccer_description/meshes/right_hip_front.dae scale=1 1 1
- added link /right_hip_side, mass 9.364e-3; collision box size=0.0485 0.022 0.0039; visual mesh filename=../soccer_description/meshes/right_hip_side.dae scale=1 1 1
- added link /right_thigh, mass 21.438e-3; collision box size=0.022 0.048 0.111; visual mesh filename=../soccer_description/meshes/right_thigh.dae scale=1 1 1
- added link /torso, mass 1.529; collision box size=0.130 0.145 0.152; visual mesh filename=../soccer_description/meshes/torso.dae scale=1 1 1
Joints:
- removed joint head_camera
- removed joint torso_imu
- added joint /head_camera: type fixed, parent /head, child /camera, origin xyz=0.015 0.00145 0.04740 rpy=0 0 0, axis 0  0  0, limit lower=0 upper=0 effort=0 velocity=0
- added joint /torso_imu: type fixed, parent /torso, child /imu_link, origin xyz=0.1 0 0.0075 rpy=0 0 0, axis 0 0 0
- joint head_motor_0: child neck -> /neck; parent torso -> /torso
- joint head_motor_1: child head -> /head; parent neck -> /neck
- joint left_arm_motor_0: child left_bicep -> /left_bicep; parent torso -> /torso
- joint left_arm_motor_1: child left_forearm -> /left_forearm; parent left_bicep -> /left_bicep
- joint left_leg_motor_0: child left_hip_side -> /left_hip_side; parent torso -> /torso
- joint left_leg_motor_1: child left_hip_front -> /left_hip_front; parent left_hip_side -> /left_hip_side
- joint left_leg_motor_2: child left_thigh -> /left_thigh; parent left_hip_front -> /left_hip_front
- joint left_leg_motor_3: child left_calve -> /left_calve; parent left_thigh -> /left_thigh
- joint left_leg_motor_4: child left_ankle -> /left_ankle; parent left_calve -> /left_calve
- joint left_leg_motor_5: child left_foot -> /left_foot; parent left_ankle -> /left_ankle
- joint right_arm_motor_0: child right_bicep -> /right_bicep; parent torso -> /torso
- joint right_arm_motor_1: child right_forearm -> /right_forearm; parent right_bicep -> /right_bicep
- joint right_leg_motor_0: child right_hip_side -> /right_hip_side; parent torso -> /torso
- joint right_leg_motor_1: child right_hip_front -> /right_hip_front; parent right_hip_side -> /right_hip_side
- joint right_leg_motor_2: child right_thigh -> /right_thigh; parent right_hip_front -> /right_hip_front
- joint right_leg_motor_3: child right_calve -> /right_calve; parent right_thigh -> /right_thigh
- joint right_leg_motor_4: child right_ankle -> /right_ankle; parent right_calve -> /right_calve
- joint right_leg_motor_5: child right_foot -> /right_foot; parent right_ankle -> /right_ankle
