Commit message: reverted mesh files + fixed collision & inertia locations of arm + added colors for PyBullet
Former-commit-id: 1e2a9715ae928bcceba143309bff2f3d25e86fe7 [formerly 30a2726f32bf9c6e7156bfb91a16cfe2a3c4895a]
Former-commit-id: f9e4a871f541f6edd088fbde6430d0e06e362878

File: soccer_description/models/arm.xacro (robot description, xacro)
@@ -20,5 +20,5 @@
                         <mesh filename="${FILE_PATH}/meshes/${name}_bicep.${MODEL_TYPE}" scale="1 1 1"/>
                     </geometry>
-                    <material name="black" />
+                    <material name="white" />
                 </visual>
             </link>
@@ -26,5 +26,5 @@
                 <inertial>
                     <mass value="45.7e-3"/>
-                    <origin rpy="0  0  0" xyz="0 0.0245 -0.0546097" />
+                    <origin rpy="0  0  0" xyz="0 ${direction * 0.0245} -0.0546097" />
                     <inertia ixx="0.113e-3" ixy="0.000" ixz="${direction * 0.001e-3}"
                              iyy="0.107e-3" iyz="${direction * 0.000}"
@@ -32,5 +32,5 @@
                 </inertial>
                 <collision name="collision">
-                    <origin rpy="0  0  0" xyz="-0.0055 0.01750 -0.0600"/>
+                    <origin rpy="0  0  0" xyz="-0.0055 ${direction * 0.01750} -0.0600"/>
                     <geometry>
                         <box size="0.035 0.049 0.144"/>
@@ -40,7 +40,7 @@
                     <origin rpy="0  0  0" xyz="0  0  0"/>
                     <geometry>
-                        <mesh filename="${FILE_PATH}/meshes/${name}_forearm.${MODEL_TYPE}" scale="0.001 0.001 0.001"/>
+                        <mesh filename="${FILE_PATH}/meshes/${name}_forearm.${MODEL_TYPE}" scale="1 1 1"/>
                     </geometry>
-                    <material name="black" />
+                    <material name="purple" />
                 </visual>
             </link>

File: soccer_description/models/head.xacro (robot description, xacro)
@@ -20,5 +20,5 @@
                     <mesh filename="${FILE_PATH}/meshes/neck.${MODEL_TYPE}" scale="1 1 1"/>
                 </geometry>
-                <material name="black" />
+                <material name="silver" />
             </visual>
         </link>
@@ -42,5 +42,5 @@
                     <mesh filename="${FILE_PATH}/meshes/head.${MODEL_TYPE}" scale="1 1 1"/>
                 </geometry>
-                <material name="black" />
+                <material name="silver" />
             </visual>
         </link>

File: soccer_description/models/leg.xacro (robot description, xacro)
@@ -20,5 +20,5 @@
                     <mesh filename="${FILE_PATH}/meshes/${name}_hip_side.${MODEL_TYPE}" scale="1 1 1"/>
                 </geometry>
-                <material name="black" />
+                <material name="cyan" />
             </visual>
         </link>
@@ -42,5 +42,5 @@
                     <mesh filename="${FILE_PATH}/meshes/${name}_hip_front.${MODEL_TYPE}" scale="1 1 1"/>
                 </geometry>
-                <material name="black" />
+                <material name="blue" />
             </visual>
         </link>
@@ -64,5 +64,5 @@
                     <mesh filename="${FILE_PATH}/meshes/${name}_thigh.${MODEL_TYPE}" scale="1 1 1"/>
                 </geometry>
-                <material name="black" />
+                <material name="red" />
             </visual>
         </link>
@@ -86,5 +86,5 @@
                     <mesh filename="${FILE_PATH}/meshes/${name}_calve.${MODEL_TYPE}" scale="1 1 1"/>
                 </geometry>
-                <material name="black" />
+                <material name="yellow" />
             </visual>
         </link>
@@ -108,5 +108,5 @@
                     <mesh filename="${FILE_PATH}/meshes/${name}_ankle.${MODEL_TYPE}" scale="1 1 1"/>
                 </geometry>
-                <material name="black" />
+                <material name="purple" />
             </visual>
         </link>
@@ -131,5 +131,5 @@
                     <mesh filename="${FILE_PATH}/meshes/${name}_foot.${MODEL_TYPE}" scale="1 1 1"/>
                 </geometry>
-                <material name="black" />
+                <material name="green" />
             </visual>
         </link>

File: soccer_description/models/parameters.xacro (robot description, xacro)
@@ -16,3 +16,27 @@
         <color rgba="0.0 0.0 0.0 1.0"/>
     </material>
+    <material name="silver">
+        <color rgba="0.7 0.7 0.7 1.0"/>
+    </material>
+    <material name="yellow">
+        <color rgba="0.9 0.9 0.0 1.0"/>
+    </material>
+    <material name="red">
+        <color rgba="0.7 0.0 0.0 1.0"/>
+    </material>
+    <material name="green">
+        <color rgba="0.0 0.7 0.0 1.0"/>
+    </material>
+    <material name="blue">
+        <color rgba="0.0 0.0 0.7 1.0"/>
+    </material>
+    <material name="purple">
+        <color rgba="0.7 0.0 0.7 1.0"/>
+    </material>
+    <material name="cyan">
+        <color rgba="0.0 0.7 0.7 1.0"/>
+    </material>
+    <material name="black">
+        <color rgba="0.2 0.2 0.2 1.0"/>
+    </material>
 </robot>

File: soccer_description/models/soccerbot.xacro (robot description, xacro)
@@ -33,4 +33,5 @@
                 <mesh filename="${FILE_PATH}/meshes/torso.${MODEL_TYPE}" scale="1 1 1"/>
             </geometry>
+            <material name="black" />
         </visual>
     </link>

File: soccer_description/models/soccerbot_stl.urdf (robot description, URDF)
Before this commit: robot soccerbot, 21 links, 20 joints
Links:
- link /left_forearm: geometry collision box size=0.035 0.049 0.144; visual mesh filename=../soccer_description/meshes/left_forearm.dae scale=1 1 1
- link /right_forearm: geometry collision box size=0.035 0.049 0.144; visual mesh filename=../soccer_description/meshes/right_forearm.dae scale=1 1 1

Commit message: Revert "Reverting & Fixing URDF bugs & Adding Colors"

File: soccer_description/models/arm.xacro (robot description, xacro)
@@ -20,5 +20,5 @@
                         <mesh filename="${FILE_PATH}/meshes/${name}_bicep.${MODEL_TYPE}" scale="1 1 1"/>
                     </geometry>
-                    <material name="white" />
+                    <material name="black" />
                 </visual>
             </link>
@@ -26,5 +26,5 @@
                 <inertial>
                     <mass value="45.7e-3"/>
-                    <origin rpy="0  0  0" xyz="0 ${direction * 0.0245} -0.0546097" />
+                    <origin rpy="0  0  0" xyz="0 0.0245 -0.0546097" />
                     <inertia ixx="0.113e-3" ixy="0.000" ixz="${direction * 0.001e-3}"
                              iyy="0.107e-3" iyz="${direction * 0.000}"
@@ -32,5 +32,5 @@
                 </inertial>
                 <collision name="collision">
-                    <origin rpy="0  0  0" xyz="-0.0055 ${direction * 0.01750} -0.0600"/>
+                    <origin rpy="0  0  0" xyz="-0.0055 0.01750 -0.0600"/>
                     <geometry>
                         <box size="0.035 0.049 0.144"/>
@@ -40,7 +40,7 @@
                     <origin rpy="0  0  0" xyz="0  0  0"/>
                     <geometry>
-                        <mesh filename="${FILE_PATH}/meshes/${name}_forearm.${MODEL_TYPE}" scale="1 1 1"/>
+                        <mesh filename="${FILE_PATH}/meshes/${name}_forearm.${MODEL_TYPE}" scale="0.001 0.001 0.001"/>
                     </geometry>
-                    <material name="purple" />
+                    <material name="black" />
                 </visual>
             </link>

File: soccer_description/models/head.xacro (robot description, xacro)
@@ -20,5 +20,5 @@
                     <mesh filename="${FILE_PATH}/meshes/neck.${MODEL_TYPE}" scale="1 1 1"/>
                 </geometry>
-                <material name="silver" />
+                <material name="black" />
             </visual>
         </link>
@@ -42,5 +42,5 @@
                     <mesh filename="${FILE_PATH}/meshes/head.${MODEL_TYPE}" scale="1 1 1"/>
                 </geometry>
-                <material name="silver" />
+                <material name="black" />
             </visual>
         </link>

File: soccer_description/models/leg.xacro (robot description, xacro)
@@ -20,5 +20,5 @@
                     <mesh filename="${FILE_PATH}/meshes/${name}_hip_side.${MODEL_TYPE}" scale="1 1 1"/>
                 </geometry>
-                <material name="cyan" />
+                <material name="black" />
             </visual>
         </link>
@@ -42,5 +42,5 @@
                     <mesh filename="${FILE_PATH}/meshes/${name}_hip_front.${MODEL_TYPE}" scale="1 1 1"/>
                 </geometry>
-                <material name="blue" />
+                <material name="black" />
             </visual>
         </link>
@@ -64,5 +64,5 @@
                     <mesh filename="${FILE_PATH}/meshes/${name}_thigh.${MODEL_TYPE}" scale="1 1 1"/>
                 </geometry>
-                <material name="red" />
+                <material name="black" />
             </visual>
         </link>
@@ -86,5 +86,5 @@
                     <mesh filename="${FILE_PATH}/meshes/${name}_calve.${MODEL_TYPE}" scale="1 1 1"/>
                 </geometry>
-                <material name="yellow" />
+                <material name="black" />
             </visual>
         </link>
@@ -108,5 +108,5 @@
                     <mesh filename="${FILE_PATH}/meshes/${name}_ankle.${MODEL_TYPE}" scale="1 1 1"/>
                 </geometry>
-                <material name="purple" />
+                <material name="black" />
             </visual>
         </link>
@@ -131,5 +131,5 @@
                     <mesh filename="${FILE_PATH}/meshes/${name}_foot.${MODEL_TYPE}" scale="1 1 1"/>
                 </geometry>
-                <material name="green" />
+                <material name="black" />
             </visual>
         </link>

File: soccer_description/models/parameters.xacro (robot description, xacro)
@@ -16,27 +16,3 @@
         <color rgba="0.0 0.0 0.0 1.0"/>
     </material>
-    <material name="silver">
-        <color rgba="0.7 0.7 0.7 1.0"/>
-    </material>
-    <material name="yellow">
-        <color rgba="0.9 0.9 0.0 1.0"/>
-    </material>
-    <material name="red">
-        <color rgba="0.7 0.0 0.0 1.0"/>
-    </material>
-    <material name="green">
-        <color rgba="0.0 0.7 0.0 1.0"/>
-    </material>
-    <material name="blue">
-        <color rgba="0.0 0.0 0.7 1.0"/>
-    </material>
-    <material name="purple">
-        <color rgba="0.7 0.0 0.7 1.0"/>
-    </material>
-    <material name="cyan">
-        <color rgba="0.0 0.7 0.7 1.0"/>
-    </material>
-    <material name="black">
-        <color rgba="0.2 0.2 0.2 1.0"/>
-    </material>
 </robot>

File: soccer_description/models/soccerbot.xacro (robot description, xacro)
@@ -33,5 +33,4 @@
                 <mesh filename="${FILE_PATH}/meshes/torso.${MODEL_TYPE}" scale="1 1 1"/>
             </geometry>
-            <material name="black" />
         </visual>
     </link>

File: soccer_description/models/soccerbot_stl.urdf (robot description, URDF)
Before this commit: robot soccerbot, 21 links, 20 joints
Links:
- link /left_forearm: geometry collision box size=0.035 0.049 0.144; visual mesh filename=../soccer_description/meshes/left_forearm.dae scale=0.001 0.001 0.001
- link /right_forearm: geometry collision box size=0.035 0.049 0.144; visual mesh filename=../soccer_description/meshes/right_forearm.dae scale=0.001 0.001 0.001
