Commit message: Added embedding
Former-commit-id: 9a2b05be7bc35ff0b41acb93bfc417c4a15df3cb [formerly 123e5be0715570c07b29a73072462fcd9066584f]
Former-commit-id: effb772e399737225a113cd5091f593b140a073a

File: soccer_description/models/imu.xacro (robot description, xacro)
@@ -13,5 +13,5 @@
             <parent link="${origin}"/>
             <child link="$(arg tf_prefix)/imu_link"/>
-            <origin rpy="0 0 0" xyz="0.1 0 0.0075"/>
+            <origin rpy="0 0 0" xyz="0.0 0 0.000"/>
             <axis xyz="0 0 0"/>
         </joint>
