Commit message: Updates ball position
Former-commit-id: 283fdd9251e814216e785cd0053db80b51ec2312 [formerly 0f167ef555ac284809a75dcf09100d78de512c21]
Former-commit-id: 32ca88834a4e677779439960ffb4da833fc24933

File: soccer_description/models/soccerbot_stl.urdf (robot description, URDF)
Before this commit: robot soccerbot, 21 links, 20 joints
Links:
- link head: geometry collision box size=0.0712 0.094 0.0779; visual mesh filename=../soccer_description/meshes/head.stl scale=1 1 1
Joints:
- joint head_camera: origin xyz=0.05295 0.00145 0.04740 rpy=0 0 0 -> xyz=0.015 0.00145 0.04740 rpy=0 0 0

Commit message: Actually Walking! + Basic IMU function added + Basic foot pressure sensor added
Former-commit-id: 9eba0d8960dc4a5e635f59e91e2ef5cac1dfabc0 [formerly 97bc45e97611a77bf46923b7669cd31661dcf896]
Former-commit-id: 4cc1b80d75dcc39f040e0855362d382047d3b583

File: soccer_description/models/soccerbot_stl.urdf (robot description, URDF)
Before this commit: robot soccerbot, 21 links, 20 joints
Links:
- link camera: mass None -> 0
- link imu_link: mass None -> 0.01

Commit message: add 4 pressure sensor on right foot
Former-commit-id: f58d9c96ec019aae39bb8d2fc6864c515bb39596 [formerly 298674e6a581d65f588b02fada4a46ab4ca2379b]
Former-commit-id: aeb71f5e322d642478d841f51b68ce7fc2472c60

File: soccer_description/models/soccerbot_stl.urdf (robot description, URDF)
Before this commit: robot soccerbot, 21 links, 20 joints
Links:
- link camera: mass 0 -> None
- link imu_link: mass 0.01 -> None

Commit message: reverted model
Former-commit-id: 6074cdb8091ec70e3dcf2be63496edff95f2a469 [formerly 5e625f6670245387c354a7b274090ddc8533fdd1]
Former-commit-id: 1d03a8584cf377b33544031a4bd5568f810eb676

File: soccer_description/models/soccerbot_stl.urdf (robot description, URDF)
Before this commit: robot soccerbot, 21 links, 20 joints
Joints:
- joint /torso_imu: origin xyz=0.1 0 0.0075 rpy=0 0 0 -> xyz=0.0 0 0.000 rpy=0 0 0
