Commit message: Update trajectories

File: soccer_description/models/parameters.xacro (robot description, xacro)
@@ -7,6 +7,6 @@
     <xacro:property name="FOREARM_MU1" value="0.2"/>
     <xacro:property name="FOREARM_MU2" value="0.2"/>
-    <xacro:property name="JOINT_FRICTION" value="0.05"/>
-    <xacro:property name="JOINT_DAMPING" value="0.02"/>
+    <xacro:property name="JOINT_FRICTION" value="0.005"/>
+    <xacro:property name="JOINT_DAMPING" value="0.005"/>
     <xacro:property name="MX28_TORQUE" value="2.5"/>
     <xacro:property name="MX28_VELOCITY" value="1"/>

Commit message: tuned parameters so that the robot stands most of the time

File: soccer_description/models/parameters.xacro (robot description, xacro)
@@ -7,6 +7,6 @@
     <xacro:property name="FOREARM_MU1" value="0.2"/>
     <xacro:property name="FOREARM_MU2" value="0.2"/>
-    <xacro:property name="JOINT_FRICTION" value="0.05"/>
-    <xacro:property name="JOINT_DAMPING" value="0.02"/>
+    <xacro:property name="JOINT_FRICTION" value="0.00"/>
+    <xacro:property name="JOINT_DAMPING" value="0.01"/>
     <xacro:property name="MX28_TORQUE" value="2.5"/>
     <xacro:property name="MX28_VELOCITY" value="1"/>

Commit message: add friction to damp away oscilations when robot is standing
Former-commit-id: 0cfbee5ba48ce7d737f939dca5b95bcaceb489d2 [formerly 8eb1d1f2324132df4b7b3632322d44d61a9257c3]
Former-commit-id: 6e581cc984106d9b3f9ea92ee45aeef6f27bf836

File: soccer_description/models/parameters.xacro (robot description, xacro)
@@ -7,5 +7,5 @@
     <xacro:property name="FOREARM_MU1" value="0.2"/>
     <xacro:property name="FOREARM_MU2" value="0.2"/>
-    <xacro:property name="JOINT_FRICTION" value="0.00"/>
+    <xacro:property name="JOINT_FRICTION" value="0.1"/>
     <xacro:property name="JOINT_DAMPING" value="0.01"/>
     <xacro:property name="MX28_TORQUE" value="2.5"/>

File: soccer_description/models/soccerbot.xacro (robot description, xacro)
@@ -5,11 +5,4 @@
     <soccerbot />
     <link name="base_link" />
-    <link name="world" />
-    <joint name="base_link_map" type="fixed">
-        <parent link="world"/>
-        <child link="base_link"/>
-        <origin rpy="0 0 0" xyz="0 0 0"/>
-        <axis xyz="1 0 0"/>
-    </joint>
     <joint name="base_link_torso" type="fixed">
         <parent link="base_link"/>

Commit message: Delete strategy
Former-commit-id: b88473400f8962aaaacf2fe57221c762a94e80dc [formerly 448d61adbe1d976206568648edbf302603035910]
Former-commit-id: bdd0381c0f5d83771d60bd5469f6c1c9f7f08cb0

File: soccer_description/models/parameters.xacro (robot description, xacro)
@@ -13,3 +13,6 @@
     <xacro:property name="AX12_TORQUE" value="1.5"/>
     <xacro:property name="AX12_VELOCITY" value="1"/>
+    <material name="black">
+        <color rgba="0.0 0.0 0.0 1.0"/>
+    </material>
 </robot>

File: soccer_description/models/soccerbot_stl.urdf (robot description, URDF)
Before this commit: robot soccerbot, 21 links, 20 joints
Links:
- link head: geometry collision box size=0.0712 0.094 0.0779; visual mesh filename=../soccer_description/meshes/head.dae scale=1 1 1
- link left_ankle: geometry collision box size=0.090769 0.042 0.0506; visual mesh filename=../soccer_description/meshes/left_ankle.dae scale=1 1 1
- link left_bicep: geometry collision box size=0.04 0.04776 0.123; visual mesh filename=../soccer_description/meshes/left_bicep.dae scale=1 1 1
- link left_calve: geometry collision box size=0.031883 0.048 0.105683; visual mesh filename=../soccer_description/meshes/left_calve.dae scale=1 1 1
- link left_foot: geometry collision box size=0.09 0.07 0.03674; visual mesh filename=../soccer_description/meshes/left_foot.dae scale=1 1 1
- link left_forearm: geometry collision box size=0.035 0.049 0.144; visual mesh filename=../soccer_description/meshes/left_forearm.dae scale=1 1 1
- link left_hip_front: geometry collision box size=0.083747 0.04885 0.0506; visual mesh filename=../soccer_description/meshes/left_hip_front.dae scale=1 1 1
- link left_hip_side: geometry collision box size=0.0485 0.022 0.0039; visual mesh filename=../soccer_description/meshes/left_hip_side.dae scale=1 1 1
- link left_thigh: geometry collision box size=0.022 0.048 0.111; visual mesh filename=../soccer_description/meshes/left_thigh.dae scale=1 1 1
- link neck: geometry collision box size=0.022 0.0523 0.033; visual mesh filename=../soccer_description/meshes/neck.dae scale=1 1 1
- link right_ankle: geometry collision box size=0.090769 0.042 0.0506; visual mesh filename=../soccer_description/meshes/right_ankle.dae scale=1 1 1
- link right_bicep: geometry collision box size=0.04 0.04776 0.123; visual mesh filename=../soccer_description/meshes/right_bicep.dae scale=1 1 1
- link right_calve: geometry collision box size=0.031883 0.048 0.105683; visual mesh filename=../soccer_description/meshes/right_calve.dae scale=1 1 1
- link right_foot: geometry collision box size=0.09 0.07 0.03674; visual mesh filename=../soccer_description/meshes/right_foot.dae scale=1 1 1
- link right_forearm: geometry collision box size=0.035 0.049 0.144; visual mesh filename=../soccer_description/meshes/right_forearm.dae scale=1 1 1
- link right_hip_front: geometry collision box size=0.083747 0.04885 0.0506; visual mesh filename=../soccer_description/meshes/right_hip_front.dae scale=1 1 1
- link right_hip_side: geometry collision box size=0.0485 0.022 0.0039; visual mesh filename=../soccer_description/meshes/right_hip_side.dae scale=1 1 1
- link right_thigh: geometry collision box size=0.022 0.048 0.111; visual mesh filename=../soccer_description/meshes/right_thigh.dae scale=1 1 1
- link torso: geometry collision box size=0.130 0.145 0.152; visual mesh filename=../soccer_description/meshes/torso.dae scale=1 1 1
Joints:
- joint head_motor_0: limit lower=-1.57079632679 upper=1.57079632679 effort=1.5 velocity=1 -> lower=-1.5707963267948966 upper=1.5707963267948966 effort=1.5 velocity=1
- joint head_motor_1: limit lower=-2.35619449019 upper=2.35619449019 effort=1.5 velocity=1 -> lower=-2.356194490192345 upper=2.356194490192345 effort=1.5 velocity=1
- joint left_arm_motor_0: limit lower=-1.57079632679 upper=3.92699081699 effort=1.5 velocity=1 -> lower=-1.5707963267948966 upper=3.9269908169872414 effort=1.5 velocity=1
- joint left_arm_motor_1: limit lower=0 upper=3.14159265359 effort=1.5 velocity=1 -> lower=0 upper=3.141592653589793 effort=1.5 velocity=1
- joint left_leg_motor_1: limit lower=-0.785398163397 upper=1.57079632679 effort=2.5 velocity=1 -> lower=-0.7853981633974483 upper=1.5707963267948966 effort=2.5 velocity=1
- joint left_leg_motor_2: limit lower=-0.785398163397 upper=2.35619449019 effort=2.5 velocity=1 -> lower=-0.7853981633974483 upper=2.356194490192345 effort=2.5 velocity=1
- joint left_leg_motor_4: limit lower=-0.785398163397 upper=1.57079632679 effort=2.5 velocity=1 -> lower=-0.7853981633974483 upper=1.5707963267948966 effort=2.5 velocity=1
- joint left_leg_motor_5: limit lower=-0.785398163397 upper=0.785398163397 effort=2.5 velocity=1 -> lower=-0.7853981633974483 upper=0.7853981633974483 effort=2.5 velocity=1
- joint right_arm_motor_0: limit lower=-1.57079632679 upper=3.92699081699 effort=1.5 velocity=1 -> lower=-1.5707963267948966 upper=3.9269908169872414 effort=1.5 velocity=1
- joint right_arm_motor_1: limit lower=0 upper=3.14159265359 effort=1.5 velocity=1 -> lower=0 upper=3.141592653589793 effort=1.5 velocity=1
- joint right_leg_motor_1: limit lower=-0.785398163397 upper=1.57079632679 effort=2.5 velocity=1 -> lower=-0.7853981633974483 upper=1.5707963267948966 effort=2.5 velocity=1
- joint right_leg_motor_2: limit lower=-0.785398163397 upper=2.35619449019 effort=2.5 velocity=1 -> lower=-0.7853981633974483 upper=2.356194490192345 effort=2.5 velocity=1
- joint right_leg_motor_4: limit lower=-0.785398163397 upper=1.57079632679 effort=2.5 velocity=1 -> lower=-0.7853981633974483 upper=1.5707963267948966 effort=2.5 velocity=1
- joint right_leg_motor_5: limit lower=-0.785398163397 upper=0.785398163397 effort=2.5 velocity=1 -> lower=-0.7853981633974483 upper=0.7853981633974483 effort=2.5 velocity=1

Commit message: fix black
Former-commit-id: 57ef82f6138dca2cfad20fc2135da1a79ffdce26 [formerly c88470feff3b887bd599d6e8ba6d0941d47ecee1]
Former-commit-id: fe14c5db4211cf614ff4ec86042bd7ebb8633492

File: soccer_description/models/parameters.xacro (robot description, xacro)
@@ -37,6 +37,3 @@
         <color rgba="0.0 0.7 0.7 1.0"/>
     </material>
-    <material name="black">
-        <color rgba="0.2 0.2 0.2 1.0"/>
-    </material>
 </robot>

Commit message: Removed Duplicate Black Color

File: soccer_description/models/parameters.xacro (robot description, xacro)
@@ -13,7 +13,4 @@
     <xacro:property name="AX12_TORQUE" value="1.5"/>
     <xacro:property name="AX12_VELOCITY" value="1"/>
-    <material name="black">
-        <color rgba="0.0 0.0 0.0 1.0"/>
-    </material>
     <material name="silver">
         <color rgba="0.7 0.7 0.7 1.0"/>

Commit message: fixed parameter.xacro

File: soccer_description/models/parameters.xacro (robot description, xacro)
@@ -34,3 +34,6 @@
         <color rgba="0.0 0.7 0.7 1.0"/>
     </material>
+    <material name="black">
+        <color rgba="0.2 0.2 0.2 1.0"/>
+    </material>
 </robot>

Commit message: Cleaned up literaly everything
Former-commit-id: 8e656e5603cddecc9886e959717af64d4a71b090 [formerly 9dde6fe28d10c54e6793a138e91079dc75c2252e]
Former-commit-id: ee1581a2ae7e9e4c7154b6e7ef42be0ae8585d1f

File: soccer_description/models/parameters.xacro (robot description, xacro)
@@ -13,4 +13,7 @@
     <xacro:property name="AX12_TORQUE" value="1.5"/>
     <xacro:property name="AX12_VELOCITY" value="1"/>
+    <material name="white">
+        <color rgba="1.0 1.0 1.0 1.0"/>
+    </material>
     <material name="black">
         <color rgba="0.0 0.0 0.0 1.0"/>
