Commit message: Added foxglove

File: bez1_description/urdf/bez1.urdf (robot description, URDF)
Before this commit: robot bez1, 21 links, 20 joints
Links:
- link /head: geometry collision box size=0.0712 0.094 0.0779; visual mesh filename=../meshes/head.dae scale=1 1 1
- link /left_ankle: geometry collision box size=0.090769 0.042 0.0506; visual mesh filename=../meshes/left_ankle.dae scale=1 1 1
- link /left_bicep: geometry collision box size=0.04 0.04776 0.123; visual mesh filename=../meshes/left_bicep.dae scale=1 1 1
- link /left_calve: geometry collision box size=0.031883 0.048 0.105683; visual mesh filename=../meshes/left_calve.dae scale=1 1 1
- link /left_foot: geometry collision box size=0.09 0.07 0.03674; visual mesh filename=../meshes/left_foot.dae scale=1 1 1
- link /left_forearm: geometry collision box size=0.035 0.049 0.144; visual mesh filename=../meshes/left_forearm.dae scale=1 1 1
- link /left_hip_front: geometry collision box size=0.083747 0.04885 0.0506; visual mesh filename=../meshes/left_hip_front.dae scale=1 1 1
- link /left_hip_side: geometry collision box size=0.0485 0.022 0.0039; visual mesh filename=../meshes/left_hip_side.dae scale=1 1 1
- link /left_thigh: geometry collision box size=0.022 0.048 0.111; visual mesh filename=../meshes/left_thigh.dae scale=1 1 1
- link /neck: geometry collision box size=0.022 0.0523 0.033; visual mesh filename=../meshes/neck.dae scale=1 1 1
- link /right_ankle: geometry collision box size=0.090769 0.042 0.0506; visual mesh filename=../meshes/right_ankle.dae scale=1 1 1
- link /right_bicep: geometry collision box size=0.04 0.04776 0.123; visual mesh filename=../meshes/right_bicep.dae scale=1 1 1
- link /right_calve: geometry collision box size=0.031883 0.048 0.105683; visual mesh filename=../meshes/right_calve.dae scale=1 1 1
- link /right_foot: geometry collision box size=0.09 0.07 0.03674; visual mesh filename=../meshes/right_foot.dae scale=1 1 1
- link /right_forearm: geometry collision box size=0.035 0.049 0.144; visual mesh filename=../meshes/right_forearm.dae scale=1 1 1
- link /right_hip_front: geometry collision box size=0.083747 0.04885 0.0506; visual mesh filename=../meshes/right_hip_front.dae scale=1 1 1
- link /right_hip_side: geometry collision box size=0.0485 0.022 0.0039; visual mesh filename=../meshes/right_hip_side.dae scale=1 1 1
- link /right_thigh: geometry collision box size=0.022 0.048 0.111; visual mesh filename=../meshes/right_thigh.dae scale=1 1 1
- link /torso: geometry collision box size=0.130 0.145 0.152; visual mesh filename=../meshes/torso.dae scale=1 1 1

Commit message: revert urdf changes back

File: bez1_description/urdf/bez1.urdf (robot description, URDF)
Before this commit: robot bez1, 21 links, 20 joints
Links:
- link /head: geometry collision box size=0.0712 0.094 0.0779; visual mesh filename=../bez1_description/meshes/head.dae scale=1 1 1
- link /left_ankle: geometry collision box size=0.090769 0.042 0.0506; visual mesh filename=../bez1_description/meshes/left_ankle.dae scale=1 1 1
- link /left_bicep: geometry collision box size=0.04 0.04776 0.123; visual mesh filename=../bez1_description/meshes/left_bicep.dae scale=1 1 1
- link /left_calve: geometry collision box size=0.031883 0.048 0.105683; visual mesh filename=../bez1_description/meshes/left_calve.dae scale=1 1 1
- link /left_foot: geometry collision box size=0.09 0.07 0.03674; visual mesh filename=../bez1_description/meshes/left_foot.dae scale=1 1 1
- link /left_forearm: geometry collision box size=0.035 0.049 0.144; visual mesh filename=../bez1_description/meshes/left_forearm.dae scale=1 1 1
- link /left_hip_front: geometry collision box size=0.083747 0.04885 0.0506; visual mesh filename=../bez1_description/meshes/left_hip_front.dae scale=1 1 1
- link /left_hip_side: geometry collision box size=0.0485 0.022 0.0039; visual mesh filename=../bez1_description/meshes/left_hip_side.dae scale=1 1 1
- link /left_thigh: geometry collision box size=0.022 0.048 0.111; visual mesh filename=../bez1_description/meshes/left_thigh.dae scale=1 1 1
- link /neck: geometry collision box size=0.022 0.0523 0.033; visual mesh filename=../bez1_description/meshes/neck.dae scale=1 1 1
- link /right_ankle: geometry collision box size=0.090769 0.042 0.0506; visual mesh filename=../bez1_description/meshes/right_ankle.dae scale=1 1 1
- link /right_bicep: geometry collision box size=0.04 0.04776 0.123; visual mesh filename=../bez1_description/meshes/right_bicep.dae scale=1 1 1
- link /right_calve: geometry collision box size=0.031883 0.048 0.105683; visual mesh filename=../bez1_description/meshes/right_calve.dae scale=1 1 1
- link /right_foot: geometry collision box size=0.09 0.07 0.03674; visual mesh filename=../bez1_description/meshes/right_foot.dae scale=1 1 1
- link /right_forearm: geometry collision box size=0.035 0.049 0.144; visual mesh filename=../bez1_description/meshes/right_forearm.dae scale=1 1 1
- link /right_hip_front: geometry collision box size=0.083747 0.04885 0.0506; visual mesh filename=../bez1_description/meshes/right_hip_front.dae scale=1 1 1
- link /right_hip_side: geometry collision box size=0.0485 0.022 0.0039; visual mesh filename=../bez1_description/meshes/right_hip_side.dae scale=1 1 1
- link /right_thigh: geometry collision box size=0.022 0.048 0.111; visual mesh filename=../bez1_description/meshes/right_thigh.dae scale=1 1 1
- link /torso: geometry collision box size=0.130 0.145 0.152; visual mesh filename=../bez1_description/meshes/torso.dae scale=1 1 1
