Commit message: Bez 3 fixed masses and inertias
Fusion model updated with more accurate material. Begin tuning walking.

File: bez3_description/urdf/bez3.urdf (robot description, URDF)
Before this commit: robot bez3, 52 links, 51 joints
Links:
- removed link JX_servo_v8_1
- removed link JX_servo_v8_11
- removed link JX_servo_v8_12
- removed link JX_servo_v8_13
- removed link JX_servo_v8_14
- removed link JX_servo_v8_15
- removed link JX_servo_v8_16
- removed link JX_servo_v8_17
- removed link JX_servo_v8_18
- removed link JX_servo_v8_19
- removed link JX_servo_v8_8
- removed link JX_servo_v8_9
- removed link custom_servo_support__lower_neck__v1_1
- added link Component32_1, mass 0.31999527000000005; collision mesh filename=package://bez3_description/meshes/Component32_1.stl scale=0.001 0.001 0.001; visual mesh filename=package://bez3_description/meshes/Component32_1.stl scale=0.001 0.001 0.001
- added link JX_servo_v12_1, mass 0.19853540350189508; collision mesh filename=package://bez3_description/meshes/JX_servo_v12_1.stl scale=0.001 0.001 0.001; visual mesh filename=package://bez3_description/meshes/JX_servo_v12_1.stl scale=0.001 0.001 0.001
- added link JX_servo_v12_11, mass 0.19853540350189508; collision mesh filename=package://bez3_description/meshes/JX_servo_v12_11.stl scale=0.001 0.001 0.001; visual mesh filename=package://bez3_description/meshes/JX_servo_v12_11.stl scale=0.001 0.001 0.001
- added link JX_servo_v12_12, mass 0.19853540350189508; collision mesh filename=package://bez3_description/meshes/JX_servo_v12_12.stl scale=0.001 0.001 0.001; visual mesh filename=package://bez3_description/meshes/JX_servo_v12_12.stl scale=0.001 0.001 0.001
- added link JX_servo_v12_13, mass 0.19853540350189508; collision mesh filename=package://bez3_description/meshes/JX_servo_v12_13.stl scale=0.001 0.001 0.001; visual mesh filename=package://bez3_description/meshes/JX_servo_v12_13.stl scale=0.001 0.001 0.001
- added link JX_servo_v12_14, mass 0.19853540350189508; collision mesh filename=package://bez3_description/meshes/JX_servo_v12_14.stl scale=0.001 0.001 0.001; visual mesh filename=package://bez3_description/meshes/JX_servo_v12_14.stl scale=0.001 0.001 0.001
- added link JX_servo_v12_15, mass 0.19853540350189508; collision mesh filename=package://bez3_description/meshes/JX_servo_v12_15.stl scale=0.001 0.001 0.001; visual mesh filename=package://bez3_description/meshes/JX_servo_v12_15.stl scale=0.001 0.001 0.001
- added link JX_servo_v12_16, mass 0.19853540350189508; collision mesh filename=package://bez3_description/meshes/JX_servo_v12_16.stl scale=0.001 0.001 0.001; visual mesh filename=package://bez3_description/meshes/JX_servo_v12_16.stl scale=0.001 0.001 0.001
- added link JX_servo_v12_17, mass 0.19853540350189508; collision mesh filename=package://bez3_description/meshes/JX_servo_v12_17.stl scale=0.001 0.001 0.001; visual mesh filename=package://bez3_description/meshes/JX_servo_v12_17.stl scale=0.001 0.001 0.001
- added link JX_servo_v12_18, mass 0.19853540350189508; collision mesh filename=package://bez3_description/meshes/JX_servo_v12_18.stl scale=0.001 0.001 0.001; visual mesh filename=package://bez3_description/meshes/JX_servo_v12_18.stl scale=0.001 0.001 0.001
- added link JX_servo_v12_19, mass 0.19853540350189508; collision mesh filename=package://bez3_description/meshes/JX_servo_v12_19.stl scale=0.001 0.001 0.001; visual mesh filename=package://bez3_description/meshes/JX_servo_v12_19.stl scale=0.001 0.001 0.001
- added link JX_servo_v12_8, mass 0.19853540350189508; collision mesh filename=package://bez3_description/meshes/JX_servo_v12_8.stl scale=0.001 0.001 0.001; visual mesh filename=package://bez3_description/meshes/JX_servo_v12_8.stl scale=0.001 0.001 0.001
- added link JX_servo_v12_9, mass 0.19853540350189508; collision mesh filename=package://bez3_description/meshes/JX_servo_v12_9.stl scale=0.001 0.001 0.001; visual mesh filename=package://bez3_description/meshes/JX_servo_v12_9.stl scale=0.001 0.001 0.001
- added link TX2_board_v2_1, mass 0.2621637298853286; collision mesh filename=package://bez3_description/meshes/TX2_board_v2_1.stl scale=0.001 0.001 0.001; visual mesh filename=package://bez3_description/meshes/TX2_board_v2_1.stl scale=0.001 0.001 0.001
- added link custom_servo_support__lower_neck__v2_1, mass 0.003136252201459725; collision mesh filename=package://bez3_description/meshes/custom_servo_support__low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 scale=0.001 0.001 0.001; visual mesh filename=package://bez3_description/meshes/custom_servo_support__low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 scale=0.001 0.001 0.001
- link 25t-servo-hub_1: mass 0.016237434875861913 -> 0.005584850212079893
- link 25t-servo-hub_2: mass 0.016237434875861913 -> 0.005584850212079893
- link 25t-servo-hub_3: mass 0.016237434875861913 -> 0.005584850212079893
- link 25t-servo-hub_4: mass 0.016237434875861913 -> 0.005584850212079893
- link 25t-servo-hub_Mirror__1: mass 0.016236664394569493 -> 0.005584585205775494
- link 25t-servo-hub_Mirror__2: mass 0.016236664394569493 -> 0.005584585205775494
- link camera_1: mass 0.17999927702289192 -> 0.094257141411043
- link elbow-attach_1: mass 0.05766200981695701 -> 0.005141835270301899
- link elbow-attach_Mirror__1: mass 0.05766200981695702 -> 0.005141835270301901
- link elbow-bearing_1: mass 0.05541781310486511 -> 0.004941715818268227
- link elbow-bearing_Mirror__1: mass 0.05541781310486507 -> 0.004941715818268223
- link gobilda-servo_1: mass 0.19736839764730799 -> 0.060587311248822606
- link gobilda-servo_3: mass 0.19736839764730799 -> 0.060587311248822606
- link gobilda-servo_4: mass 0.19736839764730799 -> 0.060587311248822606
- link gobilda-servo_5: mass 0.19736839764730799 -> 0.060587311248822606
- link gobilda-servo_Mirror__1: mass 0.197368397647308 -> 0.06058731124882261
- link gobilda-servo_Mirror__2: mass 0.197368397647308 -> 0.06058731124882261
- link head_1: mass 0.08583116046555261 -> 0.007653734054253099
- link left_bicep_1: mass 0.017347091316258258 -> 0.011455626340925264
- link left_calve_1: mass 0.514989606773696 -> 0.035688451730559324
- link left_foot_1: mass 0.34210600833439103 -> 0.03704332574321432
- link left_forearm_1: mass 0.306954483317309 -> 0.027371737365874692
- link left_hip_front_1: mass 0.2801003105283029 -> 0.025976181664280836
- link left_hip_front_2: mass 0.2801003105283029 -> 0.025976181664280836
- link left_hip_side_1: mass 0.21965915789216364 -> 0.018999817606213904
- link left_thigh_1: mass 0.5622725416559319 -> 0.04698736144283967
- link neck_1: mass 0.1451172084285195 -> 0.012940388012734224
- link right_ankle_1: mass 0.2801003105283028 -> 0.025976181664280826
- link right_ankle_2: mass 0.2801003105283028 -> 0.025976181664280826
- link right_bicep_1: mass 0.017347091316258265 -> 0.011455626340925269
- link right_calve_1: mass 0.5149901707605673 -> 0.03568840560735723
- link right_foot_1: mass 0.3421060083343909 -> 0.037043325743214305
- link right_forearm_1: mass 0.306954483317309 -> 0.027371737365874692
- link right_hip_side_1: mass 0.2196591578921638 -> 0.018999817606213918
- link right_thigh_1: mass 0.5622720012981443 -> 0.04698731628682583
- link torso_1: mass 3.328477451240261 -> 0.2968069064800233
Joints:
- added joint Rigid52: type fixed, parent torso_1, child Component32_1, origin xyz=-0.012 -0.004667 -0.005 rpy=0 0 0
- added joint Rigid53: type fixed, parent Component32_1, child TX2_board_v2_1, origin xyz=0.0 0.0 -0.047 rpy=0 0 0
- joint Rigid11: parent JX_servo_v8_12 -> JX_servo_v12_12
- joint Rigid12: child JX_servo_v8_13 -> JX_servo_v12_13
- joint Rigid14: child JX_servo_v8_14 -> JX_servo_v12_14
- joint Rigid17: parent JX_servo_v8_15 -> JX_servo_v12_15
- joint Rigid18: child JX_servo_v8_16 -> JX_servo_v12_16
- joint Rigid2: child JX_servo_v8_1 -> JX_servo_v12_1
- joint Rigid21: origin xyz=0.0085 0.0225 -0.0549 rpy=0 0 0 -> xyz=0.0085 0.0264 -0.0549 rpy=0 0 0; parent JX_servo_v8_17 -> JX_servo_v12_17
- joint Rigid23: parent JX_servo_v8_18 -> JX_servo_v12_18
- joint Rigid24: child JX_servo_v8_19 -> JX_servo_v12_19
- joint Rigid42: child custom_servo_support__lower_neck__v1_1 -> custom_servo_support__lower_neck__v2_1
- joint Rigid43: parent custom_servo_support__lower_neck__v1_1 -> custom_servo_support__lower_neck__v2_1
- joint Rigid5: parent JX_servo_v8_8 -> JX_servo_v12_8
- joint Rigid6: child JX_servo_v8_9 -> JX_servo_v12_9
- joint Rigid9: parent JX_servo_v8_11 -> JX_servo_v12_11
- joint left_arm_motor_1: axis -0.0 1.0 -0.0 -> -0.0 -1.0 -0.0
- joint left_leg_motor_0: parent JX_servo_v8_1 -> JX_servo_v12_1
- joint left_leg_motor_1: child JX_servo_v8_8 -> JX_servo_v12_8
- joint left_leg_motor_2: parent JX_servo_v8_9 -> JX_servo_v12_9
- joint left_leg_motor_3: child JX_servo_v8_11 -> JX_servo_v12_11
- joint left_leg_motor_4: child JX_servo_v8_12 -> JX_servo_v12_12
- joint left_leg_motor_5: parent JX_servo_v8_13 -> JX_servo_v12_13
- joint right_arm_motor_1: axis -0.0 1.0 0.0 -> -0.0 -1.0 0.0
- joint right_leg_motor_0: axis -0.0 0.0 -1.0 -> -0.0 0.0 1.0; parent JX_servo_v8_14 -> JX_servo_v12_14
- joint right_leg_motor_1: child JX_servo_v8_15 -> JX_servo_v12_15
- joint right_leg_motor_2: parent JX_servo_v8_16 -> JX_servo_v12_16
- joint right_leg_motor_3: child JX_servo_v8_17 -> JX_servo_v12_17
- joint right_leg_motor_4: child JX_servo_v8_18 -> JX_servo_v12_18
- joint right_leg_motor_5: parent JX_servo_v8_19 -> JX_servo_v12_19
