Commit message: Bez 3 fixed masses and inertias
Fusion model updated with more accurate material. Begin tuning walking.

File: bez3_description/urdf/bez3.xacro (robot description, xacro)
@@ -26,7 +26,7 @@
 <link name="torso_1">
   <inertial>
-    <origin xyz="-0.003658211229359205 -0.006167940664238083 -0.07338742094913073" rpy="0 0 0"/>
-    <mass value="3.328477451240261"/>
-    <inertia ixx="0.029875" iyy="0.013936" izz="0.024705" ixy="5.6e-05" iyz="5e-06" ixz="0.000674"/>
+    <origin xyz="-0.003658211229359205 -0.006167940664238083 -0.07338742094913071" rpy="0 0 0"/>
+    <mass value="0.2968069064800233"/>
+    <inertia ixx="0.002664" iyy="0.001243" izz="0.002203" ixy="5e-06" iyz="0.0" ixz="6e-05"/>
   </inertial>
   <visual>
@@ -44,21 +44,21 @@
   </collision>
 </link>
-<link name="JX_servo_v8_1">
-  <inertial>
-    <origin xyz="0.0002196166185167714 -2.643121901901857e-10 0.014139939556201991" rpy="0 0 0"/>
-    <mass value="1.0848385350345584"/>
-    <inertia ixx="0.00045" iyy="0.000785" izz="0.000503" ixy="-0.0" iyz="0.0" ixz="4.6e-05"/>
+<link name="JX_servo_v12_1">
+  <inertial>
+    <origin xyz="0.00027407227629309625 4.531028330312381e-13 0.012509678934478005" rpy="0 0 0"/>
+    <mass value="0.19853540350189508"/>
+    <inertia ixx="7.7e-05" iyy="0.000137" izz="9e-05" ixy="0.0" iyz="0.0" ixz="6e-06"/>
   </inertial>
   <visual>
     <origin xyz="0.0225 -0.0545 0.13699" rpy="0 0 0"/>
     <geometry>
-      <mesh filename="package://bez3_description/meshes/JX_servo_v8_1.stl" scale="0.001 0.001 0.001"/>
-    </geometry>
-    <material name="copper_polished"/>
+      <mesh filename="package://bez3_description/meshes/JX_servo_v12_1.stl" scale="0.001 0.001 0.001"/>
+    </geometry>
+    <material name="plastic_matte_black"/>
   </visual>
   <collision>
     <origin xyz="0.0225 -0.0545 0.13699" rpy="0 0 0"/>
     <geometry>
-      <mesh filename="package://bez3_description/meshes/JX_servo_v8_1.stl" scale="0.001 0.001 0.001"/>
+      <mesh filename="package://bez3_description/meshes/JX_servo_v12_1.stl" scale="0.001 0.001 0.001"/>
     </geometry>
   </collision>
@@ -67,6 +67,6 @@
   <inertial>
     <origin xyz="-0.0006601764265435524 7.984241046088414e-10 -0.021141547194982763" rpy="0 0 0"/>
-    <mass value="0.21965915789216364"/>
-    <inertia ixx="0.000107" iyy="0.000213" izz="0.000165" ixy="0.0" iyz="0.0" ixz="-2e-06"/>
+    <mass value="0.018999817606213904"/>
+    <inertia ixx="9e-06" iyy="1.8e-05" izz="1.4e-05" ixy="0.0" iyz="0.0" ixz="-0.0"/>
   </inertial>
   <visual>
@@ -75,5 +75,5 @@
       <mesh filename="package://bez3_description/meshes/left_hip_side_1.stl" scale="0.001 0.001 0.001"/>
     </geometry>
-    <material name="steel_satin"/>
+    <material name="plastic_glossy_black"/>
   </visual>
   <collision>
@@ -84,21 +84,21 @@
   </collision>
 </link>
-<link name="JX_servo_v8_8">
-  <inertial>
-    <origin xyz="-0.04053993955620194 -2.643123636625333e-10 -0.017780294556127285" rpy="0 0 0"/>
-    <mass value="1.0848385350345584"/>
-    <inertia ixx="0.000503" iyy="0.000785" izz="0.00045" ixy="-0.0" iyz="-0.0" ixz="-4.6e-05"/>
+<link name="JX_servo_v12_8">
+  <inertial>
+    <origin xyz="-0.03890967893447789 4.529293606836404e-13 -0.017725838898350915" rpy="0 0 0"/>
+    <mass value="0.19853540350189508"/>
+    <inertia ixx="9e-05" iyy="0.000137" izz="7.7e-05" ixy="-0.0" iyz="0.0" ixz="-6e-06"/>
   </inertial>
   <visual>
     <origin xyz="0.0345 -0.0545 0.198726" rpy="0 0 0"/>
     <geometry>
-      <mesh filename="package://bez3_description/meshes/JX_servo_v8_8.stl" scale="0.001 0.001 0.001"/>
-    </geometry>
-    <material name="copper_polished"/>
+      <mesh filename="package://bez3_description/meshes/JX_servo_v12_8.stl" scale="0.001 0.001 0.001"/>
+    </geometry>
+    <material name="plastic_matte_black"/>
   </visual>
   <collision>
     <origin xyz="0.0345 -0.0545 0.198726" rpy="0 0 0"/>
     <geometry>
-      <mesh filename="package://bez3_description/meshes/JX_servo_v8_8.stl" scale="0.001 0.001 0.001"/>
+      <mesh filename="package://bez3_description/meshes/JX_servo_v12_8.stl" scale="0.001 0.001 0.001"/>
     </geometry>
   </collision>
@@ -106,7 +106,7 @@
 <link name="left_hip_front_1">
   <inertial>
-    <origin xyz="0.02375859039821049 0.009336273295607947 -0.06494791715192266" rpy="0 0 0"/>
-    <mass value="0.2801003105283029"/>
-    <inertia ixx="0.00024" iyy="0.000331" izz="0.000219" ixy="2e-06" iyz="-3e-06" ixz="8.6e-05"/>
+    <origin xyz="0.023758590398210495 0.009336273295607947 -0.06494791715192266" rpy="0 0 0"/>
+    <mass value="0.025976181664280836"/>
+    <inertia ixx="2.2e-05" iyy="3.1e-05" izz="2e-05" ixy="0.0" iyz="-0.0" ixz="8e-06"/>
   </inertial>
   <visual>
@@ -115,5 +115,5 @@
       <mesh filename="package://bez3_description/meshes/left_hip_front_1.stl" scale="0.001 0.001 0.001"/>
     </geometry>
-    <material name="steel_satin"/>
+    <material name="plastic_glossy_black"/>
   </visual>
   <collision>
@@ -124,21 +124,21 @@
   </collision>
 </link>
-<link name="JX_servo_v8_9">
-  <inertial>
-    <origin xyz="-0.008499999392960884 -0.01803993921347575 0.037119705443873385" rpy="0 0 0"/>
-    <mass value="1.0848385350345584"/>
-    <inertia ixx="0.000785" iyy="0.000503" izz="0.00045" ixy="0.0" iyz="-4.6e-05" ixz="0.0"/>
+<link name="JX_servo_v12_9">
+  <inertial>
+    <origin xyz="-0.008499999657726187 -0.016409678591751728 0.03717416110164981" rpy="0 0 0"/>
+    <mass value="0.19853540350189508"/>
+    <inertia ixx="0.000137" iyy="9e-05" izz="7.7e-05" ixy="0.0" iyz="-6e-06" ixz="-0.0"/>
   </inertial>
   <visual>
     <origin xyz="-0.0035 -0.0699 0.253626" rpy="0 0 0"/>
     <geometry>
-      <mesh filename="package://bez3_description/meshes/JX_servo_v8_9.stl" scale="0.001 0.001 0.001"/>
-    </geometry>
-    <material name="copper_polished"/>
+      <mesh filename="package://bez3_description/meshes/JX_servo_v12_9.stl" scale="0.001 0.001 0.001"/>
+    </geometry>
+    <material name="plastic_matte_black"/>
   </visual>
   <collision>
     <origin xyz="-0.0035 -0.0699 0.253626" rpy="0 0 0"/>
     <geometry>
-      <mesh filename="package://bez3_description/meshes/JX_servo_v8_9.stl" scale="0.001 0.001 0.001"/>
+      <mesh filename="package://bez3_description/meshes/JX_servo_v12_9.stl" scale="0.001 0.001 0.001"/>
     </geometry>
   </collision>
@@ -147,6 +147,6 @@
   <inertial>
     <origin xyz="0.0035522308946802695 -0.037286001427951104 -0.06738530321679864" rpy="0 0 0"/>
-    <mass value="0.5622725416559319"/>
-    <inertia ixx="0.001718" iyy="0.00106" izz="0.00082" ixy="-1e-06" iyz="2e-06" ixz="3.8e-05"/>
+    <mass value="0.04698736144283967"/>
+    <inertia ixx="0.000144" iyy="8.9e-05" izz="6.9e-05" ixy="-0.0" iyz="0.0" ixz="3e-06"/>
   </inertial>
   <visual>
@@ -155,5 +155,5 @@
       <mesh filename="package://bez3_description/meshes/left_thigh_1.stl" scale="0.001 0.001 0.001"/>
     </geometry>
-    <material name="steel_satin"/>
+    <material name="plastic_glossy_black"/>
   </visual>
   <collision>
@@ -164,21 +164,21 @@
   </collision>
 </link>
-<link name="JX_servo_v8_11">
-  <inertial>
-    <origin xyz="6.070390318885233e-10 -0.04053993921347642 -0.017780294556126508" rpy="0 0 0"/>
-    <mass value="1.0848385350345584"/>
-    <inertia ixx="0.000785" iyy="0.000503" izz="0.00045" ixy="0.0" iyz="-4.6e-05" ixz="0.0"/>
+<link name="JX_servo_v12_11">
+  <inertial>
+    <origin xyz="3.422737293243272e-10 -0.03890967859175239 -0.017725838898350055" rpy="0 0 0"/>
+    <mass value="0.19853540350189508"/>
+    <inertia ixx="0.000137" iyy="9e-05" izz="7.7e-05" ixy="0.0" iyz="-6e-06" ixz="-0.0"/>
   </inertial>
   <visual>
     <origin xyz="0.005 -0.0924 0.322726" rpy="0 0 0"/>
     <geometry>
-      <mesh filename="package://bez3_description/meshes/JX_servo_v8_11.stl" scale="0.001 0.001 0.001"/>
-    </geometry>
-    <material name="copper_polished"/>
+      <mesh filename="package://bez3_description/meshes/JX_servo_v12_11.stl" scale="0.001 0.001 0.001"/>
+    </geometry>
+    <material name="plastic_matte_black"/>
   </visual>
   <collision>
     <origin xyz="0.005 -0.0924 0.322726" rpy="0 0 0"/>
     <geometry>
-      <mesh filename="package://bez3_description/meshes/JX_servo_v8_11.stl" scale="0.001 0.001 0.001"/>
+      <mesh filename="package://bez3_description/meshes/JX_servo_v12_11.stl" scale="0.001 0.001 0.001"/>
     </geometry>
   </collision>
@@ -187,6 +187,6 @@
   <inertial>
     <origin xyz="-0.008549992578499489 -0.011776675554452998 -0.0353123749558687" rpy="0 0 0"/>
-    <mass value="0.514989606773696"/>
-    <inertia ixx="0.001057" iyy="0.00057" izz="0.000621" ixy="-0.0" iyz="-2.9e-05" ixz="0.0"/>
+    <mass value="0.035688451730559324"/>
+    <inertia ixx="7.3e-05" iyy="3.9e-05" izz="4.3e-05" ixy="-0.0" iyz="-2e-06" ixz="0.0"/>
   </inertial>
   <visual>
@@ -195,5 +195,5 @@
       <mesh filename="package://bez3_description/meshes/left_calve_1.stl" scale="0.001 0.001 0.001"/>
     </geometry>
-    <material name="steel_satin"/>
+    <material name="plastic_glossy_black"/>
   </visual>
   <collision>
@@ -204,21 +204,21 @@
   </collision>
 </link>
-<link name="JX_servo_v8_12">
-  <inertial>
-    <origin xyz="7.841479028602993e-11 -0.040539939213477115 0.01778050548278931" rpy="0 0 0"/>
-    <mass value="1.0848385350345584"/>
-    <inertia ixx="0.000785" iyy="0.000503" izz="0.00045" ixy="-0.0" iyz="4.6e-05" ixz="0.0"/>
+<link name="JX_servo_v12_12">
+  <inertial>
+    <origin xyz="3.43180092850226e-10 -0.0389096785917531 0.01772604982501308" rpy="0 0 0"/>
+    <mass value="0.19853540350189508"/>
+    <inertia ixx="0.000137" iyy="9e-05" izz="7.7e-05" ixy="-0.0" iyz="6e-06" ixz="-0.0"/>
   </inertial>
   <visual>
     <origin xyz="0.00505 -0.094 0.462631" rpy="0 0 0"/>
     <geometry>
-      <mesh filename="package://bez3_description/meshes/JX_servo_v8_12.stl" scale="0.001 0.001 0.001"/>
-    </geometry>
-    <material name="copper_polished"/>
+      <mesh filename="package://bez3_description/meshes/JX_servo_v12_12.stl" scale="0.001 0.001 0.001"/>
+    </geometry>
+    <material name="plastic_matte_black"/>
   </visual>
   <collision>
     <origin xyz="0.00505 -0.094 0.462631" rpy="0 0 0"/>
     <geometry>
-      <mesh filename="package://bez3_description/meshes/JX_servo_v8_12.stl" scale="0.001 0.001 0.001"/>
+      <mesh filename="package://bez3_description/meshes/JX_servo_v12_12.stl" scale="0.001 0.001 0.001"/>
     </geometry>
   </collision>
@@ -226,7 +226,7 @@
 <link name="left_hip_front_2">
   <inertial>
-    <origin xyz="-0.04064140960179005 -0.017336272610156404 -0.008851871921414733" rpy="0 0 0"/>
-    <mass value="0.2801003105283029"/>
-    <inertia ixx="0.00024" iyy="0.000331" izz="0.000219" ixy="-2e-06" iyz="-3e-06" ixz="-8.6e-05"/>
+    <origin xyz="-0.040641409601790045 -0.017336272610156404 -0.008851871921414733" rpy="0 0 0"/>
+    <mass value="0.025976181664280836"/>
+    <inertia ixx="2.2e-05" iyy="3.1e-05" izz="2e-05" ixy="-0.0" iyz="-0.0" ixz="-8e-06"/>
   </inertial>
   <visual>
@@ -235,5 +235,5 @@
       <mesh filename="package://bez3_description/meshes/left_hip_front_2.stl" scale="0.001 0.001 0.001"/>
     </geometry>
-    <material name="steel_satin"/>
+    <material name="plastic_glossy_black"/>
   </visual>
   <collision>
@@ -244,21 +244,21 @@
   </collision>
 </link>
-<link name="JX_servo_v8_13">
-  <inertial>
-    <origin xyz="-0.014139939556202498 0.008500000949764205 -0.037119494517210805" rpy="0 0 0"/>
-    <mass value="1.0848385350345584"/>
-    <inertia ixx="0.000503" iyy="0.000785" izz="0.00045" ixy="0.0" iyz="-0.0" ixz="4.6e-05"/>
+<link name="JX_servo_v12_13">
+  <inertial>
+    <origin xyz="-0.01250967893447847 0.008500000684998912 -0.0371739501749872" rpy="0 0 0"/>
+    <mass value="0.19853540350189508"/>
+    <inertia ixx="9e-05" iyy="0.000137" izz="7.7e-05" ixy="0.0" iyz="0.0" ixz="6e-06"/>
   </inertial>
   <visual>
     <origin xyz="0.06095 -0.0465 0.407731" rpy="0 0 0"/>
     <geometry>
-      <mesh filename="package://bez3_description/meshes/JX_servo_v8_13.stl" scale="0.001 0.001 0.001"/>
-    </geometry>
-    <material name="copper_polished"/>
+      <mesh filename="package://bez3_description/meshes/JX_servo_v12_13.stl" scale="0.001 0.001 0.001"/>
+    </geometry>
+    <material name="plastic_matte_black"/>
   </visual>
   <collision>
     <origin xyz="0.06095 -0.0465 0.407731" rpy="0 0 0"/>
     <geometry>
-      <mesh filename="package://bez3_description/meshes/JX_servo_v8_13.stl" scale="0.001 0.001 0.001"/>
+      <mesh filename="package://bez3_description/meshes/JX_servo_v12_13.stl" scale="0.001 0.001 0.001"/>
     </geometry>
   </collision>
@@ -266,7 +266,7 @@
 <link name="left_foot_1">
   <inertial>
-    <origin xyz="0.03678225489457133 -0.0014130788744076417 -0.021045237827845176" rpy="0 0 0"/>
-    <mass value="0.34210600833439103"/>
-    <inertia ixx="0.000178" iyy="0.00044" izz="0.000406" ixy="-8e-06" iyz="-6e-06" ixz="3.3e-05"/>
+    <origin xyz="0.03678225489457133 -0.0014130788744076417 -0.02104523782784523" rpy="0 0 0"/>
+    <mass value="0.03704332574321432"/>
+    <inertia ixx="1.9e-05" iyy="4.8e-05" izz="4.4e-05" ixy="-1e-06" iyz="-1e-06" ixz="4e-06"/>
   </inertial>
   <visual>
@@ -275,5 +275,5 @@
       <mesh filename="package://bez3_description/meshes/left_foot_1.stl" scale="0.001 0.001 0.001"/>
     </geometry>
-    <material name="steel_satin"/>
+    <material name="plastic_glossy_black"/>
   </visual>
   <collision>
@@ -284,21 +284,21 @@
   </collision>
 </link>
-<link name="JX_servo_v8_14">
-  <inertial>
-    <origin xyz="0.0002196166185167714 -2.643122040679735e-10 0.014139939556201936" rpy="0 0 0"/>
-    <mass value="1.0848385350345584"/>
-    <inertia ixx="0.00045" iyy="0.000785" izz="0.000503" ixy="-0.0" iyz="0.0" ixz="4.6e-05"/>
+<link name="JX_servo_v12_14">
+  <inertial>
+    <origin xyz="0.00027407227629309625 4.531167108190459e-13 0.012509678934477936" rpy="0 0 0"/>
+    <mass value="0.19853540350189508"/>
+    <inertia ixx="7.7e-05" iyy="0.000137" izz="9e-05" ixy="0.0" iyz="0.0" ixz="6e-06"/>
   </inertial>
   <visual>
     <origin xyz="0.0225 0.0545 0.137" rpy="0 0 0"/>
     <geometry>
-      <mesh filename="package://bez3_description/meshes/JX_servo_v8_14.stl" scale="0.001 0.001 0.001"/>
-    </geometry>
-    <material name="copper_polished"/>
+      <mesh filename="package://bez3_description/meshes/JX_servo_v12_14.stl" scale="0.001 0.001 0.001"/>
+    </geometry>
+    <material name="plastic_matte_black"/>
   </visual>
   <collision>
     <origin xyz="0.0225 0.0545 0.137" rpy="0 0 0"/>
     <geometry>
-      <mesh filename="package://bez3_description/meshes/JX_servo_v8_14.stl" scale="0.001 0.001 0.001"/>
+      <mesh filename="package://bez3_description/meshes/JX_servo_v12_14.stl" scale="0.001 0.001 0.001"/>
     </geometry>
   </collision>
@@ -306,7 +306,7 @@
 <link name="right_hip_side_1">
   <inertial>
-    <origin xyz="-0.0006601764265435368 -7.984240837921597e-10 -0.021141552658250296" rpy="0 0 0"/>
-    <mass value="0.2196591578921638"/>
-    <inertia ixx="0.000107" iyy="0.000213" izz="0.000165" ixy="-0.0" iyz="-0.0" ixz="-2e-06"/>
+    <origin xyz="-0.0006601764265435368 -7.984240907310536e-10 -0.021141552658250296" rpy="0 0 0"/>
+    <mass value="0.018999817606213918"/>
+    <inertia ixx="9e-06" iyy="1.8e-05" izz="1.4e-05" ixy="-0.0" iyz="-0.0" ixz="-0.0"/>
   </inertial>
   <visual>
@@ -315,5 +315,5 @@
       <mesh filename="package://bez3_description/meshes/right_hip_side_1.stl" scale="0.001 0.001 0.001"/>
     </geometry>
-    <material name="steel_satin"/>
+    <material name="plastic_glossy_black"/>
   </visual>
   <collision>
@@ -324,21 +324,21 @@
   </collision>
 </link>
-<link name="JX_servo_v8_15">
-  <inertial>
-    <origin xyz="-0.04053993955620186 -2.643120514123076e-10 -0.017780294556127257" rpy="0 0 0"/>
-    <mass value="1.0848385350345584"/>
-    <inertia ixx="0.000503" iyy="0.000785" izz="0.00045" ixy="-0.0" iyz="-0.0" ixz="-4.6e-05"/>
+<link name="JX_servo_v12_15">
+  <inertial>
+    <origin xyz="-0.03890967893447782 4.5325548869712406e-13 -0.017725838898350943" rpy="0 0 0"/>
+    <mass value="0.19853540350189508"/>
+    <inertia ixx="9e-05" iyy="0.000137" izz="7.7e-05" ixy="-0.0" iyz="0.0" ixz="-6e-06"/>
   </inertial>
   <visual>
     <origin xyz="0.0345 0.0545 0.198736" rpy="0 0 0"/>
     <geometry>
-      <mesh filename="package://bez3_description/meshes/JX_servo_v8_15.stl" scale="0.001 0.001 0.001"/>
-    </geometry>
-    <material name="copper_polished"/>
+      <mesh filename="package://bez3_description/meshes/JX_servo_v12_15.stl" scale="0.001 0.001 0.001"/>
+    </geometry>
+    <material name="plastic_matte_black"/>
   </visual>
   <collision>
     <origin xyz="0.0345 0.0545 0.198736" rpy="0 0 0"/>
     <geometry>
-      <mesh filename="package://bez3_description/meshes/JX_servo_v8_15.stl" scale="0.001 0.001 0.001"/>
+      <mesh filename="package://bez3_description/meshes/JX_servo_v12_15.stl" scale="0.001 0.001 0.001"/>
     </geometry>
   </collision>
@@ -347,6 +347,6 @@
   <inertial>
     <origin xyz="0.02375859039821196 -0.00933627329560792 -0.06494791715192275" rpy="0 0 0"/>
-    <mass value="0.2801003105283028"/>
-    <inertia ixx="0.00024" iyy="0.000331" izz="0.000219" ixy="-2e-06" iyz="3e-06" ixz="8.6e-05"/>
+    <mass value="0.025976181664280826"/>
+    <inertia ixx="2.2e-05" iyy="3.1e-05" izz="2e-05" ixy="-0.0" iyz="0.0" ixz="8e-06"/>
   </inertial>
   <visual>
@@ -355,5 +355,5 @@
       <mesh filename="package://bez3_description/meshes/right_ankle_1.stl" scale="0.001 0.001 0.001"/>
     </geometry>
-    <material name="steel_satin"/>
+    <material name="plastic_glossy_black"/>
   </visual>
   <collision>
@@ -364,21 +364,21 @@
   </collision>
 </link>
-<link name="JX_servo_v8_16">
-  <inertial>
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
File: bez3_description/urdf/materials.xacro (robot description, xacro)
@@ -7,15 +7,21 @@
   <color rgba="0.6274509803921569 0.6274509803921569 0.6274509803921569 1.0"/>
 </material>
+<material name="plastic_matte_black">
+  <color rgba="0.09803921568627451 0.09803921568627451 0.09803921568627451 1.0"/>
+</material>
+<material name="plastic_glossy_black">
+  <color rgba="0.9058823529411765 0.0 0.0 1.0"/>
+</material>
+<material name="aluminum_satin">
+  <color rgba="0.9607843137254902 0.9607843137254902 0.9647058823529412 1.0"/>
+</material>
+<material name="plastic_glossy_grey">
+  <color rgba="0.2901960784313726 0.2901960784313726 0.2901960784313726 1.0"/>
+</material>
 <material name="polymide_kapton">
   <color rgba="0.7843137254901961 0.5568627450980392 0.027450980392156862 1.0"/>
 </material>
-<material name="copper_polished">
-  <color rgba="0.9294117647058824 0.807843137254902 0.7647058823529411 1.0"/>
-</material>
-<material name="abs_white">
-  <color rgba="0.9647058823529412 0.9647058823529412 0.9529411764705882 1.0"/>
-</material>
-<material name="plastic_glossy_black">
-  <color rgba="0.09803921568627451 0.09803921568627451 0.09803921568627451 1.0"/>
+<material name="plastic_matte_blue">
+  <color rgba="0.1607843137254902 0.5058823529411764 0.807843137254902 1.0"/>
 </material>
 </robot>
