Commit message: wip

File: bez3_description/urdf/bez3.urdf (robot description, URDF)
Before this commit: robot bez3, 54 links, 53 joints
Links:
- removed link 25t-servo-hub_1
- removed link 25t-servo-hub_2
- removed link 25t-servo-hub_3
- removed link 25t-servo-hub_4
- removed link 25t-servo-hub_Mirror__1
- removed link 25t-servo-hub_Mirror__2
- removed link Component32_1
- removed link JX_servo_v12_1
- removed link JX_servo_v12_11
- removed link JX_servo_v12_12
- removed link JX_servo_v12_13
- removed link JX_servo_v12_14
- removed link JX_servo_v12_15
- removed link JX_servo_v12_16
- removed link JX_servo_v12_17
- removed link JX_servo_v12_18
- removed link JX_servo_v12_19
- removed link JX_servo_v12_8
- removed link JX_servo_v12_9
- removed link TX2_board_v2_1
- removed link base_link
- removed link camera-link_1
- removed link camera_1
- removed link custom_servo_support__lower_neck__v2_1
- removed link elbow-attach_1
- removed link elbow-attach_Mirror__1
- removed link elbow-bearing_1
- removed link elbow-bearing_Mirror__1
- removed link gobilda-servo_1
- removed link gobilda-servo_3
- removed link gobilda-servo_4
- removed link gobilda-servo_5
- removed link gobilda-servo_Mirror__1
- removed link gobilda-servo_Mirror__2
- removed link head_1
- removed link imu-link_1
- removed link left_bicep_1
- removed link left_calve_1
- removed link left_foot_1
- removed link left_forearm_1
- removed link left_hip_front_1
- removed link left_hip_front_2
- removed link left_hip_side_1
- removed link left_thigh_1
- removed link neck_1
- removed link right_ankle_1
- removed link right_ankle_2
- removed link right_bicep_1
- removed link right_calve_1
- removed link right_foot_1
- removed link right_forearm_1
- removed link right_hip_side_1
- removed link right_thigh_1
- removed link torso_1
- added link /25t-servo-hub_1, mass 0.005584850212079893; collision mesh filename=package://bez3_description/meshes/25t-servo-hub_1.stl scale=0.001 0.001 0.001; visual mesh filename=package://bez3_description/meshes/25t-servo-hub_1.stl scale=0.001 0.001 0.001
- added link /25t-servo-hub_2, mass 0.005584850212079893; collision mesh filename=package://bez3_description/meshes/25t-servo-hub_2.stl scale=0.001 0.001 0.001; visual mesh filename=package://bez3_description/meshes/25t-servo-hub_2.stl scale=0.001 0.001 0.001
- added link /25t-servo-hub_3, mass 0.005584850212079893; collision mesh filename=package://bez3_description/meshes/25t-servo-hub_3.stl scale=0.001 0.001 0.001; visual mesh filename=package://bez3_description/meshes/25t-servo-hub_3.stl scale=0.001 0.001 0.001
- added link /25t-servo-hub_4, mass 0.005584850212079893; collision mesh filename=package://bez3_description/meshes/25t-servo-hub_4.stl scale=0.001 0.001 0.001; visual mesh filename=package://bez3_description/meshes/25t-servo-hub_4.stl scale=0.001 0.001 0.001
- added link /25t-servo-hub_Mirror__1, mass 0.005584585205775494; collision mesh filename=package://bez3_description/meshes/25t-servo-hub_Mirror__1.s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 scale=0.001 0.001 0.001; visual mesh filename=package://bez3_description/meshes/25t-servo-hub_Mirror__1.s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 scale=0.001 0.001 0.001
- added link /25t-servo-hub_Mirror__2, mass 0.005584585205775494; collision mesh filename=package://bez3_description/meshes/25t-servo-hub_Mirror__2.s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 scale=0.001 0.001 0.001; visual mesh filename=package://bez3_description/meshes/25t-servo-hub_Mirror__2.s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 scale=0.001 0.001 0.001
- added link /Component32_1, mass 0.31999527000000005; collision mesh filename=package://bez3_description/meshes/Component32_1.stl scale=0.001 0.001 0.001; visual mesh filename=package://bez3_description/meshes/Component32_1.stl scale=0.001 0.001 0.001
- added link /JX_servo_v12_1, mass 0.19853540350189508; collision mesh filename=package://bez3_description/meshes/JX_servo_v12_1.stl scale=0.001 0.001 0.001; visual mesh filename=package://bez3_description/meshes/JX_servo_v12_1.stl scale=0.001 0.001 0.001
- added link /JX_servo_v12_11, mass 0.19853540350189508; collision mesh filename=package://bez3_description/meshes/JX_servo_v12_11.stl scale=0.001 0.001 0.001; visual mesh filename=package://bez3_description/meshes/JX_servo_v12_11.stl scale=0.001 0.001 0.001
- added link /JX_servo_v12_12, mass 0.19853540350189508; collision mesh filename=package://bez3_description/meshes/JX_servo_v12_12.stl scale=0.001 0.001 0.001; visual mesh filename=package://bez3_description/meshes/JX_servo_v12_12.stl scale=0.001 0.001 0.001
- added link /JX_servo_v12_13, mass 0.19853540350189508; collision mesh filename=package://bez3_description/meshes/JX_servo_v12_13.stl scale=0.001 0.001 0.001; visual mesh filename=package://bez3_description/meshes/JX_servo_v12_13.stl scale=0.001 0.001 0.001
- added link /JX_servo_v12_14, mass 0.19853540350189508; collision mesh filename=package://bez3_description/meshes/JX_servo_v12_14.stl scale=0.001 0.001 0.001; visual mesh filename=package://bez3_description/meshes/JX_servo_v12_14.stl scale=0.001 0.001 0.001
- added link /JX_servo_v12_15, mass 0.19853540350189508; collision mesh filename=package://bez3_description/meshes/JX_servo_v12_15.stl scale=0.001 0.001 0.001; visual mesh filename=package://bez3_description/meshes/JX_servo_v12_15.stl scale=0.001 0.001 0.001
- added link /JX_servo_v12_16, mass 0.19853540350189508; collision mesh filename=package://bez3_description/meshes/JX_servo_v12_16.stl scale=0.001 0.001 0.001; visual mesh filename=package://bez3_description/meshes/JX_servo_v12_16.stl scale=0.001 0.001 0.001
- added link /JX_servo_v12_17, mass 0.19853540350189508; collision mesh filename=package://bez3_description/meshes/JX_servo_v12_17.stl scale=0.001 0.001 0.001; visual mesh filename=package://bez3_description/meshes/JX_servo_v12_17.stl scale=0.001 0.001 0.001
- added link /JX_servo_v12_18, mass 0.19853540350189508; collision mesh filename=package://bez3_description/meshes/JX_servo_v12_18.stl scale=0.001 0.001 0.001; visual mesh filename=package://bez3_description/meshes/JX_servo_v12_18.stl scale=0.001 0.001 0.001
- added link /JX_servo_v12_19, mass 0.19853540350189508; collision mesh filename=package://bez3_description/meshes/JX_servo_v12_19.stl scale=0.001 0.001 0.001; visual mesh filename=package://bez3_description/meshes/JX_servo_v12_19.stl scale=0.001 0.001 0.001
- added link /JX_servo_v12_8, mass 0.19853540350189508; collision mesh filename=package://bez3_description/meshes/JX_servo_v12_8.stl scale=0.001 0.001 0.001; visual mesh filename=package://bez3_description/meshes/JX_servo_v12_8.stl scale=0.001 0.001 0.001
- added link /JX_servo_v12_9, mass 0.19853540350189508; collision mesh filename=package://bez3_description/meshes/JX_servo_v12_9.stl scale=0.001 0.001 0.001; visual mesh filename=package://bez3_description/meshes/JX_servo_v12_9.stl scale=0.001 0.001 0.001
- added link /TX2_board_v2_1, mass 0.2621637298853286; collision mesh filename=package://bez3_description/meshes/TX2_board_v2_1.stl scale=0.001 0.001 0.001; visual mesh filename=package://bez3_description/meshes/TX2_board_v2_1.stl scale=0.001 0.001 0.001
- added link /base_link, mass 0.00785; collision mesh filename=package://bez3_description/meshes/base_link.stl scale=0.001 0.001 0.001; visual mesh filename=package://bez3_description/meshes/base_link.stl scale=0.001 0.001 0.001
- added link /camera-link_1, mass 0.00019624999999999932; collision mesh filename=package://bez3_description/meshes/camera-link_1.stl scale=0.001 0.001 0.001; visual mesh filename=package://bez3_description/meshes/camera-link_1.stl scale=0.001 0.001 0.001
- added link /camera_1, mass 0.094257141411043; collision mesh filename=package://bez3_description/meshes/camera_1.stl scale=0.001 0.001 0.001; visual mesh filename=package://bez3_description/meshes/camera_1.stl scale=0.001 0.001 0.001
- added link /custom_servo_support__lower_neck__v2_1, mass 0.003136252201459725; collision mesh filename=package://bez3_description/meshes/custom_servo_support__low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 scale=0.001 0.001 0.001; visual mesh filename=package://bez3_description/meshes/custom_servo_support__low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 scale=0.001 0.001 0.001
- added link /elbow-attach_1, mass 0.005141835270301899; collision mesh filename=package://bez3_description/meshes/elbow-attach_1.stl scale=0.001 0.001 0.001; visual mesh filename=package://bez3_description/meshes/elbow-attach_1.stl scale=0.001 0.001 0.001
- added link /elbow-attach_Mirror__1, mass 0.005141835270301901; collision mesh filename=package://bez3_description/meshes/elbow-attach_Mirror__1.stl scale=0.001 0.001 0.001; visual mesh filename=package://bez3_description/meshes/elbow-attach_Mirror__1.stl scale=0.001 0.001 0.001
- added link /elbow-bearing_1, mass 0.004941715818268227; collision mesh filename=package://bez3_description/meshes/elbow-bearing_1.stl scale=0.001 0.001 0.001; visual mesh filename=package://bez3_description/meshes/elbow-bearing_1.stl scale=0.001 0.001 0.001
- added link /elbow-bearing_Mirror__1, mass 0.004941715818268223; collision mesh filename=package://bez3_description/meshes/elbow-bearing_Mirror__1.s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 scale=0.001 0.001 0.001; visual mesh filename=package://bez3_description/meshes/elbow-bearing_Mirror__1.s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 scale=0.001 0.001 0.001
- added link /gobilda-servo_1, mass 0.060587311248822606; collision mesh filename=package://bez3_description/meshes/gobilda-servo_1.stl scale=0.001 0.001 0.001; visual mesh filename=package://bez3_description/meshes/gobilda-servo_1.stl scale=0.001 0.001 0.001
- added link /gobilda-servo_3, mass 0.060587311248822606; collision mesh filename=package://bez3_description/meshes/gobilda-servo_3.stl scale=0.001 0.001 0.001; visual mesh filename=package://bez3_description/meshes/gobilda-servo_3.stl scale=0.001 0.001 0.001
- added link /gobilda-servo_4, mass 0.060587311248822606; collision mesh filename=package://bez3_description/meshes/gobilda-servo_4.stl scale=0.001 0.001 0.001; visual mesh filename=package://bez3_description/meshes/gobilda-servo_4.stl scale=0.001 0.001 0.001
- added link /gobilda-servo_5, mass 0.060587311248822606; collision mesh filename=package://bez3_description/meshes/gobilda-servo_5.stl scale=0.001 0.001 0.001; visual mesh filename=package://bez3_description/meshes/gobilda-servo_5.stl scale=0.001 0.001 0.001
- added link /gobilda-servo_Mirror__1, mass 0.06058731124882261; collision mesh filename=package://bez3_description/meshes/gobilda-servo_Mirror__1.s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 scale=0.001 0.001 0.001; visual mesh filename=package://bez3_description/meshes/gobilda-servo_Mirror__1.s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 scale=0.001 0.001 0.001
- added link /gobilda-servo_Mirror__2, mass 0.06058731124882261; collision mesh filename=package://bez3_description/meshes/gobilda-servo_Mirror__2.s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 scale=0.001 0.001 0.001; visual mesh filename=package://bez3_description/meshes/gobilda-servo_Mirror__2.s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 scale=0.001 0.001 0.001
- added link /head_1, mass 0.007653734054253099; collision mesh filename=package://bez3_description/meshes/head_1.stl scale=0.001 0.001 0.001; visual mesh filename=package://bez3_description/meshes/head_1.stl scale=0.001 0.001 0.001
- added link /imu-link_1, mass 0.00019625; collision mesh filename=package://bez3_description/meshes/imu-link_1.stl scale=0.001 0.001 0.001; visual mesh filename=package://bez3_description/meshes/imu-link_1.stl scale=0.001 0.001 0.001
- added link /left_bicep_1, mass 0.011455626340925264; collision mesh filename=package://bez3_description/meshes/left_bicep_1.stl scale=0.001 0.001 0.001; visual mesh filename=package://bez3_description/meshes/left_bicep_1.stl scale=0.001 0.001 0.001
- added link /left_calve_1, mass 0.035688451730559324; collision mesh filename=package://bez3_description/meshes/left_calve_1.stl scale=0.001 0.001 0.001; visual mesh filename=package://bez3_description/meshes/left_calve_1.stl scale=0.001 0.001 0.001
- added link /left_foot_1, mass 0.03704332574321432; collision mesh filename=package://bez3_description/meshes/left_foot_1.stl scale=0.001 0.001 0.001; visual mesh filename=package://bez3_description/meshes/left_foot_1.stl scale=0.001 0.001 0.001
- added link /left_forearm_1, mass 0.027371737365874692; collision mesh filename=package://bez3_description/meshes/left_forearm_1.stl scale=0.001 0.001 0.001; visual mesh filename=package://bez3_description/meshes/left_forearm_1.stl scale=0.001 0.001 0.001
- added link /left_hip_front_1, mass 0.025976181664280836; collision mesh filename=package://bez3_description/meshes/left_hip_front_1.stl scale=0.001 0.001 0.001; visual mesh filename=package://bez3_description/meshes/left_hip_front_1.stl scale=0.001 0.001 0.001
- added link /left_hip_front_2, mass 0.025976181664280836; collision mesh filename=package://bez3_description/meshes/left_hip_front_2.stl scale=0.001 0.001 0.001; visual mesh filename=package://bez3_description/meshes/left_hip_front_2.stl scale=0.001 0.001 0.001
- added link /left_hip_side_1, mass 0.018999817606213904; collision mesh filename=package://bez3_description/meshes/left_hip_side_1.stl scale=0.001 0.001 0.001; visual mesh filename=package://bez3_description/meshes/left_hip_side_1.stl scale=0.001 0.001 0.001
- added link /left_thigh_1, mass 0.04698736144283967; collision mesh filename=package://bez3_description/meshes/left_thigh_1.stl scale=0.001 0.001 0.001; visual mesh filename=package://bez3_description/meshes/left_thigh_1.stl scale=0.001 0.001 0.001
- added link /neck_1, mass 0.012940388012734224; collision mesh filename=package://bez3_description/meshes/neck_1.stl scale=0.001 0.001 0.001; visual mesh filename=package://bez3_description/meshes/neck_1.stl scale=0.001 0.001 0.001
- added link /right_ankle_1, mass 0.025976181664280826; collision mesh filename=package://bez3_description/meshes/right_ankle_1.stl scale=0.001 0.001 0.001; visual mesh filename=package://bez3_description/meshes/right_ankle_1.stl scale=0.001 0.001 0.001
- added link /right_ankle_2, mass 0.025976181664280826; collision mesh filename=package://bez3_description/meshes/right_ankle_2.stl scale=0.001 0.001 0.001; visual mesh filename=package://bez3_description/meshes/right_ankle_2.stl scale=0.001 0.001 0.001
- added link /right_bicep_1, mass 0.011455626340925269; collision mesh filename=package://bez3_description/meshes/right_bicep_1.stl scale=0.001 0.001 0.001; visual mesh filename=package://bez3_description/meshes/right_bicep_1.stl scale=0.001 0.001 0.001
- added link /right_calve_1, mass 0.03568840560735723; collision mesh filename=package://bez3_description/meshes/right_calve_1.stl scale=0.001 0.001 0.001; visual mesh filename=package://bez3_description/meshes/right_calve_1.stl scale=0.001 0.001 0.001
- added link /right_foot_1, mass 0.037043325743214305; collision mesh filename=package://bez3_description/meshes/right_foot_1.stl scale=0.001 0.001 0.001; visual mesh filename=package://bez3_description/meshes/right_foot_1.stl scale=0.001 0.001 0.001
- added link /right_forearm_1, mass 0.027371737365874692; collision mesh filename=package://bez3_description/meshes/right_forearm_1.stl scale=0.001 0.001 0.001; visual mesh filename=package://bez3_description/meshes/right_forearm_1.stl scale=0.001 0.001 0.001
- added link /right_hip_side_1, mass 0.018999817606213918; collision mesh filename=package://bez3_description/meshes/right_hip_side_1.stl scale=0.001 0.001 0.001; visual mesh filename=package://bez3_description/meshes/right_hip_side_1.stl scale=0.001 0.001 0.001
- added link /right_thigh_1, mass 0.04698731628682583; collision mesh filename=package://bez3_description/meshes/right_thigh_1.stl scale=0.001 0.001 0.001; visual mesh filename=package://bez3_description/meshes/right_thigh_1.stl scale=0.001 0.001 0.001
- added link /torso_1, mass 0.2968069064800233; collision mesh filename=package://bez3_description/meshes/torso_1.stl scale=0.001 0.001 0.001; visual mesh filename=package://bez3_description/meshes/torso_1.stl scale=0.001 0.001 0.001
Joints:
- joint Rigid1: child torso_1 -> /torso_1; parent base_link -> /base_link
- joint Rigid11: child left_hip_front_2 -> /left_hip_front_2; parent JX_servo_v12_12 -> /JX_servo_v12_12
- joint Rigid12: child JX_servo_v12_13 -> /JX_servo_v12_13; parent left_hip_front_2 -> /left_hip_front_2
- joint Rigid14: child JX_servo_v12_14 -> /JX_servo_v12_14; parent torso_1 -> /torso_1
- joint Rigid17: child right_ankle_1 -> /right_ankle_1; parent JX_servo_v12_15 -> /JX_servo_v12_15
- joint Rigid18: child JX_servo_v12_16 -> /JX_servo_v12_16; parent right_ankle_1 -> /right_ankle_1
- joint Rigid2: child JX_servo_v12_1 -> /JX_servo_v12_1; parent torso_1 -> /torso_1
- joint Rigid21: child right_calve_1 -> /right_calve_1; parent JX_servo_v12_17 -> /JX_servo_v12_17
- joint Rigid23: child right_ankle_2 -> /right_ankle_2; parent JX_servo_v12_18 -> /JX_servo_v12_18
- joint Rigid24: child JX_servo_v12_19 -> /JX_servo_v12_19; parent right_ankle_2 -> /right_ankle_2
- joint Rigid26: child 25t-servo-hub_1 -> /25t-servo-hub_1; parent torso_1 -> /torso_1
- joint Rigid28: child left_bicep_1 -> /left_bicep_1; parent gobilda-servo_1 -> /gobilda-servo_1
- joint Rigid29: child gobilda-servo_3 -> /gobilda-servo_3; parent left_bicep_1 -> /left_bicep_1
- joint Rigid31: child elbow-attach_1 -> /elbow-attach_1; parent 25t-servo-hub_2 -> /25t-servo-hub_2
- joint Rigid32: child left_forearm_1 -> /left_forearm_1; parent elbow-attach_1 -> /elbow-attach_1
- joint Rigid33: child elbow-bearing_1 -> /elbow-bearing_1; parent left_forearm_1 -> /left_forearm_1
- joint Rigid34: child 25t-servo-hub_Mirror__1 -> /25t-servo-hub_Mirror__1; parent torso_1 -> /torso_1
- joint Rigid36: child right_bicep_1 -> /right_bicep_1; parent gobilda-servo_Mirror__1 -> /gobilda-servo_Mirror__1
- joint Rigid37: child gobilda-servo_Mirror__2 -> /gobilda-servo_Mirror__2; parent right_bicep_1 -> /right_bicep_1
- joint Rigid39: child elbow-attach_Mirror__1 -> /elbow-attach_Mirror__1; parent 25t-servo-hub_Mirror__2 -> /25t-servo-hub_Mirror__2
- joint Rigid40: child right_forearm_1 -> /right_forearm_1; parent elbow-attach_Mirror__1 -> /elbow-attach_Mirror__1
- joint Rigid41: child elbow-bearing_Mirror__1 -> /elbow-bearing_Mirror__1; parent right_forearm_1 -> /right_forearm_1
- joint Rigid42: child custom_servo_support__lower_neck__v2_1 -> /custom_servo_support__lower_neck__v2_1; parent torso_1 -> /torso_1
- joint Rigid43: child gobilda-servo_4 -> /gobilda-servo_4; parent custom_servo_support__lower_neck__v2_1 -> /custom_servo_support__lower_neck__v2_1
- joint Rigid45: child neck_1 -> /neck_1; parent 25t-servo-hub_3 -> /25t-servo-hub_3
- joint Rigid46: child 25t-servo-hub_4 -> /25t-servo-hub_4; parent neck_1 -> /neck_1
- joint Rigid48: child head_1 -> /head_1; parent gobilda-servo_5 -> /gobilda-servo_5
- joint Rigid49: child camera_1 -> /camera_1; parent head_1 -> /head_1
- joint Rigid5: child left_hip_front_1 -> /left_hip_front_1; parent JX_servo_v12_8 -> /JX_servo_v12_8
- joint Rigid52: child Component32_1 -> /Component32_1; parent torso_1 -> /torso_1
- joint Rigid53: child TX2_board_v2_1 -> /TX2_board_v2_1; parent Component32_1 -> /Component32_1
- joint Rigid6: child JX_servo_v12_9 -> /JX_servo_v12_9; parent left_hip_front_1 -> /left_hip_front_1
- joint Rigid9: child left_calve_1 -> /left_calve_1; parent JX_servo_v12_11 -> /JX_servo_v12_11
- joint camera_joint: child camera-link_1 -> /camera-link_1; parent camera_1 -> /camera_1
- joint head_motor_0: child 25t-servo-hub_3 -> /25t-servo-hub_3; parent gobilda-servo_4 -> /gobilda-servo_4
- joint head_motor_1: child gobilda-servo_5 -> /gobilda-servo_5; parent 25t-servo-hub_4 -> /25t-servo-hub_4
- joint imu_joint: child imu-link_1 -> /imu-link_1; parent torso_1 -> /torso_1
- joint left_arm_motor_0: child gobilda-servo_1 -> /gobilda-servo_1; parent 25t-servo-hub_1 -> /25t-servo-hub_1
- joint left_arm_motor_1: child 25t-servo-hub_2 -> /25t-servo-hub_2; parent gobilda-servo_3 -> /gobilda-servo_3
- joint left_leg_motor_0: child left_hip_side_1 -> /left_hip_side_1; parent JX_servo_v12_1 -> /JX_servo_v12_1
- joint left_leg_motor_1: child JX_servo_v12_8 -> /JX_servo_v12_8; parent left_hip_side_1 -> /left_hip_side_1
- joint left_leg_motor_2: child left_thigh_1 -> /left_thigh_1; parent JX_servo_v12_9 -> /JX_servo_v12_9
- joint left_leg_motor_3: child JX_servo_v12_11 -> /JX_servo_v12_11; parent left_thigh_1 -> /left_thigh_1
- joint left_leg_motor_4: child JX_servo_v12_12 -> /JX_servo_v12_12; parent left_calve_1 -> /left_calve_1
- joint left_leg_motor_5: child left_foot_1 -> /left_foot_1; parent JX_servo_v12_13 -> /JX_servo_v12_13
- joint right_arm_motor_0: child gobilda-servo_Mirror__1 -> /gobilda-servo_Mirror__1; parent 25t-servo-hub_Mirror__1 -> /25t-servo-hub_Mirror__1
- joint right_arm_motor_1: child 25t-servo-hub_Mirror__2 -> /25t-servo-hub_Mirror__2; parent gobilda-servo_Mirror__2 -> /gobilda-servo_Mirror__2
- joint right_leg_motor_0: child right_hip_side_1 -> /right_hip_side_1; parent JX_servo_v12_14 -> /JX_servo_v12_14
- joint right_leg_motor_1: child JX_servo_v12_15 -> /JX_servo_v12_15; parent right_hip_side_1 -> /right_hip_side_1
- joint right_leg_motor_2: child right_thigh_1 -> /right_thigh_1; parent JX_servo_v12_16 -> /JX_servo_v12_16
- joint right_leg_motor_3: child JX_servo_v12_17 -> /JX_servo_v12_17; parent right_thigh_1 -> /right_thigh_1
- joint right_leg_motor_4: child JX_servo_v12_18 -> /JX_servo_v12_18; parent right_calve_1 -> /right_calve_1
- joint right_leg_motor_5: child right_foot_1 -> /right_foot_1; parent JX_servo_v12_19 -> /JX_servo_v12_19
