Commit message: wip

File: bez3_description/urdf/bez3.xacro (robot description, xacro)
@@ -1,8 +1,9 @@
 <?xml version="1.0" ?>
 <robot name="bez3" xmlns:xacro="http://www.ros.org/wiki/xacro">
+<xacro:arg name="tf_prefix" default="" />
 <xacro:include filename="$(find bez3_description)/urdf/materials.xacro" />
 <xacro:include filename="$(find bez3_description)/urdf/bez3.trans" />
 <xacro:include filename="$(find bez3_description)/urdf/bez3.gazebo" />
-<link name="base_link">
+<link name="$(arg tf_prefix)/base_link">
   <inertial>
     <origin xyz="0.005 0.005 0.005" rpy="0 0 0"/>
@@ -24,5 +25,5 @@
   </collision>
 </link>
-<link name="torso_1">
+<link name="$(arg tf_prefix)/torso">
   <inertial>
     <origin xyz="-0.003658211229359205 -0.006167940664238083 -0.07338742094913071" rpy="0 0 0"/>
@@ -44,5 +45,5 @@
   </collision>
 </link>
-<link name="JX_servo_v12_1">
+<link name="$(arg tf_prefix)/JX_servo_v12_1">
   <inertial>
     <origin xyz="0.00027407227629309625 4.531028330312381e-13 0.012509678934478005" rpy="0 0 0"/>
@@ -64,5 +65,5 @@
   </collision>
 </link>
-<link name="left_hip_side_1">
+<link name="$(arg tf_prefix)/left_hip_side_1">
   <inertial>
     <origin xyz="-0.0006601764265435524 7.984241046088414e-10 -0.021141547194982763" rpy="0 0 0"/>
@@ -84,5 +85,5 @@
   </collision>
 </link>
-<link name="JX_servo_v12_8">
+<link name="$(arg tf_prefix)/JX_servo_v12_8">
   <inertial>
     <origin xyz="-0.03890967893447789 4.529293606836404e-13 -0.017725838898350915" rpy="0 0 0"/>
@@ -104,5 +105,5 @@
   </collision>
 </link>
-<link name="left_hip_front_1">
+<link name="$(arg tf_prefix)/left_hip_front_1">
   <inertial>
     <origin xyz="0.023758590398210495 0.009336273295607947 -0.06494791715192266" rpy="0 0 0"/>
@@ -124,5 +125,5 @@
   </collision>
 </link>
-<link name="JX_servo_v12_9">
+<link name="$(arg tf_prefix)/JX_servo_v12_9">
   <inertial>
     <origin xyz="-0.008499999657726187 -0.016409678591751728 0.03717416110164981" rpy="0 0 0"/>
@@ -144,5 +145,5 @@
   </collision>
 </link>
-<link name="left_thigh_1">
+<link name="$(arg tf_prefix)/left_thigh_1">
   <inertial>
     <origin xyz="0.0035522308946802695 -0.037286001427951104 -0.06738530321679864" rpy="0 0 0"/>
@@ -164,5 +165,5 @@
   </collision>
 </link>
-<link name="JX_servo_v12_11">
+<link name="$(arg tf_prefix)/JX_servo_v12_11">
   <inertial>
     <origin xyz="3.422737293243272e-10 -0.03890967859175239 -0.017725838898350055" rpy="0 0 0"/>
@@ -184,5 +185,5 @@
   </collision>
 </link>
-<link name="left_calve_1">
+<link name="$(arg tf_prefix)/left_calve_1">
   <inertial>
     <origin xyz="-0.008549992578499489 -0.011776675554452998 -0.0353123749558687" rpy="0 0 0"/>
@@ -204,5 +205,5 @@
   </collision>
 </link>
-<link name="JX_servo_v12_12">
+<link name="$(arg tf_prefix)/JX_servo_v12_12">
   <inertial>
     <origin xyz="3.43180092850226e-10 -0.0389096785917531 0.01772604982501308" rpy="0 0 0"/>
@@ -224,5 +225,5 @@
   </collision>
 </link>
-<link name="left_hip_front_2">
+<link name="$(arg tf_prefix)/left_hip_front_2">
   <inertial>
     <origin xyz="-0.040641409601790045 -0.017336272610156404 -0.008851871921414733" rpy="0 0 0"/>
@@ -244,5 +245,5 @@
   </collision>
 </link>
-<link name="JX_servo_v12_13">
+<link name="$(arg tf_prefix)/JX_servo_v12_13">
   <inertial>
     <origin xyz="-0.01250967893447847 0.008500000684998912 -0.0371739501749872" rpy="0 0 0"/>
@@ -264,5 +265,5 @@
   </collision>
 </link>
-<link name="left_foot_1">
+<link name="$(arg tf_prefix)/left_foot_1">
   <inertial>
     <origin xyz="0.03678225489457133 -0.0014130788744076417 -0.02104523782784523" rpy="0 0 0"/>
@@ -284,5 +285,5 @@
   </collision>
 </link>
-<link name="JX_servo_v12_14">
+<link name="$(arg tf_prefix)/JX_servo_v12_14">
   <inertial>
     <origin xyz="0.00027407227629309625 4.531167108190459e-13 0.012509678934477936" rpy="0 0 0"/>
@@ -304,5 +305,5 @@
   </collision>
 </link>
-<link name="right_hip_side_1">
+<link name="$(arg tf_prefix)/right_hip_side_1">
   <inertial>
     <origin xyz="-0.0006601764265435368 -7.984240907310536e-10 -0.021141552658250296" rpy="0 0 0"/>
@@ -324,5 +325,5 @@
   </collision>
 </link>
-<link name="JX_servo_v12_15">
+<link name="$(arg tf_prefix)/JX_servo_v12_15">
   <inertial>
     <origin xyz="-0.03890967893447782 4.5325548869712406e-13 -0.017725838898350943" rpy="0 0 0"/>
@@ -344,5 +345,5 @@
   </collision>
 </link>
-<link name="right_ankle_1">
+<link name="$(arg tf_prefix)/right_ankle_1">
   <inertial>
     <origin xyz="0.02375859039821196 -0.00933627329560792 -0.06494791715192275" rpy="0 0 0"/>
@@ -364,5 +365,5 @@
   </collision>
 </link>
-<link name="JX_servo_v12_16">
+<link name="$(arg tf_prefix)/JX_servo_v12_16">
   <inertial>
     <origin xyz="-0.008499999656819584 0.016409678591751596 0.03717416110164953" rpy="0 0 0"/>
@@ -384,5 +385,5 @@
   </collision>
 </link>
-<link name="right_thigh_1">
+<link name="$(arg tf_prefix)/right_thigh_1">
   <inertial>
     <origin xyz="0.0035522343275843837 0.03728602282125167 -0.06738525640624529" rpy="0 0 0"/>
@@ -404,5 +405,5 @@
   </collision>
 </link>
-<link name="JX_servo_v12_17">
+<link name="$(arg tf_prefix)/JX_servo_v12_17">
   <inertial>
     <origin xyz="3.431804328560273e-10 0.038909678591752296 -0.017725838898350554" rpy="0 0 0"/>
@@ -424,5 +425,5 @@
   </collision>
 </link>
-<link name="right_calve_1">
+<link name="$(arg tf_prefix)/right_calve_1">
   <inertial>
     <origin xyz="-0.00854999027881307 0.011776733864301954 -0.035312401211175015" rpy="0 0 0"/>
@@ -444,5 +445,5 @@
   </collision>
 </link>
-<link name="JX_servo_v12_18">
+<link name="$(arg tf_prefix)/JX_servo_v12_18">
   <inertial>
     <origin xyz="3.422741994343892e-10 0.03890967859175305 0.017726049825012857" rpy="0 0 0"/>
@@ -464,5 +465,5 @@
   </collision>
 </link>
-<link name="right_ankle_2">
+<link name="$(arg tf_prefix)/right_ankle_2">
   <inertial>
     <origin xyz="-0.040641409601788116 0.017336272610156585 -0.008851871921415178" rpy="0 0 0"/>
@@ -484,5 +485,5 @@
   </collision>
 </link>
-<link name="JX_servo_v12_19">
+<link name="$(arg tf_prefix)/JX_servo_v12_19">
   <inertial>
     <origin xyz="-0.012509678934477693 -0.00850000068590498 -0.03717395017498715" rpy="0 0 0"/>
@@ -504,5 +505,5 @@
   </collision>
 </link>
-<link name="right_foot_1">
+<link name="$(arg tf_prefix)/right_foot_1">
   <inertial>
     <origin xyz="0.03678225489457156 0.001413078874407711 -0.021045237827845564" rpy="0 0 0"/>
@@ -524,5 +525,5 @@
   </collision>
 </link>
-<link name="25t-servo-hub_1">
+<link name="$(arg tf_prefix)/25t-servo-hub_1">
   <inertial>
     <origin xyz="-4.77893450374911e-07 0.003136191852991313 1.6215494567234368e-07" rpy="0 0 0"/>
@@ -544,5 +545,5 @@
   </collision>
 </link>
-<link name="gobilda-servo_1">
+<link name="$(arg tf_prefix)/gobilda-servo_1">
   <inertial>
     <origin xyz="1.3433243441218767e-09 0.021117732524250116 -0.00976910769495494" rpy="0 0 0"/>
@@ -564,5 +565,5 @@
   </collision>
 </link>
-<link name="left_bicep_1">
+<link name="$(arg tf_prefix)/left_bicep_1">
   <inertial>
     <origin xyz="0.007500000000005787 -0.003484179384329711 -0.06115545050144429" rpy="0 0 0"/>
@@ -584,5 +585,5 @@
   </collision>
 </link>
-<link name="gobilda-servo_3">
+<link name="$(arg tf_prefix)/gobilda-servo_3">
   <inertial>
     <origin xyz="0.007500001343324372 -0.015782267475749873 -0.01726910769495492" rpy="0 0 0"/>
@@ -604,5 +605,5 @@
   </collision>
 </link>
-<link name="25t-servo-hub_2">
+<link name="$(arg tf_prefix)/25t-servo-hub_2">
   <inertial>
     <origin xyz="-4.77893450343686e-07 0.000342191852934437 1.6215494560989363e-07" rpy="0 0 0"/>
@@ -624,5 +625,5 @@
   </collision>
 </link>
-<link name="elbow-attach_1">
+<link name="$(arg tf_prefix)/elbow-attach_1">
   <inertial>
     <origin xyz="-0.009233924925004727 -0.0015151372970110405 -0.002548115188024211" rpy="0 0 0"/>
@@ -644,5 +645,5 @@
   </collision>
 </link>
-<link name="left_forearm_1">
+<link name="$(arg tf_prefix)/left_forearm_1">
   <inertial>
     <origin xyz="0.00223843912986596 0.02233699999994311 -0.06792564077352817" rpy="0 0 0"/>
@@ -664,5 +665,5 @@
   </collision>
 </link>
-<link name="elbow-bearing_1">
+<link name="$(arg tf_prefix)/elbow-bearing_1">
   <inertial>
     <origin xyz="0.017892138559024794 0.003495502323537125 -0.012651303520558516" rpy="0 0 0"/>
@@ -684,5 +685,5 @@
   </collision>
 </link>
-<link name="25t-servo-hub_Mirror__1">
+<link name="$(arg tf_prefix)/25t-servo-hub_Mirror__1">
   <inertial>
     <origin xyz="8.974977877482249e-07 -0.0031361151897775635 1.0845728465602722e-06" rpy="0 0 0"/>
@@ -704,5 +705,5 @@
   </collision>
 </link>
-<link name="gobilda-servo_Mirror__1">
+<link name="$(arg tf_prefix)/gobilda-servo_Mirror__1">
   <inertial>
     <origin xyz="1.3433243441218767e-09 -0.02111773252430696 -0.009769107694954933" rpy="0 0 0"/>
@@ -724,5 +725,5 @@
   </collision>
 </link>
-<link name="right_bicep_1">
+<link name="$(arg tf_prefix)/right_bicep_1">
   <inertial>
     <origin xyz="0.00750000000000579 0.0034841793842728674 -0.06115545050144429" rpy="0 0 0"/>
@@ -744,5 +745,5 @@
   </collision>
 </link>
-<link name="gobilda-servo_Mirror__2">
+<link name="$(arg tf_prefix)/gobilda-servo_Mirror__2">
   <inertial>
     <origin xyz="0.007500001343324372 0.015782267475693 -0.017269107694954933" rpy="0 0 0"/>
@@ -764,5 +765,5 @@
   </collision>
 </link>
-<link name="25t-servo-hub_Mirror__2">
+<link name="$(arg tf_prefix)/25t-servo-hub_Mirror__2">
   <inertial>
     <origin xyz="8.97497787772511e-07 -0.00034211518977761424 1.0845728465325166e-06" rpy="0 0 0"/>
@@ -784,5 +785,5 @@
   </collision>
 </link>
-<link name="elbow-attach_Mirror__1">
+<link name="$(arg tf_prefix)/elbow-attach_Mirror__1">
   <inertial>
     <origin xyz="-0.009233924925004636 0.001515137296954086 -0.0025481151880241137" rpy="0 0 0"/>
@@ -804,5 +805,5 @@
   </collision>
 </link>
-<link name="right_forearm_1">
+<link name="$(arg tf_prefix)/right_forearm_1">
   <inertial>
     <origin xyz="0.0022384391298659947 -0.02233700000000001 -0.06792564077352811" rpy="0 0 0"/>
@@ -824,5 +825,5 @@
   </collision>
 </link>
-<link name="elbow-bearing_Mirror__1">
+<link name="$(arg tf_prefix)/elbow-bearing_Mirror__1">
   <inertial>
     <origin xyz="0.01789213855902462 -0.003495502323594024 -0.012651303520558488" rpy="0 0 0"/>
@@ -844,5 +845,5 @@
   </collision>
 </link>
-<link name="custom_servo_support__lower_neck__v2_1">
+<link name="$(arg tf_prefix)/custom_servo_support__lower_neck__v2_1">
   <inertial>
     <origin xyz="-0.0001818603745370151 4.095612737842203e-15 0.001967193599301919" rpy="0 0 0"/>
@@ -864,5 +865,5 @@
   </collision>
 </link>
-<link name="gobilda-servo_4">
+<link name="$(arg tf_prefix)/gobilda-servo_4">
   <inertial>
     <origin xyz="0.017269107739658406 0.007500001343324397 0.015782267475689782" rpy="0 0 0"/>
@@ -884,5 +885,5 @@
   </collision>
 </link>
-<link name="25t-servo-hub_3">
+<link name="$(arg tf_prefix)/25t-servo-hub_3">
   <inertial>
     <origin xyz="-4.778487469048187e-07 1.6215494569815637e-07 -0.0003421918530514406" rpy="0 0 0"/>
@@ -904,5 +905,5 @@
   </collision>
 </link>
-<link name="neck_1">
+<link name="$(arg tf_prefix)/neck_1">
   <inertial>
     <origin xyz="4.4703468357609744e-11 0.0015600923125218369 0.014702901470170587" rpy="0 0 0"/>
@@ -924,5 +925,5 @@
   </collision>
 </link>
-<link name="25t-servo-hub_4">
+<link name="$(arg tf_prefix)/25t-servo-hub_4">
   <inertial>
     <origin xyz="-4.77848746903084e-07 0.003136191852991365 6.322169145839274e-07" rpy="0 0 0"/>
@@ -944,5 +945,5 @@
   </collision>
 </link>
-<link name="gobilda-servo_5">
+<link name="$(arg tf_prefix)/gobilda-servo_5">
   <inertial>
     <origin xyz="0.009769107739658408 0.021117732524250185 4.714052932869306e-07" rpy="0 0 0"/>
@@ -964,5 +965,5 @@
   </collision>
 </link>
-<link name="head_1">
+<link name="$(arg tf_prefix)/head_1">
   <inertial>
     <origin xyz="0.017762050405363966 -0.005180173125019489 5.450273398273364e-05" rpy="0 0 0"/>
@@ -984,5 +985,5 @@
   </collision>
 </link>
-<link name="camera_1">
+<link name="$(arg tf_prefix)/camera">
   <inertial>
     <origin xyz="0.014184398578565184 -1.0759407732763727e-05 0.019215618136865634" rpy="0 0 0"/>
@@ -1004,5 +1005,5 @@
   </collision>
 </link>
-<link name="camera-link_1">
+<link name="$(arg tf_prefix)/camera-link_1">
   <inertial>
     <origin xyz="0.0005000006258488593 -3.1298447384156547e-10 4.7006196884913365e-07" rpy="0 0 0"/>
@@ -1024,5 +1025,5 @@
   </collision>
 </link>
-<link name="imu-link_1">
+<link name="$(arg tf_prefix)/imu">
   <inertial>
     <origin xyz="-4.440892098500626e-18 -1.7763568394002505e-17 -0.0495" rpy="0 0 0"/>
@@ -1044,5 +1045,5 @@
   </collision>
 </link>
-<link name="Component32_1">
+<link name="$(arg tf_prefix)/Component32_1">
   <inertial>
     <origin xyz="-8.673617379884035e-18 3.3333333333211267e-07 -0.0235" rpy="0 0 0"/>
@@ -1064,5 +1065,5 @@
   </collision>
 </link>
-<link name="TX2_board_v2_1">
+<link name="$(arg tf_prefix)/TX2_board_v2_1">
   <inertial>
     <origin xyz="0.0007727737790098402 -3.4264823634152304e-05 -0.015294861644822792" rpy="0 0 0"/>
@@ -1086,286 +1087,286 @@
 <joint name="Rigid1" type="fixed">
   <origin xyz="0.0 0.005 0.0" rpy="0 0 0"/>
-  <parent link="base_link"/>
-  <child link="torso_1"/>
+  <parent link="$(arg tf_prefix)/base_link"/>
+  <child link="$(arg tf_prefix)/torso"/>
 </joint>
 <joint name="Rigid2" type="fixed">
   <origin xyz="-0.0225 0.0495 -0.13699" rpy="0 0 0"/>
-  <parent link="torso_1"/>
-  <child link="JX_servo_v12_1"/>
+  <parent link="$(arg tf_prefix)/torso"/>
+  <child link="$(arg tf_prefix)/JX_servo_v12_1"/>
 </joint>
 <joint name="left_leg_motor_0" type="continuous">
   <origin xyz="0.018 0.0 -0.0264" rpy="0 0 0"/>
-  <parent link="JX_servo_v12_1"/>
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