Commit message: fix imu issue
- imu link name was wrong in xacro -> messes with tf tree stuff
- fixed initial height that caused sudden jump

File: bez3_description/urdf/bez3.urdf (robot description, URDF)
Before this commit: robot bez3, 54 links, 53 joints
Links:
- removed link /camera_1
- removed link /imu-link_1
- removed link /torso_1
- added link /camera, mass 0.094257141411043; collision mesh filename=package://bez3_description/meshes/camera_1.stl scale=1 1 1; visual mesh filename=package://bez3_description/meshes/camera_1.stl scale=1 1 1
- added link /imu_link, mass 0.00019625; collision mesh filename=package://bez3_description/meshes/imu-link_1.stl scale=1 1 1; visual mesh filename=package://bez3_description/meshes/imu-link_1.stl scale=1 1 1
- added link /torso, mass 0.2968069064800233; collision mesh filename=package://bez3_description/meshes/torso_1.stl scale=1 1 1; visual mesh filename=package://bez3_description/meshes/torso_1.stl scale=1 1 1
- link /25t-servo-hub_1: geometry collision mesh filename=package://bez3_description/meshes/25t-servo-hub_1.stl scale=1 1 1; visual mesh filename=package://bez3_description/meshes/25t-servo-hub_1.stl scale=1 1 1
- link /25t-servo-hub_2: geometry collision mesh filename=package://bez3_description/meshes/25t-servo-hub_2.stl scale=1 1 1; visual mesh filename=package://bez3_description/meshes/25t-servo-hub_2.stl scale=1 1 1
- link /25t-servo-hub_3: geometry collision mesh filename=package://bez3_description/meshes/25t-servo-hub_3.stl scale=1 1 1; visual mesh filename=package://bez3_description/meshes/25t-servo-hub_3.stl scale=1 1 1
- link /25t-servo-hub_4: geometry collision mesh filename=package://bez3_description/meshes/25t-servo-hub_4.stl scale=1 1 1; visual mesh filename=package://bez3_description/meshes/25t-servo-hub_4.stl scale=1 1 1
- link /25t-servo-hub_Mirror__1: geometry collision mesh filename=package://bez3_description/meshes/25t-servo-hub_Mirror__1.s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 scale=1 1 1; visual mesh filename=package://bez3_description/meshes/25t-servo-hub_Mirror__1.s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 scale=1 1 1
- link /25t-servo-hub_Mirror__2: geometry collision mesh filename=package://bez3_description/meshes/25t-servo-hub_Mirror__2.s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 scale=1 1 1; visual mesh filename=package://bez3_description/meshes/25t-servo-hub_Mirror__2.s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 scale=1 1 1
- link /Component32_1: geometry collision mesh filename=package://bez3_description/meshes/Component32_1.stl scale=1 1 1; visual mesh filename=package://bez3_description/meshes/Component32_1.stl scale=1 1 1
- link /JX_servo_v12_1: geometry collision mesh filename=package://bez3_description/meshes/JX_servo_v12_1.stl scale=1 1 1; visual mesh filename=package://bez3_description/meshes/JX_servo_v12_1.stl scale=1 1 1
- link /JX_servo_v12_11: geometry collision mesh filename=package://bez3_description/meshes/JX_servo_v12_11.stl scale=1 1 1; visual mesh filename=package://bez3_description/meshes/JX_servo_v12_11.stl scale=1 1 1
- link /JX_servo_v12_12: geometry collision mesh filename=package://bez3_description/meshes/JX_servo_v12_12.stl scale=1 1 1; visual mesh filename=package://bez3_description/meshes/JX_servo_v12_12.stl scale=1 1 1
- link /JX_servo_v12_13: geometry collision mesh filename=package://bez3_description/meshes/JX_servo_v12_13.stl scale=1 1 1; visual mesh filename=package://bez3_description/meshes/JX_servo_v12_13.stl scale=1 1 1
- link /JX_servo_v12_14: geometry collision mesh filename=package://bez3_description/meshes/JX_servo_v12_14.stl scale=1 1 1; visual mesh filename=package://bez3_description/meshes/JX_servo_v12_14.stl scale=1 1 1
- link /JX_servo_v12_15: geometry collision mesh filename=package://bez3_description/meshes/JX_servo_v12_15.stl scale=1 1 1; visual mesh filename=package://bez3_description/meshes/JX_servo_v12_15.stl scale=1 1 1
- link /JX_servo_v12_16: geometry collision mesh filename=package://bez3_description/meshes/JX_servo_v12_16.stl scale=1 1 1; visual mesh filename=package://bez3_description/meshes/JX_servo_v12_16.stl scale=1 1 1
- link /JX_servo_v12_17: geometry collision mesh filename=package://bez3_description/meshes/JX_servo_v12_17.stl scale=1 1 1; visual mesh filename=package://bez3_description/meshes/JX_servo_v12_17.stl scale=1 1 1
- link /JX_servo_v12_18: geometry collision mesh filename=package://bez3_description/meshes/JX_servo_v12_18.stl scale=1 1 1; visual mesh filename=package://bez3_description/meshes/JX_servo_v12_18.stl scale=1 1 1
- link /JX_servo_v12_19: geometry collision mesh filename=package://bez3_description/meshes/JX_servo_v12_19.stl scale=1 1 1; visual mesh filename=package://bez3_description/meshes/JX_servo_v12_19.stl scale=1 1 1
- link /JX_servo_v12_8: geometry collision mesh filename=package://bez3_description/meshes/JX_servo_v12_8.stl scale=1 1 1; visual mesh filename=package://bez3_description/meshes/JX_servo_v12_8.stl scale=1 1 1
- link /JX_servo_v12_9: geometry collision mesh filename=package://bez3_description/meshes/JX_servo_v12_9.stl scale=1 1 1; visual mesh filename=package://bez3_description/meshes/JX_servo_v12_9.stl scale=1 1 1
- link /TX2_board_v2_1: geometry collision mesh filename=package://bez3_description/meshes/TX2_board_v2_1.stl scale=1 1 1; visual mesh filename=package://bez3_description/meshes/TX2_board_v2_1.stl scale=1 1 1
- link /base_link: geometry collision mesh filename=package://bez3_description/meshes/base_link.stl scale=1 1 1; visual mesh filename=package://bez3_description/meshes/base_link.stl scale=1 1 1
- link /camera-link_1: geometry collision mesh filename=package://bez3_description/meshes/camera-link_1.stl scale=1 1 1; visual mesh filename=package://bez3_description/meshes/camera-link_1.stl scale=1 1 1
- link /custom_servo_support__lower_neck__v2_1: geometry collision mesh filename=package://bez3_description/meshes/custom_servo_support__low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 scale=1 1 1; visual mesh filename=package://bez3_description/meshes/custom_servo_support__low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 scale=1 1 1
- link /elbow-attach_1: geometry collision mesh filename=package://bez3_description/meshes/elbow-attach_1.stl scale=1 1 1; visual mesh filename=package://bez3_description/meshes/elbow-attach_1.stl scale=1 1 1
- link /elbow-attach_Mirror__1: geometry collision mesh filename=package://bez3_description/meshes/elbow-attach_Mirror__1.stl scale=1 1 1; visual mesh filename=package://bez3_description/meshes/elbow-attach_Mirror__1.stl scale=1 1 1
- link /elbow-bearing_1: geometry collision mesh filename=package://bez3_description/meshes/elbow-bearing_1.stl scale=1 1 1; visual mesh filename=package://bez3_description/meshes/elbow-bearing_1.stl scale=1 1 1
- link /elbow-bearing_Mirror__1: geometry collision mesh filename=package://bez3_description/meshes/elbow-bearing_Mirror__1.s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 scale=1 1 1; visual mesh filename=package://bez3_description/meshes/elbow-bearing_Mirror__1.s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 scale=1 1 1
- link /gobilda-servo_1: geometry collision mesh filename=package://bez3_description/meshes/gobilda-servo_1.stl scale=1 1 1; visual mesh filename=package://bez3_description/meshes/gobilda-servo_1.stl scale=1 1 1
- link /gobilda-servo_3: geometry collision mesh filename=package://bez3_description/meshes/gobilda-servo_3.stl scale=1 1 1; visual mesh filename=package://bez3_description/meshes/gobilda-servo_3.stl scale=1 1 1
- link /gobilda-servo_4: geometry collision mesh filename=package://bez3_description/meshes/gobilda-servo_4.stl scale=1 1 1; visual mesh filename=package://bez3_description/meshes/gobilda-servo_4.stl scale=1 1 1
- link /gobilda-servo_5: geometry collision mesh filename=package://bez3_description/meshes/gobilda-servo_5.stl scale=1 1 1; visual mesh filename=package://bez3_description/meshes/gobilda-servo_5.stl scale=1 1 1
- link /gobilda-servo_Mirror__1: geometry collision mesh filename=package://bez3_description/meshes/gobilda-servo_Mirror__1.s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 scale=1 1 1; visual mesh filename=package://bez3_description/meshes/gobilda-servo_Mirror__1.s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 scale=1 1 1
- link /gobilda-servo_Mirror__2: geometry collision mesh filename=package://bez3_description/meshes/gobilda-servo_Mirror__2.s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 scale=1 1 1; visual mesh filename=package://bez3_description/meshes/gobilda-servo_Mirror__2.s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 scale=1 1 1
- link /head_1: geometry collision mesh filename=package://bez3_description/meshes/head_1.stl scale=1 1 1; visual mesh filename=package://bez3_description/meshes/head_1.stl scale=1 1 1
- link /left_bicep_1: geometry collision mesh filename=package://bez3_description/meshes/left_bicep_1.stl scale=1 1 1; visual mesh filename=package://bez3_description/meshes/left_bicep_1.stl scale=1 1 1
- link /left_calve_1: geometry collision mesh filename=package://bez3_description/meshes/left_calve_1.stl scale=1 1 1; visual mesh filename=package://bez3_description/meshes/left_calve_1.stl scale=1 1 1
- link /left_foot_1: geometry collision mesh filename=package://bez3_description/meshes/left_foot_1.stl scale=1 1 1; visual mesh filename=package://bez3_description/meshes/left_foot_1.stl scale=1 1 1
- link /left_forearm_1: geometry collision mesh filename=package://bez3_description/meshes/left_forearm_1.stl scale=1 1 1; visual mesh filename=package://bez3_description/meshes/left_forearm_1.stl scale=1 1 1
- link /left_hip_front_1: geometry collision mesh filename=package://bez3_description/meshes/left_hip_front_1.stl scale=1 1 1; visual mesh filename=package://bez3_description/meshes/left_hip_front_1.stl scale=1 1 1
- link /left_hip_front_2: geometry collision mesh filename=package://bez3_description/meshes/left_hip_front_2.stl scale=1 1 1; visual mesh filename=package://bez3_description/meshes/left_hip_front_2.stl scale=1 1 1
- link /left_hip_side_1: geometry collision mesh filename=package://bez3_description/meshes/left_hip_side_1.stl scale=1 1 1; visual mesh filename=package://bez3_description/meshes/left_hip_side_1.stl scale=1 1 1
- link /left_thigh_1: geometry collision mesh filename=package://bez3_description/meshes/left_thigh_1.stl scale=1 1 1; visual mesh filename=package://bez3_description/meshes/left_thigh_1.stl scale=1 1 1
- link /neck_1: geometry collision mesh filename=package://bez3_description/meshes/neck_1.stl scale=1 1 1; visual mesh filename=package://bez3_description/meshes/neck_1.stl scale=1 1 1
- link /right_ankle_1: geometry collision mesh filename=package://bez3_description/meshes/right_ankle_1.stl scale=1 1 1; visual mesh filename=package://bez3_description/meshes/right_ankle_1.stl scale=1 1 1
- link /right_ankle_2: geometry collision mesh filename=package://bez3_description/meshes/right_ankle_2.stl scale=1 1 1; visual mesh filename=package://bez3_description/meshes/right_ankle_2.stl scale=1 1 1
- link /right_bicep_1: geometry collision mesh filename=package://bez3_description/meshes/right_bicep_1.stl scale=1 1 1; visual mesh filename=package://bez3_description/meshes/right_bicep_1.stl scale=1 1 1
- link /right_calve_1: geometry collision mesh filename=package://bez3_description/meshes/right_calve_1.stl scale=1 1 1; visual mesh filename=package://bez3_description/meshes/right_calve_1.stl scale=1 1 1
- link /right_foot_1: geometry collision mesh filename=package://bez3_description/meshes/right_foot_1.stl scale=1 1 1; visual mesh filename=package://bez3_description/meshes/right_foot_1.stl scale=1 1 1
- link /right_forearm_1: geometry collision mesh filename=package://bez3_description/meshes/right_forearm_1.stl scale=1 1 1; visual mesh filename=package://bez3_description/meshes/right_forearm_1.stl scale=1 1 1
- link /right_hip_side_1: geometry collision mesh filename=package://bez3_description/meshes/right_hip_side_1.stl scale=1 1 1; visual mesh filename=package://bez3_description/meshes/right_hip_side_1.stl scale=1 1 1
- link /right_thigh_1: geometry collision mesh filename=package://bez3_description/meshes/right_thigh_1.stl scale=1 1 1; visual mesh filename=package://bez3_description/meshes/right_thigh_1.stl scale=1 1 1
Joints:
- joint Rigid1: child /torso_1 -> /torso
- joint Rigid14: parent /torso_1 -> /torso
- joint Rigid2: parent /torso_1 -> /torso
- joint Rigid26: parent /torso_1 -> /torso
- joint Rigid34: parent /torso_1 -> /torso
- joint Rigid42: parent /torso_1 -> /torso
- joint Rigid49: child /camera_1 -> /camera
- joint Rigid52: parent /torso_1 -> /torso
- joint camera_joint: parent /camera_1 -> /camera
- joint imu_joint: child /imu-link_1 -> /imu_link; parent /torso_1 -> /torso
