Commit message: fix imu issue
- imu link name was wrong in xacro -> messes with tf tree stuff
- fixed initial height that caused sudden jump

File: bez3_description/urdf/bez3.xacro (robot description, xacro)
@@ -14,5 +14,5 @@
     <origin xyz="0 0 0" rpy="0 0 0"/>
     <geometry>
-      <mesh filename="package://bez3_description/meshes/base_link.stl" scale="0.001 0.001 0.001"/>
+      <mesh filename="package://bez3_description/meshes/base_link.stl" scale="1 1 1"/>
     </geometry>
     <material name="steel_satin"/>
@@ -21,5 +21,5 @@
     <origin xyz="0 0 0" rpy="0 0 0"/>
     <geometry>
-      <mesh filename="package://bez3_description/meshes/base_link.stl" scale="0.001 0.001 0.001"/>
+      <mesh filename="package://bez3_description/meshes/base_link.stl" scale="1 1 1"/>
     </geometry>
   </collision>
@@ -34,5 +34,5 @@
     <origin xyz="-0.0 -0.005 -0.0" rpy="0 0 0"/>
     <geometry>
-      <mesh filename="package://bez3_description/meshes/torso_1.stl" scale="0.001 0.001 0.001"/>
+      <mesh filename="package://bez3_description/meshes/torso_1.stl" scale="1 1 1"/>
     </geometry>
     <material name="polymide_kapton"/>
@@ -41,5 +41,5 @@
     <origin xyz="-0.0 -0.005 -0.0" rpy="0 0 0"/>
     <geometry>
-      <mesh filename="package://bez3_description/meshes/torso_1.stl" scale="0.001 0.001 0.001"/>
+      <mesh filename="package://bez3_description/meshes/torso_1.stl" scale="1 1 1"/>
     </geometry>
   </collision>
@@ -54,5 +54,5 @@
     <origin xyz="0.0225 -0.0545 0.13699" rpy="0 0 0"/>
     <geometry>
-      <mesh filename="package://bez3_description/meshes/JX_servo_v12_1.stl" scale="0.001 0.001 0.001"/>
+      <mesh filename="package://bez3_description/meshes/JX_servo_v12_1.stl" scale="1 1 1"/>
     </geometry>
     <material name="plastic_matte_black"/>
@@ -61,5 +61,5 @@
     <origin xyz="0.0225 -0.0545 0.13699" rpy="0 0 0"/>
     <geometry>
-      <mesh filename="package://bez3_description/meshes/JX_servo_v12_1.stl" scale="0.001 0.001 0.001"/>
+      <mesh filename="package://bez3_description/meshes/JX_servo_v12_1.stl" scale="1 1 1"/>
     </geometry>
   </collision>
@@ -74,5 +74,5 @@
     <origin xyz="0.0045 -0.0545 0.16339" rpy="0 0 0"/>
     <geometry>
-      <mesh filename="package://bez3_description/meshes/left_hip_side_1.stl" scale="0.001 0.001 0.001"/>
+      <mesh filename="package://bez3_description/meshes/left_hip_side_1.stl" scale="1 1 1"/>
     </geometry>
     <material name="plastic_glossy_black"/>
@@ -81,5 +81,5 @@
     <origin xyz="0.0045 -0.0545 0.16339" rpy="0 0 0"/>
     <geometry>
-      <mesh filename="package://bez3_description/meshes/left_hip_side_1.stl" scale="0.001 0.001 0.001"/>
+      <mesh filename="package://bez3_description/meshes/left_hip_side_1.stl" scale="1 1 1"/>
     </geometry>
   </collision>
@@ -94,5 +94,5 @@
     <origin xyz="0.0345 -0.0545 0.198726" rpy="0 0 0"/>
     <geometry>
-      <mesh filename="package://bez3_description/meshes/JX_servo_v12_8.stl" scale="0.001 0.001 0.001"/>
+      <mesh filename="package://bez3_description/meshes/JX_servo_v12_8.stl" scale="1 1 1"/>
     </geometry>
     <material name="plastic_matte_black"/>
@@ -101,5 +101,5 @@
     <origin xyz="0.0345 -0.0545 0.198726" rpy="0 0 0"/>
     <geometry>
-      <mesh filename="package://bez3_description/meshes/JX_servo_v12_8.stl" scale="0.001 0.001 0.001"/>
+      <mesh filename="package://bez3_description/meshes/JX_servo_v12_8.stl" scale="1 1 1"/>
     </geometry>
   </collision>
@@ -114,5 +114,5 @@
     <origin xyz="0.0609 -0.046 0.179826" rpy="0 0 0"/>
     <geometry>
-      <mesh filename="package://bez3_description/meshes/left_hip_front_1.stl" scale="0.001 0.001 0.001"/>
+      <mesh filename="package://bez3_description/meshes/left_hip_front_1.stl" scale="1 1 1"/>
     </geometry>
     <material name="plastic_glossy_black"/>
@@ -121,5 +121,5 @@
     <origin xyz="0.0609 -0.046 0.179826" rpy="0 0 0"/>
     <geometry>
-      <mesh filename="package://bez3_description/meshes/left_hip_front_1.stl" scale="0.001 0.001 0.001"/>
+      <mesh filename="package://bez3_description/meshes/left_hip_front_1.stl" scale="1 1 1"/>
     </geometry>
   </collision>
@@ -134,5 +134,5 @@
     <origin xyz="-0.0035 -0.0699 0.253626" rpy="0 0 0"/>
     <geometry>
-      <mesh filename="package://bez3_description/meshes/JX_servo_v12_9.stl" scale="0.001 0.001 0.001"/>
+      <mesh filename="package://bez3_description/meshes/JX_servo_v12_9.stl" scale="1 1 1"/>
     </geometry>
     <material name="plastic_matte_black"/>
@@ -141,5 +141,5 @@
     <origin xyz="-0.0035 -0.0699 0.253626" rpy="0 0 0"/>
     <geometry>
-      <mesh filename="package://bez3_description/meshes/JX_servo_v12_9.stl" scale="0.001 0.001 0.001"/>
+      <mesh filename="package://bez3_description/meshes/JX_servo_v12_9.stl" scale="1 1 1"/>
     </geometry>
   </collision>
@@ -154,5 +154,5 @@
     <origin xyz="0.005 -0.0924 0.198726" rpy="0 0 0"/>
     <geometry>
-      <mesh filename="package://bez3_description/meshes/left_thigh_1.stl" scale="0.001 0.001 0.001"/>
+      <mesh filename="package://bez3_description/meshes/left_thigh_1.stl" scale="1 1 1"/>
     </geometry>
     <material name="plastic_glossy_black"/>
@@ -161,5 +161,5 @@
     <origin xyz="0.005 -0.0924 0.198726" rpy="0 0 0"/>
     <geometry>
-      <mesh filename="package://bez3_description/meshes/left_thigh_1.stl" scale="0.001 0.001 0.001"/>
+      <mesh filename="package://bez3_description/meshes/left_thigh_1.stl" scale="1 1 1"/>
     </geometry>
   </collision>
@@ -174,5 +174,5 @@
     <origin xyz="0.005 -0.0924 0.322726" rpy="0 0 0"/>
     <geometry>
-      <mesh filename="package://bez3_description/meshes/JX_servo_v12_11.stl" scale="0.001 0.001 0.001"/>
+      <mesh filename="package://bez3_description/meshes/JX_servo_v12_11.stl" scale="1 1 1"/>
     </geometry>
     <material name="plastic_matte_black"/>
@@ -181,5 +181,5 @@
     <origin xyz="0.005 -0.0924 0.322726" rpy="0 0 0"/>
     <geometry>
-      <mesh filename="package://bez3_description/meshes/JX_servo_v12_11.stl" scale="0.001 0.001 0.001"/>
+      <mesh filename="package://bez3_description/meshes/JX_servo_v12_11.stl" scale="1 1 1"/>
     </geometry>
   </collision>
@@ -194,5 +194,5 @@
     <origin xyz="-0.0035 -0.066 0.377626" rpy="0 0 0"/>
     <geometry>
-      <mesh filename="package://bez3_description/meshes/left_calve_1.stl" scale="0.001 0.001 0.001"/>
+      <mesh filename="package://bez3_description/meshes/left_calve_1.stl" scale="1 1 1"/>
     </geometry>
     <material name="plastic_glossy_black"/>
@@ -201,5 +201,5 @@
     <origin xyz="-0.0035 -0.066 0.377626" rpy="0 0 0"/>
     <geometry>
-      <mesh filename="package://bez3_description/meshes/left_calve_1.stl" scale="0.001 0.001 0.001"/>
+      <mesh filename="package://bez3_description/meshes/left_calve_1.stl" scale="1 1 1"/>
     </geometry>
   </collision>
@@ -214,5 +214,5 @@
     <origin xyz="0.00505 -0.094 0.462631" rpy="0 0 0"/>
     <geometry>
-      <mesh filename="package://bez3_description/meshes/JX_servo_v12_12.stl" scale="0.001 0.001 0.001"/>
+      <mesh filename="package://bez3_description/meshes/JX_servo_v12_12.stl" scale="1 1 1"/>
     </geometry>
     <material name="plastic_matte_black"/>
@@ -221,5 +221,5 @@
     <origin xyz="0.00505 -0.094 0.462631" rpy="0 0 0"/>
     <geometry>
-      <mesh filename="package://bez3_description/meshes/JX_servo_v12_12.stl" scale="0.001 0.001 0.001"/>
+      <mesh filename="package://bez3_description/meshes/JX_servo_v12_12.stl" scale="1 1 1"/>
     </geometry>
   </collision>
@@ -234,5 +234,5 @@
     <origin xyz="-0.00345 -0.0715 0.407731" rpy="0 0 0"/>
     <geometry>
-      <mesh filename="package://bez3_description/meshes/left_hip_front_2.stl" scale="0.001 0.001 0.001"/>
+      <mesh filename="package://bez3_description/meshes/left_hip_front_2.stl" scale="1 1 1"/>
     </geometry>
     <material name="plastic_glossy_black"/>
@@ -241,5 +241,5 @@
     <origin xyz="-0.00345 -0.0715 0.407731" rpy="0 0 0"/>
     <geometry>
-      <mesh filename="package://bez3_description/meshes/left_hip_front_2.stl" scale="0.001 0.001 0.001"/>
+      <mesh filename="package://bez3_description/meshes/left_hip_front_2.stl" scale="1 1 1"/>
     </geometry>
   </collision>
@@ -254,5 +254,5 @@
     <origin xyz="0.06095 -0.0465 0.407731" rpy="0 0 0"/>
     <geometry>
-      <mesh filename="package://bez3_description/meshes/JX_servo_v12_13.stl" scale="0.001 0.001 0.001"/>
+      <mesh filename="package://bez3_description/meshes/JX_servo_v12_13.stl" scale="1 1 1"/>
     </geometry>
     <material name="plastic_matte_black"/>
@@ -261,5 +261,5 @@
     <origin xyz="0.06095 -0.0465 0.407731" rpy="0 0 0"/>
     <geometry>
-      <mesh filename="package://bez3_description/meshes/JX_servo_v12_13.stl" scale="0.001 0.001 0.001"/>
+      <mesh filename="package://bez3_description/meshes/JX_servo_v12_13.stl" scale="1 1 1"/>
     </geometry>
   </collision>
@@ -274,5 +274,5 @@
     <origin xyz="0.03455 -0.055 0.462631" rpy="0 0 0"/>
     <geometry>
-      <mesh filename="package://bez3_description/meshes/left_foot_1.stl" scale="0.001 0.001 0.001"/>
+      <mesh filename="package://bez3_description/meshes/left_foot_1.stl" scale="1 1 1"/>
     </geometry>
     <material name="plastic_glossy_black"/>
@@ -281,5 +281,5 @@
     <origin xyz="0.03455 -0.055 0.462631" rpy="0 0 0"/>
     <geometry>
-      <mesh filename="package://bez3_description/meshes/left_foot_1.stl" scale="0.001 0.001 0.001"/>
+      <mesh filename="package://bez3_description/meshes/left_foot_1.stl" scale="1 1 1"/>
     </geometry>
   </collision>
@@ -294,5 +294,5 @@
     <origin xyz="0.0225 0.0545 0.137" rpy="0 0 0"/>
     <geometry>
-      <mesh filename="package://bez3_description/meshes/JX_servo_v12_14.stl" scale="0.001 0.001 0.001"/>
+      <mesh filename="package://bez3_description/meshes/JX_servo_v12_14.stl" scale="1 1 1"/>
     </geometry>
     <material name="plastic_matte_black"/>
@@ -301,5 +301,5 @@
     <origin xyz="0.0225 0.0545 0.137" rpy="0 0 0"/>
     <geometry>
-      <mesh filename="package://bez3_description/meshes/JX_servo_v12_14.stl" scale="0.001 0.001 0.001"/>
+      <mesh filename="package://bez3_description/meshes/JX_servo_v12_14.stl" scale="1 1 1"/>
     </geometry>
   </collision>
@@ -314,5 +314,5 @@
     <origin xyz="0.0045 0.0545 0.1634" rpy="0 0 0"/>
     <geometry>
-      <mesh filename="package://bez3_description/meshes/right_hip_side_1.stl" scale="0.001 0.001 0.001"/>
+      <mesh filename="package://bez3_description/meshes/right_hip_side_1.stl" scale="1 1 1"/>
     </geometry>
     <material name="plastic_glossy_black"/>
@@ -321,5 +321,5 @@
     <origin xyz="0.0045 0.0545 0.1634" rpy="0 0 0"/>
     <geometry>
-      <mesh filename="package://bez3_description/meshes/right_hip_side_1.stl" scale="0.001 0.001 0.001"/>
+      <mesh filename="package://bez3_description/meshes/right_hip_side_1.stl" scale="1 1 1"/>
     </geometry>
   </collision>
@@ -334,5 +334,5 @@
     <origin xyz="0.0345 0.0545 0.198736" rpy="0 0 0"/>
     <geometry>
-      <mesh filename="package://bez3_description/meshes/JX_servo_v12_15.stl" scale="0.001 0.001 0.001"/>
+      <mesh filename="package://bez3_description/meshes/JX_servo_v12_15.stl" scale="1 1 1"/>
     </geometry>
     <material name="plastic_matte_black"/>
@@ -341,5 +341,5 @@
     <origin xyz="0.0345 0.0545 0.198736" rpy="0 0 0"/>
     <geometry>
-      <mesh filename="package://bez3_description/meshes/JX_servo_v12_15.stl" scale="0.001 0.001 0.001"/>
+      <mesh filename="package://bez3_description/meshes/JX_servo_v12_15.stl" scale="1 1 1"/>
     </geometry>
   </collision>
@@ -354,5 +354,5 @@
     <origin xyz="0.0609 0.046 0.179836" rpy="0 0 0"/>
     <geometry>
-      <mesh filename="package://bez3_description/meshes/right_ankle_1.stl" scale="0.001 0.001 0.001"/>
+      <mesh filename="package://bez3_description/meshes/right_ankle_1.stl" scale="1 1 1"/>
     </geometry>
     <material name="plastic_glossy_black"/>
@@ -361,5 +361,5 @@
     <origin xyz="0.0609 0.046 0.179836" rpy="0 0 0"/>
     <geometry>
-      <mesh filename="package://bez3_description/meshes/right_ankle_1.stl" scale="0.001 0.001 0.001"/>
+      <mesh filename="package://bez3_description/meshes/right_ankle_1.stl" scale="1 1 1"/>
     </geometry>
   </collision>
@@ -374,5 +374,5 @@
     <origin xyz="-0.0035 0.0699 0.253636" rpy="0 0 0"/>
     <geometry>
-      <mesh filename="package://bez3_description/meshes/JX_servo_v12_16.stl" scale="0.001 0.001 0.001"/>
+      <mesh filename="package://bez3_description/meshes/JX_servo_v12_16.stl" scale="1 1 1"/>
     </geometry>
     <material name="plastic_matte_black"/>
@@ -381,5 +381,5 @@
     <origin xyz="-0.0035 0.0699 0.253636" rpy="0 0 0"/>
     <geometry>
-      <mesh filename="package://bez3_description/meshes/JX_servo_v12_16.stl" scale="0.001 0.001 0.001"/>
+      <mesh filename="package://bez3_description/meshes/JX_servo_v12_16.stl" scale="1 1 1"/>
     </geometry>
   </collision>
@@ -394,5 +394,5 @@
     <origin xyz="0.005 0.0924 0.198736" rpy="0 0 0"/>
     <geometry>
-      <mesh filename="package://bez3_description/meshes/right_thigh_1.stl" scale="0.001 0.001 0.001"/>
+      <mesh filename="package://bez3_description/meshes/right_thigh_1.stl" scale="1 1 1"/>
     </geometry>
     <material name="plastic_glossy_black"/>
@@ -401,5 +401,5 @@
     <origin xyz="0.005 0.0924 0.198736" rpy="0 0 0"/>
     <geometry>
-      <mesh filename="package://bez3_description/meshes/right_thigh_1.stl" scale="0.001 0.001 0.001"/>
+      <mesh filename="package://bez3_description/meshes/right_thigh_1.stl" scale="1 1 1"/>
     </geometry>
   </collision>
@@ -414,5 +414,5 @@
     <origin xyz="0.005 0.0924 0.322736" rpy="0 0 0"/>
     <geometry>
-      <mesh filename="package://bez3_description/meshes/JX_servo_v12_17.stl" scale="0.001 0.001 0.001"/>
+      <mesh filename="package://bez3_description/meshes/JX_servo_v12_17.stl" scale="1 1 1"/>
     </geometry>
     <material name="plastic_matte_black"/>
@@ -421,5 +421,5 @@
     <origin xyz="0.005 0.0924 0.322736" rpy="0 0 0"/>
     <geometry>
-      <mesh filename="package://bez3_description/meshes/JX_servo_v12_17.stl" scale="0.001 0.001 0.001"/>
+      <mesh filename="package://bez3_description/meshes/JX_servo_v12_17.stl" scale="1 1 1"/>
     </geometry>
   </collision>
@@ -434,5 +434,5 @@
     <origin xyz="-0.0035 0.066 0.377636" rpy="0 0 0"/>
     <geometry>
-      <mesh filename="package://bez3_description/meshes/right_calve_1.stl" scale="0.001 0.001 0.001"/>
+      <mesh filename="package://bez3_description/meshes/right_calve_1.stl" scale="1 1 1"/>
     </geometry>
     <material name="plastic_glossy_black"/>
@@ -441,5 +441,5 @@
     <origin xyz="-0.0035 0.066 0.377636" rpy="0 0 0"/>
     <geometry>
-      <mesh filename="package://bez3_description/meshes/right_calve_1.stl" scale="0.001 0.001 0.001"/>
+      <mesh filename="package://bez3_description/meshes/right_calve_1.stl" scale="1 1 1"/>
     </geometry>
   </collision>
@@ -454,5 +454,5 @@
     <origin xyz="0.00505 0.094 0.462641" rpy="0 0 0"/>
     <geometry>
-      <mesh filename="package://bez3_description/meshes/JX_servo_v12_18.stl" scale="0.001 0.001 0.001"/>
+      <mesh filename="package://bez3_description/meshes/JX_servo_v12_18.stl" scale="1 1 1"/>
     </geometry>
     <material name="plastic_matte_black"/>
@@ -461,5 +461,5 @@
     <origin xyz="0.00505 0.094 0.462641" rpy="0 0 0"/>
     <geometry>
-      <mesh filename="package://bez3_description/meshes/JX_servo_v12_18.stl" scale="0.001 0.001 0.001"/>
+      <mesh filename="package://bez3_description/meshes/JX_servo_v12_18.stl" scale="1 1 1"/>
     </geometry>
   </collision>
@@ -474,5 +474,5 @@
     <origin xyz="-0.00345 0.0715 0.407741" rpy="0 0 0"/>
     <geometry>
-      <mesh filename="package://bez3_description/meshes/right_ankle_2.stl" scale="0.001 0.001 0.001"/>
+      <mesh filename="package://bez3_description/meshes/right_ankle_2.stl" scale="1 1 1"/>
     </geometry>
     <material name="plastic_glossy_black"/>
@@ -481,5 +481,5 @@
     <origin xyz="-0.00345 0.0715 0.407741" rpy="0 0 0"/>
     <geometry>
-      <mesh filename="package://bez3_description/meshes/right_ankle_2.stl" scale="0.001 0.001 0.001"/>
+      <mesh filename="package://bez3_description/meshes/right_ankle_2.stl" scale="1 1 1"/>
     </geometry>
   </collision>
@@ -494,5 +494,5 @@
     <origin xyz="0.06095 0.0465 0.407741" rpy="0 0 0"/>
     <geometry>
-      <mesh filename="package://bez3_description/meshes/JX_servo_v12_19.stl" scale="0.001 0.001 0.001"/>
+      <mesh filename="package://bez3_description/meshes/JX_servo_v12_19.stl" scale="1 1 1"/>
     </geometry>
     <material name="plastic_matte_black"/>
@@ -501,5 +501,5 @@
     <origin xyz="0.06095 0.0465 0.407741" rpy="0 0 0"/>
     <geometry>
-      <mesh filename="package://bez3_description/meshes/JX_servo_v12_19.stl" scale="0.001 0.001 0.001"/>
+      <mesh filename="package://bez3_description/meshes/JX_servo_v12_19.stl" scale="1 1 1"/>
     </geometry>
   </collision>
@@ -514,5 +514,5 @@
     <origin xyz="0.03455 0.055 0.462641" rpy="0 0 0"/>
     <geometry>
-      <mesh filename="package://bez3_description/meshes/right_foot_1.stl" scale="0.001 0.001 0.001"/>
+      <mesh filename="package://bez3_description/meshes/right_foot_1.stl" scale="1 1 1"/>
     </geometry>
     <material name="plastic_glossy_black"/>
@@ -521,5 +521,5 @@
     <origin xyz="0.03455 0.055 0.462641" rpy="0 0 0"/>
     <geometry>
-      <mesh filename="package://bez3_description/meshes/right_foot_1.stl" scale="0.001 0.001 0.001"/>
+      <mesh filename="package://bez3_description/meshes/right_foot_1.stl" scale="1 1 1"/>
     </geometry>
   </collision>
@@ -534,5 +534,5 @@
     <origin xyz="0.021 -0.1075 0.0365" rpy="0 0 0"/>
     <geometry>
-      <mesh filename="package://bez3_description/meshes/25t-servo-hub_1.stl" scale="0.001 0.001 0.001"/>
+      <mesh filename="package://bez3_description/meshes/25t-servo-hub_1.stl" scale="1 1 1"/>
     </geometry>
     <material name="aluminum_satin"/>
@@ -541,5 +541,5 @@
     <origin xyz="0.021 -0.1075 0.0365" rpy="0 0 0"/>
     <geometry>
-      <mesh filename="package://bez3_description/meshes/25t-servo-hub_1.stl" scale="0.001 0.001 0.001"/>
+      <mesh filename="package://bez3_description/meshes/25t-servo-hub_1.stl" scale="1 1 1"/>
     </geometry>
   </collision>
@@ -554,5 +554,5 @@
     <origin xyz="0.021 -0.110294 0.0365" rpy="0 0 0"/>
     <geometry>
-      <mesh filename="package://bez3_description/meshes/gobilda-servo_1.stl" scale="0.001 0.001 0.001"/>
+      <mesh filename="package://bez3_description/meshes/gobilda-servo_1.stl" scale="1 1 1"/>
     </geometry>
     <material name="plastic_glossy_grey"/>
@@ -561,5 +561,5 @@
     <origin xyz="0.021 -0.110294 0.0365" rpy="0 0 0"/>
     <geometry>
-      <mesh filename="package://bez3_description/meshes/gobilda-servo_1.stl" scale="0.001 0.001 0.001"/>
+      <mesh filename="package://bez3_description/meshes/gobilda-servo_1.stl" scale="1 1 1"/>
     </geometry>
   </collision>
@@ -574,5 +574,5 @@
     <origin xyz="0.0285 -0.147194 0.029" rpy="0 0 0"/>
     <geometry>
-      <mesh filename="package://bez3_description/meshes/left_bicep_1.stl" scale="0.001 0.001 0.001"/>
+      <mesh filename="package://bez3_description/meshes/left_bicep_1.stl" scale="1 1 1"/>
     </geometry>
     <material name="plastic_glossy_black"/>
@@ -581,5 +581,5 @@
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