Commit message: make camera/imu joints fixed, generate simple box collisions

File: bez3_description/urdf/bez3.xacro (robot description, xacro)
@@ -1347,5 +1347,5 @@
   <child link="camera_1"/>
 </joint>
-<joint name="camera_joint" type="continuous">
+<joint name="camera_joint" type="fixed">
   <origin xyz="0.0372 0.0 0.027" rpy="0 0 0"/>
   <parent link="camera_1"/>
@@ -1353,5 +1353,5 @@
   <axis xyz="1.0 -0.0 0.0"/>
 </joint>
-<joint name="imu_joint" type="continuous">
+<joint name="imu_joint" type="fixed">
   <origin xyz="0.0 -0.005 -0.005" rpy="0 0 0"/>
   <parent link="torso_1"/>

File: bez3_description/urdf/bez3_simple.urdf (robot description, URDF)
Before this commit: robot bez3, 54 links, 53 joints
Links:
- link 25t-servo-hub_1: geometry collision box size=0.006378183021786476 0.025251950007364292 0.025379984451465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; visual mesh filename=package://bez3_description/meshes/25t-servo-hub_1.stl scale=1e-06 1e-06 1e-06
- link 25t-servo-hub_2: geometry collision box size=0.00640692776428926 0.025662782879393775 0.0256669522471851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; visual mesh filename=package://bez3_description/meshes/25t-servo-hub_2.stl scale=1e-06 1e-06 1e-06
- link 25t-servo-hub_3: geometry collision box size=0.006369504964453446 0.025233453945395844 0.025357520863662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; visual mesh filename=package://bez3_description/meshes/25t-servo-hub_3.stl scale=1e-06 1e-06 1e-06
- link 25t-servo-hub_4: geometry collision box size=0.006378195737828646 0.02525196060038335 0.025380002425038; visual mesh filename=package://bez3_description/meshes/25t-servo-hub_4.stl scale=1e-06 1e-06 1e-06
- link 25t-servo-hub_Mirror__1: geometry collision box size=0.006413470648793196 0.02520474876690182 0.0253029056805054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; visual mesh filename=package://bez3_description/meshes/25t-servo-hub_Mirror__1.s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 scale=1e-06 1e-06 1e-06
- link 25t-servo-hub_Mirror__2: geometry collision box size=0.006413470600263925 0.025204755950700975 0.025302910742906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; visual mesh filename=package://bez3_description/meshes/25t-servo-hub_Mirror__2.s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 scale=1e-06 1e-06 1e-06
- link Component32_1: geometry collision box size=0.03500000014901161 0.04700000118464232 0.10700000077486038; visual mesh filename=package://bez3_description/meshes/Component32_1.stl scale=1e-06 1e-06 1e-06
- link JX_servo_v12_1: geometry collision box size=0.04054670823531333 0.07320708274687829 0.08278942044884; visual mesh filename=package://bez3_description/meshes/JX_servo_v12_1.stl scale=1e-06 1e-06 1e-06
- link JX_servo_v12_11: geometry collision box size=0.04000845578282203 0.07278502398499857 0.0818383861167361; visual mesh filename=package://bez3_description/meshes/JX_servo_v12_11.stl scale=1e-06 1e-06 1e-06
- link JX_servo_v12_12: geometry collision box size=0.040008453871064664 0.07278503718039667 0.08183838867335402; visual mesh filename=package://bez3_description/meshes/JX_servo_v12_12.stl scale=1e-06 1e-06 1e-06
- link JX_servo_v12_13: geometry collision box size=0.040546708572980955 0.07320709080496267 0.08278945243235761; visual mesh filename=package://bez3_description/meshes/JX_servo_v12_13.stl scale=1e-06 1e-06 1e-06
- link JX_servo_v12_14: geometry collision box size=0.04054670816493613 0.07320708270345652 0.08278942078053159; visual mesh filename=package://bez3_description/meshes/JX_servo_v12_14.stl scale=1e-06 1e-06 1e-06
- link JX_servo_v12_15: geometry collision box size=0.04000845479340684 0.07278504140539158 0.0818383886353029; visual mesh filename=package://bez3_description/meshes/JX_servo_v12_15.stl scale=1e-06 1e-06 1e-06
- link JX_servo_v12_16: geometry collision box size=0.040008452927453524 0.07278503955894784 0.08183838859725273; visual mesh filename=package://bez3_description/meshes/JX_servo_v12_16.stl scale=1e-06 1e-06 1e-06
- link JX_servo_v12_17: geometry collision box size=0.04000845301114797 0.07278502246569804 0.081838386116736; visual mesh filename=package://bez3_description/meshes/JX_servo_v12_17.stl scale=1e-06 1e-06 1e-06
- link JX_servo_v12_18: geometry collision box size=0.04000845386164336 0.07278503585588014 0.0818383588728816; visual mesh filename=package://bez3_description/meshes/JX_servo_v12_18.stl scale=1e-06 1e-06 1e-06
- link JX_servo_v12_19: geometry collision box size=0.04054672375968531 0.07320709212991403 0.08278942267814574; visual mesh filename=package://bez3_description/meshes/JX_servo_v12_19.stl scale=1e-06 1e-06 1e-06
- link JX_servo_v12_8: geometry collision box size=0.040008454801080326 0.07278504123650459 0.08183837373506664; visual mesh filename=package://bez3_description/meshes/JX_servo_v12_8.stl scale=1e-06 1e-06 1e-06
- link JX_servo_v12_9: geometry collision box size=0.04000845479936067 0.07278504123672407 0.08183837369701641; visual mesh filename=package://bez3_description/meshes/JX_servo_v12_9.stl scale=1e-06 1e-06 1e-06
- link base_link: geometry collision box size=0.009999999776482584 0.009999999776482584 0.009999999776482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; visual mesh filename=package://bez3_description/meshes/base_link.stl scale=1e-06 1e-06 1e-06
- link camera-link_1: geometry collision box size=0.0009999983012676248 0.005000000004656614 0.00500001013278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; visual mesh filename=package://bez3_description/meshes/camera-link_1.stl scale=1e-06 1e-06 1e-06
- link camera_1: geometry collision box size=0.04150000214576721 0.07098785349728846 0.09400000048161036; visual mesh filename=package://bez3_description/meshes/camera_1.stl scale=1e-06 1e-06 1e-06
- link custom_servo_support__lower_neck__v2_1: geometry collision box size=0.007049533893643815 0.04002735960495628 0.04114593061934336; visual mesh filename=package://bez3_description/meshes/custom_servo_support__low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 scale=1e-06 1e-06 1e-06
- link elbow-attach_1: geometry collision box size=0.009114717533457157 0.03501314090504535 0.04993097391197541; visual mesh filename=package://bez3_description/meshes/elbow-attach_1.stl scale=1e-06 1e-06 1e-06
- link elbow-attach_Mirror__1: geometry collision box size=0.009758820468505985 0.035006274132078054 0.049820451491883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; visual mesh filename=package://bez3_description/meshes/elbow-attach_Mirror__1.stl scale=1e-06 1e-06 1e-06
- link elbow-bearing_1: geometry collision box size=0.009762054381294787 0.03500627413562576 0.0499665474924589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; visual mesh filename=package://bez3_description/meshes/elbow-bearing_1.stl scale=1e-06 1e-06 1e-06
- link elbow-bearing_Mirror__1: geometry collision box size=0.009221219110703038 0.034999996423721313 0.049866950105174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; visual mesh filename=package://bez3_description/meshes/elbow-bearing_Mirror__1.s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 scale=1e-06 1e-06 1e-06
- link gobilda-servo_1: geometry collision box size=0.01999999955296517 0.0399826830600124 0.05437307046998198; visual mesh filename=package://bez3_description/meshes/gobilda-servo_1.stl scale=1e-06 1e-06 1e-06
- link gobilda-servo_3: geometry collision box size=0.019999999552965168 0.03998268930005222 0.0543730750677536; visual mesh filename=package://bez3_description/meshes/gobilda-servo_3.stl scale=1e-06 1e-06 1e-06
- link gobilda-servo_4: geometry collision box size=0.019999999552965175 0.03998267586685512 0.0543730767931727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; visual mesh filename=package://bez3_description/meshes/gobilda-servo_4.stl scale=1e-06 1e-06 1e-06
- link gobilda-servo_5: geometry collision box size=0.01999999582767487 0.03998267775876498 0.05437307478927776; visual mesh filename=package://bez3_description/meshes/gobilda-servo_5.stl scale=1e-06 1e-06 1e-06
- link gobilda-servo_Mirror__1: geometry collision box size=0.019999999552965164 0.04047670997108249 0.0543730704699819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; visual mesh filename=package://bez3_description/meshes/gobilda-servo_Mirror__1.s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 scale=1e-06 1e-06 1e-06
- link gobilda-servo_Mirror__2: geometry collision box size=0.019999999552965168 0.040476712084511424 0.054373081899480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; visual mesh filename=package://bez3_description/meshes/gobilda-servo_Mirror__2.s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 scale=1e-06 1e-06 1e-06
- link head_1: geometry collision box size=0.033965209499001524 0.03509340922727139 0.0608510607274505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; visual mesh filename=package://bez3_description/meshes/head_1.stl scale=1e-06 1e-06 1e-06
- link imu-link_1: geometry collision box size=0.0009999983012676241 0.004999999888241291 0.00499999988824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; visual mesh filename=package://bez3_description/meshes/imu-link_1.stl scale=1e-06 1e-06 1e-06
- link left_bicep_1: geometry collision box size=0.03570982710179357 0.0428372093610371 0.110695531807019; visual mesh filename=package://bez3_description/meshes/left_bicep_1.stl scale=1e-06 1e-06 1e-06
- link left_calve_1: geometry collision box size=0.04009244410387435 0.08934971823335128 0.1090484024603223; visual mesh filename=package://bez3_description/meshes/left_calve_1.stl scale=1e-06 1e-06 1e-06
- link left_foot_1: geometry collision box size=0.06015777061157024 0.06334595847485622 0.11811981933807195; visual mesh filename=package://bez3_description/meshes/left_foot_1.stl scale=1e-06 1e-06 1e-06
- link left_forearm_1: geometry collision box size=0.02753307769937075 0.050673991441726726 0.14429567831080597; visual mesh filename=package://bez3_description/meshes/left_forearm_1.stl scale=1e-06 1e-06 1e-06
- link left_hip_front_1: geometry collision box size=0.04100000113248826 0.07840000372380018 0.08820788562297821; visual mesh filename=package://bez3_description/meshes/left_hip_front_1.stl scale=1e-06 1e-06 1e-06
- link left_hip_front_2: geometry collision box size=0.04105894538917622 0.07915189064439027 0.08831298710238125; visual mesh filename=package://bez3_description/meshes/left_hip_front_2.stl scale=1e-06 1e-06 1e-06
- link left_hip_side_1: geometry collision box size=0.040000002831220634 0.05924370884895324 0.06200983002781868; visual mesh filename=package://bez3_description/meshes/left_hip_side_1.stl scale=1e-06 1e-06 1e-06
- link left_thigh_1: geometry collision box size=0.04007143189170146 0.08883423336978291 0.1640051519072386; visual mesh filename=package://bez3_description/meshes/left_thigh_1.stl scale=1e-06 1e-06 1e-06
- link neck_1: geometry collision box size=0.034999999217689065 0.048414763063192374 0.056374000385403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; visual mesh filename=package://bez3_description/meshes/neck_1.stl scale=1e-06 1e-06 1e-06
- link right_ankle_1: geometry collision box size=0.041000001132488265 0.07860071677714586 0.08820787072181702; visual mesh filename=package://bez3_description/meshes/right_ankle_1.stl scale=1e-06 1e-06 1e-06
- link right_ankle_2: geometry collision box size=0.04099999740719798 0.07860070932656528 0.08820787072181702; visual mesh filename=package://bez3_description/meshes/right_ankle_2.stl scale=1e-06 1e-06 1e-06
- link right_bicep_1: geometry collision box size=0.03504697431706887 0.0429835820897832 0.11071014669788423; visual mesh filename=package://bez3_description/meshes/right_bicep_1.stl scale=1e-06 1e-06 1e-06
- link right_calve_1: geometry collision box size=0.04005597184791974 0.0893443198546015 0.10905559176825397; visual mesh filename=package://bez3_description/meshes/right_calve_1.stl scale=1e-06 1e-06 1e-06
- link right_foot_1: geometry collision box size=0.05934509962590004 0.06383469121587682 0.11762418282986051; visual mesh filename=package://bez3_description/meshes/right_foot_1.stl scale=1e-06 1e-06 1e-06
- link right_forearm_1: geometry collision box size=0.027546153323796983 0.050673991441726685 0.144205829409862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; visual mesh filename=package://bez3_description/meshes/right_forearm_1.stl scale=1e-06 1e-06 1e-06
- link right_hip_side_1: geometry collision box size=0.040058424427170426 0.059198398432720914 0.062009830027818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; visual mesh filename=package://bez3_description/meshes/right_hip_side_1.stl scale=1e-06 1e-06 1e-06
- link right_thigh_1: geometry collision box size=0.04031622705210779 0.08885990114706975 0.16419299183864544; visual mesh filename=package://bez3_description/meshes/right_thigh_1.stl scale=1e-06 1e-06 1e-06
- link torso_1: geometry collision box size=0.12413852661848071 0.13700000673917856 0.21500000357627866; visual mesh filename=package://bez3_description/meshes/torso_1.stl scale=1e-06 1e-06 1e-06
Joints:
- joint Rigid1: origin xyz=0.0 0.005 0.0 rpy=0 0 0 -> xyz=0.0 0.005 0.0 rpy=0.0 0.0 0.0
- joint Rigid11: origin xyz=0.0085 -0.0225 0.0549 rpy=0 0 0 -> xyz=0.0085 -0.0225 0.0549 rpy=0.0 0.0 0.0
- joint Rigid12: origin xyz=-0.0644 -0.025 0.0 rpy=0 0 0 -> xyz=-0.0644 -0.025 0.0 rpy=0.0 0.0 0.0
- joint Rigid14: origin xyz=-0.0225 -0.0595 -0.137 rpy=0 0 0 -> xyz=-0.0225 -0.0595 -0.137 rpy=0.0 0.0 0.0
- joint Rigid17: origin xyz=-0.0264 0.0085 0.0189 rpy=0 0 0 -> xyz=-0.0264 0.0085 0.0189 rpy=0.0 0.0 0.0
- joint Rigid18: origin xyz=0.0644 -0.0239 -0.0738 rpy=0 0 0 -> xyz=0.0644 -0.0239 -0.0738 rpy=0.0 0.0 0.0
- joint Rigid2: origin xyz=-0.0225 0.0495 -0.13699 rpy=0 0 0 -> xyz=-0.0225 0.0495 -0.13699 rpy=0.0 0.0 0.0
- joint Rigid21: origin xyz=0.0085 0.0264 -0.0549 rpy=0 0 0 -> xyz=0.0085 0.0264 -0.0549 rpy=0.0 0.0 0.0
- joint Rigid23: origin xyz=0.0085 0.0225 0.0549 rpy=0 0 0 -> xyz=0.0085 0.0225 0.0549 rpy=0.0 0.0 0.0
- joint Rigid24: origin xyz=-0.0644 0.025 0.0 rpy=0 0 0 -> xyz=-0.0644 0.025 0.0 rpy=0.0 0.0 0.0
- joint Rigid26: origin xyz=-0.021 0.1025 -0.0365 rpy=0 0 0 -> xyz=-0.021 0.1025 -0.0365 rpy=0.0 0.0 0.0
- joint Rigid28: origin xyz=-0.0075 0.0369 0.0075 rpy=0 0 0 -> xyz=-0.0075 0.0369 0.0075 rpy=0.0 0.0 0.0
- joint Rigid29: origin xyz=0.0 0.0 -0.0703 rpy=0 0 0 -> xyz=0.0 0.0 -0.0703 rpy=0.0 0.0 0.0
- joint Rigid31: origin xyz=0.0 -0.002794 0.0 rpy=0 0 0 -> xyz=0.0 -0.002794 0.0 rpy=0.0 0.0 0.0
- joint Rigid32: origin xyz=-0.0275 0.002 0.01 rpy=0 0 0 -> xyz=-0.0275 0.002 0.01 rpy=0.0 0.0 0.0
- joint Rigid33: origin xyz=0.0 0.044674 0.0 rpy=0 0 0 -> xyz=0.0 0.044674 0.0 rpy=0.0 0.0 0.0
- joint Rigid34: origin xyz=-0.021 -0.1125 -0.0365 rpy=0 0 0 -> xyz=-0.021 -0.1125 -0.0365 rpy=0.0 0.0 0.0
- joint Rigid36: origin xyz=-0.0075 -0.0369 0.0075 rpy=0 0 0 -> xyz=-0.0075 -0.0369 0.0075 rpy=0.0 0.0 0.0
- joint Rigid37: origin xyz=0.0 0.0 -0.0703 rpy=0 0 0 -> xyz=0.0 0.0 -0.0703 rpy=0.0 0.0 0.0
- joint Rigid39: origin xyz=0.0 0.002794 0.0 rpy=0 0 0 -> xyz=0.0 0.002794 0.0 rpy=0.0 0.0 0.0
- joint Rigid40: origin xyz=-0.0275 -0.002 0.01 rpy=0 0 0 -> xyz=-0.0275 -0.002 0.01 rpy=0.0 0.0 0.0
- joint Rigid41: origin xyz=0.0 -0.044674 0.0 rpy=0 0 0 -> xyz=0.0 -0.044674 0.0 rpy=0.0 0.0 0.0
- joint Rigid42: origin xyz=0.0 -0.005 -1e-05 rpy=0 0 0 -> xyz=0.0 -0.005 -1e-05 rpy=0.0 0.0 0.0
- joint Rigid43: origin xyz=-0.01715 -0.0075 0.00698 rpy=0 0 0 -> xyz=-0.01715 -0.0075 0.00698 rpy=0.0 0.0 0.0
- joint Rigid45: origin xyz=0.0 0.0 0.002794 rpy=0 0 0 -> xyz=0.0 0.0 0.002794 rpy=0.0 0.0 0.0
- joint Rigid46: origin xyz=0.0 -0.022187 0.033817 rpy=0 0 0 -> xyz=0.0 -0.022187 0.033817 rpy=0.0 0.0 0.0
- joint Rigid48: origin xyz=-0.0075 0.0369 0.0075 rpy=0 0 0 -> xyz=-0.0075 0.0369 0.0075 rpy=0.0 0.0 0.0
- joint Rigid49: origin xyz=0.024 -0.01402 0.0135 rpy=0 0 0 -> xyz=0.024 -0.01402 0.0135 rpy=0.0 0.0 0.0
- joint Rigid5: origin xyz=-0.0264 -0.0085 0.0189 rpy=0 0 0 -> xyz=-0.0264 -0.0085 0.0189 rpy=0.0 0.0 0.0
- joint Rigid52: origin xyz=-0.012 -0.004667 -0.005 rpy=0 0 0 -> xyz=-0.012 -0.004667 -0.005 rpy=0.0 0.0 0.0
- joint Rigid53: origin xyz=0.0 0.0 -0.047 rpy=0 0 0 -> xyz=0.0 0.0 -0.047 rpy=0.0 0.0 0.0
- joint Rigid6: origin xyz=0.0644 0.0239 -0.0738 rpy=0 0 0 -> xyz=0.0644 0.0239 -0.0738 rpy=0.0 0.0 0.0
- joint Rigid9: origin xyz=0.0085 -0.0264 -0.0549 rpy=0 0 0 -> xyz=0.0085 -0.0264 -0.0549 rpy=0.0 0.0 0.0
- joint camera_joint: origin xyz=0.0372 0.0 0.027 rpy=0 0 0 -> xyz=0.0372 0.0 0.027 rpy=0.0 0.0 0.0
- joint head_motor_0: origin xyz=0.0075 0.0075 0.0369 rpy=0 0 0 -> xyz=0.0075 0.0075 0.0369 rpy=0.0 0.0 0.0
- joint head_motor_1: origin xyz=0.0 0.002794 0.0 rpy=0 0 0 -> xyz=0.0 0.002794 0.0 rpy=0.0 0.0 0.0
- joint imu_joint: origin xyz=0.0 -0.005 -0.005 rpy=0 0 0 -> xyz=0.0 -0.005 -0.005 rpy=0.0 0.0 0.0
- joint left_arm_motor_0: origin xyz=0.0 0.002794 0.0 rpy=0 0 0 -> xyz=0.0 0.002794 0.0 rpy=0.0 0.0 0.0
- joint left_arm_motor_1: origin xyz=0.0075 -0.0369 -0.0075 rpy=0 0 0 -> xyz=0.0075 -0.0369 -0.0075 rpy=0.0 0.0 0.0
- joint left_leg_motor_0: origin xyz=0.018 0.0 -0.0264 rpy=0 0 0 -> xyz=0.018 0.0 -0.0264 rpy=0.0 0.0 0.0
- joint left_leg_motor_1: origin xyz=-0.03 0.0 -0.035336 rpy=0 0 0 -> xyz=-0.03 0.0 -0.035336 rpy=0.0 0.0 0.0
- joint left_leg_motor_2: origin xyz=-0.0085 0.0225 0.0549 rpy=0 0 0 -> xyz=-0.0085 0.0225 0.0549 rpy=0.0 0.0 0.0
- joint left_leg_motor_3: origin xyz=0.0 0.0 -0.124 rpy=0 0 0 -> xyz=0.0 0.0 -0.124 rpy=0.0 0.0 0.0
- joint left_leg_motor_4: origin xyz=-0.00855 0.028 -0.085005 rpy=0 0 0 -> xyz=-0.00855 0.028 -0.085005 rpy=0.0 0.0 0.0
- joint left_leg_motor_5: origin xyz=0.0264 0.0085 -0.0549 rpy=0 0 0 -> xyz=0.0264 0.0085 -0.0549 rpy=0.0 0.0 0.0
- joint right_arm_motor_0: origin xyz=0.0 -0.002794 0.0 rpy=0 0 0 -> xyz=0.0 -0.002794 0.0 rpy=0.0 0.0 0.0
- joint right_arm_motor_1: origin xyz=0.0075 0.0369 -0.0075 rpy=0 0 0 -> xyz=0.0075 0.0369 -0.0075 rpy=0.0 0.0 0.0
- joint right_leg_motor_0: origin xyz=0.018 0.0 -0.0264 rpy=0 0 0 -> xyz=0.018 0.0 -0.0264 rpy=0.0 0.0 0.0
- joint right_leg_motor_1: origin xyz=-0.03 0.0 -0.035336 rpy=0 0 0 -> xyz=-0.03 0.0 -0.035336 rpy=0.0 0.0 0.0
- joint right_leg_motor_2: origin xyz=-0.0085 -0.0225 0.0549 rpy=0 0 0 -> xyz=-0.0085 -0.0225 0.0549 rpy=0.0 0.0 0.0
- joint right_leg_motor_3: origin xyz=0.0 0.0 -0.124 rpy=0 0 0 -> xyz=0.0 0.0 -0.124 rpy=0.0 0.0 0.0
- joint right_leg_motor_4: origin xyz=-0.00855 -0.028 -0.085005 rpy=0 0 0 -> xyz=-0.00855 -0.028 -0.085005 rpy=0.0 0.0 0.0
- joint right_leg_motor_5: origin xyz=0.0264 -0.0085 -0.0549 rpy=0 0 0 -> xyz=0.0264 -0.0085 -0.0549 rpy=0.0 0.0 0.0
