Commit message: generated urdf and initial proto
- order of links and joints was manually changed to make pybullet read correct order
- meshes were simplified already
- proto freshly generated needs manual fixes to make work

File: bez2_description/urdf/bez2.urdf (robot description, URDF)
Before this commit: robot bez2, 22 links, 21 joints
Links:
- removed link neck_v4_1
- link base_link: mass 1.3874949527504563 -> 1.4940527908480117
- link camera_point_1: mass 0.0005023999999999976 -> 0.0005023999999999989
Joints:
- removed joint Rigid19
- removed joint camera_joint
- removed joint imu_joint
- added joint head_camera: type continuous, parent head_v4_1, child camera_point_1, origin xyz=0.0344 0.025674 0.048 rpy=0 0 0, axis 1.0 0.0 -0.0
- added joint torso_imu: type continuous, parent base_link, child imu_1, origin xyz=0.013 0.0 0.02895 rpy=0 0 0, axis 0.0 0.0 1.0
- joint head_motor_0: axis 0.0 -0.0 1.0 -> 0.0 0.0 -1.0; origin xyz=0.015 0.0045 0.046674 rpy=0 0 0 -> xyz=0.03325 -0.000333 0.075624 rpy=0 0 0; parent neck_v4_1 -> base_link
- joint head_motor_1: axis -1.0 0.0 0.0 -> -0.0 1.0 0.0; origin xyz=-0.022187 0.0 0.033818 rpy=0 0 0 -> xyz=0.0 -0.022187 0.033817 rpy=0 0 0
- joint left_arm_motor_0: axis -1.0 0.0 0.0 -> -0.0 -1.0 0.0; origin xyz=0.144659 0.075444 0.072056 rpy=0 0 0 -> xyz=0.0 0.0725 0.00045 rpy=0 0 0
- joint left_arm_motor_1: axis -1.0 -0.0 0.0 -> 0.0 -1.0 0.0; origin xyz=0.008 0.0 -0.0906 rpy=0 0 0 -> xyz=0.0 0.008 -0.0906 rpy=0 0 0
- joint left_leg_motor_0: axis 0.0 0.0 -1.0 -> -0.0 0.0 -1.0; origin xyz=0.109859 0.059474 -0.072444 rpy=0 0 0 -> xyz=0.01597 0.0377 -0.14405 rpy=0 0 0
- joint left_leg_motor_1: axis -0.0 -1.0 -0.0 -> 1.0 -0.0 -0.0; origin xyz=0.0 0.025 -0.032 rpy=0 0 0 -> xyz=-0.025 0.0 -0.032 rpy=0 0 0
- joint left_leg_motor_2: axis -1.0 -0.0 0.0 -> 0.0 -1.0 0.0; origin xyz=-0.02 -0.02365 0.0 rpy=0 0 0 -> xyz=0.02365 -0.02 0.0 rpy=0 0 0
- joint left_leg_motor_3: axis -1.0 -0.0 0.0 -> 0.0 -1.0 0.0; origin xyz=-0.0045 0.0 -0.0917 rpy=0 0 0 -> xyz=0.0 -0.0045 -0.0917 rpy=0 0 0
- joint left_leg_motor_4: axis -1.0 0.0 0.0 -> 0.0 -1.0 0.0; origin xyz=-0.0005 0.0 -0.1083 rpy=0 0 0 -> xyz=0.0 -0.0005 -0.1083 rpy=0 0 0
- joint left_leg_motor_5: axis 0.0 -1.0 -0.0 -> -1.0 0.0 0.0; origin xyz=0.0233 0.0843 0.0 rpy=0 0 0 -> xyz=-0.0843 0.0233 0.0 rpy=0 0 0
- joint right_arm_motor_0: axis 1.0 -0.0 -0.0 -> 0.0 -1.0 0.0; origin xyz=-0.000341 0.075444 0.072056 rpy=0 0 0 -> xyz=0.0 -0.0725 0.00045 rpy=0 0 0
- joint right_arm_motor_1: axis 1.0 0.0 0.0 -> -0.0 -1.0 0.0; origin xyz=-0.008 0.0 -0.0906 rpy=0 0 0 -> xyz=-0.0 -0.008 -0.0906 rpy=0 0 0
- joint right_leg_motor_0: axis 0.0 0.0 -1.0 -> -0.0 -0.0 1.0; origin xyz=0.035359 0.059474 -0.072444 rpy=0 0 0 -> xyz=0.01597 -0.0368 -0.14405 rpy=0 0 0
- joint right_leg_motor_1: axis -0.0 -1.0 -0.0 -> -1.0 0.0 0.0; origin xyz=0.0 0.0235 -0.032 rpy=0 0 0 -> xyz=-0.0235 0.0 -0.032 rpy=0 0 0
- joint right_leg_motor_2: axis 1.0 0.0 0.0 -> 0.0 -1.0 0.0; origin xyz=0.02 -0.02365 0.0 rpy=0 0 0 -> xyz=0.02365 0.02 0.0 rpy=0 0 0
- joint right_leg_motor_3: axis 1.0 0.0 0.0 -> 0.0 -1.0 0.0; origin xyz=0.0045 0.0 -0.0917 rpy=0 0 0 -> xyz=0.0 0.0045 -0.0917 rpy=0 0 0
- joint right_leg_motor_4: axis 1.0 -0.0 0.0 -> 0.0 -1.0 0.0; origin xyz=0.0005 0.0 -0.1083 rpy=0 0 0 -> xyz=0.0 0.0005 -0.1083 rpy=0 0 0
- joint right_leg_motor_5: axis 0.0 -1.0 -0.0 -> 1.0 0.0 0.0; origin xyz=-0.0233 0.0843 0.0 rpy=0 0 0 -> xyz=-0.0843 -0.0233 0.0 rpy=0 0 0

File: bez2_description/urdf/bez2.xacro (robot description, xacro)
@@ -6,7 +6,7 @@
 <link name="base_link">
   <inertial>
-    <origin xyz="0.07343372628291743 0.07159927292954832 0.020872010814779768" rpy="0 0 0"/>
-    <mass value="1.3874949527504563"/>
-    <inertia ixx="0.004586" iyy="0.005498" izz="0.00387" ixy="-8e-06" iyz="0.000146" ixz="0.000118"/>
+    <origin xyz="0.005344203942179857 0.0011597330599576942 -0.04327601296104891" rpy="0 0 0"/>
+    <mass value="1.4940527908480117"/>
+    <inertia ixx="0.006599" iyy="0.005741" izz="0.003932" ixy="0" iyz="0" ixz="0"/>
   </inertial>
   <visual>
@@ -26,10 +26,10 @@
 <link name="biceps_v3_1">
   <inertial>
-    <origin xyz="0.026300253416251113 -1.0338235605089618e-07 -0.03838594777031868" rpy="0 0 0"/>
+    <origin xyz="-4.857598999001871e-13 0.026299931386057934 -0.038386051153163035" rpy="0 0 0"/>
     <mass value="0.25825416029102555"/>
-    <inertia ixx="0.000394" iyy="0.000437" izz="6.4e-05" ixy="-0.0" iyz="0.0" ixz="3.3e-05"/>
-  </inertial>
-  <visual>
-    <origin xyz="-0.144659 -0.075444 -0.072056" rpy="0 0 0"/>
+    <inertia ixx="0.000437" iyy="0.000394" izz="6.4e-05" ixy="0.0" iyz="3.3e-05" ixz="-0.0"/>
+  </inertial>
+  <visual>
+    <origin xyz="-0.0 -0.0725 -0.00045" rpy="0 0 0"/>
     <geometry>
       <mesh filename="package://bez2_description/meshes/biceps_v3_1.stl" scale="0.001 0.001 0.001"/>
@@ -38,5 +38,5 @@
   </visual>
   <collision>
-    <origin xyz="-0.144659 -0.075444 -0.072056" rpy="0 0 0"/>
+    <origin xyz="-0.0 -0.0725 -0.00045" rpy="0 0 0"/>
     <geometry>
       <mesh filename="package://bez2_description/meshes/biceps_v3_1.stl" scale="0.001 0.001 0.001"/>
@@ -46,10 +46,10 @@
 <link name="Arm_Assembly-bez3_v12_2">
   <inertial>
-    <origin xyz="0.02284504145700883 0.005329912793864702 0.029751383749166617" rpy="0 0 0"/>
+    <origin xyz="-0.005330016176706751 0.022844719426815346 0.029751280366322262" rpy="0 0 0"/>
     <mass value="0.32110352957731503"/>
-    <inertia ixx="0.002137" iyy="0.002148" izz="0.000103" ixy="-3e-06" iyz="0.000175" ixz="1.6e-05"/>
-  </inertial>
-  <visual>
-    <origin xyz="-0.152659 -0.075444 0.018544" rpy="0 0 0"/>
+    <inertia ixx="0.002148" iyy="0.002137" izz="0.000103" ixy="3e-06" iyz="1.6e-05" ixz="-0.000175"/>
+  </inertial>
+  <visual>
+    <origin xyz="-0.0 -0.0805 0.09015" rpy="0 0 0"/>
     <geometry>
       <mesh filename="package://bez2_description/meshes/Arm_Assembly-bez3_v12_2.stl" scale="0.001 0.001 0.001"/>
@@ -58,5 +58,5 @@
   </visual>
   <collision>
-    <origin xyz="-0.152659 -0.075444 0.018544" rpy="0 0 0"/>
+    <origin xyz="-0.0 -0.0805 0.09015" rpy="0 0 0"/>
     <geometry>
       <mesh filename="package://bez2_description/meshes/Arm_Assembly-bez3_v12_2.stl" scale="0.001 0.001 0.001"/>
@@ -66,10 +66,10 @@
 <link name="biceps_v3_2">
   <inertial>
-    <origin xyz="-0.026299609355872014 -1.0338333342185813e-07 -0.03838594777031868" rpy="0 0 0"/>
+    <origin xyz="4.933084310590376e-13 -0.026299931386065484 -0.038386051153161384" rpy="0 0 0"/>
     <mass value="0.25825416029102555"/>
-    <inertia ixx="0.000394" iyy="0.000437" izz="6.4e-05" ixy="-0.0" iyz="-0.0" ixz="-3.3e-05"/>
-  </inertial>
-  <visual>
-    <origin xyz="0.000341 -0.075444 -0.072056" rpy="0 0 0"/>
+    <inertia ixx="0.000437" iyy="0.000394" izz="6.4e-05" ixy="0.0" iyz="-3.3e-05" ixz="0.0"/>
+  </inertial>
+  <visual>
+    <origin xyz="-0.0 0.0725 -0.00045" rpy="0 0 0"/>
     <geometry>
       <mesh filename="package://bez2_description/meshes/biceps_v3_2.stl" scale="0.001 0.001 0.001"/>
@@ -78,5 +78,5 @@
   </visual>
   <collision>
-    <origin xyz="0.000341 -0.075444 -0.072056" rpy="0 0 0"/>
+    <origin xyz="-0.0 0.0725 -0.00045" rpy="0 0 0"/>
     <geometry>
       <mesh filename="package://bez2_description/meshes/biceps_v3_2.stl" scale="0.001 0.001 0.001"/>
@@ -86,10 +86,10 @@
 <link name="Arm_Assembly-bez3_v12_1">
   <inertial>
-    <origin xyz="-0.025828958542993025 0.005329912793873015 0.02975138374916475" rpy="0 0 0"/>
+    <origin xyz="-0.005330016176713268 -0.02582928057318666 0.02975128036632215" rpy="0 0 0"/>
     <mass value="0.32110352957731503"/>
-    <inertia ixx="0.002137" iyy="0.002148" izz="0.000103" ixy="-3e-06" iyz="0.000175" ixz="1.6e-05"/>
-  </inertial>
-  <visual>
-    <origin xyz="0.008341 -0.075444 0.018544" rpy="0 0 0"/>
+    <inertia ixx="0.002148" iyy="0.002137" izz="0.000103" ixy="3e-06" iyz="1.6e-05" ixz="-0.000175"/>
+  </inertial>
+  <visual>
+    <origin xyz="0.0 0.0805 0.09015" rpy="0 0 0"/>
     <geometry>
       <mesh filename="package://bez2_description/meshes/Arm_Assembly-bez3_v12_1.stl" scale="0.001 0.001 0.001"/>
@@ -98,5 +98,5 @@
   </visual>
   <collision>
-    <origin xyz="0.008341 -0.075444 0.018544" rpy="0 0 0"/>
+    <origin xyz="0.0 0.0805 0.09015" rpy="0 0 0"/>
     <geometry>
       <mesh filename="package://bez2_description/meshes/Arm_Assembly-bez3_v12_1.stl" scale="0.001 0.001 0.001"/>
@@ -104,12 +104,232 @@
   </collision>
 </link>
+<link name="Hip_Printable_v2_v10_2">
+  <inertial>
+    <origin xyz="4.21754180706356e-05 -3.2154834350706096e-14 -0.014017367581241474" rpy="0 0 0"/>
+    <mass value="0.010089224750638792"/>
+    <inertia ixx="2e-06" iyy="6e-06" izz="5e-06" ixy="0.0" iyz="-0.0" ixz="0.0"/>
+  </inertial>
+  <visual>
+    <origin xyz="-0.01597 -0.0377 0.14405" rpy="0 0 0"/>
+    <geometry>
+      <mesh filename="package://bez2_description/meshes/Hip_Printable_v2_v10_2.stl" scale="0.001 0.001 0.001"/>
+    </geometry>
+    <material name="abs_white"/>
+  </visual>
+  <collision>
+    <origin xyz="-0.01597 -0.0377 0.14405" rpy="0 0 0"/>
+    <geometry>
+      <mesh filename="package://bez2_description/meshes/Hip_Printable_v2_v10_2.stl" scale="0.001 0.001 0.001"/>
+    </geometry>
+  </collision>
+</link>
+<link name="hip_motors_v4_1">
+  <inertial>
+    <origin xyz="0.00908799649277551 -7.287744503703397e-08 -0.011907384768018503" rpy="0 0 0"/>
+    <mass value="0.2728199051639206"/>
+    <inertia ixx="7.4e-05" iyy="0.000178" izz="0.000153" ixy="-0.0" iyz="0.0" ixz="-1e-06"/>
+  </inertial>
+  <visual>
+    <origin xyz="0.00753 0.0368 0.17605" rpy="0 0 0"/>
+    <geometry>
+      <mesh filename="package://bez2_description/meshes/hip_motors_v4_1.stl" scale="0.001 0.001 0.001"/>
+    </geometry>
+    <material name="silver_default"/>
+  </visual>
+  <collision>
+    <origin xyz="0.00753 0.0368 0.17605" rpy="0 0 0"/>
+    <geometry>
+      <mesh filename="package://bez2_description/meshes/hip_motors_v4_1.stl" scale="0.001 0.001 0.001"/>
+    </geometry>
+  </collision>
+</link>
+<link name="hip_motors_v4_2">
+  <inertial>
+    <origin xyz="0.009087996492779226 -7.28774387503961e-08 -0.011907384768019141" rpy="0 0 0"/>
+    <mass value="0.2728199051639206"/>
+    <inertia ixx="7.4e-05" iyy="0.000178" izz="0.000153" ixy="-0.0" iyz="0.0" ixz="-1e-06"/>
+  </inertial>
+  <visual>
+    <origin xyz="0.00903 -0.0377 0.17605" rpy="0 0 0"/>
+    <geometry>
+      <mesh filename="package://bez2_description/meshes/hip_motors_v4_2.stl" scale="0.001 0.001 0.001"/>
+    </geometry>
+    <material name="silver_default"/>
+  </visual>
+  <collision>
+    <origin xyz="0.00903 -0.0377 0.17605" rpy="0 0 0"/>
+    <geometry>
+      <mesh filename="package://bez2_description/meshes/hip_motors_v4_2.stl" scale="0.001 0.001 0.001"/>
+    </geometry>
+  </collision>
+</link>
+<link name="Upper_left_leg_support__bottom__v8_1">
+  <inertial>
+    <origin xyz="-5.513384106897723e-10 0.019462494401918447 -0.048113787355149845" rpy="0 0 0"/>
+    <mass value="0.027169463894965433"/>
+    <inertia ixx="3.2e-05" iyy="2.2e-05" izz="1.3e-05" ixy="0.0" iyz="-0.0" ixz="-0.0"/>
+  </inertial>
+  <visual>
+    <origin xyz="-0.01462 -0.0177 0.17605" rpy="0 0 0"/>
+    <geometry>
+      <mesh filename="package://bez2_description/meshes/Upper_left_leg_support__bottom__v8_1.stl" scale="0.001 0.001 0.001"/>
+    </geometry>
+    <material name="abs_white"/>
+  </visual>
+  <collision>
+    <origin xyz="-0.01462 -0.0177 0.17605" rpy="0 0 0"/>
+    <geometry>
+      <mesh filename="package://bez2_description/meshes/Upper_left_leg_support__bottom__v8_1.stl" scale="0.001 0.001 0.001"/>
+    </geometry>
+  </collision>
+</link>
+<link name="Upper_left_leg_support__bottom__v8_2">
+  <inertial>
+    <origin xyz="-5.513428880110638e-10 -0.019537505598094276 -0.04811378735514921" rpy="0 0 0"/>
+    <mass value="0.027169463894965433"/>
+    <inertia ixx="3.2e-05" iyy="2.2e-05" izz="1.3e-05" ixy="0.0" iyz="-0.0" ixz="-0.0"/>
+  </inertial>
+  <visual>
+    <origin xyz="-0.01612 0.0168 0.17605" rpy="0 0 0"/>
+    <geometry>
+      <mesh filename="package://bez2_description/meshes/Upper_left_leg_support__bottom__v8_2.stl" scale="0.001 0.001 0.001"/>
+    </geometry>
+    <material name="abs_white"/>
+  </visual>
+  <collision>
+    <origin xyz="-0.01612 0.0168 0.17605" rpy="0 0 0"/>
+    <geometry>
+      <mesh filename="package://bez2_description/meshes/Upper_left_leg_support__bottom__v8_2.stl" scale="0.001 0.001 0.001"/>
+    </geometry>
+  </collision>
+</link>
+<link name="New_left_foot_upperhalf_v5_1">
+  <inertial>
+    <origin xyz="0.05139344311503742 -0.01218090675701626 -0.02177657679768813" rpy="0 0 0"/>
+    <mass value="0.0588564551543425"/>
+    <inertia ixx="3.9e-05" iyy="0.000149" izz="0.000178" ixy="-0.0" iyz="-3e-06" ixz="-0.0"/>
+  </inertial>
+  <visual>
+    <origin xyz="0.06818 0.0351 0.37605" rpy="0 0 0"/>
+    <geometry>
+      <mesh filename="package://bez2_description/meshes/New_left_foot_upperhalf_v5_1.stl" scale="0.001 0.001 0.001"/>
+    </geometry>
+    <material name="abs_white"/>
+  </visual>
+  <collision>
+    <origin xyz="0.06818 0.0351 0.37605" rpy="0 0 0"/>
+    <geometry>
+      <mesh filename="package://bez2_description/meshes/New_left_foot_upperhalf_v5_1.stl" scale="0.001 0.001 0.001"/>
+    </geometry>
+  </collision>
+</link>
+<link name="New_right_foot_upperhalf_v3_1">
+  <inertial>
+    <origin xyz="0.05139344394950704 0.060000000000004765 -0.02177657679768963" rpy="0 0 0"/>
+    <mass value="0.117712910308685"/>
+    <inertia ixx="0.000348" iyy="0.000297" izz="0.000625" ixy="0.0" iyz="0.0" ixz="-1e-06"/>
+  </inertial>
+  <visual>
+    <origin xyz="0.06968 -0.036 0.37605" rpy="0 0 0"/>
+    <geometry>
+      <mesh filename="package://bez2_description/meshes/New_right_foot_upperhalf_v3_1.stl" scale="0.001 0.001 0.001"/>
+    </geometry>
+    <material name="abs_white"/>
+  </visual>
+  <collision>
+    <origin xyz="0.06968 -0.036 0.37605" rpy="0 0 0"/>
+    <geometry>
+      <mesh filename="package://bez2_description/meshes/New_right_foot_upperhalf_v3_1.stl" scale="0.001 0.001 0.001"/>
+    </geometry>
+  </collision>
+</link>
+<link name="lower_leg_v4_1">
+  <inertial>
+    <origin xyz="-7.555562408362304e-09 -0.023191925057663376 -0.02213350063265468" rpy="0 0 0"/>
+    <mass value="0.1476733120184745"/>
+    <inertia ixx="0.000124" iyy="0.000107" izz="4.1e-05" ixy="0.0" iyz="-2e-06" ixz="-0.0"/>
+  </inertial>
+  <visual>
+    <origin xyz="-0.01612 0.0123 0.26775" rpy="0 0 0"/>
+    <geometry>
+      <mesh filename="package://bez2_description/meshes/lower_leg_v4_1.stl" scale="0.001 0.001 0.001"/>
+    </geometry>
+    <material name="abs_white"/>
+  </visual>
+  <collision>
+    <origin xyz="-0.01612 0.0123 0.26775" rpy="0 0 0"/>
+    <geometry>
+      <mesh filename="package://bez2_description/meshes/lower_leg_v4_1.stl" scale="0.001 0.001 0.001"/>
+    </geometry>
+  </collision>
+</link>
+<link name="lower_leg_v4_2">
+  <inertial>
+    <origin xyz="6.452880308219222e-09 0.023191925057662998 -0.02213350063265551" rpy="0 0 0"/>
+    <mass value="0.1476733120184745"/>
+    <inertia ixx="0.000124" iyy="0.000107" izz="4.1e-05" ixy="0.0" iyz="2e-06" ixz="0.0"/>
+  </inertial>
+  <visual>
+    <origin xyz="-0.01462 -0.0132 0.26775" rpy="0 0 0"/>
+    <geometry>
+      <mesh filename="package://bez2_description/meshes/lower_leg_v4_2.stl" scale="0.001 0.001 0.001"/>
+    </geometry>
+    <material name="abs_white"/>
+  </visual>
+  <collision>
+    <origin xyz="-0.01462 -0.0132 0.26775" rpy="0 0 0"/>
+    <geometry>
+      <mesh filename="package://bez2_description/meshes/lower_leg_v4_2.stl" scale="0.001 0.001 0.001"/>
+    </geometry>
+  </collision>
+</link>
+<link name="ankle_motors_v4_1">
+  <inertial>
+    <origin xyz="-0.020543373941361492 0.023300002595937435 0.015062549801947933" rpy="0 0 0"/>
+    <mass value="0.3955604131597503"/>
+    <inertia ixx="0.000155" iyy="0.000468" izz="0.000419" ixy="0.0" iyz="-0.0" ixz="-2e-06"/>
+  </inertial>
+  <visual>
+    <origin xyz="-0.01462 -0.0127 0.37605" rpy="0 0 0"/>
+    <geometry>
+      <mesh filename="package://bez2_description/meshes/ankle_motors_v4_1.stl" scale="0.001 0.001 0.001"/>
+    </geometry>
+    <material name="steel_satin"/>
+  </visual>
+  <collision>
+    <origin xyz="-0.01462 -0.0127 0.37605" rpy="0 0 0"/>
+    <geometry>
+      <mesh filename="package://bez2_description/meshes/ankle_motors_v4_1.stl" scale="0.001 0.001 0.001"/>
+    </geometry>
+  </collision>
+</link>
+<link name="ankle_motors_v4_2">
+  <inertial>
+    <origin xyz="-0.020543374775831007 -0.023299997404074242 0.015062549801948433" rpy="0 0 0"/>
+    <mass value="0.3955604131597503"/>
+    <inertia ixx="0.000155" iyy="0.000468" izz="0.000419" ixy="0.0" iyz="-0.0" ixz="-2e-06"/>
+  </inertial>
+  <visual>
+    <origin xyz="-0.01612 0.0118 0.37605" rpy="0 0 0"/>
+    <geometry>
+      <mesh filename="package://bez2_description/meshes/ankle_motors_v4_2.stl" scale="0.001 0.001 0.001"/>
+    </geometry>
+    <material name="steel_satin"/>
+  </visual>
+  <collision>
+    <origin xyz="-0.01612 0.0118 0.37605" rpy="0 0 0"/>
+    <geometry>
+      <mesh filename="package://bez2_description/meshes/ankle_motors_v4_2.stl" scale="0.001 0.001 0.001"/>
+    </geometry>
+  </collision>
+</link>
 <link name="Hip_Printable_v2_v10_1">
   <inertial>
-    <origin xyz="3.220301637574252e-07 -4.2278800908499004e-05 -0.014017264198397453" rpy="0 0 0"/>
+    <origin xyz="4.217541806686084e-05 -3.049643870767227e-14 -0.014017367581240808" rpy="0 0 0"/>
     <mass value="0.010089224750638792"/>
-    <inertia ixx="6e-06" iyy="2e-06" izz="5e-06" ixy="-0.0" iyz="-0.0" ixz="-0.0"/>
-  </inertial>
-  <visual>
-    <origin xyz="-0.035359 -0.059474 0.072444" rpy="0 0 0"/>
+    <inertia ixx="2e-06" iyy="6e-06" izz="5e-06" ixy="0.0" iyz="-0.0" ixz="0.0"/>
+  </inertial>
+  <visual>
+    <origin xyz="-0.01597 0.0368 0.14405" rpy="0 0 0"/>
     <geometry>
       <mesh filename="package://bez2_description/meshes/Hip_Printable_v2_v10_1.stl" scale="0.001 0.001 0.001"/>
@@ -118,5 +338,5 @@
   </visual>
   <collision>
-    <origin xyz="-0.035359 -0.059474 0.072444" rpy="0 0 0"/>
+    <origin xyz="-0.01597 0.0368 0.14405" rpy="0 0 0"/>
     <geometry>
       <mesh filename="package://bez2_description/meshes/Hip_Printable_v2_v10_1.stl" scale="0.001 0.001 0.001"/>
@@ -124,161 +344,21 @@
   </collision>
 </link>
-<link name="Hip_Printable_v2_v10_2">
-  <inertial>
-    <origin xyz="3.220301620365795e-07 -4.227880091287051e-05 -0.01401726419839748" rpy="0 0 0"/>
-    <mass value="0.010089224750638792"/>
-    <inertia ixx="6e-06" iyy="2e-06" izz="5e-06" ixy="-0.0" iyz="-0.0" ixz="-0.0"/>
-  </inertial>
-  <visual>
-    <origin xyz="-0.109859 -0.059474 0.072444" rpy="0 0 0"/>
-    <geometry>
-      <mesh filename="package://bez2_description/meshes/Hip_Printable_v2_v10_2.stl" scale="0.001 0.001 0.001"/>
-    </geometry>
-    <material name="abs_white"/>
-  </visual>
-  <collision>
-    <origin xyz="-0.109859 -0.059474 0.072444" rpy="0 0 0"/>
-    <geometry>
-      <mesh filename="package://bez2_description/meshes/Hip_Printable_v2_v10_2.stl" scale="0.001 0.001 0.001"/>
-    </geometry>
-  </collision>
-</link>
-<link name="hip_motors_v4_1">
-  <inertial>
-    <origin xyz="2.491527500980695e-07 -0.009088099875617373 -0.011907281385175342" rpy="0 0 0"/>
-    <mass value="0.2728199051639206"/>
-    <inertia ixx="0.000178" iyy="7.4e-05" izz="0.000153" ixy="0.0" iyz="1e-06" ixz="0.0"/>
-  </inertial>
-  <visual>
-    <origin xyz="-0.035359 -0.082974 0.104444" rpy="0 0 0"/>
-    <geometry>
-      <mesh filename="package://bez2_description/meshes/hip_motors_v4_1.stl" scale="0.001 0.001 0.001"/>
-    </geometry>
-    <material name="silver_default"/>
-  </visual>
-  <collision>
-    <origin xyz="-0.035359 -0.082974 0.104444" rpy="0 0 0"/>
-    <geometry>
-      <mesh filename="package://bez2_description/meshes/hip_motors_v4_1.stl" scale="0.001 0.001 0.001"/>
-    </geometry>
-  </collision>
-</link>
-<link name="hip_motors_v4_2">
-  <inertial>
-    <origin xyz="2.491527557740847e-07 -0.009088099875621716 -0.011907281385175342" rpy="0 0 0"/>
-    <mass value="0.2728199051639206"/>
-    <inertia ixx="0.000178" iyy="7.4e-05" izz="0.000153" ixy="0.0" iyz="1e-06" ixz="0.0"/>
-  </inertial>
-  <visual>
-    <origin xyz="-0.109859 -0.084474 0.104444" rpy="0 0 0"/>
-    <geometry>
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