Commit message: generated urdf and initial proto
- order of links and joints was manually changed to make pybullet read correct order
- meshes were simplified already
- proto freshly generated needs manual fixes to make work

File: bez2_description/urdf/bez2_simple.urdf (robot description, URDF)
Before this commit: robot bez2, 22 links, 21 joints
Links:
- removed link neck_v4_1
- link Arm_Assembly-bez3_v12_1: geometry collision box size=50.00000000000001 56.673995971679695 197.48017120361328; visual mesh filename=package://bez2_description/meshes/Arm_Assembly-bez3_v12_1.s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 scale=0.001 0.001 0.001
- link Arm_Assembly-bez3_v12_2: geometry collision box size=50.00000000000001 56.673995971679695 197.48017120361328; visual mesh filename=package://bez2_description/meshes/Arm_Assembly-bez3_v12_2.s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 scale=0.001 0.001 0.001
- link Hip_Printable_v2_v10_1: geometry collision box size=26.000000000000004 45.0 50.00000190734863; visual mesh filename=package://bez2_description/meshes/Hip_Printable_v2_v10_1.stl scale=0.001 0.001 0.001
- link Hip_Printable_v2_v10_2: geometry collision box size=26.000000000000004 45.0 50.00000190734863; visual mesh filename=package://bez2_description/meshes/Hip_Printable_v2_v10_2.stl scale=0.001 0.001 0.001
- link New_left_foot_upperhalf_v5_1: geometry collision box size=43.000000000000014 89.99999856948854 169.99999999999997; visual mesh filename=package://bez2_description/meshes/New_left_foot_upperhalf_v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 scale=0.001 0.001 0.001
- link New_right_foot_upperhalf_v3_1: geometry collision box size=43.00000000000002 90.00000000000003 170.0; visual mesh filename=package://bez2_description/meshes/New_right_foot_upperhalf_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 scale=0.001 0.001 0.001
- link Upper_left_leg_support__bottom__v8_1: geometry collision box size=27.999999463558208 53.999997138977065 119.55892944335938; visual mesh filename=package://bez2_description/meshes/Upper_left_leg_support__b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 scale=0.001 0.001 0.001
- link Upper_left_leg_support__bottom__v8_2: geometry collision box size=27.99999952316284 53.99999904632569 119.55892944335936; visual mesh filename=package://bez2_description/meshes/Upper_left_leg_support__b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 scale=0.001 0.001 0.001
- link ankle_motors_v4_1: geometry collision box size=51.45655939157668 62.08892822265624 109.9148508877624; visual mesh filename=package://bez2_description/meshes/ankle_motors_v4_1.stl scale=0.001 0.001 0.001
- link ankle_motors_v4_2: geometry collision box size=51.45655811656067 62.08892822265625 109.91484706541547; visual mesh filename=package://bez2_description/meshes/ankle_motors_v4_2.stl scale=0.001 0.001 0.001
- link base_link: mass 1.3874949527504563 -> 1.4940527908480117; geometry collision box size=124.00000000000003 145.0 220.6740036010742; visual mesh filename=package://bez2_description/meshes/base_link.stl scale=0.001 0.001 0.001
- link biceps_v3_1: geometry collision box size=36.0 56.67399597167968 125.19999694824219; visual mesh filename=package://bez2_description/meshes/biceps_v3_1.stl scale=0.001 0.001 0.001
- link biceps_v3_2: geometry collision box size=35.99999999999999 56.67399597167968 125.19999694824219; visual mesh filename=package://bez2_description/meshes/biceps_v3_2.stl scale=0.001 0.001 0.001
- link camera_point_1: mass 0.0005023999999999976 -> 0.0005023999999999989; geometry collision box size=4.000000000000001 4.000000000000001 4.0000001192092896; visual mesh filename=package://bez2_description/meshes/camera_point_1.stl scale=0.001 0.001 0.001
- link custom_servo_support__middle_neck__v9_1: geometry collision box size=35.0 48.24042510986328 56.374000549316406; visual mesh filename=package://bez2_description/meshes/custom_servo_support__mid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 scale=0.001 0.001 0.001
- link head_v4_1: geometry collision box size=76.10000085830688 76.50000000000003 94.00000000000001; visual mesh filename=package://bez2_description/meshes/head_v4_1.stl scale=0.001 0.001 0.001
- link hip_motors_v4_1: geometry collision box size=40.999999046325684 46.50000000000001 76.89999771118164; visual mesh filename=package://bez2_description/meshes/hip_motors_v4_1.stl scale=0.001 0.001 0.001
- link hip_motors_v4_2: geometry collision box size=41.000000953674316 46.50000000000001 76.89999771118164; visual mesh filename=package://bez2_description/meshes/hip_motors_v4_2.stl scale=0.001 0.001 0.001
- link imu_1: geometry collision box size=3.9999990463256845 4.000000000000001 4.0; visual mesh filename=package://bez2_description/meshes/imu_1.stl scale=0.001 0.001 0.001
- link lower_leg_v4_1: geometry collision box size=40.200001716613784 54.6036782992241 137.71416301334767; visual mesh filename=package://bez2_description/meshes/lower_leg_v4_1.stl scale=0.001 0.001 0.001
- link lower_leg_v4_2: geometry collision box size=40.200001716613784 54.60368020650708 137.71416302916919; visual mesh filename=package://bez2_description/meshes/lower_leg_v4_2.stl scale=0.001 0.001 0.001
Joints:
- removed joint Rigid19
- removed joint camera_joint
- removed joint imu_joint
- added joint head_camera: type continuous, parent head_v4_1, child camera_point_1, origin xyz=0.0344 0.025674 0.048 rpy=0.0 0.0 0.0, axis 1.0 0.0 -0.0
- added joint torso_imu: type continuous, parent base_link, child imu_1, origin xyz=0.013 0.0 0.02895 rpy=0.0 0.0 0.0, axis 0.0 0.0 1.0
- joint head_motor_0: axis 0.0 -0.0 1.0 -> 0.0 0.0 -1.0; origin xyz=0.015 0.0045 0.046674 rpy=0.0 0.0 0.0 -> xyz=0.03325 -0.000333 0.075624 rpy=0.0 0.0 0.0; parent neck_v4_1 -> base_link
- joint head_motor_1: axis -1.0 0.0 0.0 -> -0.0 1.0 0.0; origin xyz=-0.022187 0.0 0.033818 rpy=0.0 0.0 0.0 -> xyz=0.0 -0.022187 0.033817 rpy=0.0 0.0 0.0
- joint left_arm_motor_0: axis -1.0 0.0 0.0 -> -0.0 -1.0 0.0; origin xyz=0.144659 0.075444 0.072056 rpy=0.0 0.0 0.0 -> xyz=0.0 0.0725 0.00045 rpy=0.0 0.0 0.0
- joint left_arm_motor_1: axis -1.0 -0.0 0.0 -> 0.0 -1.0 0.0; origin xyz=0.008 0.0 -0.0906 rpy=0.0 0.0 0.0 -> xyz=0.0 0.008 -0.0906 rpy=0.0 0.0 0.0
- joint left_leg_motor_0: axis 0.0 0.0 -1.0 -> -0.0 0.0 -1.0; origin xyz=0.109859 0.059474 -0.072444 rpy=0.0 0.0 0.0 -> xyz=0.01597 0.0377 -0.14405 rpy=0.0 0.0 0.0
- joint left_leg_motor_1: axis -0.0 -1.0 -0.0 -> 1.0 -0.0 -0.0; origin xyz=0.0 0.025 -0.032 rpy=0.0 0.0 0.0 -> xyz=-0.025 0.0 -0.032 rpy=0.0 0.0 0.0
- joint left_leg_motor_2: axis -1.0 -0.0 0.0 -> 0.0 -1.0 0.0; origin xyz=-0.02 -0.02365 0.0 rpy=0.0 0.0 0.0 -> xyz=0.02365 -0.02 0.0 rpy=0.0 0.0 0.0
- joint left_leg_motor_3: axis -1.0 -0.0 0.0 -> 0.0 -1.0 0.0; origin xyz=-0.0045 0.0 -0.0917 rpy=0.0 0.0 0.0 -> xyz=0.0 -0.0045 -0.0917 rpy=0.0 0.0 0.0
- joint left_leg_motor_4: axis -1.0 0.0 0.0 -> 0.0 -1.0 0.0; origin xyz=-0.0005 0.0 -0.1083 rpy=0.0 0.0 0.0 -> xyz=0.0 -0.0005 -0.1083 rpy=0.0 0.0 0.0
- joint left_leg_motor_5: axis 0.0 -1.0 -0.0 -> -1.0 0.0 0.0; origin xyz=0.0233 0.0843 0.0 rpy=0.0 0.0 0.0 -> xyz=-0.0843 0.0233 0.0 rpy=0.0 0.0 0.0
- joint right_arm_motor_0: axis 1.0 -0.0 -0.0 -> 0.0 -1.0 0.0; origin xyz=-0.000341 0.075444 0.072056 rpy=0.0 0.0 0.0 -> xyz=0.0 -0.0725 0.00045 rpy=0.0 0.0 0.0
- joint right_arm_motor_1: axis 1.0 0.0 0.0 -> -0.0 -1.0 0.0; origin xyz=-0.008 0.0 -0.0906 rpy=0.0 0.0 0.0 -> xyz=-0.0 -0.008 -0.0906 rpy=0.0 0.0 0.0
- joint right_leg_motor_0: axis 0.0 0.0 -1.0 -> -0.0 -0.0 1.0; origin xyz=0.035359 0.059474 -0.072444 rpy=0.0 0.0 0.0 -> xyz=0.01597 -0.0368 -0.14405 rpy=0.0 0.0 0.0
- joint right_leg_motor_1: axis -0.0 -1.0 -0.0 -> -1.0 0.0 0.0; origin xyz=0.0 0.0235 -0.032 rpy=0.0 0.0 0.0 -> xyz=-0.0235 0.0 -0.032 rpy=0.0 0.0 0.0
- joint right_leg_motor_2: axis 1.0 0.0 0.0 -> 0.0 -1.0 0.0; origin xyz=0.02 -0.02365 0.0 rpy=0.0 0.0 0.0 -> xyz=0.02365 0.02 0.0 rpy=0.0 0.0 0.0
- joint right_leg_motor_3: axis 1.0 0.0 0.0 -> 0.0 -1.0 0.0; origin xyz=0.0045 0.0 -0.0917 rpy=0.0 0.0 0.0 -> xyz=0.0 0.0045 -0.0917 rpy=0.0 0.0 0.0
- joint right_leg_motor_4: axis 1.0 -0.0 0.0 -> 0.0 -1.0 0.0; origin xyz=0.0005 0.0 -0.1083 rpy=0.0 0.0 0.0 -> xyz=0.0 0.0005 -0.1083 rpy=0.0 0.0 0.0
- joint right_leg_motor_5: axis 0.0 -1.0 -0.0 -> 1.0 0.0 0.0; origin xyz=-0.0233 0.0843 0.0 rpy=0.0 0.0 0.0 -> xyz=-0.0843 -0.0233 0.0 rpy=0.0 0.0 0.0

Commit message: fixed bounding boxes error

File: bez2_description/urdf/bez2.urdf (robot description, URDF)
Before this commit: robot bez2, 21 links, 20 joints
Links:
- link Arm_Assembly-bez3_v12_1: geometry collision mesh filename=package://bez2_description/meshes/Arm_Assembly-bez3_v12_1.s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 scale=1 1 1; visual mesh filename=package://bez2_description/meshes/Arm_Assembly-bez3_v12_1.s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 scale=1 1 1
- link Arm_Assembly-bez3_v12_2: geometry collision mesh filename=package://bez2_description/meshes/Arm_Assembly-bez3_v12_2.s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 scale=1 1 1; visual mesh filename=package://bez2_description/meshes/Arm_Assembly-bez3_v12_2.s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 scale=1 1 1
- link Hip_Printable_v2_v10_1: geometry collision mesh filename=package://bez2_description/meshes/Hip_Printable_v2_v10_1.stl scale=1 1 1; visual mesh filename=package://bez2_description/meshes/Hip_Printable_v2_v10_1.stl scale=1 1 1
- link Hip_Printable_v2_v10_2: geometry collision mesh filename=package://bez2_description/meshes/Hip_Printable_v2_v10_2.stl scale=1 1 1; visual mesh filename=package://bez2_description/meshes/Hip_Printable_v2_v10_2.stl scale=1 1 1
- link New_left_foot_upperhalf_v5_1: geometry collision mesh filename=package://bez2_description/meshes/New_left_foot_upperhalf_v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 scale=1 1 1; visual mesh filename=package://bez2_description/meshes/New_left_foot_upperhalf_v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 scale=1 1 1
- link New_right_foot_upperhalf_v3_1: geometry collision mesh filename=package://bez2_description/meshes/New_right_foot_upperhalf_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 scale=1 1 1; visual mesh filename=package://bez2_description/meshes/New_right_foot_upperhalf_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 scale=1 1 1
- link Upper_left_leg_support__bottom__v8_1: geometry collision mesh filename=package://bez2_description/meshes/Upper_left_leg_support__b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 scale=1 1 1; visual mesh filename=package://bez2_description/meshes/Upper_left_leg_support__b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 scale=1 1 1
- link Upper_left_leg_support__bottom__v8_2: geometry collision mesh filename=package://bez2_description/meshes/Upper_left_leg_support__b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 scale=1 1 1; visual mesh filename=package://bez2_description/meshes/Upper_left_leg_support__b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 scale=1 1 1
- link ankle_motors_v4_1: geometry collision mesh filename=package://bez2_description/meshes/ankle_motors_v4_1.stl scale=1 1 1; visual mesh filename=package://bez2_description/meshes/ankle_motors_v4_1.stl scale=1 1 1
- link ankle_motors_v4_2: geometry collision mesh filename=package://bez2_description/meshes/ankle_motors_v4_2.stl scale=1 1 1; visual mesh filename=package://bez2_description/meshes/ankle_motors_v4_2.stl scale=1 1 1
- link base_link: geometry collision mesh filename=package://bez2_description/meshes/base_link.stl scale=1 1 1; visual mesh filename=package://bez2_description/meshes/base_link.stl scale=1 1 1
- link biceps_v3_1: geometry collision mesh filename=package://bez2_description/meshes/biceps_v3_1.stl scale=1 1 1; visual mesh filename=package://bez2_description/meshes/biceps_v3_1.stl scale=1 1 1
- link biceps_v3_2: geometry collision mesh filename=package://bez2_description/meshes/biceps_v3_2.stl scale=1 1 1; visual mesh filename=package://bez2_description/meshes/biceps_v3_2.stl scale=1 1 1
- link camera_point_1: geometry collision mesh filename=package://bez2_description/meshes/camera_point_1.stl scale=1 1 1; visual mesh filename=package://bez2_description/meshes/camera_point_1.stl scale=1 1 1
- link custom_servo_support__middle_neck__v9_1: geometry collision mesh filename=package://bez2_description/meshes/custom_servo_support__mid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 scale=1 1 1; visual mesh filename=package://bez2_description/meshes/custom_servo_support__mid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 scale=1 1 1
- link head_v4_1: geometry collision mesh filename=package://bez2_description/meshes/head_v4_1.stl scale=1 1 1; visual mesh filename=package://bez2_description/meshes/head_v4_1.stl scale=1 1 1
- link hip_motors_v4_1: geometry collision mesh filename=package://bez2_description/meshes/hip_motors_v4_1.stl scale=1 1 1; visual mesh filename=package://bez2_description/meshes/hip_motors_v4_1.stl scale=1 1 1
- link hip_motors_v4_2: geometry collision mesh filename=package://bez2_description/meshes/hip_motors_v4_2.stl scale=1 1 1; visual mesh filename=package://bez2_description/meshes/hip_motors_v4_2.stl scale=1 1 1
- link imu_1: geometry collision mesh filename=package://bez2_description/meshes/imu_1.stl scale=1 1 1; visual mesh filename=package://bez2_description/meshes/imu_1.stl scale=1 1 1
- link lower_leg_v4_1: geometry collision mesh filename=package://bez2_description/meshes/lower_leg_v4_1.stl scale=1 1 1; visual mesh filename=package://bez2_description/meshes/lower_leg_v4_1.stl scale=1 1 1
- link lower_leg_v4_2: geometry collision mesh filename=package://bez2_description/meshes/lower_leg_v4_2.stl scale=1 1 1; visual mesh filename=package://bez2_description/meshes/lower_leg_v4_2.stl scale=1 1 1

File: bez2_description/urdf/bez2_simple.urdf (robot description, URDF)
Before this commit: robot bez2, 21 links, 20 joints
Links:
- link Arm_Assembly-bez3_v12_1: geometry collision box size=0.05000000074505806 0.05667400360107422 0.19749999791383743; visual mesh filename=package://bez2_description/meshes/Arm_Assembly-bez3_v12_1.s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 scale=1.0 1.0 1.0
- link Arm_Assembly-bez3_v12_2: geometry collision box size=0.05000000074505807 0.056674003601074226 0.19749999791383743; visual mesh filename=package://bez2_description/meshes/Arm_Assembly-bez3_v12_2.s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 scale=1.0 1.0 1.0
- link Hip_Printable_v2_v10_1: geometry collision box size=0.0260000005364418 0.04500000178813934 0.04999999795109033; visual mesh filename=package://bez2_description/meshes/Hip_Printable_v2_v10_1.stl scale=1.0 1.0 1.0
- link Hip_Printable_v2_v10_2: geometry collision box size=0.0260000005364418 0.04500000178813934 0.04999999795109033; visual mesh filename=package://bez2_description/meshes/Hip_Printable_v2_v10_2.stl scale=1.0 1.0 1.0
- link New_left_foot_upperhalf_v5_1: geometry collision box size=0.04300001263618469 0.0900000003166497 0.17000000178813934; visual mesh filename=package://bez2_description/meshes/New_left_foot_upperhalf_v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 scale=1.0 1.0 1.0
- link New_right_foot_upperhalf_v3_1: geometry collision box size=0.04300001263618471 0.09000000078231099 0.16999999433755875; visual mesh filename=package://bez2_description/meshes/New_right_foot_upperhalf_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 scale=1.0 1.0 1.0
- link Upper_left_leg_support__bottom__v8_1: geometry collision box size=0.027999999641906474 0.053999998606741435 0.119600012898445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; visual mesh filename=package://bez2_description/meshes/Upper_left_leg_support__b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 scale=1.0 1.0 1.0
- link Upper_left_leg_support__bottom__v8_2: geometry collision box size=0.02800000086426735 0.05399999860674143 0.11960001289844512; visual mesh filename=package://bez2_description/meshes/Upper_left_leg_support__b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 scale=1.0 1.0 1.0
- link ankle_motors_v4_1: geometry collision box size=0.05145662496933042 0.06209999322891237 0.109915084847917; visual mesh filename=package://bez2_description/meshes/ankle_motors_v4_1.stl scale=1.0 1.0 1.0
- link ankle_motors_v4_2: geometry collision box size=0.051475384296038096 0.06242990907162086 0.11020424060664373; visual mesh filename=package://bez2_description/meshes/ankle_motors_v4_2.stl scale=1.0 1.0 1.0
- link base_link: geometry collision box size=0.12400000542402269 0.1449999958276749 0.22067400068044662; visual mesh filename=package://bez2_description/meshes/base_link.stl scale=1.0 1.0 1.0
- link biceps_v3_1: geometry collision box size=0.035999998450279236 0.056673996150493615 0.125200001522898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; visual mesh filename=package://bez2_description/meshes/biceps_v3_1.stl scale=1.0 1.0 1.0
- link biceps_v3_2: geometry collision box size=0.035999998450279236 0.056673996150493615 0.125200001522898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; visual mesh filename=package://bez2_description/meshes/biceps_v3_2.stl scale=1.0 1.0 1.0
- link camera_point_1: geometry collision box size=0.00399999984074384 0.0040000006556510925 0.004000008106231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; visual mesh filename=package://bez2_description/meshes/camera_point_1.stl scale=1.0 1.0 1.0
- link custom_servo_support__middle_neck__v9_1: geometry collision box size=0.034999998286366456 0.04825326800346374 0.0563740003854036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; visual mesh filename=package://bez2_description/meshes/custom_servo_support__mid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 scale=1.0 1.0 1.0
- link head_v4_1: geometry collision box size=0.07609999924898148 0.07650000602006911 0.09400000050663948; visual mesh filename=package://bez2_description/meshes/head_v4_1.stl scale=1.0 1.0 1.0
- link hip_motors_v4_1: geometry collision box size=0.04099999833852053 0.04649999737739564 0.07689999975264072; visual mesh filename=package://bez2_description/meshes/hip_motors_v4_1.stl scale=1.0 1.0 1.0
- link hip_motors_v4_2: geometry collision box size=0.040999999269843095 0.04649999737739564 0.07689999975264071; visual mesh filename=package://bez2_description/meshes/hip_motors_v4_2.stl scale=1.0 1.0 1.0
- link imu_1: geometry collision box size=0.003999999724328519 0.004000000189989805 0.004000000655651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; visual mesh filename=package://bez2_description/meshes/imu_1.stl scale=1.0 1.0 1.0
- link lower_leg_v4_1: geometry collision box size=0.04019999969750644 0.05460367704768601 0.1377141897100448; visual mesh filename=package://bez2_description/meshes/lower_leg_v4_1.stl scale=1.0 1.0 1.0
- link lower_leg_v4_2: geometry collision box size=0.040200000628829016 0.05460367704768602 0.13771418971004487; visual mesh filename=package://bez2_description/meshes/lower_leg_v4_2.stl scale=1.0 1.0 1.0
