Commit message: Added meshes and fixed boundary problem

File: bez2_description/urdf/bez2_simple.urdf (robot description, URDF)
Before this commit: robot bez2, 21 links, 20 joints
Links:
- link Arm_Assembly-bez3_v12_1: geometry collision box size=50.000000000000014 56.67403535785024 197.51995458409905; visual mesh filename=package://bez2_description/meshes/Arm_Assembly-bez3_v12_1.s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 scale=0.001 0.001 0.001
- link Arm_Assembly-bez3_v12_2: geometry collision box size=50.00222408295757 56.67594349399609 197.51990509033203; visual mesh filename=package://bez2_description/meshes/Arm_Assembly-bez3_v12_2.s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 scale=0.001 0.001 0.001
- link Hip_Printable_v2_v10_1: geometry collision box size=26.002658349065094 45.24937726384439 50.00474032362708; visual mesh filename=package://bez2_description/meshes/Hip_Printable_v2_v10_1.stl scale=0.001 0.001 0.001
- link Hip_Printable_v2_v10_2: geometry collision box size=26.000967879521202 45.01321288741608 50.00136462741593; visual mesh filename=package://bez2_description/meshes/Hip_Printable_v2_v10_2.stl scale=0.001 0.001 0.001
- link New_left_foot_upperhalf_v5_1: geometry collision box size=43.000000000000014 89.99999856948855 169.99999999999997; visual mesh filename=package://bez2_description/meshes/New_left_foot_upperhalf_v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 scale=0.001 0.001 0.001
- link Upper_left_leg_support__bottom__v8_1: geometry collision box size=28.000522899514664 54.00099828050638 120.1605903833068; visual mesh filename=package://bez2_description/meshes/Upper_left_leg_support__b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 scale=0.001 0.001 0.001
- link Upper_left_leg_support__bottom__v8_2: geometry collision box size=28.000651388620067 54.00030139771184 119.7835903507593; visual mesh filename=package://bez2_description/meshes/Upper_left_leg_support__b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 scale=0.001 0.001 0.001
- link ankle_motors_v4_1: geometry collision box size=51.47627155047293 62.213952265043645 109.92561296712472; visual mesh filename=package://bez2_description/meshes/ankle_motors_v4_1.stl scale=0.001 0.001 0.001
- link ankle_motors_v4_2: geometry collision box size=51.48890161606914 62.4720331612971 110.02951674639873; visual mesh filename=package://bez2_description/meshes/ankle_motors_v4_2.stl scale=0.001 0.001 0.001
- link custom_servo_support__middle_neck__v9_1: geometry collision box size=35.0 48.321075440803114 56.375022169987524; visual mesh filename=package://bez2_description/meshes/custom_servo_support__mid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 scale=0.001 0.001 0.001
- link head_v4_1: geometry collision box size=76.10000085830688 76.5 94.0; visual mesh filename=package://bez2_description/meshes/head_v4_1.stl scale=0.001 0.001 0.001
- link hip_motors_v4_1: geometry collision box size=41.0000051077346 46.50000000000001 76.90002646425684; visual mesh filename=package://bez2_description/meshes/hip_motors_v4_1.stl scale=0.001 0.001 0.001
- link hip_motors_v4_2: geometry collision box size=41.00000603095625 46.50000000000001 76.90002806270799; visual mesh filename=package://bez2_description/meshes/hip_motors_v4_2.stl scale=0.001 0.001 0.001
- link lower_leg_v4_1: geometry collision box size=40.240934093771955 54.63939599062199 137.7149307458541; visual mesh filename=package://bez2_description/meshes/lower_leg_v4_1.stl scale=0.001 0.001 0.001
- link lower_leg_v4_2: geometry collision box size=40.50708316639091 54.63906611085356 137.7663535953382; visual mesh filename=package://bez2_description/meshes/lower_leg_v4_2.stl scale=0.001 0.001 0.001

Commit message: Updating webots

File: bez2_description/urdf/bez2_simple.urdf (robot description, URDF)
Before this commit: robot bez2, 21 links, 20 joints
Links:
- link Arm_Assembly-bez3_v12_1: geometry collision box size=0.05000000074505806 0.05667400360107422 0.19749999791383743; visual mesh filename=package://bez2_description/meshes/Arm_Assembly-bez3_v12_1.d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 scale=1.0 1.0 1.0
- link Arm_Assembly-bez3_v12_2: geometry collision box size=0.05000000074505807 0.056674003601074226 0.19749999791383743; visual mesh filename=package://bez2_description/meshes/Arm_Assembly-bez3_v12_2.d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 scale=1.0 1.0 1.0
- link Hip_Printable_v2_v10_1: geometry collision box size=0.0260000005364418 0.04500000178813934 0.04999999795109033; visual mesh filename=package://bez2_description/meshes/Hip_Printable_v2_v10_1.dae scale=1.0 1.0 1.0
- link Hip_Printable_v2_v10_2: geometry collision box size=0.0260000005364418 0.04500000178813934 0.04999999795109033; visual mesh filename=package://bez2_description/meshes/Hip_Printable_v2_v10_2.dae scale=1.0 1.0 1.0
- link ankle_motors_v4_1: geometry collision box size=0.05145662496933042 0.06209999322891237 0.109915084847917; visual mesh filename=package://bez2_description/meshes/ankle_motors_v4_1.dae scale=1.0 1.0 1.0
- link ankle_motors_v4_2: geometry collision box size=0.051475384296038096 0.06242990907162086 0.11020424060664373; visual mesh filename=package://bez2_description/meshes/ankle_motors_v4_2.dae scale=1.0 1.0 1.0
- link base_link: geometry collision box size=0.12400000542402269 0.1449999958276749 0.22067400068044662; visual mesh filename=package://bez2_description/meshes/base_link.dae scale=1.0 1.0 1.0
- link biceps_v3_1: geometry collision box size=0.035999998450279236 0.056673996150493615 0.125200001522898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; visual mesh filename=package://bez2_description/meshes/biceps_v3_1.dae scale=1.0 1.0 1.0
- link biceps_v3_2: geometry collision box size=0.035999998450279236 0.056673996150493615 0.125200001522898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; visual mesh filename=package://bez2_description/meshes/biceps_v3_2.dae scale=1.0 1.0 1.0
- link camera_point_1: geometry collision box size=0.00399999984074384 0.0040000006556510925 0.004000008106231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; visual mesh filename=package://bez2_description/meshes/camera_point_1.dae scale=1.0 1.0 1.0
- link head_v4_1: geometry collision box size=0.07609999924898148 0.07650000602006911 0.09400000050663948; visual mesh filename=package://bez2_description/meshes/head_v4_1.dae scale=1.0 1.0 1.0
- link hip_motors_v4_1: geometry collision box size=0.04099999833852053 0.04649999737739564 0.07689999975264072; visual mesh filename=package://bez2_description/meshes/hip_motors_v4_1.dae scale=1.0 1.0 1.0
- link hip_motors_v4_2: geometry collision box size=0.040999999269843095 0.04649999737739564 0.07689999975264071; visual mesh filename=package://bez2_description/meshes/hip_motors_v4_2.dae scale=1.0 1.0 1.0
- link imu_1: geometry collision box size=0.003999999724328519 0.004000000189989805 0.004000000655651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; visual mesh filename=package://bez2_description/meshes/imu_1.dae scale=1.0 1.0 1.0
- link lower_leg_v4_1: geometry collision box size=0.04019999969750644 0.05460367704768601 0.1377141897100448; visual mesh filename=package://bez2_description/meshes/lower_leg_v4_1.dae scale=1.0 1.0 1.0
- link lower_leg_v4_2: geometry collision box size=0.040200000628829016 0.05460367704768602 0.13771418971004487; visual mesh filename=package://bez2_description/meshes/lower_leg_v4_2.dae scale=1.0 1.0 1.0

Commit message: Finished updating webots

File: bez2_description/urdf/bez2_simple.urdf (robot description, URDF)
Before this commit: robot bez2, 21 links, 20 joints
Links:
- link Arm_Assembly-bez3_v12_1: geometry collision box size=0.05000000074505806 0.05667400360107422 0.19749999791383743; visual mesh filename=package://bez2_description/meshes/Arm_Assembly-bez3_v12_1.s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 scale=1.0 1.0 1.0
- link Arm_Assembly-bez3_v12_2: geometry collision box size=0.05000000074505807 0.056674003601074226 0.19749999791383743; visual mesh filename=package://bez2_description/meshes/Arm_Assembly-bez3_v12_2.s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 scale=1.0 1.0 1.0
- link Hip_Printable_v2_v10_1: geometry collision box size=0.0260000005364418 0.04500000178813934 0.04999999795109033; visual mesh filename=package://bez2_description/meshes/Hip_Printable_v2_v10_1.stl scale=1.0 1.0 1.0
- link Hip_Printable_v2_v10_2: geometry collision box size=0.0260000005364418 0.04500000178813934 0.04999999795109033; visual mesh filename=package://bez2_description/meshes/Hip_Printable_v2_v10_2.stl scale=1.0 1.0 1.0
- link ankle_motors_v4_1: geometry collision box size=0.05145662496933042 0.06209999322891237 0.109915084847917; visual mesh filename=package://bez2_description/meshes/ankle_motors_v4_1.stl scale=1.0 1.0 1.0
- link ankle_motors_v4_2: geometry collision box size=0.051475384296038096 0.06242990907162086 0.11020424060664373; visual mesh filename=package://bez2_description/meshes/ankle_motors_v4_2.stl scale=1.0 1.0 1.0
- link base_link: geometry collision box size=0.12400000542402269 0.1449999958276749 0.22067400068044662; visual mesh filename=package://bez2_description/meshes/base_link.stl scale=1.0 1.0 1.0
- link biceps_v3_1: geometry collision box size=0.035999998450279236 0.056673996150493615 0.125200001522898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; visual mesh filename=package://bez2_description/meshes/biceps_v3_1.stl scale=1.0 1.0 1.0
- link biceps_v3_2: geometry collision box size=0.035999998450279236 0.056673996150493615 0.125200001522898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; visual mesh filename=package://bez2_description/meshes/biceps_v3_2.stl scale=1.0 1.0 1.0
- link camera_point_1: geometry collision box size=0.00399999984074384 0.0040000006556510925 0.004000008106231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; visual mesh filename=package://bez2_description/meshes/camera_point_1.stl scale=1.0 1.0 1.0
- link head_v4_1: geometry collision box size=0.07609999924898148 0.07650000602006911 0.09400000050663948; visual mesh filename=package://bez2_description/meshes/head_v4_1.stl scale=1.0 1.0 1.0
- link hip_motors_v4_1: geometry collision box size=0.04099999833852053 0.04649999737739564 0.07689999975264072; visual mesh filename=package://bez2_description/meshes/hip_motors_v4_1.stl scale=1.0 1.0 1.0
- link hip_motors_v4_2: geometry collision box size=0.040999999269843095 0.04649999737739564 0.07689999975264071; visual mesh filename=package://bez2_description/meshes/hip_motors_v4_2.stl scale=1.0 1.0 1.0
- link imu_1: geometry collision box size=0.003999999724328519 0.004000000189989805 0.004000000655651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; visual mesh filename=package://bez2_description/meshes/imu_1.stl scale=1.0 1.0 1.0
- link lower_leg_v4_1: geometry collision box size=0.04019999969750644 0.05460367704768601 0.1377141897100448; visual mesh filename=package://bez2_description/meshes/lower_leg_v4_1.stl scale=1.0 1.0 1.0
- link lower_leg_v4_2: geometry collision box size=0.040200000628829016 0.05460367704768602 0.13771418971004487; visual mesh filename=package://bez2_description/meshes/lower_leg_v4_2.stl scale=1.0 1.0 1.0
