Commit message: regenerate fusion model
- updated masses to be more accurate
- update joint names
- added imu and camera joints
- names of stl files changed

File: bez2_description/urdf/bez2_simple.urdf (robot description, URDF)
Before this commit: robot bez2, 20 links, 19 joints
Links:
- removed link Arm_Assembly-bez3_v10_1
- removed link Arm_Assembly-bez3_v10_2
- removed link Hip_Printable_v2_v9_1
- removed link Hip_Printable_v2_v9_2
- removed link New_left_foot_upperhalf_v4_1
- removed link New_right_foot_upperhalf_v2_1
- removed link Upper_left_leg_support__bottom__v7_1
- removed link Upper_left_leg_support__bottom__v7_2
- removed link ankle_motors_v3_1
- removed link ankle_motors_v3_2
- removed link biceps_v2_1
- removed link biceps_v2_2
- removed link custom_servo_support__middle_neck__v8_1
- removed link head_v2_1
- removed link hip_motors_v3_1
- removed link hip_motors_v3_2
- removed link lower_leg_v2_1
- removed link lower_leg_v2_2
- removed link neck_v2_1
- added link Arm_Assembly-bez3_v12_1, mass 0.32110352957731503; collision box size=0.05000000074505806 0.05667400034144522 0.19750000373460352; visual mesh filename=package://bez2_description/meshes/Arm_Assembly-bez3_v12_1.s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 scale=0.001 0.001 0.001
- added link Arm_Assembly-bez3_v12_2, mass 0.32110352957731503; collision box size=0.05000000074505805 0.056674003601074226 0.19750000373460352; visual mesh filename=package://bez2_description/meshes/Arm_Assembly-bez3_v12_2.s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 scale=0.001 0.001 0.001
- added link Hip_Printable_v2_v10_1, mass 0.010089224750638792; collision box size=0.026000000536441806 0.04500000178813934 0.05000000447034835; visual mesh filename=package://bez2_description/meshes/Hip_Printable_v2_v10_1.stl scale=0.001 0.001 0.001
- added link Hip_Printable_v2_v10_2, mass 0.010089224750638792; collision box size=0.02600000053644181 0.04500000178813934 0.05000000447034836; visual mesh filename=package://bez2_description/meshes/Hip_Printable_v2_v10_2.stl scale=0.001 0.001 0.001
- added link New_left_foot_upperhalf_v5_1, mass 0.0588564551543425; collision box size=0.043000012636184706 0.09000000171363354 0.17000000458210707; visual mesh filename=package://bez2_description/meshes/New_left_foot_upperhalf_v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 scale=0.001 0.001 0.001
- added link New_right_foot_upperhalf_v3_1, mass 0.117712910308685; collision box size=0.0430000126361847 0.08999999612569809 0.17000000085681677; visual mesh filename=package://bez2_description/meshes/New_right_foot_upperhalf_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 scale=0.001 0.001 0.001
- added link Upper_left_leg_support__bottom__v8_1, mass 0.027169463894965433; collision box size=0.02799999713897706 0.05399999767541887 0.11959999799728394; visual mesh filename=package://bez2_description/meshes/Upper_left_leg_support__b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 scale=0.001 0.001 0.001
- added link Upper_left_leg_support__bottom__v8_2, mass 0.027169463894965433; collision box size=0.028000000864267387 0.05399999674409628 0.11959999799728395; visual mesh filename=package://bez2_description/meshes/Upper_left_leg_support__b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 scale=0.001 0.001 0.001
- added link ankle_motors_v4_1, mass 0.3955604131597503; collision box size=0.05145662812639435 0.06209999322891235 0.10991508842745541; visual mesh filename=package://bez2_description/meshes/ankle_motors_v4_1.stl scale=0.001 0.001 0.001
- added link ankle_motors_v4_2, mass 0.3955604131597503; collision box size=0.05145662430256209 0.06209999322891237 0.109915078070939; visual mesh filename=package://bez2_description/meshes/ankle_motors_v4_2.stl scale=0.001 0.001 0.001
- added link biceps_v3_1, mass 0.25825416029102555; collision box size=0.03599999472498894 0.05667400360107421 0.12519999966025352; visual mesh filename=package://bez2_description/meshes/biceps_v3_1.stl scale=0.001 0.001 0.001
- added link biceps_v3_2, mass 0.25825416029102555; collision box size=0.03599999472498894 0.05667399970116094 0.12519999966025352; visual mesh filename=package://bez2_description/meshes/biceps_v3_2.stl scale=0.001 0.001 0.001
- added link camera_point_1, mass 0.0005023999999999976; collision box size=0.0039999932050704965 0.004000000189989806 0.00400000065565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; visual mesh filename=package://bez2_description/meshes/camera_point_1.stl scale=0.001 0.001 0.001
- added link custom_servo_support__middle_neck__v9_1, mass 0.01959544470499754; collision box size=0.034999998286366456 0.048253268003463745 0.056374002248048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; visual mesh filename=package://bez2_description/meshes/custom_servo_support__mid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 scale=0.001 0.001 0.001
- added link head_v4_1, mass 0.29338454987270446; collision box size=0.07609999692067504 0.07649999856948851 0.09399999678134917; visual mesh filename=package://bez2_description/meshes/head_v4_1.stl scale=0.001 0.001 0.001
- added link hip_motors_v4_1, mass 0.2728199051639206; collision box size=0.04100000113248826 0.04650000482797623 0.07689999788999557; visual mesh filename=package://bez2_description/meshes/hip_motors_v4_1.stl scale=0.001 0.001 0.001
- added link hip_motors_v4_2, mass 0.2728199051639206; collision box size=0.04100000113248826 0.04650000482797622 0.07690000161528589; visual mesh filename=package://bez2_description/meshes/hip_motors_v4_2.stl scale=0.001 0.001 0.001
- added link imu_1, mass 0.0005024000000000008; collision box size=0.0040000006556511 0.004000000655651093 0.00400000065565109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; visual mesh filename=package://bez2_description/meshes/imu_1.stl scale=0.001 0.001 0.001
- added link lower_leg_v4_1, mass 0.1476733120184745; collision box size=0.04019999876618386 0.05460367809420252 0.13771419042204602; visual mesh filename=package://bez2_description/meshes/lower_leg_v4_1.stl scale=0.001 0.001 0.001
- added link lower_leg_v4_2, mass 0.1476733120184745; collision box size=0.040200002491474186 0.05460368554452673 0.13771419048384892; visual mesh filename=package://bez2_description/meshes/lower_leg_v4_2.stl scale=0.001 0.001 0.001
- added link neck_v4_1, mass 0.10655783809755558; collision box size=0.040000002831220606 0.04667399823665619 0.0543000008910894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; visual mesh filename=package://bez2_description/meshes/neck_v4_1.stl scale=0.001 0.001 0.001
- link base_link: mass 19.222054389299405 -> 1.3874949527504563; geometry collision box size=0.12400000635534526 0.14500000345287845 0.17400000244379044; visual mesh filename=package://bez2_description/meshes/base_link.stl scale=0.001 0.001 0.001
Joints:
- removed joint Rev1
- removed joint Rev10
- removed joint Rev17
- removed joint Rev18
- removed joint Rev2
- removed joint Rev20
- removed joint Rev21
- removed joint Rev22
- removed joint Rev23
- removed joint Rev25
- removed joint Rev26
- removed joint Rev3
- removed joint Rev4
- removed joint Rev5
- removed joint Rev6
- removed joint Rev7
- removed joint Rev8
- removed joint Rev9
- added joint camera_joint: type continuous, parent head_v4_1, child camera_point_1, origin xyz=0.025674 -0.0344 0.048 rpy=0.0 0.0 0.0, axis -0.0 -1.0 -0.0
- added joint head_motor_0: type continuous, parent neck_v4_1, child custom_servo_support__middle_neck__v9_1, origin xyz=0.015 0.0045 0.046674 rpy=0.0 0.0 0.0, axis 0.0 -0.0 1.0
- added joint head_motor_1: type continuous, parent custom_servo_support__middle_neck__v9_1, child head_v4_1, origin xyz=-0.022187 0.0 0.033818 rpy=0.0 0.0 0.0, axis -1.0 0.0 0.0
- added joint imu_joint: type continuous, parent base_link, child imu_1, origin xyz=0.072159 0.062444 0.100556 rpy=0.0 0.0 0.0, axis -0.0 -0.0 1.0
- added joint left_arm_motor_0: type continuous, parent base_link, child biceps_v3_1, origin xyz=0.144659 0.075444 0.072056 rpy=0.0 0.0 0.0, axis -1.0 0.0 0.0
- added joint left_arm_motor_1: type continuous, parent biceps_v3_1, child Arm_Assembly-bez3_v12_2, origin xyz=0.008 0.0 -0.0906 rpy=0.0 0.0 0.0, axis -1.0 -0.0 0.0
- added joint left_leg_motor_0: type continuous, parent base_link, child Hip_Printable_v2_v10_2, origin xyz=0.109859 0.059474 -0.072444 rpy=0.0 0.0 0.0, axis 0.0 0.0 -1.0
- added joint left_leg_motor_1: type continuous, parent Hip_Printable_v2_v10_2, child hip_motors_v4_2, origin xyz=0.0 0.025 -0.032 rpy=0.0 0.0 0.0, axis -0.0 -1.0 -0.0
- added joint left_leg_motor_2: type continuous, parent hip_motors_v4_2, child Upper_left_leg_support__bottom__v8_1, origin xyz=-0.02 -0.02365 0.0 rpy=0.0 0.0 0.0, axis -1.0 -0.0 0.0
- added joint left_leg_motor_3: type continuous, parent Upper_left_leg_support__bottom__v8_1, child lower_leg_v4_2, origin xyz=-0.0045 0.0 -0.0917 rpy=0.0 0.0 0.0, axis -1.0 -0.0 0.0
- added joint left_leg_motor_4: type continuous, parent lower_leg_v4_2, child ankle_motors_v4_1, origin xyz=-0.0005 0.0 -0.1083 rpy=0.0 0.0 0.0, axis -1.0 0.0 0.0
- added joint left_leg_motor_5: type continuous, parent ankle_motors_v4_1, child New_right_foot_upperhalf_v3_1, origin xyz=0.0233 0.0843 0.0 rpy=0.0 0.0 0.0, axis 0.0 -1.0 -0.0
- added joint right_arm_motor_0: type continuous, parent base_link, child biceps_v3_2, origin xyz=-0.000341 0.075444 0.072056 rpy=0.0 0.0 0.0, axis 1.0 -0.0 -0.0
- added joint right_arm_motor_1: type continuous, parent biceps_v3_2, child Arm_Assembly-bez3_v12_1, origin xyz=-0.008 0.0 -0.0906 rpy=0.0 0.0 0.0, axis 1.0 0.0 0.0
- added joint right_leg_motor_0: type continuous, parent base_link, child Hip_Printable_v2_v10_1, origin xyz=0.035359 0.059474 -0.072444 rpy=0.0 0.0 0.0, axis 0.0 0.0 -1.0
- added joint right_leg_motor_1: type continuous, parent Hip_Printable_v2_v10_1, child hip_motors_v4_1, origin xyz=0.0 0.0235 -0.032 rpy=0.0 0.0 0.0, axis -0.0 -1.0 -0.0
- added joint right_leg_motor_2: type continuous, parent hip_motors_v4_1, child Upper_left_leg_support__bottom__v8_2, origin xyz=0.02 -0.02365 0.0 rpy=0.0 0.0 0.0, axis 1.0 0.0 0.0
- added joint right_leg_motor_3: type continuous, parent Upper_left_leg_support__bottom__v8_2, child lower_leg_v4_1, origin xyz=0.0045 0.0 -0.0917 rpy=0.0 0.0 0.0, axis 1.0 0.0 0.0
- added joint right_leg_motor_4: type continuous, parent lower_leg_v4_1, child ankle_motors_v4_2, origin xyz=0.0005 0.0 -0.1083 rpy=0.0 0.0 0.0, axis 1.0 -0.0 0.0
- added joint right_leg_motor_5: type continuous, parent ankle_motors_v4_2, child New_left_foot_upperhalf_v5_1, origin xyz=-0.0233 0.0843 0.0 rpy=0.0 0.0 0.0, axis 0.0 -1.0 -0.0
- joint Rigid19: child neck_v2_1 -> neck_v4_1

File: bez2_description/urdf/materials.xacro (robot description, xacro)
@@ -7,12 +7,12 @@
   <color rgba="0.7843137254901961 0.5568627450980392 0.027450980392156862 1.0"/>
 </material>
+<material name="plastic_glossy_black">
+  <color rgba="0.09803921568627451 0.09803921568627451 0.09803921568627451 1.0"/>
+</material>
+<material name="abs_white">
+  <color rgba="0.9647058823529412 0.9647058823529412 0.9529411764705882 1.0"/>
+</material>
 <material name="steel_satin">
   <color rgba="0.6274509803921569 0.6274509803921569 0.6274509803921569 1.0"/>
 </material>
-<material name="abs_white">
-  <color rgba="0.37254901960784315 0.3607843137254902 0.34509803921568627 1.0"/>
-</material>
-<material name="plastic_glossy_black">
-  <color rgba="0.09803921568627451 0.09803921568627451 0.09803921568627451 1.0"/>
-</material>
 </robot>
