Commit message: working on it

File: soccer_description/bez1_description/urdf/bez1_old.urdf (robot description, URDF)
Before this commit: robot bez1, 20 links, 19 joints
Links:
- added link /camera, mass 0.01
Joints:
- added joint /head_camera: type fixed, parent /head, child /camera, origin xyz=0.015 0.00145 0.04740 rpy=0 0 0, axis 0  0  0, limit lower=0 upper=0 effort=0 velocity=0

File: soccer_description/bez2_description/urdf/bez2.urdf (robot description, URDF)
Before this commit: robot bez2, 22 links, 21 joints
Joints:
- joint left_leg_motor_0: axis 0.0 0.0 1.0 -> 0.0 0.0 -1.0
- joint right_leg_motor_0: axis -0.0 -0.0 -1.0 -> -0.0 -0.0 1.0

File: soccer_description/bez2_description/urdf/bez2.xacro (robot description, xacro)
@@ -469,5 +469,5 @@
 <parent link="torso"/>
 <child link="left_hip_side"/>
-<axis xyz="0.0 0.0 1.0"/>
+<axis xyz="0.0 0.0 -1.0"/>
   <dynamics damping="${XM430_DAMPING}" friction="${XM430_FRICTION}" />
 <limit effort="${XM430_TORQUE}" lower="-1.309" upper="0.524" velocity="${XM430_VELOCITY}"/>
@@ -541,5 +541,5 @@
   <parent link="torso"/>
   <child link="right_hip_side"/>
-  <axis xyz="-0.0 -0.0 -1.0"/>
+  <axis xyz="-0.0 -0.0 1.0"/>
     <dynamics damping="${XM430_DAMPING}" friction="${XM430_FRICTION}" />
   <limit effort="${XM430_TORQUE}" lower="-1.309" upper="0.524" velocity="${XM430_VELOCITY}"/>
