Commit message: experimenting with placo

File: soccer_description/bez1_description/urdf/bez1_b.urdf (robot description, URDF)
Before this commit: robot bez1, 19 links, 18 joints
Links:
- added link /imu_link, mass 0.01
Joints:
- added joint /torso_imu: type fixed, parent /torso, child /imu_link, origin xyz=0.0 0 0.000 rpy=0 0 0, axis 0 0 0
