Commit message: Fixed someproblems in the webots bridge and urdf/xacro. integrated placo as a walk engine alternative

File: soccer_description/bez1_description/urdf/arm.xacro (robot description, xacro)
@@ -45,5 +45,5 @@
                 </visual>
             </link>
-            <joint name="${name}_arm_motor_0" type="revolute">
+            <joint name="${name}_shoulder_pitch" type="revolute">
                 <parent link="${origin}"/>
                 <child link="$(arg tf_prefix)/${name}_bicep"/>
@@ -53,5 +53,5 @@
                 <limit effort="${AX12_TORQUE}" lower="-${PI/2}" upper="${PI*5/4}" velocity="${AX12_VELOCITY}"/>
             </joint>
-            <joint name="${name}_arm_motor_1" type="revolute">
+            <joint name="${name}_elbow" type="revolute">
                 <parent link="$(arg tf_prefix)/${name}_bicep"/>
                 <child link="$(arg tf_prefix)/${name}_forearm"/>
@@ -65,20 +65,20 @@
                 <mu2>${FOREARM_MU2}</mu2>
             </gazebo>
-            <transmission name="${name}_arm_motor_0">
+            <transmission name="${name}_shoulder_pitch">
                 <type>transmission_interface/SimpleTransmission</type>
-                <joint name="${name}_arm_motor_0">
+                <joint name="${name}_shoulder_pitch">
                     <hardwareInterface>hardware_interface/EffortJointInterface</hardwareInterface>
                 </joint>
-                <actuator name="${name}_arm_motor_0">
+                <actuator name="${name}_shoulder_pitch">
                     <hardwareInterface>hardware_interface/EffortJointInterface</hardwareInterface>
                     <mechanicalReduction>1</mechanicalReduction>
                 </actuator>
             </transmission>
-            <transmission name="${name}_arm_motor_1">
+            <transmission name="${name}_elbow">
                 <type>transmission_interface/SimpleTransmission</type>
-                <joint name="${name}_arm_motor_1">
+                <joint name="${name}_elbow">
                     <hardwareInterface>hardware_interface/EffortJointInterface</hardwareInterface>
                 </joint>
-                <actuator name="${name}_arm_motor_1">
+                <actuator name="${name}_elbow">
                     <hardwareInterface>hardware_interface/EffortJointInterface</hardwareInterface>
                     <mechanicalReduction>1</mechanicalReduction>

File: soccer_description/bez1_description/urdf/head.xacro (robot description, xacro)
@@ -45,5 +45,5 @@
             </visual>
         </link>
-        <joint name="head_motor_0" type="revolute">
+        <joint name="head_yaw" type="revolute">
             <parent link="${origin}"/>
             <child link="$(arg tf_prefix)/neck"/>
@@ -53,5 +53,5 @@
             <limit effort="${AX12_TORQUE}" lower="-${PI/2}" upper="${PI/2}" velocity="${AX12_VELOCITY}"/>
         </joint>
-        <joint name="head_motor_1" type="revolute">
+        <joint name="head_pitch" type="revolute">
             <parent link="$(arg tf_prefix)/neck"/>
             <child link="$(arg tf_prefix)/head"/>
@@ -61,20 +61,20 @@
             <limit effort="${AX12_TORQUE}" lower="-${PI*3/4}" upper="${PI*3/4}" velocity="${AX12_VELOCITY}"/>
         </joint>
-        <transmission name="head_motor_0">
+        <transmission name="head_yaw">
             <type>transmission_interface/SimpleTransmission</type>
-            <joint name="head_motor_0">
+            <joint name="head_yaw">
                 <hardwareInterface>hardware_interface/EffortJointInterface</hardwareInterface>
             </joint>
-            <actuator name="head_motor_0">
+            <actuator name="head_yaw">
                 <hardwareInterface>hardware_interface/EffortJointInterface</hardwareInterface>
                 <mechanicalReduction>1</mechanicalReduction>
             </actuator>
         </transmission>
-        <transmission name="head_motor_1">
+        <transmission name="head_pitch">
             <type>transmission_interface/SimpleTransmission</type>
-            <joint name="head_motor_1">
+            <joint name="head_pitch">
                 <hardwareInterface>hardware_interface/EffortJointInterface</hardwareInterface>
             </joint>
-            <actuator name="head_motor_1">
+            <actuator name="head_pitch">
                 <hardwareInterface>hardware_interface/EffortJointInterface</hardwareInterface>
                 <mechanicalReduction>1</mechanicalReduction>

File: soccer_description/bez1_description/urdf/leg.xacro (robot description, xacro)
@@ -134,5 +134,5 @@
             </visual>
         </link>
-        <joint name="${name}_leg_motor_0" type="revolute">
+        <joint name="${name}_hip_yaw" type="revolute">
             <parent link="$(arg tf_prefix)/torso"/>
             <child link="$(arg tf_prefix)/${name}_hip_side"/>
@@ -142,5 +142,5 @@
             <limit effort="${MX28_TORQUE}" lower="-1.309" upper="0.524" velocity="${MX28_VELOCITY}"/>
         </joint>
-        <joint name="${name}_leg_motor_1" type="revolute">
+        <joint name="${name}_hip_roll" type="revolute">
             <parent link="$(arg tf_prefix)/${name}_hip_side"/>
             <child link="$(arg tf_prefix)/${name}_hip_front"/>
@@ -150,5 +150,5 @@
             <limit effort="${MX28_TORQUE}" lower="-${PI/4}" upper="${PI/2}" velocity="${MX28_VELOCITY}"/>
         </joint>
-        <joint name="${name}_leg_motor_2" type="revolute">
+        <joint name="${name}_hip_pitch" type="revolute">
             <parent link="$(arg tf_prefix)/${name}_hip_front"/>
             <child link="$(arg tf_prefix)/${name}_thigh"/>
@@ -158,5 +158,5 @@
             <limit effort="${MX28_TORQUE}" lower="-${PI/4}" upper="${PI*3/4}" velocity="${MX28_VELOCITY}"/>
         </joint>
-        <joint name="${name}_leg_motor_3" type="revolute">
+        <joint name="${name}_knee" type="revolute">
             <parent link="$(arg tf_prefix)/${name}_thigh"/>
             <child link="$(arg tf_prefix)/${name}_calve"/>
@@ -166,5 +166,5 @@
             <limit effort="${MX28_TORQUE}" lower="-2.793" upper="0" velocity="${MX28_VELOCITY}"/>
         </joint>
-        <joint name="${name}_leg_motor_4" type="revolute">
+        <joint name="${name}_ankle_pitch" type="revolute">
             <parent link="$(arg tf_prefix)/${name}_calve"/>
             <child link="$(arg tf_prefix)/${name}_ankle"/>
@@ -174,5 +174,5 @@
             <limit effort="${MX28_TORQUE}" lower="-${PI/4}" upper="${PI/2}" velocity="${MX28_VELOCITY}"/>
         </joint>
-        <joint name="${name}_leg_motor_5" type="revolute">
+        <joint name="${name}_ankle_roll" type="revolute">
             <parent link="$(arg tf_prefix)/${name}_ankle"/>
             <child link="$(arg tf_prefix)/${name}_foot"/>
@@ -182,60 +182,60 @@
             <limit effort="${MX28_TORQUE}" lower="-${PI/4}" upper="${PI/4}" velocity="${MX28_VELOCITY}"/>
         </joint>
-        <transmission name="${name}_leg_motor_0">
-            <type>transmission_interface/SimpleTransmission</type>
-            <joint name="${name}_leg_motor_0">
-                <hardwareInterface>hardware_interface/EffortJointInterface</hardwareInterface>
-            </joint>
-            <actuator name="${name}_leg_motor_0">
-                <hardwareInterface>hardware_interface/EffortJointInterface</hardwareInterface>
-                <mechanicalReduction>1</mechanicalReduction>
-            </actuator>
-        </transmission>
-        <transmission name="${name}_leg_motor_1">
-            <type>transmission_interface/SimpleTransmission</type>
-            <joint name="${name}_leg_motor_1">
-                <hardwareInterface>hardware_interface/EffortJointInterface</hardwareInterface>
-            </joint>
-            <actuator name="${name}_leg_motor_1">
-                <hardwareInterface>hardware_interface/EffortJointInterface</hardwareInterface>
-                <mechanicalReduction>1</mechanicalReduction>
-            </actuator>
-        </transmission>
-        <transmission name="${name}_leg_motor_2">
-            <type>transmission_interface/SimpleTransmission</type>
-            <joint name="${name}_leg_motor_2">
-                <hardwareInterface>hardware_interface/EffortJointInterface</hardwareInterface>
-            </joint>
-            <actuator name="${name}_leg_motor_2">
-                <hardwareInterface>hardware_interface/EffortJointInterface</hardwareInterface>
-                <mechanicalReduction>1</mechanicalReduction>
-            </actuator>
-        </transmission>
-        <transmission name="${name}_leg_motor_3">
-            <type>transmission_interface/SimpleTransmission</type>
-            <joint name="${name}_leg_motor_3">
-                <hardwareInterface>hardware_interface/EffortJointInterface</hardwareInterface>
-            </joint>
-            <actuator name="${name}_leg_motor_3">
-                <hardwareInterface>hardware_interface/EffortJointInterface</hardwareInterface>
-                <mechanicalReduction>1</mechanicalReduction>
-            </actuator>
-        </transmission>
-        <transmission name="${name}_leg_motor_4">
-            <type>transmission_interface/SimpleTransmission</type>
-            <joint name="${name}_leg_motor_4">
-                <hardwareInterface>hardware_interface/EffortJointInterface</hardwareInterface>
-            </joint>
-            <actuator name="${name}_leg_motor_4">
-                <hardwareInterface>hardware_interface/EffortJointInterface</hardwareInterface>
-                <mechanicalReduction>1</mechanicalReduction>
-            </actuator>
-        </transmission>
-        <transmission name="${name}_leg_motor_5">
-            <type>transmission_interface/SimpleTransmission</type>
-            <joint name="${name}_leg_motor_5">
-                <hardwareInterface>hardware_interface/EffortJointInterface</hardwareInterface>
-            </joint>
-            <actuator name="${name}_leg_motor_5">
+        <transmission name="${name}_hip_yaw">
+            <type>transmission_interface/SimpleTransmission</type>
+            <joint name="${name}_hip_yaw">
+                <hardwareInterface>hardware_interface/EffortJointInterface</hardwareInterface>
+            </joint>
+            <actuator name="${name}_hip_yaw">
+                <hardwareInterface>hardware_interface/EffortJointInterface</hardwareInterface>
+                <mechanicalReduction>1</mechanicalReduction>
+            </actuator>
+        </transmission>
+        <transmission name="${name}_hip_roll">
+            <type>transmission_interface/SimpleTransmission</type>
+            <joint name="${name}_hip_roll">
+                <hardwareInterface>hardware_interface/EffortJointInterface</hardwareInterface>
+            </joint>
+            <actuator name="${name}_hip_roll">
+                <hardwareInterface>hardware_interface/EffortJointInterface</hardwareInterface>
+                <mechanicalReduction>1</mechanicalReduction>
+            </actuator>
+        </transmission>
+        <transmission name="${name}_hip_pitch">
+            <type>transmission_interface/SimpleTransmission</type>
+            <joint name="${name}_hip_pitch">
+                <hardwareInterface>hardware_interface/EffortJointInterface</hardwareInterface>
+            </joint>
+            <actuator name="${name}_hip_pitch">
+                <hardwareInterface>hardware_interface/EffortJointInterface</hardwareInterface>
+                <mechanicalReduction>1</mechanicalReduction>
+            </actuator>
+        </transmission>
+        <transmission name="${name}_knee">
+            <type>transmission_interface/SimpleTransmission</type>
+            <joint name="${name}_knee">
+                <hardwareInterface>hardware_interface/EffortJointInterface</hardwareInterface>
+            </joint>
+            <actuator name="${name}_knee">
+                <hardwareInterface>hardware_interface/EffortJointInterface</hardwareInterface>
+                <mechanicalReduction>1</mechanicalReduction>
+            </actuator>
+        </transmission>
+        <transmission name="${name}_ankle_pitch">
+            <type>transmission_interface/SimpleTransmission</type>
+            <joint name="${name}_ankle_pitch">
+                <hardwareInterface>hardware_interface/EffortJointInterface</hardwareInterface>
+            </joint>
+            <actuator name="${name}_ankle_pitch">
+                <hardwareInterface>hardware_interface/EffortJointInterface</hardwareInterface>
+                <mechanicalReduction>1</mechanicalReduction>
+            </actuator>
+        </transmission>
+        <transmission name="${name}_ankle_roll">
+            <type>transmission_interface/SimpleTransmission</type>
+            <joint name="${name}_ankle_roll">
+                <hardwareInterface>hardware_interface/EffortJointInterface</hardwareInterface>
+            </joint>
+            <actuator name="${name}_ankle_roll">
                 <hardwareInterface>hardware_interface/EffortJointInterface</hardwareInterface>
                 <mechanicalReduction>1</mechanicalReduction>

File: soccer_description/bez2_description/urdf/robot.urdf (robot description, URDF)
Before this commit: robot bez2, 22 links, 21 joints
Joints:
- joint left_ankle_roll: origin xyz=-0.0645 -0.0235 -0.036 rpy=0 0 0 -> xyz=0 -0.025 0  rpy=0 0 0
- joint right_ankle_roll: origin xyz=-0.0645 -0.0235 -0.036 rpy=0 0 0 -> xyz=0 -0.025 0 rpy=0 0 0
