Commit message: removed old walk engine and replaced with placo. reworked the ros layer and removed redundent parameter sharing. General clean up. Got walking loop to work from same code regardless of sim or ros. Fixed parameters and general plumbing. removed sigmanban and other description stuff to make it nicer. Fixed bez2 xacro and some improvements to firmware interface tests. should be ready to go.

File: soccer_description/bez1_description/urdf/robot.urdf (robot description, URDF)
Before this commit: robot bez1, 20 links, 19 joints
Links:
- link /head: geometry collision box size=0.0712 0.094 0.0779; visual mesh filename=../meshes/head.stl scale=1.0 1.0 1.0
- link /left_ankle: geometry collision box size=0.090769 0.042 0.0506; visual mesh filename=../meshes/left_ankle.stl scale=1.0 1.0 1.0
- link /left_bicep: geometry collision box size=0.04 0.04776 0.123; visual mesh filename=../meshes/left_bicep.stl scale=1.0 1.0 1.0
- link /left_calve: geometry collision box size=0.031883 0.048 0.105683; visual mesh filename=../meshes/left_calve.stl scale=1.0 1.0 1.0
- link /left_forearm: geometry collision box size=0.035 0.049 0.144; visual mesh filename=../meshes/left_forearm.stl scale=1.0 1.0 1.0
- link /left_hip_front: geometry collision box size=0.083747 0.04885 0.0506; visual mesh filename=../meshes/left_hip_front.stl scale=1.0 1.0 1.0
- link /left_hip_side: geometry collision box size=0.0485 0.022 0.0039; visual mesh filename=../meshes/left_hip_side.stl scale=1.0 1.0 1.0
- link /left_thigh: geometry collision box size=0.022 0.048 0.111; visual mesh filename=../meshes/left_thigh.stl scale=1.0 1.0 1.0
- link /right_ankle: geometry collision box size=0.090769 0.042 0.0506; visual mesh filename=../meshes/right_ankle.stl scale=1.0 1.0 1.0
- link /right_bicep: geometry collision box size=0.04 0.04776 0.123; visual mesh filename=../meshes/right_bicep.stl scale=1.0 1.0 1.0
- link /right_calve: geometry collision box size=0.031883 0.048 0.105683; visual mesh filename=../meshes/right_calve.stl scale=1.0 1.0 1.0
- link /right_forearm: geometry collision box size=0.035 0.049 0.144; visual mesh filename=../meshes/right_forearm.stl scale=1.0 1.0 1.0
- link /right_hip_front: geometry collision box size=0.083747 0.04885 0.0506; visual mesh filename=../meshes/right_hip_front.stl scale=1.0 1.0 1.0
- link /right_hip_side: geometry collision box size=0.0485 0.022 0.0039; visual mesh filename=../meshes/right_hip_side.stl scale=1.0 1.0 1.0
- link /right_thigh: geometry collision box size=0.022 0.048 0.111; visual mesh filename=../meshes/right_thigh.stl scale=1.0 1.0 1.0
- link head_base: geometry collision box size=0.022 0.0523 0.033; visual mesh filename=../meshes/neck.stl scale=1.0 1.0 1.0
- link left_foot: geometry collision box size=0.09 0.07 0.03674; visual mesh filename=../meshes/left_foot.stl scale=1.0 1.0 1.0
- link right_foot: geometry collision box size=0.09 0.07 0.03674; visual mesh filename=../meshes/right_foot.stl scale=1.0 1.0 1.0
- link trunk: geometry collision box size=0.13 0.145 0.152; visual mesh filename=../meshes/torso.stl scale=1.0 1.0 1.0

File: soccer_description/bez2_description/urdf/bez2.xacro (robot description, xacro)
@@ -5,5 +5,5 @@
 <xacro:include filename="$(find bez2_description)/urdf/bez2.trans" />
 <xacro:include filename="$(find bez2_description)/urdf/bez2.gazebo" />
-<link name="torso">
+<link name="trunk">
   <inertial>
     <origin xyz="-2.6182166493521018e-05 0.0037391632790891283 -0.07310917852477573" rpy="0 0 0"/>
@@ -425,5 +425,5 @@
   </collision>
 </link>
-<joint name="head_motor_0" type="revolute">
+<joint name="head_yaw" type="revolute">
   <origin xyz="0.009539 0.002537 0.03138" rpy="0 0 0"/>
   <parent link="torso"/>
@@ -433,5 +433,5 @@
           <limit effort="${XL430_TORQUE}" lower="-${PI/2}" upper="${PI/2}" velocity="${XL430_VELOCITY}"/>
 </joint>
-<joint name="head_motor_1" type="revolute">
+<joint name="head_pitch" type="revolute">
   <origin xyz="0.0 -0.0195 0.025" rpy="0 0 0"/>
   <parent link="neck"/>
@@ -441,5 +441,5 @@
             <limit effort="${XL430_TORQUE}" lower="0" upper="${PI*2/4}" velocity="${XL430_VELOCITY}"/>
 </joint>
-<joint name="left_arm_motor_0" type="revolute">
+<joint name="left_shoulder_pitch" type="revolute">
   <origin xyz="0.006539 0.112237 -0.00062" rpy="0 0 0"/>
   <parent link="torso"/>
@@ -449,5 +449,5 @@
 <limit effort="${XM430_TORQUE}" lower="-${PI}" upper="${PI*5/4}" velocity="${XM430_VELOCITY}"/>
 </joint>
-<joint name="left_arm_motor_1" type="revolute">
+<joint name="left_shoulder_roll" type="revolute">
   <origin xyz="0.0205 0.0295 -0.021" rpy="0 0 0"/>
   <parent link="left_shoulder"/>
@@ -457,5 +457,5 @@
                 <limit effort="${MX28_TORQUE}" lower="0" upper="${PI/2}" velocity="${MX28_VELOCITY}"/>
 </joint>
-<joint name="left_arm_motor_2" type="revolute">
+<joint name="left_elbow" type="revolute">
 <origin xyz="-0.018688 0.021938 -0.08675" rpy="0 0 0"/>
 <parent link="left_bicep"/>
@@ -465,5 +465,5 @@
               <limit effort="${MX28_TORQUE}" lower="0" upper="${PI}" velocity="${MX28_VELOCITY}"/>
 </joint>
-<joint name="left_leg_motor_0" type="revolute">
+<joint name="left_hip_yaw" type="revolute">
 <origin xyz="0.018839 0.067737 -0.20662" rpy="0 0 0"/>
 <parent link="torso"/>
@@ -473,5 +473,5 @@
 <limit effort="${XM430_TORQUE}" lower="-1.309" upper="0.524" velocity="${XM430_VELOCITY}"/>
 </joint>
-<joint name="left_leg_motor_1" type="revolute">
+<joint name="left_hip_roll" type="revolute">
 <origin xyz="-0.0205 0.0 -0.028" rpy="0 0 0"/>
 <parent link="left_hip_side"/>
@@ -481,5 +481,5 @@
           <limit effort="${XM430_TORQUE}" lower="-${PI/4}" upper="${PI/2}" velocity="${XM430_VELOCITY}"/>
 </joint>
-<joint name="left_leg_motor_2" type="revolute">
+<joint name="left_hip_pitch" type="revolute">
 <origin xyz="0.020771 0.0203 0.0" rpy="0 0 0"/>
 <parent link="left_hip_front"/>
@@ -489,5 +489,5 @@
             <limit effort="${XM430_TORQUE}" lower="-${PI/4}" upper="${PI*3/4}" velocity="${XM430_VELOCITY}"/>
 </joint>
-<joint name="left_leg_motor_3" type="revolute">
+<joint name="left_knee" type="revolute">
   <origin xyz="0.0 0.005269 -0.116" rpy="0 0 0"/>
   <parent link="left_thigh"/>
@@ -497,5 +497,5 @@
             <limit effort="${MX64_TORQUE}" lower="-2.793" upper="0" velocity="${MX64_VELOCITY}"/>
 </joint>
-<joint name="left_leg_motor_4" type="revolute">
+<joint name="left_ankle_pitch" type="revolute">
   <origin xyz="0.0013 0.0 -0.088" rpy="0 0 0"/>
   <parent link="left_calve"/>
@@ -505,5 +505,5 @@
             <limit effort="${MX64_TORQUE}" lower="-${PI/4}" upper="${PI/2}" velocity="${MX64_VELOCITY}"/>
 </joint>
-<joint name="left_leg_motor_5" type="revolute">
+<joint name="left_ankle_roll" type="revolute">
 <origin xyz="-0.0645 -0.0235 -0.036" rpy="0 0 0"/>
 <parent link="left_ankle"/>
@@ -513,5 +513,5 @@
             <limit effort="${MX64_TORQUE}" lower="-${PI/4}" upper="${PI/4}" velocity="${MX64_VELOCITY}"/>
 </joint>
-<joint name="right_arm_motor_0" type="revolute">
+<joint name="right_shoulder_pitch" type="revolute">
   <origin xyz="0.006539 -0.107163 -0.00062" rpy="0 0 0"/>
   <parent link="torso"/>
@@ -521,5 +521,5 @@
               <limit effort="${XM430_TORQUE}" lower="-${PI}" upper="${PI*5/4}" velocity="${XM430_VELOCITY}"/>
 </joint>
-<joint name="right_arm_motor_1" type="revolute">
+<joint name="right_shoulder_roll" type="revolute">
   <origin xyz="0.021 -0.0295 -0.021" rpy="0 0 0"/>
   <parent link="right_shoulder"/>
@@ -529,5 +529,5 @@
                 <limit effort="${MX28_TORQUE}" lower="0" upper="${PI/2}" velocity="${MX28_VELOCITY}"/>
 </joint>
-<joint name="right_arm_motor_2" type="revolute">
+<joint name="right_elbow" type="revolute">
   <origin xyz="-0.021312 -0.021937 -0.08675" rpy="0 0 0"/>
   <parent link="right_bicep"/>
@@ -537,5 +537,5 @@
                 <limit effort="${MX28_TORQUE}" lower="0" upper="${PI}" velocity="${MX28_VELOCITY}"/>
 </joint>
-<joint name="right_leg_motor_0" type="revolute">
+<joint name="right_hip_yaw" type="revolute">
   <origin xyz="0.018839 -0.062663 -0.20662" rpy="0 0 0"/>
   <parent link="torso"/>
@@ -545,5 +545,5 @@
   <limit effort="${XM430_TORQUE}" lower="-1.309" upper="0.524" velocity="${XM430_VELOCITY}"/>
 </joint>
-<joint name="right_leg_motor_1" type="revolute">
+<joint name="right_hip_roll" type="revolute">
   <origin xyz="-0.0205 0.0 -0.028" rpy="0 0 0"/>
   <parent link="right_hip_side"/>
@@ -553,5 +553,5 @@
             <limit effort="${XM430_TORQUE}" lower="-${PI/4}" upper="${PI/2}" velocity="${XM430_VELOCITY}"/>
 </joint>
-<joint name="right_leg_motor_2" type="revolute">
+<joint name="right_hip_pitch" type="revolute">
   <origin xyz="0.020771 0.0203 0.0" rpy="0 0 0"/>
   <parent link="right_hip_front"/>
@@ -561,5 +561,5 @@
             <limit effort="${XM430_TORQUE}" lower="-${PI/4}" upper="${PI*3/4}" velocity="${XM430_VELOCITY}"/>
 </joint>
-<joint name="right_leg_motor_3" type="revolute">
+<joint name="right_knee" type="revolute">
   <origin xyz="0.0 0.005269 -0.116" rpy="0 0 0"/>
   <parent link="right_thigh"/>
@@ -569,5 +569,5 @@
             <limit effort="${MX64_TORQUE}" lower="-2.793" upper="0" velocity="${MX64_VELOCITY}"/>
 </joint>
-<joint name="right_leg_motor_4" type="revolute">
+<joint name="right_ankle_pitch" type="revolute">
   <origin xyz="0.0013 0.0 -0.088" rpy="0 0 0"/>
   <parent link="right_calve"/>
@@ -577,5 +577,5 @@
             <limit effort="${MX64_TORQUE}" lower="-${PI/4}" upper="${PI/2}" velocity="${MX64_VELOCITY}"/>
 </joint>
-<joint name="right_leg_motor_5" type="revolute">
+<joint name="right_ankle_roll" type="revolute">
   <origin xyz="-0.0645 -0.0235 -0.036" rpy="0 0 0"/>
   <parent link="right_ankle"/>
