Commit message: added box collisions and fixed motor problem due to improper static and damping

File: soccer_description/bez1_description/urdf/bez1.urdf (robot description, URDF)
Before this commit: robot bez1, 20 links, 19 joints
Links:
- link /head: geometry collision box size=0.0712 0.094 0.0779; visual mesh filename=package://bez1_description/meshes/head.dae scale=1 1 1
- link /left_ankle: geometry collision box size=0.090769 0.042 0.0506; visual mesh filename=package://bez1_description/meshes/left_ankle.dae scale=1 1 1
- link /left_bicep: geometry collision box size=0.04 0.04776 0.123; visual mesh filename=package://bez1_description/meshes/left_bicep.dae scale=1 1 1
- link /left_calve: geometry collision box size=0.031883 0.048 0.105683; visual mesh filename=package://bez1_description/meshes/left_calve.dae scale=1 1 1
- link /left_foot: geometry collision box size=0.09 0.07 0.03674; visual mesh filename=package://bez1_description/meshes/left_foot.dae scale=1 1 1
- link /left_forearm: geometry collision box size=0.035 0.049 0.144; visual mesh filename=package://bez1_description/meshes/left_forearm.dae scale=1 1 1
- link /left_hip_front: geometry collision box size=0.083747 0.04885 0.0506; visual mesh filename=package://bez1_description/meshes/left_hip_front.dae scale=1 1 1
- link /left_hip_side: geometry collision box size=0.0485 0.022 0.0039; visual mesh filename=package://bez1_description/meshes/left_hip_side.dae scale=1 1 1
- link /left_thigh: geometry collision box size=0.022 0.048 0.111; visual mesh filename=package://bez1_description/meshes/left_thigh.dae scale=1 1 1
- link /neck: geometry collision box size=0.022 0.0523 0.033; visual mesh filename=package://bez1_description/meshes/neck.dae scale=1 1 1
- link /right_ankle: geometry collision box size=0.090769 0.042 0.0506; visual mesh filename=package://bez1_description/meshes/right_ankle.dae scale=1 1 1
- link /right_bicep: geometry collision box size=0.04 0.04776 0.123; visual mesh filename=package://bez1_description/meshes/right_bicep.dae scale=1 1 1
- link /right_calve: geometry collision box size=0.031883 0.048 0.105683; visual mesh filename=package://bez1_description/meshes/right_calve.dae scale=1 1 1
- link /right_foot: geometry collision box size=0.09 0.07 0.03674; visual mesh filename=package://bez1_description/meshes/right_foot.dae scale=1 1 1
- link /right_forearm: geometry collision box size=0.035 0.049 0.144; visual mesh filename=package://bez1_description/meshes/right_forearm.dae scale=1 1 1
- link /right_hip_front: geometry collision box size=0.083747 0.04885 0.0506; visual mesh filename=package://bez1_description/meshes/right_hip_front.dae scale=1 1 1
- link /right_hip_side: geometry collision box size=0.0485 0.022 0.0039; visual mesh filename=package://bez1_description/meshes/right_hip_side.dae scale=1 1 1
- link /right_thigh: geometry collision box size=0.022 0.048 0.111; visual mesh filename=package://bez1_description/meshes/right_thigh.dae scale=1 1 1
- link /torso: geometry collision box size=0.130 0.145 0.152; visual mesh filename=package://bez1_description/meshes/torso.dae scale=1 1 1

File: soccer_description/bez2_urdf_description/urdf/bez2_urdf.urdf (robot description, URDF)
Before this commit: robot bez2_urdf, 22 links, 21 joints
Links:
- link head: geometry collision box size=0.07120 0.09400 0.07530; visual mesh filename=package://bez2_urdf_description/meshes/Head_Pitch_Assembly_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 scale=0.001 0.001 0.001
- link left_ankle: geometry collision box size=0.08910 0.05000 0.06398; visual mesh filename=package://bez2_urdf_description/meshes/ankle_v2_1.stl scale=0.001 0.001 0.001
- link left_bicep: geometry collision box size=0.05000 0.04703 0.11202; visual mesh filename=package://bez2_urdf_description/meshes/bicep_v1_1.stl scale=0.001 0.001 0.001
- link left_calve: geometry collision box size=0.04030 0.05350 0.10500; visual mesh filename=package://bez2_urdf_description/meshes/calf_v1_1.stl scale=0.001 0.001 0.001
- link left_foot: geometry collision box size=0.17000 0.09000 0.03300; visual mesh filename=package://bez2_urdf_description/meshes/left_foot_v2_1.stl scale=0.001 0.001 0.001
- link left_forearm: geometry collision box size=0.04800 0.05300 0.18838; visual mesh filename=package://bez2_urdf_description/meshes/Bez1_forearm_v7_1.stl scale=0.001 0.001 0.001
- link left_hip_front: geometry collision box size=0.07402 0.04100 0.04650; visual mesh filename=package://bez2_urdf_description/meshes/hip_v1_1.stl scale=0.001 0.001 0.001
- link left_hip_side: geometry collision box size=0.04100 0.02400 0.03050; visual mesh filename=package://bez2_urdf_description/meshes/fr12_h101_v1_2.stl scale=0.001 0.001 0.001
- link left_shoulder: geometry collision box size=0.04360 0.04730 0.05100; visual mesh filename=package://bez2_urdf_description/meshes/left_shoulder_v1_1.s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 scale=0.001 0.001 0.001
- link left_thigh: geometry collision box size=0.03300 0.05100 0.12150; visual mesh filename=package://bez2_urdf_description/meshes/thigh_v1_1.stl scale=0.001 0.001 0.001
- link neck: geometry collision box size=0.02200 0.05100 0.03800; visual mesh filename=package://bez2_urdf_description/meshes/Head_Yaw_Assembly_v1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 scale=0.001 0.001 0.001
- link right_ankle: geometry collision box size=0.08910 0.05000 0.06398; visual mesh filename=package://bez2_urdf_description/meshes/ankle_v2_2.stl scale=0.001 0.001 0.001
- link right_bicep: geometry collision box size=0.05000 0.04703 0.11202; visual mesh filename=package://bez2_urdf_description/meshes/bicep_v1_2.stl scale=0.001 0.001 0.001
- link right_calve: geometry collision box size=0.04030 0.05350 0.10500; visual mesh filename=package://bez2_urdf_description/meshes/calf_v1_2.stl scale=0.001 0.001 0.001
- link right_foot: geometry collision box size=0.17000 0.09000 0.03300; visual mesh filename=package://bez2_urdf_description/meshes/right_foot_v2_1.stl scale=0.001 0.001 0.001
- link right_forearm: geometry collision box size=0.04800 0.05300 0.18838; visual mesh filename=package://bez2_urdf_description/meshes/Bez1_forearm_v7_2.stl scale=0.001 0.001 0.001
- link right_hip_front: geometry collision box size=0.07402 0.04100 0.04650; visual mesh filename=package://bez2_urdf_description/meshes/hip_v1_2.stl scale=0.001 0.001 0.001
- link right_hip_side: geometry collision box size=0.04100 0.02400 0.03050; visual mesh filename=package://bez2_urdf_description/meshes/fr12_h101_v1_1.stl scale=0.001 0.001 0.001
- link right_shoulder: geometry collision box size=0.04435 0.04730 0.05100; visual mesh filename=package://bez2_urdf_description/meshes/right_shoulder_v2_1.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 scale=0.001 0.001 0.001
- link right_thigh: geometry collision box size=0.03300 0.05100 0.12150; visual mesh filename=package://bez2_urdf_description/meshes/thigh_v1_2.stl scale=0.001 0.001 0.001
- link torso: geometry collision box size=0.14440 0.20843 0.19912; visual mesh filename=package://bez2_urdf_description/meshes/base_link.stl scale=0.001 0.001 0.001

File: soccer_description/bez2_urdf_description/urdf/bez2_urdf.xacro (robot description, xacro)
@@ -18,9 +18,9 @@
     <material name="steel_satin"/>
   </visual>
-  <collision>
-    <origin xyz="0 0 0" rpy="0 0 0"/>
-    <geometry>
-      <mesh filename="package://bez2_urdf_description/meshes/base_link.stl" scale="0.001 0.001 0.001"/>
-    </geometry>
+  <collision name="collision">
+      <origin rpy="0.00000 0.00000 0.00000" xyz="0.00154 0.00254 -0.07057"/>
+      <geometry>
+        <box size="0.14440 0.20843 0.19912"/>
+      </geometry>
   </collision>
 </link>
@@ -39,8 +39,8 @@
   </visual>
   <collision>
-    <origin xyz="-0.009539 -0.002537 -0.03138" rpy="0 0 0"/>
-    <geometry>
-      <mesh filename="package://bez2_urdf_description/meshes/Head_Yaw_Assembly_v1_1.stl" scale="0.001 0.001 0.001"/>
-    </geometry>
+    <origin rpy="0.00000 0.00000 0.00000" xyz="0.00000 0.00000 0.01900"/>
+      <geometry>
+        <box size="0.02200 0.05100 0.03800"/>
+      </geometry>
   </collision>
 </link>
@@ -59,8 +59,8 @@
   </visual>
   <collision>
-    <origin xyz="-0.009539 0.016963 -0.05638" rpy="0 0 0"/>
-    <geometry>
-      <mesh filename="package://bez2_urdf_description/meshes/Head_Pitch_Assembly_v4_1.stl" scale="0.001 0.001 0.001"/>
-    </geometry>
+    <origin rpy="0.00000 0.00000 0.00000" xyz="-0.00950 0.01920 0.02340"/>
+      <geometry>
+        <box size="0.07120 0.09400 0.07530"/>
+      </geometry>
   </collision>
 </link>
@@ -79,8 +79,8 @@
   </visual>
   <collision>
-    <origin xyz="-0.006539 -0.112237 0.00062" rpy="0 0 0"/>
-    <geometry>
-      <mesh filename="package://bez2_urdf_description/meshes/left_shoulder_v1_1.stl" scale="0.001 0.001 0.001"/>
-    </geometry>
+    <origin rpy="0.00000 0.00000 0.00000" xyz="0.00155 0.02365 -0.00750"/>
+      <geometry>
+        <box size="0.04360 0.04730 0.05100"/>
+      </geometry>
   </collision>
 </link>
@@ -99,8 +99,8 @@
   </visual>
   <collision>
-    <origin xyz="-0.027039 -0.141737 0.02162" rpy="0 0 0"/>
-    <geometry>
-      <mesh filename="package://bez2_urdf_description/meshes/bicep_v1_1.stl" scale="0.001 0.001 0.001"/>
-    </geometry>
+    <origin rpy="0.00000 0.00000 0.00000" xyz="-0.02000 0.00127 -0.04274"/>
+      <geometry>
+        <box size="0.05000 0.04703 0.11202"/>
+      </geometry>
   </collision>
 </link>
@@ -119,8 +119,8 @@
   </visual>
   <collision>
-    <origin xyz="-0.008351 -0.163675 0.10837" rpy="0 0 0"/>
-    <geometry>
-      <mesh filename="package://bez2_urdf_description/meshes/Bez1_forearm_v7_1.stl" scale="0.001 0.001 0.001"/>
-    </geometry>
+    <origin rpy="0.00000 0.00000 0.00000" xyz="-0.01200 -0.02050 -0.08119"/>
+      <geometry>
+        <box size="0.04800 0.05300 0.18838"/>
+      </geometry>
   </collision>
 </link>
@@ -139,8 +139,8 @@
   </visual>
   <collision>
-    <origin xyz="-0.018839 -0.067737 0.20662" rpy="0 0 0"/>
-    <geometry>
-      <mesh filename="package://bez2_urdf_description/meshes/fr12_h101_v1_2.stl" scale="0.001 0.001 0.001"/>
-    </geometry>
+    <origin rpy="0.00000 0.00000 0.00000" xyz="0.00000 0.00000 -0.01525"/>
+      <geometry>
+        <box size="0.04100 0.02400 0.03050"/>
+      </geometry>
   </collision>
 </link>
@@ -159,8 +159,8 @@
 </visual>
 <collision>
-  <origin xyz="0.001661 -0.067737 0.23462" rpy="0 0 0"/>
-  <geometry>
-    <mesh filename="package://bez2_urdf_description/meshes/hip_v1_1.stl" scale="0.001 0.001 0.001"/>
-  </geometry>
+  <origin rpy="0.00000 0.00000 0.00000" xyz="-0.00199 0.00180 -0.01200"/>
+      <geometry>
+        <box size="0.07402 0.04100 0.04650"/>
+      </geometry>
 </collision>
 </link>
@@ -179,8 +179,8 @@
   </visual>
   <collision>
-    <origin xyz="-0.01911 -0.088037 0.23462" rpy="0 0 0"/>
-    <geometry>
-      <mesh filename="package://bez2_urdf_description/meshes/thigh_v1_1.stl" scale="0.001 0.001 0.001"/>
-    </geometry>
+    <origin rpy="0.00000 0.00000 0.00000" xyz="0.00000 -0.01823 -0.05825"/>
+      <geometry>
+        <box size="0.03300 0.05100 0.12150"/>
+      </geometry>
   </collision>
 </link>
@@ -199,8 +199,8 @@
   </visual>
   <collision>
-    <origin xyz="-0.01911 -0.093306 0.35062" rpy="0 0 0"/>
-    <geometry>
-      <mesh filename="package://bez2_urdf_description/meshes/calf_v1_1.stl" scale="0.001 0.001 0.001"/>
-    </geometry>
+    <origin rpy="0.00000 0.00000 0.00000" xyz="-0.00005 -0.02225 -0.03850"/>
+      <geometry>
+        <box size="0.04030 0.05350 0.10500"/>
+      </geometry>
   </collision>
 </link>
@@ -219,8 +219,8 @@
   </visual>
   <collision>
-    <origin xyz="-0.02041 -0.093306 0.43862" rpy="0 0 0"/>
-    <geometry>
-      <mesh filename="package://bez2_urdf_description/meshes/ankle_v2_1.stl" scale="0.001 0.001 0.001"/>
-    </geometry>
+    <origin rpy="0.00000 0.00000 0.00000" xyz="-0.02445 -0.02050 -0.01800"/>
+      <geometry>
+        <box size="0.08910 0.05000 0.06398"/>
+      </geometry>
   </collision>
 </link>
@@ -239,8 +239,8 @@
   </visual>
   <collision>
-    <origin xyz="0.04409 -0.069806 0.47462" rpy="0 0 0"/>
-    <geometry>
-      <mesh filename="package://bez2_urdf_description/meshes/left_foot_v2_1.stl" scale="0.001 0.001 0.001"/>
-    </geometry>
+    <origin rpy="0.00000 0.00000 0.00000" xyz="0.05150 0.01936 -0.00550"/>
+      <geometry>
+        <box size="0.17000 0.09000 0.03300"/>
+      </geometry>
   </collision>
 </link>
@@ -259,8 +259,8 @@
   </visual>
   <collision>
-    <origin xyz="-0.018839 0.062663 0.20662" rpy="0 0 0"/>
-    <geometry>
-      <mesh filename="package://bez2_urdf_description/meshes/fr12_h101_v1_1.stl" scale="0.001 0.001 0.001"/>
-    </geometry>
+    <origin rpy="0.00000 0.00000 0.00000" xyz="0.00000 0.00000 -0.01525"/>
+      <geometry>
+        <box size="0.04100 0.02400 0.03050"/>
+      </geometry>
   </collision>
 </link>
@@ -279,8 +279,8 @@
   </visual>
   <collision>
-    <origin xyz="0.001661 0.062663 0.23462" rpy="0 0 0"/>
-    <geometry>
-      <mesh filename="package://bez2_urdf_description/meshes/hip_v1_2.stl" scale="0.001 0.001 0.001"/>
-    </geometry>
+    <origin rpy="0.00000 0.00000 0.00000" xyz="-0.00199 0.00180 -0.01200"/>
+      <geometry>
+        <box size="0.07402 0.04100 0.04650"/>
+      </geometry>
   </collision>
 </link>
@@ -299,8 +299,8 @@
   </visual>
   <collision>
-    <origin xyz="-0.01911 0.042363 0.23462" rpy="0 0 0"/>
-    <geometry>
-      <mesh filename="package://bez2_urdf_description/meshes/thigh_v1_2.stl" scale="0.001 0.001 0.001"/>
-    </geometry>
+    <origin rpy="0.00000 0.00000 0.00000" xyz="0.00000 -0.01823 -0.05825"/>
+      <geometry>
+        <box size="0.03300 0.05100 0.12150"/>
+      </geometry>
   </collision>
 </link>
@@ -319,8 +319,8 @@
   </visual>
   <collision>
-    <origin xyz="-0.01911 0.037094 0.35062" rpy="0 0 0"/>
-    <geometry>
-      <mesh filename="package://bez2_urdf_description/meshes/calf_v1_2.stl" scale="0.001 0.001 0.001"/>
-    </geometry>
+    <origin rpy="0.00000 0.00000 0.00000" xyz="-0.00005 -0.02225 -0.03850"/>
+      <geometry>
+        <box size="0.04030 0.05350 0.10500"/>
+      </geometry>
   </collision>
 </link>
@@ -339,8 +339,8 @@
   </visual>
   <collision>
-    <origin xyz="-0.02041 0.037094 0.43862" rpy="0 0 0"/>
-    <geometry>
-      <mesh filename="package://bez2_urdf_description/meshes/ankle_v2_2.stl" scale="0.001 0.001 0.001"/>
-    </geometry>
+    <origin rpy="0.00000 0.00000 0.00000" xyz="-0.02445 -0.02050 -0.01800"/>
+      <geometry>
+        <box size="0.08910 0.05000 0.06398"/>
+      </geometry>
   </collision>
 </link>
@@ -359,8 +359,8 @@
   </visual>
   <collision>
-    <origin xyz="0.04409 0.060594 0.47462" rpy="0 0 0"/>
-    <geometry>
-      <mesh filename="package://bez2_urdf_description/meshes/right_foot_v2_1.stl" scale="0.001 0.001 0.001"/>
-    </geometry>
+    <origin rpy="0.00000 0.00000 0.00000" xyz="0.05150 -0.01936 -0.00550"/>
+      <geometry>
+        <box size="0.17000 0.09000 0.03300"/>
+      </geometry>
   </collision>
 </link>
@@ -379,8 +379,8 @@
   </visual>
   <collision>
-    <origin xyz="-0.006539 0.107163 0.00062" rpy="0 0 0"/>
-    <geometry>
-      <mesh filename="package://bez2_urdf_description/meshes/right_shoulder_v2_1.stl" scale="0.001 0.001 0.001"/>
-    </geometry>
+    <origin rpy="0.00000 0.00000 0.00000" xyz="0.00168 -0.02365 -0.00750"/>
+      <geometry>
+        <box size="0.04435 0.04730 0.05100"/>
+      </geometry>
   </collision>
 </link>
@@ -399,8 +399,8 @@
   </visual>
   <collision>
-    <origin xyz="-0.027539 0.136663 0.02162" rpy="0 0 0"/>
-    <geometry>
-      <mesh filename="package://bez2_urdf_description/meshes/bicep_v1_2.stl" scale="0.001 0.001 0.001"/>
-    </geometry>
+    <origin rpy="0.00000 0.00000 0.00000" xyz="-0.02000 -0.00127 -0.04274"/>
+      <geometry>
+        <box size="0.05000 0.04703 0.11202"/>
+      </geometry>
   </collision>
 </link>
@@ -419,8 +419,8 @@
   </visual>
   <collision>
-    <origin xyz="-0.006227 0.1586 0.10837" rpy="0 0 0"/>
-    <geometry>
-      <mesh filename="package://bez2_urdf_description/meshes/Bez1_forearm_v7_2.stl" scale="0.001 0.001 0.001"/>
-    </geometry>
+    <origin rpy="0.00000 0.00000 0.00000" xyz="-0.01200 0.02050 -0.08119"/>
+      <geometry>
+        <box size="0.04800 0.05300 0.18838"/>
+      </geometry>
   </collision>
 </link>

File: soccer_description/bez2_urdf_description/urdf/parameters.xacro (robot description, xacro)
@@ -9,20 +9,21 @@
     <xacro:property name="JOINT_FRICTION" value="0.1"/>
     <xacro:property name="JOINT_DAMPING" value="0.01"/>
+<!--TODO figure out why damping and friction mess with it so much-->
     <xacro:property name="MX28_TORQUE" value="2.5"/>
     <xacro:property name="MX28_VELOCITY" value="5.76"/>
-    <xacro:property name="MX28_DAMPING" value="0.3"/>
-    <xacro:property name="MX28_FRICTION" value="0.83"/>
+    <xacro:property name="MX28_DAMPING" value="${JOINT_DAMPING}"/>
+    <xacro:property name="MX28_FRICTION" value="${JOINT_FRICTION}"/>
     <xacro:property name="MX64_TORQUE" value="6.0"/>
     <xacro:property name="MX64_VELOCITY" value="6.6"/>
-    <xacro:property name="MX64_DAMPING" value="0.66"/>
-    <xacro:property name="MX64_FRICTION" value="1.42"/>
+    <xacro:property name="MX64_DAMPING" value="${JOINT_DAMPING}"/>
+    <xacro:property name="MX64_FRICTION" value="${JOINT_FRICTION}"/>
     <xacro:property name="XM430_TORQUE" value="4.1"/>
     <xacro:property name="XM430_VELOCITY" value="4.82"/>
-    <xacro:property name="XM430_DAMPING" value="0.721165"/>
-    <xacro:property name="XM430_FRICTION" value="0.721165"/>
+    <xacro:property name="XM430_DAMPING" value="${JOINT_DAMPING}"/>
+    <xacro:property name="XM430_FRICTION" value="${JOINT_FRICTION}"/>
     <xacro:property name="XL430_TORQUE" value="1.5"/>
     <xacro:property name="XL430_VELOCITY" value="6.39"/>
-    <xacro:property name="XL430_DAMPING" value="0.16"/>
-    <xacro:property name="XL430_FRICTION" value="0.6"/>
+    <xacro:property name="XL430_DAMPING" value="${JOINT_DAMPING}"/>
+    <xacro:property name="XL430_FRICTION" value="${JOINT_FRICTION}"/>
     <xacro:property name="y_offset" value="0.21571129429326383"/>
     <xacro:property name="z_offset" value="0.05556097822952673"/>

Commit message: fixing merge issues

File: soccer_description/bez1_description/urdf/bez1.urdf (robot description, URDF)
Before this commit: robot bez1, 20 links, 19 joints
Links:
- link /head: geometry collision box size=0.0712 0.094 0.0779; visual mesh filename=package://bez1_description/meshes/head.dae scale=1 1 1
- link /left_ankle: geometry collision box size=0.090769 0.042 0.0506; visual mesh filename=package://bez1_description/meshes/left_ankle.dae scale=1 1 1
- link /left_bicep: geometry collision box size=0.04 0.04776 0.123; visual mesh filename=package://bez1_description/meshes/left_bicep.dae scale=1 1 1
- link /left_calve: geometry collision box size=0.031883 0.048 0.105683; visual mesh filename=package://bez1_description/meshes/left_calve.dae scale=1 1 1
- link /left_foot: geometry collision box size=0.09 0.07 0.03674; visual mesh filename=package://bez1_description/meshes/left_foot.dae scale=1 1 1
- link /left_forearm: geometry collision box size=0.035 0.049 0.144; visual mesh filename=package://bez1_description/meshes/left_forearm.dae scale=1 1 1
- link /left_hip_front: geometry collision box size=0.083747 0.04885 0.0506; visual mesh filename=package://bez1_description/meshes/left_hip_front.dae scale=1 1 1
- link /left_hip_side: geometry collision box size=0.0485 0.022 0.0039; visual mesh filename=package://bez1_description/meshes/left_hip_side.dae scale=1 1 1
- link /left_thigh: geometry collision box size=0.022 0.048 0.111; visual mesh filename=package://bez1_description/meshes/left_thigh.dae scale=1 1 1
- link /neck: geometry collision box size=0.022 0.0523 0.033; visual mesh filename=package://bez1_description/meshes/neck.dae scale=1 1 1
- link /right_ankle: geometry collision box size=0.090769 0.042 0.0506; visual mesh filename=package://bez1_description/meshes/right_ankle.dae scale=1 1 1
- link /right_bicep: geometry collision box size=0.04 0.04776 0.123; visual mesh filename=package://bez1_description/meshes/right_bicep.dae scale=1 1 1
- link /right_calve: geometry collision box size=0.031883 0.048 0.105683; visual mesh filename=package://bez1_description/meshes/right_calve.dae scale=1 1 1
- link /right_foot: geometry collision box size=0.09 0.07 0.03674; visual mesh filename=package://bez1_description/meshes/right_foot.dae scale=1 1 1
- link /right_forearm: geometry collision box size=0.035 0.049 0.144; visual mesh filename=package://bez1_description/meshes/right_forearm.dae scale=1 1 1
- link /right_hip_front: geometry collision box size=0.083747 0.04885 0.0506; visual mesh filename=package://bez1_description/meshes/right_hip_front.dae scale=1 1 1
- link /right_hip_side: geometry collision box size=0.0485 0.022 0.0039; visual mesh filename=package://bez1_description/meshes/right_hip_side.dae scale=1 1 1
- link /right_thigh: geometry collision box size=0.022 0.048 0.111; visual mesh filename=package://bez1_description/meshes/right_thigh.dae scale=1 1 1
- link /torso: geometry collision box size=0.130 0.145 0.152; visual mesh filename=package://bez1_description/meshes/torso.dae scale=1 1 1
