Commit message: working on adding placo as the main walk engine

File: soccer_description/bez1_description/urdf/bez1.urdf (robot description, URDF)
Before this commit: robot bez1, 19 links, 18 joints
Links:
- added link /imu_link, mass 0.01
Joints:
- added joint /torso_imu: type fixed, parent /torso, child /imu_link, origin xyz=0.0 0 0.000 rpy=0 0 0, axis 0 0 0
- joint head_pitch: limit lower=-2.356194490192345 upper=2.356194490192345 effort=1.5 velocity=1 -> lower=-2.356194490192345 upper=2.356194490192345 effort=1.5 velocity=5.76
- joint head_yaw: limit lower=-1.5707963267948966 upper=1.5707963267948966 effort=1.5 velocity=1 -> lower=-1.5707963267948966 upper=1.5707963267948966 effort=1.5 velocity=5.76
- joint left_ankle_pitch: limit lower=-0.7853981633974483 upper=1.5707963267948966 effort=2.5 velocity=1 -> lower=-0.7853981633974483 upper=1.5707963267948966 effort=2.5 velocity=5.76
- joint left_ankle_roll: limit lower=-0.7853981633974483 upper=0.7853981633974483 effort=2.5 velocity=1 -> lower=-0.7853981633974483 upper=0.7853981633974483 effort=2.5 velocity=5.76
- joint left_elbow: limit lower=0 upper=3.141592653589793 effort=1.5 velocity=1 -> lower=0 upper=3.141592653589793 effort=1.5 velocity=5.76
- joint left_hip_pitch: limit lower=-0.7853981633974483 upper=2.356194490192345 effort=2.5 velocity=1 -> lower=-0.7853981633974483 upper=2.356194490192345 effort=2.5 velocity=5.76
- joint left_hip_roll: limit lower=-0.7853981633974483 upper=1.5707963267948966 effort=2.5 velocity=1 -> lower=-0.7853981633974483 upper=1.5707963267948966 effort=2.5 velocity=5.76
- joint left_hip_yaw: limit lower=-1.309 upper=0.524 effort=2.5 velocity=1 -> lower=-1.309 upper=0.524 effort=2.5 velocity=5.76
- joint left_knee: limit lower=-2.793 upper=0 effort=2.5 velocity=1 -> lower=-2.793 upper=0 effort=2.5 velocity=5.76
- joint left_shoulder_pitch: limit lower=-1.5707963267948966 upper=3.9269908169872414 effort=1.5 velocity=1 -> lower=-1.5707963267948966 upper=3.9269908169872414 effort=1.5 velocity=5.76
- joint right_ankle_pitch: limit lower=-0.7853981633974483 upper=1.5707963267948966 effort=2.5 velocity=1 -> lower=-0.7853981633974483 upper=1.5707963267948966 effort=2.5 velocity=5.76
- joint right_ankle_roll: limit lower=-0.7853981633974483 upper=0.7853981633974483 effort=2.5 velocity=1 -> lower=-0.7853981633974483 upper=0.7853981633974483 effort=2.5 velocity=5.76
- joint right_elbow: limit lower=0 upper=3.141592653589793 effort=1.5 velocity=1 -> lower=0 upper=3.141592653589793 effort=1.5 velocity=5.76
- joint right_hip_pitch: limit lower=-0.7853981633974483 upper=2.356194490192345 effort=2.5 velocity=1 -> lower=-0.7853981633974483 upper=2.356194490192345 effort=2.5 velocity=5.76
- joint right_hip_roll: limit lower=-0.7853981633974483 upper=1.5707963267948966 effort=2.5 velocity=1 -> lower=-0.7853981633974483 upper=1.5707963267948966 effort=2.5 velocity=5.76
- joint right_hip_yaw: limit lower=-1.309 upper=0.524 effort=2.5 velocity=1 -> lower=-1.309 upper=0.524 effort=2.5 velocity=5.76
- joint right_knee: limit lower=-2.793 upper=0 effort=2.5 velocity=1 -> lower=-2.793 upper=0 effort=2.5 velocity=5.76
- joint right_shoulder_pitch: limit lower=-1.5707963267948966 upper=3.9269908169872414 effort=1.5 velocity=1 -> lower=-1.5707963267948966 upper=3.9269908169872414 effort=1.5 velocity=5.76

File: soccer_description/bez1_description/urdf/robot.urdf (robot description, URDF)
Before this commit: robot bez1, 20 links, 19 joints
Joints:
- joint head_pitch: limit lower=-2.356194490192345 upper=2.356194490192345 effort=1.5 velocity=1.0 -> lower=-2.356194490192345 upper=2.356194490192345 effort=1.5 velocity=5.76
- joint head_yaw: limit lower=-1.5707963267948966 upper=1.5707963267948966 effort=1.5 velocity=1.0 -> lower=-1.5707963267948966 upper=1.5707963267948966 effort=1.5 velocity=5.76
- joint left_ankle_pitch: limit lower=-0.7853981633974483 upper=1.5707963267948966 effort=2.5 velocity=1.0 -> lower=-0.7853981633974483 upper=1.5707963267948966 effort=2.5 velocity=5.76
- joint left_ankle_roll: limit lower=-0.7853981633974483 upper=0.7853981633974483 effort=2.5 velocity=1.0 -> lower=-0.7853981633974483 upper=0.7853981633974483 effort=2.5 velocity=5.76
- joint left_elbow: limit lower=0.0 upper=3.141592653589793 effort=1.5 velocity=1.0 -> lower=0.0 upper=3.141592653589793 effort=1.5 velocity=5.76
- joint left_hip_pitch: limit lower=-0.7853981633974483 upper=2.356194490192345 effort=2.5 velocity=1.0 -> lower=-0.7853981633974483 upper=2.356194490192345 effort=2.5 velocity=5.76
- joint left_hip_roll: limit lower=-0.7853981633974483 upper=1.5707963267948966 effort=2.5 velocity=1.0 -> lower=-0.7853981633974483 upper=1.5707963267948966 effort=2.5 velocity=5.76
- joint left_hip_yaw: limit lower=-1.309 upper=0.524 effort=2.5 velocity=1.0 -> lower=-1.309 upper=0.524 effort=2.5 velocity=5.76
- joint left_knee: limit lower=-2.793 upper=0.0 effort=2.5 velocity=1.0 -> lower=-2.793 upper=0.0 effort=2.5 velocity=5.76
- joint left_shoulder_pitch: limit lower=-1.5707963267948966 upper=3.9269908169872414 effort=1.5 velocity=1.0 -> lower=-1.5707963267948966 upper=3.9269908169872414 effort=1.5 velocity=5.76
- joint right_ankle_pitch: limit lower=-0.7853981633974483 upper=1.5707963267948966 effort=2.5 velocity=1.0 -> lower=-0.7853981633974483 upper=1.5707963267948966 effort=2.5 velocity=5.76
- joint right_ankle_roll: limit lower=-0.7853981633974483 upper=0.7853981633974483 effort=2.5 velocity=1.0 -> lower=-0.7853981633974483 upper=0.7853981633974483 effort=2.5 velocity=5.76
- joint right_elbow: limit lower=0.0 upper=3.141592653589793 effort=1.5 velocity=1.0 -> lower=0.0 upper=3.141592653589793 effort=1.5 velocity=5.76
- joint right_hip_pitch: limit lower=-0.7853981633974483 upper=2.356194490192345 effort=2.5 velocity=1.0 -> lower=-0.7853981633974483 upper=2.356194490192345 effort=2.5 velocity=5.76
- joint right_hip_roll: limit lower=-0.7853981633974483 upper=1.5707963267948966 effort=2.5 velocity=1.0 -> lower=-0.7853981633974483 upper=1.5707963267948966 effort=2.5 velocity=5.76
- joint right_hip_yaw: limit lower=-1.309 upper=0.524 effort=2.5 velocity=1.0 -> lower=-1.309 upper=0.524 effort=2.5 velocity=5.76
- joint right_knee: limit lower=-2.793 upper=0.0 effort=2.5 velocity=1.0 -> lower=-2.793 upper=0.0 effort=2.5 velocity=5.76
- joint right_shoulder_pitch: limit lower=-1.5707963267948966 upper=3.9269908169872414 effort=1.5 velocity=1.0 -> lower=-1.5707963267948966 upper=3.9269908169872414 effort=1.5 velocity=5.76

File: soccer_description/bez2_description/urdf/robot.urdf (robot description, URDF)
Before this commit: robot bez2, 23 links, 22 joints
Links:
- removed link torso
- removed link torso_cylinder
- added link trunk, mass 1.62191101903404; collision box size=0.14440 0.20843 0.19912; visual mesh filename=/home/jonathan/catkin_ws/src/soccerbot/soccer_description/b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 scale=0.001 0.001 0.001
- link head: geometry collision box size=0.07120 0.09400 0.07530; visual mesh filename=/home/jonathan/catkin_ws/src/soccerbot/soccer_description/b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 scale=0.001 0.001 0.001
- link left_ankle: geometry collision box size=0.08910 0.05000 0.06398; visual mesh filename=/home/jonathan/catkin_ws/src/soccerbot/soccer_description/b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 scale=0.001 0.001 0.001
- link left_bicep: geometry collision box size=0.05000 0.04703 0.11202; visual mesh filename=/home/jonathan/catkin_ws/src/soccerbot/soccer_description/b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 scale=0.001 0.001 0.001
- link left_calve: geometry collision box size=0.04030 0.05350 0.10500; visual mesh filename=/home/jonathan/catkin_ws/src/soccerbot/soccer_description/b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 scale=0.001 0.001 0.001
- link left_foot: geometry collision box size=0.17000 0.09000 0.03300; visual mesh filename=/home/jonathan/catkin_ws/src/soccerbot/soccer_description/b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 scale=0.001 0.001 0.001
- link left_forearm: geometry collision box size=0.04800 0.05300 0.18838; visual mesh filename=/home/jonathan/catkin_ws/src/soccerbot/soccer_description/b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 scale=0.001 0.001 0.001
- link left_hip_front: geometry collision box size=0.07402 0.04100 0.04650; visual mesh filename=/home/jonathan/catkin_ws/src/soccerbot/soccer_description/b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 scale=0.001 0.001 0.001
- link left_hip_side: geometry collision box size=0.04100 0.02400 0.03050; visual mesh filename=/home/jonathan/catkin_ws/src/soccerbot/soccer_description/b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 scale=0.001 0.001 0.001
- link left_shoulder: geometry collision box size=0.04360 0.04730 0.05100; visual mesh filename=/home/jonathan/catkin_ws/src/soccerbot/soccer_description/b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 scale=0.001 0.001 0.001
- link left_thigh: geometry collision box size=0.03300 0.05100 0.12150; visual mesh filename=/home/jonathan/catkin_ws/src/soccerbot/soccer_description/b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 scale=0.001 0.001 0.001
- link neck: geometry collision box size=0.02200 0.05100 0.03800; visual mesh filename=/home/jonathan/catkin_ws/src/soccerbot/soccer_description/b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 scale=0.001 0.001 0.001
- link right_ankle: geometry collision box size=0.08910 0.05000 0.06398; visual mesh filename=/home/jonathan/catkin_ws/src/soccerbot/soccer_description/b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 scale=0.001 0.001 0.001
- link right_bicep: geometry collision box size=0.05000 0.04703 0.11202; visual mesh filename=/home/jonathan/catkin_ws/src/soccerbot/soccer_description/b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 scale=0.001 0.001 0.001
- link right_calve: geometry collision box size=0.04030 0.05350 0.10500; visual mesh filename=/home/jonathan/catkin_ws/src/soccerbot/soccer_description/b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 scale=0.001 0.001 0.001
- link right_foot: geometry collision box size=0.17000 0.09000 0.03300; visual mesh filename=/home/jonathan/catkin_ws/src/soccerbot/soccer_description/b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 scale=0.001 0.001 0.001
- link right_forearm: geometry collision box size=0.04800 0.05300 0.18838; visual mesh filename=/home/jonathan/catkin_ws/src/soccerbot/soccer_description/b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 scale=0.001 0.001 0.001
- link right_hip_front: geometry collision box size=0.07402 0.04100 0.04650; visual mesh filename=/home/jonathan/catkin_ws/src/soccerbot/soccer_description/b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 scale=0.001 0.001 0.001
- link right_hip_side: geometry collision box size=0.04100 0.02400 0.03050; visual mesh filename=/home/jonathan/catkin_ws/src/soccerbot/soccer_description/b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 scale=0.001 0.001 0.001
- link right_shoulder: geometry collision box size=0.04435 0.04730 0.05100; visual mesh filename=/home/jonathan/catkin_ws/src/soccerbot/soccer_description/b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 scale=0.001 0.001 0.001
- link right_thigh: geometry collision box size=0.03300 0.05100 0.12150; visual mesh filename=/home/jonathan/catkin_ws/src/soccerbot/soccer_description/b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 scale=0.001 0.001 0.001
Joints:
- removed joint torso_cylinder_joint
- joint head_yaw: parent torso -> trunk
- joint left_hip_yaw: parent torso -> trunk
- joint left_shoulder_pitch: parent torso -> trunk
- joint right_hip_yaw: parent torso -> trunk
- joint right_shoulder_pitch: parent torso -> trunk
- joint torso_imu: parent torso -> trunk

Commit message: Js placo (#879)
* moved localization and firmware into folders where they belong. playing with order of folders. added an ros example that makes sense for camera. setting up a ros example that makes sense with walk but the ros layer needs some work

* experimenting with placo

* working on adding placo as the main walk engine

* Fixed someproblems in the webots bridge and urdf/xacro. integrated placo as a walk engine alternative

* added a rough draft of ros layer for placo and it works great out of the box

* removed old walk engine and replaced with placo. reworked the ros layer and removed redundent parameter sharing. General clean up. Got walking loop to work from same code regardless of sim or ros. Fixed parameters and general plumbing. removed sigmanban and other description stuff to make it nicer. Fixed bez2 xacro and some improvements to firmware interface tests. should be ready to go.

File: soccer_description/bez1_description/urdf/bez1.urdf (robot description, URDF)
Before this commit: robot bez1, 20 links, 19 joints
Joints:
- removed joint head_motor_0
- removed joint head_motor_1
- removed joint left_arm_motor_0
- removed joint left_arm_motor_1
- removed joint left_leg_motor_0
- removed joint left_leg_motor_1
- removed joint left_leg_motor_2
- removed joint left_leg_motor_3
- removed joint left_leg_motor_4
- removed joint left_leg_motor_5
- removed joint right_arm_motor_0
- removed joint right_arm_motor_1
- removed joint right_leg_motor_0
- removed joint right_leg_motor_1
- removed joint right_leg_motor_2
- removed joint right_leg_motor_3
- removed joint right_leg_motor_4
- removed joint right_leg_motor_5
- added joint head_pitch: type revolute, parent /neck, child /head, origin xyz=0 0 0.024 rpy=0 0 0, axis 0 1 0, limit lower=-2.356194490192345 upper=2.356194490192345 effort=1.5 velocity=5.76
- added joint head_yaw: type revolute, parent /torso, child /neck, origin xyz=0.024 0 0.05875 rpy=0 0 0, axis 0 0 1, limit lower=-1.5707963267948966 upper=1.5707963267948966 effort=1.5 velocity=5.76
- added joint left_ankle_pitch: type revolute, parent /left_calve, child /left_ankle, origin xyz=0 0 -0.0827 rpy=0 0 0, axis 0 -1 0, limit lower=-0.7853981633974483 upper=1.5707963267948966 effort=2.5 velocity=5.76
- added joint left_ankle_roll: type revolute, parent /left_ankle, child /left_foot, origin xyz=0 0 0 rpy=0 0 0, axis 1 0 0, limit lower=-0.7853981633974483 upper=0.7853981633974483 effort=2.5 velocity=5.76
- added joint left_elbow: type revolute, parent /left_bicep, child /left_forearm, origin xyz=0 0 -0.10 rpy=0 0 0, axis 0 -1 0, limit lower=0 upper=3.141592653589793 effort=1.5 velocity=5.76
- added joint left_hip_pitch: type revolute, parent /left_hip_front, child /left_thigh, origin xyz=0 0 0 rpy=0 0 0, axis 0 -1 0, limit lower=-0.7853981633974483 upper=2.356194490192345 effort=2.5 velocity=5.76
- added joint left_hip_roll: type revolute, parent /left_hip_side, child /left_hip_front, origin xyz=0 0 0 rpy=0 0 0, axis 1 0 0, limit lower=-0.7853981633974483 upper=1.5707963267948966 effort=2.5 velocity=5.76
- added joint left_hip_yaw: type revolute, parent /torso, child /left_hip_side, origin xyz=0.0135 0.035 -0.156 rpy=0 0 0, axis 0 0 -1, limit lower=-1.309 upper=0.524 effort=2.5 velocity=5.76
- added joint left_knee: type revolute, parent /left_thigh, child /left_calve, origin xyz=0 0 -0.0890 rpy=0 0 0, axis 0 -1 0, limit lower=-2.793 upper=0 effort=2.5 velocity=5.76
- added joint left_shoulder_pitch: type revolute, parent /torso, child /left_bicep, origin xyz=-0.0157 0.0725 0 rpy=0 0 0, axis 0 -1 0, limit lower=-1.5707963267948966 upper=3.9269908169872414 effort=1.5 velocity=5.76
- added joint right_ankle_pitch: type revolute, parent /right_calve, child /right_ankle, origin xyz=0 0 -0.0827 rpy=0 0 0, axis 0 -1 0, limit lower=-0.7853981633974483 upper=1.5707963267948966 effort=2.5 velocity=5.76
- added joint right_ankle_roll: type revolute, parent /right_ankle, child /right_foot, origin xyz=0 0 0 rpy=0 0 0, axis -1 0 0, limit lower=-0.7853981633974483 upper=0.7853981633974483 effort=2.5 velocity=5.76
- added joint right_elbow: type revolute, parent /right_bicep, child /right_forearm, origin xyz=0 0 -0.10 rpy=0 0 0, axis 0 -1 0, limit lower=0 upper=3.141592653589793 effort=1.5 velocity=5.76
- added joint right_hip_pitch: type revolute, parent /right_hip_front, child /right_thigh, origin xyz=0 0 0 rpy=0 0 0, axis 0 -1 0, limit lower=-0.7853981633974483 upper=2.356194490192345 effort=2.5 velocity=5.76
- added joint right_hip_roll: type revolute, parent /right_hip_side, child /right_hip_front, origin xyz=0 0 0 rpy=0 0 0, axis -1 0 0, limit lower=-0.7853981633974483 upper=1.5707963267948966 effort=2.5 velocity=5.76
- added joint right_hip_yaw: type revolute, parent /torso, child /right_hip_side, origin xyz=0.0135 -0.035 -0.156 rpy=0 0 0, axis 0 0 1, limit lower=-1.309 upper=0.524 effort=2.5 velocity=5.76
- added joint right_knee: type revolute, parent /right_thigh, child /right_calve, origin xyz=0 0 -0.0890 rpy=0 0 0, axis 0 -1 0, limit lower=-2.793 upper=0 effort=2.5 velocity=5.76
- added joint right_shoulder_pitch: type revolute, parent /torso, child /right_bicep, origin xyz=-0.0157 -0.0725 0 rpy=0 0 0, axis 0 -1 0, limit lower=-1.5707963267948966 upper=3.9269908169872414 effort=1.5 velocity=5.76

File: soccer_description/bez2_description/urdf/bez2.urdf (robot description, URDF)
Before this commit: robot bez2, 23 links, 22 joints
Joints:
- removed joint head_motor_0
- removed joint head_motor_1
- removed joint left_arm_motor_0
- removed joint left_arm_motor_1
- removed joint left_arm_motor_2
- removed joint left_leg_motor_0
- removed joint left_leg_motor_1
- removed joint left_leg_motor_2
- removed joint left_leg_motor_3
- removed joint left_leg_motor_4
- removed joint left_leg_motor_5
- removed joint right_arm_motor_0
- removed joint right_arm_motor_1
- removed joint right_arm_motor_2
- removed joint right_leg_motor_0
- removed joint right_leg_motor_1
- removed joint right_leg_motor_2
- removed joint right_leg_motor_3
- removed joint right_leg_motor_4
- removed joint right_leg_motor_5
- added joint head_pitch: type revolute, parent neck, child head, origin xyz=0.0 -0.0195 0.025 rpy=0 0 0, axis 0.0 1.0 0.0, limit lower=0 upper=1.5707963267948966 effort=1.5 velocity=6.39
- added joint head_yaw: type revolute, parent torso, child neck, origin xyz=0.009539 0.002537 0.03138 rpy=0 0 0, axis 0.0 0.0 -1.0, limit lower=-1.5707963267948966 upper=1.5707963267948966 effort=1.5 velocity=6.39
- added joint left_ankle_pitch: type revolute, parent left_calve, child left_ankle, origin xyz=0.0013 0.0 -0.088 rpy=0 0 0, axis -0.0 -1.0 0.0, limit lower=-0.7853981633974483 upper=1.5707963267948966 effort=6.0 velocity=6.6
- added joint left_ankle_roll: type revolute, parent left_ankle, child left_foot, origin xyz=-0.0645 -0.0235 -0.036 rpy=0 0 0, axis 1.0 0.0 0.0, limit lower=-0.7853981633974483 upper=0.7853981633974483 effort=6.0 velocity=6.6
- added joint left_elbow: type revolute, parent left_bicep, child left_forearm, origin xyz=-0.018688 0.021938 -0.08675 rpy=0 0 0, axis -0.0 -1.0 -0.0, limit lower=0 upper=3.141592653589793 effort=2.5 velocity=5.76
- added joint left_hip_pitch: type revolute, parent left_hip_front, child left_thigh, origin xyz=0.020771 0.0203 0.0 rpy=0 0 0, axis -0.0 -1.0 0.0, limit lower=-0.7853981633974483 upper=2.356194490192345 effort=4.1 velocity=4.82
- added joint left_hip_roll: type revolute, parent left_hip_side, child left_hip_front, origin xyz=-0.0205 0.0 -0.028 rpy=0 0 0, axis 1.0 0.0 0.0, limit lower=-0.7853981633974483 upper=1.5707963267948966 effort=4.1 velocity=4.82
- added joint left_hip_yaw: type revolute, parent torso, child left_hip_side, origin xyz=0.018839 0.067737 -0.20662 rpy=0 0 0, axis 0.0 0.0 -1.0, limit lower=-1.309 upper=0.524 effort=4.1 velocity=4.82
- added joint left_knee: type revolute, parent left_thigh, child left_calve, origin xyz=0.0 0.005269 -0.116 rpy=0 0 0, axis -0.0 -1.0 0.0, limit lower=-2.793 upper=0 effort=6.0 velocity=6.6
- added joint left_shoulder_pitch: type revolute, parent torso, child left_shoulder, origin xyz=0.006539 0.112237 -0.00062 rpy=0 0 0, axis -0.0 -1.0 0.0, limit lower=-3.141592653589793 upper=3.9269908169872414 effort=4.1 velocity=4.82
- added joint left_shoulder_roll: type revolute, parent left_shoulder, child left_bicep, origin xyz=0.0205 0.0295 -0.021 rpy=0 0 0, axis 1.0 -0.0 0.0, limit lower=0 upper=1.5707963267948966 effort=2.5 velocity=5.76
- added joint right_ankle_pitch: type revolute, parent right_calve, child right_ankle, origin xyz=0.0013 0.0 -0.088 rpy=0 0 0, axis -0.0 -1.0 0.0, limit lower=-0.7853981633974483 upper=1.5707963267948966 effort=6.0 velocity=6.6
- added joint right_ankle_roll: type revolute, parent right_ankle, child right_foot, origin xyz=-0.0645 -0.0235 -0.036 rpy=0 0 0, axis -1.0 0.0 0.0, limit lower=-0.7853981633974483 upper=0.7853981633974483 effort=6.0 velocity=6.6
- added joint right_elbow: type revolute, parent right_bicep, child right_forearm, origin xyz=-0.021312 -0.021937 -0.08675 rpy=0 0 0, axis 0.0 -1.0 0.0, limit lower=0 upper=3.141592653589793 effort=2.5 velocity=5.76
- added joint right_hip_pitch: type revolute, parent right_hip_front, child right_thigh, origin xyz=0.020771 0.0203 0.0 rpy=0 0 0, axis -0.0 -1.0 0.0, limit lower=-0.7853981633974483 upper=2.356194490192345 effort=4.1 velocity=4.82
- added joint right_hip_roll: type revolute, parent right_hip_side, child right_hip_front, origin xyz=-0.0205 0.0 -0.028 rpy=0 0 0, axis -1.0 0.0 0.0, limit lower=-0.7853981633974483 upper=1.5707963267948966 effort=4.1 velocity=4.82
- added joint right_hip_yaw: type revolute, parent torso, child right_hip_side, origin xyz=0.018839 -0.062663 -0.20662 rpy=0 0 0, axis -0.0 -0.0 1.0, limit lower=-1.309 upper=0.524 effort=4.1 velocity=4.82
- added joint right_knee: type revolute, parent right_thigh, child right_calve, origin xyz=0.0 0.005269 -0.116 rpy=0 0 0, axis -0.0 -1.0 0.0, limit lower=-2.793 upper=0 effort=6.0 velocity=6.6
- added joint right_shoulder_pitch: type revolute, parent torso, child right_shoulder, origin xyz=0.006539 -0.107163 -0.00062 rpy=0 0 0, axis 0.0 -1.0 -0.0, limit lower=-3.141592653589793 upper=3.9269908169872414 effort=4.1 velocity=4.82
- added joint right_shoulder_roll: type revolute, parent right_shoulder, child right_bicep, origin xyz=0.021 -0.0295 -0.021 rpy=0 0 0, axis -1.0 0.0 0.0, limit lower=0 upper=1.5707963267948966 effort=2.5 velocity=5.76
