Commit message: Started rough drafts of flowcharts. Found issue with bez2 and will wait till new version is done. Removed pybullet as engine to calculate kinematic data and switched to using pinnocio to be more light weight and modular. Removed ik_data and replaced with kinematic data to group all common data . cleaned up handle_urdf and merged set_pose into it and renamed it. Cleaned up IK moving functions around to make more sense based on how they are used. General clean up and renaming. Got test_ik to work with refactor and ready & sweep in pybullet to work.

File: soccer_description/bez2_description/urdf/bez2.urdf (robot description, URDF)
Before this commit: robot bez2, 21 links, 20 joints
Links:
- removed link Arm_Assembly-bez3_v12_2
- removed link base_link
- removed link biceps_v3_1
- removed link imu_1
- added link /imu_link, mass 0.0005024000000000008; collision mesh filename=../bez2_description/meshes/imu_1.stl scale=1 1 1; visual mesh filename=../bez2_description/meshes/imu_1.stl scale=1 1 1
- added link /left_bicep, mass 0.25825416029102555; collision mesh filename=../bez2_description/meshes/biceps_v3_1.stl scale=1 1 1; visual mesh filename=../bez2_description/meshes/biceps_v3_1.stl scale=1 1 1
- added link /left_forearm, mass 0.32110352957731503; collision mesh filename=../bez2_description/meshes/Arm_Assembly-bez3_v12_2.stl scale=1 1 1; visual mesh filename=../bez2_description/meshes/Arm_Assembly-bez3_v12_2.stl scale=1 1 1
- added link /torso, mass 1.4940527908480117; collision mesh filename=../bez2_description/meshes/base_link.stl scale=1 1 1; visual mesh filename=../bez2_description/meshes/base_link.stl scale=1 1 1
- link Arm_Assembly-bez3_v12_1: geometry collision mesh filename=../bez2_description/meshes/Arm_Assembly-bez3_v12_1.stl scale=1 1 1; visual mesh filename=../bez2_description/meshes/Arm_Assembly-bez3_v12_1.stl scale=1 1 1
- link Hip_Printable_v2_v10_1: geometry collision mesh filename=../bez2_description/meshes/Hip_Printable_v2_v10_1.stl scale=1 1 1; visual mesh filename=../bez2_description/meshes/Hip_Printable_v2_v10_1.stl scale=1 1 1
- link Hip_Printable_v2_v10_2: geometry collision mesh filename=../bez2_description/meshes/Hip_Printable_v2_v10_2.stl scale=1 1 1; visual mesh filename=../bez2_description/meshes/Hip_Printable_v2_v10_2.stl scale=1 1 1
- link New_left_foot_upperhalf_v5_1: geometry collision mesh filename=../bez2_description/meshes/New_left_foot_upperhalf_v5_1.stl scale=1 1 1; visual mesh filename=../bez2_description/meshes/New_left_foot_upperhalf_v5_1.stl scale=1 1 1
- link New_right_foot_upperhalf_v3_1: geometry collision mesh filename=../bez2_description/meshes/New_right_foot_upperhalf_v3_1.stl scale=1 1 1; visual mesh filename=../bez2_description/meshes/New_right_foot_upperhalf_v3_1.stl scale=1 1 1
- link Upper_left_leg_support__bottom__v8_1: geometry collision mesh filename=../bez2_description/meshes/Upper_left_leg_support__bottom__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 scale=1 1 1; visual mesh filename=../bez2_description/meshes/Upper_left_leg_support__bottom__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 scale=1 1 1
- link Upper_left_leg_support__bottom__v8_2: geometry collision mesh filename=../bez2_description/meshes/Upper_left_leg_support__bottom__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 scale=1 1 1; visual mesh filename=../bez2_description/meshes/Upper_left_leg_support__bottom__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 scale=1 1 1
- link ankle_motors_v4_1: geometry collision mesh filename=../bez2_description/meshes/ankle_motors_v4_1.stl scale=1 1 1; visual mesh filename=../bez2_description/meshes/ankle_motors_v4_1.stl scale=1 1 1
- link ankle_motors_v4_2: geometry collision mesh filename=../bez2_description/meshes/ankle_motors_v4_2.stl scale=1 1 1; visual mesh filename=../bez2_description/meshes/ankle_motors_v4_2.stl scale=1 1 1
- link biceps_v3_2: geometry collision mesh filename=../bez2_description/meshes/biceps_v3_2.stl scale=1 1 1; visual mesh filename=../bez2_description/meshes/biceps_v3_2.stl scale=1 1 1
- link camera_point_1: geometry collision mesh filename=../bez2_description/meshes/camera_point_1.stl scale=1 1 1; visual mesh filename=../bez2_description/meshes/camera_point_1.stl scale=1 1 1
- link custom_servo_support__middle_neck__v9_1: geometry collision mesh filename=../bez2_description/meshes/custom_servo_support__middle_nec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 scale=1 1 1; visual mesh filename=../bez2_description/meshes/custom_servo_support__middle_nec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 scale=1 1 1
- link head_v4_1: geometry collision mesh filename=../bez2_description/meshes/head_v4_1.stl scale=1 1 1; visual mesh filename=../bez2_description/meshes/head_v4_1.stl scale=1 1 1
- link hip_motors_v4_1: geometry collision mesh filename=../bez2_description/meshes/hip_motors_v4_1.stl scale=1 1 1; visual mesh filename=../bez2_description/meshes/hip_motors_v4_1.stl scale=1 1 1
- link hip_motors_v4_2: geometry collision mesh filename=../bez2_description/meshes/hip_motors_v4_2.stl scale=1 1 1; visual mesh filename=../bez2_description/meshes/hip_motors_v4_2.stl scale=1 1 1
- link lower_leg_v4_1: geometry collision mesh filename=../bez2_description/meshes/lower_leg_v4_1.stl scale=1 1 1; visual mesh filename=../bez2_description/meshes/lower_leg_v4_1.stl scale=1 1 1
- link lower_leg_v4_2: geometry collision mesh filename=../bez2_description/meshes/lower_leg_v4_2.stl scale=1 1 1; visual mesh filename=../bez2_description/meshes/lower_leg_v4_2.stl scale=1 1 1
Joints:
- joint head_camera: type continuous -> fixed
- joint head_motor_0: parent base_link -> /torso
- joint left_arm_motor_0: child biceps_v3_1 -> /left_bicep; parent base_link -> /torso
- joint left_arm_motor_1: child Arm_Assembly-bez3_v12_2 -> /left_forearm; parent biceps_v3_1 -> /left_bicep
- joint left_leg_motor_0: parent base_link -> /torso
- joint right_arm_motor_0: parent base_link -> /torso
- joint right_leg_motor_0: parent base_link -> /torso
- joint torso_imu: child imu_1 -> /imu_link; parent base_link -> /torso; type continuous -> fixed

Commit message: renamed and got rid of unnessary desrciption packages

File: soccer_description/bez2_description/urdf/bez2.urdf (robot description, URDF)
Before this commit: robot bez2, 21 links, 20 joints
Links:
- removed link /imu_link
- removed link /left_bicep
- removed link /left_forearm
- removed link /torso
- removed link Arm_Assembly-bez3_v12_1
- removed link Hip_Printable_v2_v10_1
- removed link Hip_Printable_v2_v10_2
- removed link New_left_foot_upperhalf_v5_1
- removed link New_right_foot_upperhalf_v3_1
- removed link Upper_left_leg_support__bottom__v8_1
- removed link Upper_left_leg_support__bottom__v8_2
- removed link ankle_motors_v4_1
- removed link ankle_motors_v4_2
- removed link biceps_v3_2
- removed link camera_point_1
- removed link custom_servo_support__middle_neck__v9_1
- removed link head_v4_1
- removed link hip_motors_v4_1
- removed link hip_motors_v4_2
- removed link lower_leg_v4_1
- removed link lower_leg_v4_2
- added link head, mass 0.5407373847724953; collision box size=0.07120 0.09400 0.07530; visual mesh filename=package://bez2_description/meshes/Head_Pitch_Assembly_v4_1.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 scale=0.001 0.001 0.001
- added link imu_link, mass 0.01
- added link left_ankle, mass 0.26345509510176346; collision box size=0.08910 0.05000 0.06398; visual mesh filename=package://bez2_description/meshes/ankle_v2_1.stl scale=0.001 0.001 0.001
- added link left_bicep, mass 0.7365391814909177; collision box size=0.05000 0.04703 0.11202; visual mesh filename=package://bez2_description/meshes/bicep_v1_1.stl scale=0.001 0.001 0.001
- added link left_calve, mass 0.20304073544640247; collision box size=0.04030 0.05350 0.10500; visual mesh filename=package://bez2_description/meshes/calf_v1_1.stl scale=0.001 0.001 0.001
- added link left_foot, mass 0.37785469138016164; collision box size=0.17000 0.09000 0.03300; visual mesh filename=package://bez2_description/meshes/left_foot_v2_1.stl scale=0.001 0.001 0.001
- added link left_forearm, mass 0.06415483406403591; collision box size=0.04800 0.05300 0.18838; visual mesh filename=package://bez2_description/meshes/Bez1_forearm_v7_1.stl scale=0.001 0.001 0.001
- added link left_hip_front, mass 0.7328385746044006; collision box size=0.07402 0.04100 0.04650; visual mesh filename=package://bez2_description/meshes/hip_v1_1.stl scale=0.001 0.001 0.001
- added link left_hip_side, mass 0.023116469719045966; collision box size=0.04100 0.02400 0.03050; visual mesh filename=package://bez2_description/meshes/fr12_h101_v1_2.stl scale=0.001 0.001 0.001
- added link left_shoulder, mass 0.42869731083494267; collision box size=0.04360 0.04730 0.05100; visual mesh filename=package://bez2_description/meshes/left_shoulder_v1_1.stl scale=0.001 0.001 0.001
- added link left_thigh, mass 0.191955361852033; collision box size=0.03300 0.05100 0.12150; visual mesh filename=package://bez2_description/meshes/thigh_v1_1.stl scale=0.001 0.001 0.001
- added link neck, mass 0.015549664333897642; collision box size=0.02200 0.05100 0.03800; visual mesh filename=package://bez2_description/meshes/Head_Yaw_Assembly_v1_1.stl scale=0.001 0.001 0.001
- added link right_ankle, mass 0.26345509510176346; collision box size=0.08910 0.05000 0.06398; visual mesh filename=package://bez2_description/meshes/ankle_v2_2.stl scale=0.001 0.001 0.001
- added link right_bicep, mass 0.7365391814909177; collision box size=0.05000 0.04703 0.11202; visual mesh filename=package://bez2_description/meshes/bicep_v1_2.stl scale=0.001 0.001 0.001
- added link right_calve, mass 0.20304073544640247; collision box size=0.04030 0.05350 0.10500; visual mesh filename=package://bez2_description/meshes/calf_v1_2.stl scale=0.001 0.001 0.001
- added link right_foot, mass 0.37785469138016164; collision box size=0.17000 0.09000 0.03300; visual mesh filename=package://bez2_description/meshes/right_foot_v2_1.stl scale=0.001 0.001 0.001
- added link right_forearm, mass 0.06415483406403591; collision box size=0.04800 0.05300 0.18838; visual mesh filename=package://bez2_description/meshes/Bez1_forearm_v7_2.stl scale=0.001 0.001 0.001
- added link right_hip_front, mass 0.7328385746044006; collision box size=0.07402 0.04100 0.04650; visual mesh filename=package://bez2_description/meshes/hip_v1_2.stl scale=0.001 0.001 0.001
- added link right_hip_side, mass 0.023116469719045966; collision box size=0.04100 0.02400 0.03050; visual mesh filename=package://bez2_description/meshes/fr12_h101_v1_1.stl scale=0.001 0.001 0.001
- added link right_shoulder, mass 0.42869731083494267; collision box size=0.04435 0.04730 0.05100; visual mesh filename=package://bez2_description/meshes/right_shoulder_v2_1.stl scale=0.001 0.001 0.001
- added link right_thigh, mass 0.191955361852033; collision box size=0.03300 0.05100 0.12150; visual mesh filename=package://bez2_description/meshes/thigh_v1_2.stl scale=0.001 0.001 0.001
- added link torso, mass 1.621911019034044; collision box size=0.14440 0.20843 0.19912; visual mesh filename=package://bez2_description/meshes/base_link.stl scale=0.001 0.001 0.001
Joints:
- removed joint head_camera
- added joint left_arm_motor_2: type revolute, parent left_bicep, child left_forearm, origin xyz=-0.018688 0.021938 -0.08675 rpy=0 0 0, axis -0.0 -1.0 -0.0, limit lower=0 upper=3.141592653589793 effort=2.5 velocity=5.76
- added joint right_arm_motor_2: type revolute, parent right_bicep, child right_forearm, origin xyz=-0.021312 -0.021937 -0.08675 rpy=0 0 0, axis 0.0 -1.0 0.0, limit lower=0 upper=3.141592653589793 effort=2.5 velocity=5.76
- joint head_motor_0: child custom_servo_support__middle_neck__v9_1 -> neck; limit (none) -> lower=-1.5707963267948966 upper=1.5707963267948966 effort=1.5 velocity=6.39; origin xyz=0.03325 -0.000333 0.075624 rpy=0 0 0 -> xyz=0.009539 0.002537 0.03138 rpy=0 0 0; parent /torso -> torso; type continuous -> revolute
- joint head_motor_1: axis -0.0 1.0 0.0 -> 0.0 1.0 0.0; child head_v4_1 -> head; limit (none) -> lower=0 upper=1.5707963267948966 effort=1.5 velocity=6.39; origin xyz=0.0 -0.022187 0.033817 rpy=0 0 0 -> xyz=0.0 -0.0195 0.025 rpy=0 0 0; parent custom_servo_support__middle_neck__v9_1 -> neck; type continuous -> revolute
- joint left_arm_motor_0: child /left_bicep -> left_shoulder; limit (none) -> lower=-1.5707963267948966 upper=3.9269908169872414 effort=2.5 velocity=5.76; origin xyz=0.0 0.0725 0.00045 rpy=0 0 0 -> xyz=0.006539 0.112237 -0.00062 rpy=0 0 0; parent /torso -> torso; type continuous -> revolute
- joint left_arm_motor_1: axis 0.0 -1.0 0.0 -> 1.0 -0.0 0.0; child /left_forearm -> left_bicep; limit (none) -> lower=0 upper=1.5707963267948966 effort=2.5 velocity=5.76; origin xyz=0.0 0.008 -0.0906 rpy=0 0 0 -> xyz=0.0205 0.0295 -0.021 rpy=0 0 0; parent /left_bicep -> left_shoulder; type continuous -> revolute
- joint left_leg_motor_0: axis -0.0 0.0 -1.0 -> 0.0 0.0 1.0; child Hip_Printable_v2_v10_2 -> left_hip_side; limit (none) -> lower=-1.309 upper=0.524 effort=4.1 velocity=4.82; origin xyz=0.01597 0.0377 -0.14405 rpy=0 0 0 -> xyz=0.018839 0.067737 -0.20662 rpy=0 0 0; parent /torso -> torso; type continuous -> revolute
- joint left_leg_motor_1: axis 1.0 -0.0 -0.0 -> 1.0 0.0 0.0; child hip_motors_v4_2 -> left_hip_front; limit (none) -> lower=-0.7853981633974483 upper=1.5707963267948966 effort=4.1 velocity=4.82; origin xyz=-0.025 0.0 -0.032 rpy=0 0 0 -> xyz=-0.0205 0.0 -0.028 rpy=0 0 0; parent Hip_Printable_v2_v10_2 -> left_hip_side; type continuous -> revolute
- joint left_leg_motor_2: axis 0.0 -1.0 0.0 -> -0.0 -1.0 0.0; child Upper_left_leg_support__bottom__v8_1 -> left_thigh; limit (none) -> lower=-0.7853981633974483 upper=2.356194490192345 effort=4.1 velocity=4.82; origin xyz=0.02365 -0.02 0.0 rpy=0 0 0 -> xyz=0.020771 0.0203 0.0 rpy=0 0 0; parent hip_motors_v4_2 -> left_hip_front; type continuous -> revolute
- joint left_leg_motor_3: axis 0.0 -1.0 0.0 -> -0.0 -1.0 0.0; child lower_leg_v4_2 -> left_calve; limit (none) -> lower=-2.793 upper=0 effort=6.0 velocity=6.6; origin xyz=0.0 -0.0045 -0.0917 rpy=0 0 0 -> xyz=0.0 0.005269 -0.116 rpy=0 0 0; parent Upper_left_leg_support__bottom__v8_1 -> left_thigh; type continuous -> revolute
- joint left_leg_motor_4: axis 0.0 -1.0 0.0 -> -0.0 -1.0 0.0; child ankle_motors_v4_1 -> left_ankle; limit (none) -> lower=-0.7853981633974483 upper=1.5707963267948966 effort=6.0 velocity=6.6; origin xyz=0.0 -0.0005 -0.1083 rpy=0 0 0 -> xyz=0.0013 0.0 -0.088 rpy=0 0 0; parent lower_leg_v4_2 -> left_calve; type continuous -> revolute
- joint left_leg_motor_5: axis -1.0 0.0 0.0 -> 1.0 0.0 0.0; child New_right_foot_upperhalf_v3_1 -> left_foot; limit (none) -> lower=-0.7853981633974483 upper=0.7853981633974483 effort=6.0 velocity=6.6; origin xyz=-0.0843 0.0233 0.0 rpy=0 0 0 -> xyz=-0.0645 -0.0235 -0.036 rpy=0 0 0; parent ankle_motors_v4_1 -> left_ankle; type continuous -> revolute
- joint right_arm_motor_0: axis 0.0 -1.0 0.0 -> 0.0 -1.0 -0.0; child biceps_v3_2 -> right_shoulder; limit (none) -> lower=-1.5707963267948966 upper=3.9269908169872414 effort=2.5 velocity=5.76; origin xyz=0.0 -0.0725 0.00045 rpy=0 0 0 -> xyz=0.006539 -0.107163 -0.00062 rpy=0 0 0; parent /torso -> torso; type continuous -> revolute
- joint right_arm_motor_1: axis -0.0 -1.0 0.0 -> -1.0 0.0 0.0; child Arm_Assembly-bez3_v12_1 -> right_bicep; limit (none) -> lower=0 upper=1.5707963267948966 effort=2.5 velocity=5.76; origin xyz=-0.0 -0.008 -0.0906 rpy=0 0 0 -> xyz=0.021 -0.0295 -0.021 rpy=0 0 0; parent biceps_v3_2 -> right_shoulder; type continuous -> revolute
- joint right_leg_motor_0: axis -0.0 -0.0 1.0 -> -0.0 -0.0 -1.0; child Hip_Printable_v2_v10_1 -> right_hip_side; limit (none) -> lower=-1.309 upper=0.524 effort=4.1 velocity=4.82; origin xyz=0.01597 -0.0368 -0.14405 rpy=0 0 0 -> xyz=0.018839 -0.062663 -0.20662 rpy=0 0 0; parent /torso -> torso; type continuous -> revolute
- joint right_leg_motor_1: child hip_motors_v4_1 -> right_hip_front; limit (none) -> lower=-0.7853981633974483 upper=1.5707963267948966 effort=4.1 velocity=4.82; origin xyz=-0.0235 0.0 -0.032 rpy=0 0 0 -> xyz=-0.0205 0.0 -0.028 rpy=0 0 0; parent Hip_Printable_v2_v10_1 -> right_hip_side; type continuous -> revolute
- joint right_leg_motor_2: axis 0.0 -1.0 0.0 -> -0.0 -1.0 0.0; child Upper_left_leg_support__bottom__v8_2 -> right_thigh; limit (none) -> lower=-0.7853981633974483 upper=2.356194490192345 effort=4.1 velocity=4.82; origin xyz=0.02365 0.02 0.0 rpy=0 0 0 -> xyz=0.020771 0.0203 0.0 rpy=0 0 0; parent hip_motors_v4_1 -> right_hip_front; type continuous -> revolute
- joint right_leg_motor_3: axis 0.0 -1.0 0.0 -> -0.0 -1.0 0.0; child lower_leg_v4_1 -> right_calve; limit (none) -> lower=-2.793 upper=0 effort=6.0 velocity=6.6; origin xyz=0.0 0.0045 -0.0917 rpy=0 0 0 -> xyz=0.0 0.005269 -0.116 rpy=0 0 0; parent Upper_left_leg_support__bottom__v8_2 -> right_thigh; type continuous -> revolute
- joint right_leg_motor_4: axis 0.0 -1.0 0.0 -> -0.0 -1.0 0.0; child ankle_motors_v4_2 -> right_ankle; limit (none) -> lower=-0.7853981633974483 upper=1.5707963267948966 effort=6.0 velocity=6.6; origin xyz=0.0 0.0005 -0.1083 rpy=0 0 0 -> xyz=0.0013 0.0 -0.088 rpy=0 0 0; parent lower_leg_v4_1 -> right_calve; type continuous -> revolute
- joint right_leg_motor_5: axis 1.0 0.0 0.0 -> -1.0 0.0 0.0; child New_left_foot_upperhalf_v5_1 -> right_foot; limit (none) -> lower=-0.7853981633974483 upper=0.7853981633974483 effort=6.0 velocity=6.6; origin xyz=-0.0843 -0.0233 0.0 rpy=0 0 0 -> xyz=-0.0645 -0.0235 -0.036 rpy=0 0 0; parent ankle_motors_v4_2 -> right_ankle; type continuous -> revolute
- joint torso_imu: axis 0.0 0.0 1.0 -> 0 0 0; child /imu_link -> imu_link; origin xyz=0.013 0.0 0.02895 rpy=0 0 0 -> xyz=0.0 0 0.000 rpy=0 0 0; parent /torso -> torso
