Commit message: renamed and got rid of unnessary desrciption packages

File: soccer_description/bez2_description/urdf/bez2.xacro (robot description, xacro)
@@ -1,14 +1,13 @@
 <?xml version="1.0" ?>
 <robot name="bez2" xmlns:xacro="http://www.ros.org/wiki/xacro">
+<xacro:include filename="$(find bez2_description)/urdf/parameters.xacro" />
 <xacro:include filename="$(find bez2_description)/urdf/materials.xacro" />
 <xacro:include filename="$(find bez2_description)/urdf/bez2.trans" />
 <xacro:include filename="$(find bez2_description)/urdf/bez2.gazebo" />
-<xacro:arg name="has_base_footprint" default="false" />
-<xacro:arg name="tf_prefix" default="" />
-<link name="$(arg tf_prefix)/torso">
-  <inertial>
-    <origin xyz="0.005344203942179857 0.0011597330599576942 -0.04327601296104891" rpy="0 0 0"/>
-    <mass value="1.4940527908480117"/>
-    <inertia ixx="0.006599" iyy="0.005741" izz="0.003932" ixy="0" iyz="0" ixz="0"/>
+<link name="torso">
+  <inertial>
+    <origin xyz="-2.6182166493521018e-05 0.0037391632790891283 -0.07310917852477573" rpy="0 0 0"/>
+    <mass value="1.621911019034044"/>
+    <inertia ixx="0.17522" iyy="0.126523" izz="0.127074" ixy="0.000499" iyz="0.000833" ixz="0.001818"/>
   </inertial>
   <visual>
@@ -17,547 +16,610 @@
       <mesh filename="package://bez2_description/meshes/base_link.stl" scale="0.001 0.001 0.001"/>
     </geometry>
-    <material name="polymide_kapton"/>
-  </visual>
-  <collision>
-    <origin xyz="0 0 0" rpy="0 0 0"/>
-    <geometry>
-      <mesh filename="package://bez2_description/meshes/base_link.stl" scale="0.001 0.001 0.001"/>
-    </geometry>
-  </collision>
-</link>
-<link name="$(arg tf_prefix)/biceps_v3_1">
-  <inertial>
-    <origin xyz="-4.857598999001871e-13 0.026299931386057934 -0.038386051153163035" rpy="0 0 0"/>
-    <mass value="0.25825416029102555"/>
-    <inertia ixx="0.000437" iyy="0.000394" izz="6.4e-05" ixy="0.0" iyz="3.3e-05" ixz="-0.0"/>
-  </inertial>
-  <visual>
-    <origin xyz="-0.0 -0.0725 -0.00045" rpy="0 0 0"/>
-    <geometry>
-      <mesh filename="package://bez2_description/meshes/biceps_v3_1.stl" scale="0.001 0.001 0.001"/>
-    </geometry>
-    <material name="plastic_glossy_black"/>
-  </visual>
-  <collision>
-    <origin xyz="-0.0 -0.0725 -0.00045" rpy="0 0 0"/>
-    <geometry>
-      <mesh filename="package://bez2_description/meshes/biceps_v3_1.stl" scale="0.001 0.001 0.001"/>
-    </geometry>
-  </collision>
-</link>
-<link name="$(arg tf_prefix)/Arm_Assembly-bez3_v12_2">
-  <inertial>
-    <origin xyz="-0.005330016176706751 0.022844719426815346 0.029751280366322262" rpy="0 0 0"/>
-    <mass value="0.32110352957731503"/>
-    <inertia ixx="0.002148" iyy="0.002137" izz="0.000103" ixy="3e-06" iyz="1.6e-05" ixz="-0.000175"/>
-  </inertial>
-  <visual>
-    <origin xyz="-0.0 -0.0805 0.09015" rpy="0 0 0"/>
-    <geometry>
-      <mesh filename="package://bez2_description/meshes/Arm_Assembly-bez3_v12_2.stl" scale="0.001 0.001 0.001"/>
-    </geometry>
-    <material name="abs_white"/>
-  </visual>
-  <collision>
-    <origin xyz="-0.0 -0.0805 0.09015" rpy="0 0 0"/>
-    <geometry>
-      <mesh filename="package://bez2_description/meshes/Arm_Assembly-bez3_v12_2.stl" scale="0.001 0.001 0.001"/>
-    </geometry>
-  </collision>
-</link>
-<link name="$(arg tf_prefix)/biceps_v3_2">
-  <inertial>
-    <origin xyz="4.933084310590376e-13 -0.026299931386065484 -0.038386051153161384" rpy="0 0 0"/>
-    <mass value="0.25825416029102555"/>
-    <inertia ixx="0.000437" iyy="0.000394" izz="6.4e-05" ixy="0.0" iyz="-3.3e-05" ixz="0.0"/>
-  </inertial>
-  <visual>
-    <origin xyz="-0.0 0.0725 -0.00045" rpy="0 0 0"/>
-    <geometry>
-      <mesh filename="package://bez2_description/meshes/biceps_v3_2.stl" scale="0.001 0.001 0.001"/>
-    </geometry>
-    <material name="plastic_glossy_black"/>
-  </visual>
-  <collision>
-    <origin xyz="-0.0 0.0725 -0.00045" rpy="0 0 0"/>
-    <geometry>
-      <mesh filename="package://bez2_description/meshes/biceps_v3_2.stl" scale="0.001 0.001 0.001"/>
-    </geometry>
-  </collision>
-</link>
-<link name="$(arg tf_prefix)/Arm_Assembly-bez3_v12_1">
-  <inertial>
-    <origin xyz="-0.005330016176713268 -0.02582928057318666 0.02975128036632215" rpy="0 0 0"/>
-    <mass value="0.32110352957731503"/>
-    <inertia ixx="0.002148" iyy="0.002137" izz="0.000103" ixy="3e-06" iyz="1.6e-05" ixz="-0.000175"/>
-  </inertial>
-  <visual>
-    <origin xyz="0.0 0.0805 0.09015" rpy="0 0 0"/>
-    <geometry>
-      <mesh filename="package://bez2_description/meshes/Arm_Assembly-bez3_v12_1.stl" scale="0.001 0.001 0.001"/>
-    </geometry>
-    <material name="abs_white"/>
-  </visual>
-  <collision>
-    <origin xyz="0.0 0.0805 0.09015" rpy="0 0 0"/>
-    <geometry>
-      <mesh filename="package://bez2_description/meshes/Arm_Assembly-bez3_v12_1.stl" scale="0.001 0.001 0.001"/>
-    </geometry>
-  </collision>
-</link>
-<link name="$(arg tf_prefix)/Hip_Printable_v2_v10_2">
-  <inertial>
-    <origin xyz="4.21754180706356e-05 -3.2154834350706096e-14 -0.014017367581241474" rpy="0 0 0"/>
-    <mass value="0.010089224750638792"/>
-    <inertia ixx="2e-06" iyy="6e-06" izz="5e-06" ixy="0.0" iyz="-0.0" ixz="0.0"/>
-  </inertial>
-  <visual>
-    <origin xyz="-0.01597 -0.0377 0.14405" rpy="0 0 0"/>
-    <geometry>
-      <mesh filename="package://bez2_description/meshes/Hip_Printable_v2_v10_2.stl" scale="0.001 0.001 0.001"/>
-    </geometry>
-    <material name="abs_white"/>
-  </visual>
-  <collision>
-    <origin xyz="-0.01597 -0.0377 0.14405" rpy="0 0 0"/>
-    <geometry>
-      <mesh filename="package://bez2_description/meshes/Hip_Printable_v2_v10_2.stl" scale="0.001 0.001 0.001"/>
-    </geometry>
-  </collision>
-</link>
-<link name="$(arg tf_prefix)/hip_motors_v4_1">
-  <inertial>
-    <origin xyz="0.00908799649277551 -7.287744503703397e-08 -0.011907384768018503" rpy="0 0 0"/>
-    <mass value="0.2728199051639206"/>
-    <inertia ixx="7.4e-05" iyy="0.000178" izz="0.000153" ixy="-0.0" iyz="0.0" ixz="-1e-06"/>
-  </inertial>
-  <visual>
-    <origin xyz="0.00753 0.0368 0.17605" rpy="0 0 0"/>
-    <geometry>
-      <mesh filename="package://bez2_description/meshes/hip_motors_v4_1.stl" scale="0.001 0.001 0.001"/>
-    </geometry>
-    <material name="silver_default"/>
-  </visual>
-  <collision>
-    <origin xyz="0.00753 0.0368 0.17605" rpy="0 0 0"/>
-    <geometry>
-      <mesh filename="package://bez2_description/meshes/hip_motors_v4_1.stl" scale="0.001 0.001 0.001"/>
-    </geometry>
-  </collision>
-</link>
-<link name="$(arg tf_prefix)/hip_motors_v4_2">
-  <inertial>
-    <origin xyz="0.009087996492779226 -7.28774387503961e-08 -0.011907384768019141" rpy="0 0 0"/>
-    <mass value="0.2728199051639206"/>
-    <inertia ixx="7.4e-05" iyy="0.000178" izz="0.000153" ixy="-0.0" iyz="0.0" ixz="-1e-06"/>
-  </inertial>
-  <visual>
-    <origin xyz="0.00903 -0.0377 0.17605" rpy="0 0 0"/>
-    <geometry>
-      <mesh filename="package://bez2_description/meshes/hip_motors_v4_2.stl" scale="0.001 0.001 0.001"/>
-    </geometry>
-    <material name="silver_default"/>
-  </visual>
-  <collision>
-    <origin xyz="0.00903 -0.0377 0.17605" rpy="0 0 0"/>
-    <geometry>
-      <mesh filename="package://bez2_description/meshes/hip_motors_v4_2.stl" scale="0.001 0.001 0.001"/>
-    </geometry>
-  </collision>
-</link>
-<link name="$(arg tf_prefix)/Upper_left_leg_support__bottom__v8_1">
-  <inertial>
-    <origin xyz="-5.513384106897723e-10 0.019462494401918447 -0.048113787355149845" rpy="0 0 0"/>
-    <mass value="0.027169463894965433"/>
-    <inertia ixx="3.2e-05" iyy="2.2e-05" izz="1.3e-05" ixy="0.0" iyz="-0.0" ixz="-0.0"/>
-  </inertial>
-  <visual>
-    <origin xyz="-0.01462 -0.0177 0.17605" rpy="0 0 0"/>
-    <geometry>
-      <mesh filename="package://bez2_description/meshes/Upper_left_leg_support__bottom__v8_1.stl" scale="0.001 0.001 0.001"/>
-    </geometry>
-    <material name="abs_white"/>
-  </visual>
-  <collision>
-    <origin xyz="-0.01462 -0.0177 0.17605" rpy="0 0 0"/>
-    <geometry>
-      <mesh filename="package://bez2_description/meshes/Upper_left_leg_support__bottom__v8_1.stl" scale="0.001 0.001 0.001"/>
-    </geometry>
-  </collision>
-</link>
-<link name="$(arg tf_prefix)/Upper_left_leg_support__bottom__v8_2">
-  <inertial>
-    <origin xyz="-5.513428880110638e-10 -0.019537505598094276 -0.04811378735514921" rpy="0 0 0"/>
-    <mass value="0.027169463894965433"/>
-    <inertia ixx="3.2e-05" iyy="2.2e-05" izz="1.3e-05" ixy="0.0" iyz="-0.0" ixz="-0.0"/>
-  </inertial>
-  <visual>
-    <origin xyz="-0.01612 0.0168 0.17605" rpy="0 0 0"/>
-    <geometry>
-      <mesh filename="package://bez2_description/meshes/Upper_left_leg_support__bottom__v8_2.stl" scale="0.001 0.001 0.001"/>
-    </geometry>
-    <material name="abs_white"/>
-  </visual>
-  <collision>
-    <origin xyz="-0.01612 0.0168 0.17605" rpy="0 0 0"/>
-    <geometry>
-      <mesh filename="package://bez2_description/meshes/Upper_left_leg_support__bottom__v8_2.stl" scale="0.001 0.001 0.001"/>
-    </geometry>
-  </collision>
-</link>
-<link name="$(arg tf_prefix)/New_left_foot_upperhalf_v5_1">
-  <inertial>
-    <origin xyz="0.05139344311503742 -0.01218090675701626 -0.02177657679768813" rpy="0 0 0"/>
-    <mass value="0.0588564551543425"/>
-    <inertia ixx="3.9e-05" iyy="0.000149" izz="0.000178" ixy="-0.0" iyz="-3e-06" ixz="-0.0"/>
-  </inertial>
-  <visual>
-    <origin xyz="0.06818 0.0351 0.37605" rpy="0 0 0"/>
-    <geometry>
-      <mesh filename="package://bez2_description/meshes/New_left_foot_upperhalf_v5_1.stl" scale="0.001 0.001 0.001"/>
-    </geometry>
-    <material name="abs_white"/>
-  </visual>
-  <collision>
-    <origin xyz="0.06818 0.0351 0.37605" rpy="0 0 0"/>
-    <geometry>
-      <mesh filename="package://bez2_description/meshes/New_left_foot_upperhalf_v5_1.stl" scale="0.001 0.001 0.001"/>
-    </geometry>
-  </collision>
-</link>
-<link name="$(arg tf_prefix)/New_right_foot_upperhalf_v3_1">
-  <inertial>
-    <origin xyz="0.05139344394950704 0.060000000000004765 -0.02177657679768963" rpy="0 0 0"/>
-    <mass value="0.117712910308685"/>
-    <inertia ixx="0.000348" iyy="0.000297" izz="0.000625" ixy="0.0" iyz="0.0" ixz="-1e-06"/>
-  </inertial>
-  <visual>
-    <origin xyz="0.06968 -0.036 0.37605" rpy="0 0 0"/>
-    <geometry>
-      <mesh filename="package://bez2_description/meshes/New_right_foot_upperhalf_v3_1.stl" scale="0.001 0.001 0.001"/>
-    </geometry>
-    <material name="abs_white"/>
-  </visual>
-  <collision>
-    <origin xyz="0.06968 -0.036 0.37605" rpy="0 0 0"/>
-    <geometry>
-      <mesh filename="package://bez2_description/meshes/New_right_foot_upperhalf_v3_1.stl" scale="0.001 0.001 0.001"/>
-    </geometry>
-  </collision>
-</link>
-<link name="$(arg tf_prefix)/lower_leg_v4_1">
-  <inertial>
-    <origin xyz="-7.555562408362304e-09 -0.023191925057663376 -0.02213350063265468" rpy="0 0 0"/>
-    <mass value="0.1476733120184745"/>
-    <inertia ixx="0.000124" iyy="0.000107" izz="4.1e-05" ixy="0.0" iyz="-2e-06" ixz="-0.0"/>
-  </inertial>
-  <visual>
-    <origin xyz="-0.01612 0.0123 0.26775" rpy="0 0 0"/>
-    <geometry>
-      <mesh filename="package://bez2_description/meshes/lower_leg_v4_1.stl" scale="0.001 0.001 0.001"/>
-    </geometry>
-    <material name="abs_white"/>
-  </visual>
-  <collision>
-    <origin xyz="-0.01612 0.0123 0.26775" rpy="0 0 0"/>
-    <geometry>
-      <mesh filename="package://bez2_description/meshes/lower_leg_v4_1.stl" scale="0.001 0.001 0.001"/>
-    </geometry>
-  </collision>
-</link>
-<link name="$(arg tf_prefix)/lower_leg_v4_2">
-  <inertial>
-    <origin xyz="6.452880308219222e-09 0.023191925057662998 -0.02213350063265551" rpy="0 0 0"/>
-    <mass value="0.1476733120184745"/>
-    <inertia ixx="0.000124" iyy="0.000107" izz="4.1e-05" ixy="0.0" iyz="2e-06" ixz="0.0"/>
-  </inertial>
-  <visual>
-    <origin xyz="-0.01462 -0.0132 0.26775" rpy="0 0 0"/>
-    <geometry>
-      <mesh filename="package://bez2_description/meshes/lower_leg_v4_2.stl" scale="0.001 0.001 0.001"/>
-    </geometry>
-    <material name="abs_white"/>
-  </visual>
-  <collision>
-    <origin xyz="-0.01462 -0.0132 0.26775" rpy="0 0 0"/>
-    <geometry>
-      <mesh filename="package://bez2_description/meshes/lower_leg_v4_2.stl" scale="0.001 0.001 0.001"/>
-    </geometry>
-  </collision>
-</link>
-<link name="$(arg tf_prefix)/ankle_motors_v4_1">
-  <inertial>
-    <origin xyz="-0.020543373941361492 0.023300002595937435 0.015062549801947933" rpy="0 0 0"/>
-    <mass value="0.3955604131597503"/>
-    <inertia ixx="0.000155" iyy="0.000468" izz="0.000419" ixy="0.0" iyz="-0.0" ixz="-2e-06"/>
-  </inertial>
-  <visual>
-    <origin xyz="-0.01462 -0.0127 0.37605" rpy="0 0 0"/>
-    <geometry>
-      <mesh filename="package://bez2_description/meshes/ankle_motors_v4_1.stl" scale="0.001 0.001 0.001"/>
-    </geometry>
-    <material name="steel_satin"/>
-  </visual>
-  <collision>
-    <origin xyz="-0.01462 -0.0127 0.37605" rpy="0 0 0"/>
-    <geometry>
-      <mesh filename="package://bez2_description/meshes/ankle_motors_v4_1.stl" scale="0.001 0.001 0.001"/>
-    </geometry>
-  </collision>
-</link>
-<link name="$(arg tf_prefix)/ankle_motors_v4_2">
-  <inertial>
-    <origin xyz="-0.020543374775831007 -0.023299997404074242 0.015062549801948433" rpy="0 0 0"/>
-    <mass value="0.3955604131597503"/>
-    <inertia ixx="0.000155" iyy="0.000468" izz="0.000419" ixy="0.0" iyz="-0.0" ixz="-2e-06"/>
-  </inertial>
-  <visual>
-    <origin xyz="-0.01612 0.0118 0.37605" rpy="0 0 0"/>
-    <geometry>
-      <mesh filename="package://bez2_description/meshes/ankle_motors_v4_2.stl" scale="0.001 0.001 0.001"/>
-    </geometry>
-    <material name="steel_satin"/>
-  </visual>
-  <collision>
-    <origin xyz="-0.01612 0.0118 0.37605" rpy="0 0 0"/>
-    <geometry>
-      <mesh filename="package://bez2_description/meshes/ankle_motors_v4_2.stl" scale="0.001 0.001 0.001"/>
-    </geometry>
-  </collision>
-</link>
-<link name="$(arg tf_prefix)/Hip_Printable_v2_v10_1">
-  <inertial>
-    <origin xyz="4.217541806686084e-05 -3.049643870767227e-14 -0.014017367581240808" rpy="0 0 0"/>
-    <mass value="0.010089224750638792"/>
-    <inertia ixx="2e-06" iyy="6e-06" izz="5e-06" ixy="0.0" iyz="-0.0" ixz="0.0"/>
-  </inertial>
-  <visual>
-    <origin xyz="-0.01597 0.0368 0.14405" rpy="0 0 0"/>
-    <geometry>
-      <mesh filename="package://bez2_description/meshes/Hip_Printable_v2_v10_1.stl" scale="0.001 0.001 0.001"/>
-    </geometry>
-    <material name="abs_white"/>
-  </visual>
-  <collision>
-    <origin xyz="-0.01597 0.0368 0.14405" rpy="0 0 0"/>
-    <geometry>
-      <mesh filename="package://bez2_description/meshes/Hip_Printable_v2_v10_1.stl" scale="0.001 0.001 0.001"/>
-    </geometry>
-  </collision>
-</link>
-<link name="$(arg tf_prefix)/head_v4_1">
-  <inertial>
-    <origin xyz="0.003748762391791026 0.024245275552457073 0.02498879678916051" rpy="0 0 0"/>
-    <mass value="0.29338454987270446"/>
-    <inertia ixx="0.00023" iyy="0.000239" izz="0.000194" ixy="-2e-06" iyz="-1.1e-05" ixz="-7.6e-05"/>
-  </inertial>
-  <visual>
-    <origin xyz="-0.03325 0.02252 -0.109441" rpy="0 0 0"/>
-    <geometry>
-      <mesh filename="package://bez2_description/meshes/head_v4_1.stl" scale="0.001 0.001 0.001"/>
-    </geometry>
-    <material name="plastic_glossy_black"/>
-  </visual>
-  <collision>
-    <origin xyz="-0.03325 0.02252 -0.109441" rpy="0 0 0"/>
-    <geometry>
-      <mesh filename="package://bez2_description/meshes/head_v4_1.stl" scale="0.001 0.001 0.001"/>
-    </geometry>
-  </collision>
-</link>
-<link name="$(arg tf_prefix)/custom_servo_support__middle_neck__v9_1">
-  <inertial>
-    <origin xyz="-4.4698224288541866e-11 0.0015597589791841214 0.014702901470227653" rpy="0 0 0"/>
-    <mass value="0.01959544470499754"/>
-    <inertia ixx="1.4e-05" iyy="6e-06" izz="1.2e-05" ixy="-0.0" iyz="0.0" ixz="-0.0"/>
-  </inertial>
-  <visual>
-    <origin xyz="-0.03325 0.000333 -0.075624" rpy="0 0 0"/>
-    <geometry>
-      <mesh filename="package://bez2_description/meshes/custom_servo_support__middle_neck__v9_1.stl" scale="0.001 0.001 0.001"/>
-    </geometry>
-    <material name="abs_white"/>
-  </visual>
-  <collision>
-    <origin xyz="-0.03325 0.000333 -0.075624" rpy="0 0 0"/>
-    <geometry>
-      <mesh filename="package://bez2_description/meshes/custom_servo_support__middle_neck__v9_1.stl" scale="0.001 0.001 0.001"/>
-    </geometry>
-  </collision>
-</link>
-<link name="$(arg tf_prefix)/camera">
-  <inertial>
-    <origin xyz="-0.000999999374146826 -3.3364626470400865e-07 4.7006202563704136e-07" rpy="0 0 0"/>
-    <mass value="0.0005023999999999989"/>
-    <inertia ixx="0.0" iyy="0.0" izz="0.0" ixy="-0.0" iyz="0.0" ixz="-0.0"/>
-  </inertial>
-  <visual>
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
File: soccer_description/bez2_description/urdf/materials.xacro (robot description, xacro)
@@ -4,15 +4,9 @@
   <color rgba="0.700 0.700 0.700 1.000"/>
 </material>
-<material name="polymide_kapton">
-  <color rgba="0.7843137254901961 0.5568627450980392 0.027450980392156862 1.0"/>
-</material>
-<material name="plastic_glossy_black">
-  <color rgba="0.09803921568627451 0.09803921568627451 0.09803921568627451 1.0"/>
-</material>
-<material name="abs_white">
-  <color rgba="0.9647058823529412 0.9647058823529412 0.9529411764705882 1.0"/>
-</material>
 <material name="steel_satin">
   <color rgba="0.6274509803921569 0.6274509803921569 0.6274509803921569 1.0"/>
 </material>
+<material name="plastic_matte_yellow">
+  <color rgba="0.9098039215686274 0.6784313725490196 0.13725490196078433 1.0"/>
+</material>
 </robot>

File: soccer_description/bez2_description/urdf/parameters.xacro (robot description, xacro)
@@ -1,3 +1,3 @@
-<robot name="bez2_urdf" xmlns:xacro="http://www.ros.org/wiki/xacro">
+<robot name="bez2" xmlns:xacro="http://www.ros.org/wiki/xacro">
     <xacro:property name="PI" value="3.1415926535897931"/>
     <xacro:property name="JOINT_KP" value="1e15"/>
@@ -9,20 +9,21 @@
     <xacro:property name="JOINT_FRICTION" value="0.1"/>
     <xacro:property name="JOINT_DAMPING" value="0.01"/>
+<!--TODO figure out why damping and friction mess with it so much-->
     <xacro:property name="MX28_TORQUE" value="2.5"/>
     <xacro:property name="MX28_VELOCITY" value="5.76"/>
-    <xacro:property name="MX28_DAMPING" value="0.3"/>
-    <xacro:property name="MX28_FRICTION" value="0.83"/>
+    <xacro:property name="MX28_DAMPING" value="${JOINT_DAMPING}"/>
+    <xacro:property name="MX28_FRICTION" value="${JOINT_FRICTION}"/>
     <xacro:property name="MX64_TORQUE" value="6.0"/>
     <xacro:property name="MX64_VELOCITY" value="6.6"/>
-    <xacro:property name="MX64_DAMPING" value="0.66"/>
-    <xacro:property name="MX64_FRICTION" value="1.42"/>
+    <xacro:property name="MX64_DAMPING" value="${JOINT_DAMPING}"/>
+    <xacro:property name="MX64_FRICTION" value="${JOINT_FRICTION}"/>
     <xacro:property name="XM430_TORQUE" value="4.1"/>
     <xacro:property name="XM430_VELOCITY" value="4.82"/>
-    <xacro:property name="XM430_DAMPING" value="0.721165"/>
-    <xacro:property name="XM430_FRICTION" value="0.721165"/>
+    <xacro:property name="XM430_DAMPING" value="${JOINT_DAMPING}"/>
+    <xacro:property name="XM430_FRICTION" value="${JOINT_FRICTION}"/>
     <xacro:property name="XL430_TORQUE" value="1.5"/>
     <xacro:property name="XL430_VELOCITY" value="6.39"/>
-    <xacro:property name="XL430_DAMPING" value="0.16"/>
-    <xacro:property name="XL430_FRICTION" value="0.6"/>
+    <xacro:property name="XL430_DAMPING" value="${JOINT_DAMPING}"/>
+    <xacro:property name="XL430_FRICTION" value="${JOINT_FRICTION}"/>
     <xacro:property name="y_offset" value="0.21571129429326383"/>
     <xacro:property name="z_offset" value="0.05556097822952673"/>

Commit message: work in progress getup back joanne

File: soccer_description/bez2_description/urdf/bez2.urdf (robot description, URDF)
Before this commit: robot bez2, 22 links, 21 joints
Joints:
- joint left_arm_motor_0: limit lower=-1.5707963267948966 upper=3.9269908169872414 effort=2.5 velocity=5.76 -> lower=-3.14 upper=3.9269908169872414 effort=2.5 velocity=5.76
- joint right_arm_motor_0: limit lower=-1.5707963267948966 upper=3.9269908169872414 effort=2.5 velocity=5.76 -> lower=-3.14 upper=3.9269908169872414 effort=2.5 velocity=5.76

Commit message: update urdf/xacro with new torques

File: soccer_description/bez2_description/urdf/bez2.urdf (robot description, URDF)
Before this commit: robot bez2, 22 links, 21 joints
Joints:
- joint left_arm_motor_0: limit lower=-3.14 upper=3.9269908169872414 effort=2.5 velocity=5.76 -> lower=-3.141592653589793 upper=3.9269908169872414 effort=4.1 velocity=4.82
- joint right_arm_motor_0: limit lower=-3.14 upper=3.9269908169872414 effort=2.5 velocity=5.76 -> lower=-3.141592653589793 upper=3.9269908169872414 effort=4.1 velocity=4.82

File: soccer_description/bez2_description/urdf/bez2.xacro (robot description, xacro)
@@ -447,5 +447,5 @@
   <axis xyz="-0.0 -1.0 0.0"/>
   <dynamics damping="${MX28_DAMPING}" friction="${MX28_FRICTION}" />
-<limit effort="${MX28_TORQUE}" lower="-${PI/2}" upper="${PI*5/4}" velocity="${MX28_VELOCITY}"/>
+<limit effort="${XM430_TORQUE}" lower="-${PI}" upper="${PI*5/4}" velocity="${XM430_VELOCITY}"/>
 </joint>
 <joint name="left_arm_motor_1" type="revolute">
@@ -519,5 +519,5 @@
   <axis xyz="0.0 -1.0 -0.0"/>
     <dynamics damping="${MX28_DAMPING}" friction="${MX28_FRICTION}" />
-              <limit effort="${MX28_TORQUE}" lower="-${PI/2}" upper="${PI*5/4}" velocity="${MX28_VELOCITY}"/>
+              <limit effort="${XM430_TORQUE}" lower="-${PI}" upper="${PI*5/4}" velocity="${XM430_VELOCITY}"/>
 </joint>
 <joint name="right_arm_motor_1" type="revolute">

Commit message: updated with getup branch

File: soccer_description/bez2_description/urdf/bez2.urdf (robot description, URDF)
Before this commit: robot bez2, 22 links, 21 joints
Joints:
- joint left_arm_motor_0: limit lower=-1.5707963267948966 upper=3.9269908169872414 effort=2.5 velocity=5.76 -> lower=-3.141592653589793 upper=3.9269908169872414 effort=4.1 velocity=4.82
- joint right_arm_motor_0: limit lower=-1.5707963267948966 upper=3.9269908169872414 effort=2.5 velocity=5.76 -> lower=-3.141592653589793 upper=3.9269908169872414 effort=4.1 velocity=4.82
