Commit message: improved model weights and physics

File: soccer_description/bez2_description/urdf/bez2.urdf (robot description, URDF)
Before this commit: robot bez2, 22 links, 21 joints
Links:
- link left_ankle: mass 0.26345509510176346 -> 0.151468601936124
- link left_bicep: mass 0.7365391814909177 -> 0.212120407883451
- link left_calve: mass 0.20304073544640247 -> 0.143723171211077
- link left_foot: mass 0.37785469138016164 -> 0.16613521684361
- link left_hip_front: mass 0.7328385746044006 -> 0.211645971103128
- link left_hip_side: mass 0.023116469719045966 -> 0.120655957656288
- link left_shoulder: mass 0.42869731083494267 -> 0.172653501389095
- link left_thigh: mass 0.191955361852033 -> 0.142301969468209
- link right_ankle: mass 0.26345509510176346 -> 0.151468601936124
- link right_bicep: mass 0.7365391814909177 -> 0.212120407883451
- link right_calve: mass 0.20304073544640247 -> 0.143723171211077
- link right_foot: mass 0.37785469138016164 -> 0.16613521684361
- link right_hip_front: mass 0.7328385746044006 -> 0.211645971103128
- link right_hip_side: mass 0.023116469719045966 -> 0.120655957656288
- link right_shoulder: mass 0.42869731083494267 -> 0.172653501389095
- link right_thigh: mass 0.191955361852033 -> 0.142301969468209
- link torso: mass 1.621911019034044 -> 1.62191101903404

File: soccer_description/bez2_description/urdf/bez2.xacro (robot description, xacro)
@@ -8,5 +8,5 @@
   <inertial>
     <origin xyz="-2.6182166493521018e-05 0.0037391632790891283 -0.07310917852477573" rpy="0 0 0"/>
-    <mass value="1.621911019034044"/>
+    <mass value="1.62191101903404"/>
     <inertia ixx="0.17522" iyy="0.126523" izz="0.127074" ixy="0.000499" iyz="0.000833" ixz="0.001818"/>
   </inertial>
@@ -68,5 +68,5 @@
   <inertial>
     <origin xyz="9.49688693072442e-05 0.025391120875814188 -0.00710009103373208" rpy="0 0 0"/>
-    <mass value="0.42869731083494267"/>
+    <mass value="0.172653501389095"/>
     <inertia ixx="0.000136" iyy="0.000137" izz="0.000116" ixy="0.0" iyz="1.8e-05" ixz="3e-06"/>
   </inertial>
@@ -88,5 +88,5 @@
   <inertial>
     <origin xyz="-0.01931620093381984 0.0008375708488899958 -0.05229697639295136" rpy="0 0 0"/>
-    <mass value="0.7365391814909177"/>
+    <mass value="0.212120407883451"/>
     <inertia ixx="0.000601" iyy="0.000616" izz="0.000236" ixy="-0.0" iyz="1.3e-05" ixz="9e-06"/>
   </inertial>
@@ -128,5 +128,5 @@
   <inertial>
     <origin xyz="2.104631423652248e-08 3.399354384647779e-07 -0.0077462434278427195" rpy="0 0 0"/>
-    <mass value="0.023116469719045966"/>
+    <mass value="0.120655957656288"/>
     <inertia ixx="3e-06" iyy="8e-06" izz="7e-06" ixy="-0.0" iyz="-0.0" ixz="0.0"/>
   </inertial>
@@ -148,5 +148,5 @@
 <inertial>
   <origin xyz="0.0004996292549223533 0.0005421424160892835 -0.012131129108951588" rpy="0 0 0"/>
-  <mass value="0.7328385746044006"/>
+  <mass value="0.211645971103128"/>
   <inertia ixx="0.000195" iyy="0.000458" izz="0.000394" ixy="-8e-06" iyz="-1e-06" ixz="-2e-06"/>
 </inertial>
@@ -168,5 +168,5 @@
   <inertial>
     <origin xyz="2.1046150922715556e-08 -0.018793706652435974 -0.06540894904468947" rpy="0 0 0"/>
-    <mass value="0.191955361852033"/>
+    <mass value="0.142301969468209"/>
     <inertia ixx="0.000159" iyy="0.000121" izz="6.9e-05" ixy="-0.0" iyz="1e-06" ixz="0.0"/>
   </inertial>
@@ -188,5 +188,5 @@
   <inertial>
     <origin xyz="0.00034959081321023905 -0.023268493362085793 -0.030853501915197812" rpy="0 0 0"/>
-    <mass value="0.20304073544640247"/>
+    <mass value="0.143723171211077"/>
     <inertia ixx="0.000176" iyy="0.00015" izz="6.2e-05" ixy="0.0" iyz="-2e-06" ixz="2e-06"/>
   </inertial>
@@ -208,5 +208,5 @@
   <inertial>
     <origin xyz="-0.02065513049536576 -0.023057637545577894 -0.017838420955393897" rpy="0 0 0"/>
-    <mass value="0.26345509510176346"/>
+    <mass value="0.151468601936124"/>
     <inertia ixx="0.000102" iyy="0.000212" izz="0.000173" ixy="-1e-06" iyz="-2e-06" ixz="-1.7e-05"/>
   </inertial>
@@ -228,5 +228,5 @@
   <inertial>
     <origin xyz="0.0476419808535605 0.018106431082562213 -0.01978200152059173" rpy="0 0 0"/>
-    <mass value="0.37785469138016164"/>
+    <mass value="0.16613521684361"/>
     <inertia ixx="0.000247" iyy="0.000905" izz="0.001142" ixy="-2.6e-05" iyz="5e-06" ixz="1.4e-05"/>
   </inertial>
@@ -248,5 +248,5 @@
   <inertial>
     <origin xyz="2.1046314309380865e-08 3.3993543878396704e-07 -0.007746243427843552" rpy="0 0 0"/>
-    <mass value="0.023116469719045966"/>
+    <mass value="0.120655957656288"/>
     <inertia ixx="3e-06" iyy="8e-06" izz="7e-06" ixy="-0.0" iyz="-0.0" ixz="0.0"/>
   </inertial>
@@ -268,5 +268,5 @@
   <inertial>
     <origin xyz="0.0004996292549223817 0.0005421424160894084 -0.01213112910895231" rpy="0 0 0"/>
-    <mass value="0.7328385746044006"/>
+    <mass value="0.211645971103128"/>
     <inertia ixx="0.000195" iyy="0.000458" izz="0.000394" ixy="-8e-06" iyz="-1e-06" ixz="-2e-06"/>
   </inertial>
@@ -288,5 +288,5 @@
   <inertial>
     <origin xyz="2.1046151002512836e-08 -0.018793706652437202 -0.0654089490446903" rpy="0 0 0"/>
-    <mass value="0.191955361852033"/>
+    <mass value="0.142301969468209"/>
     <inertia ixx="0.000159" iyy="0.000121" izz="6.9e-05" ixy="-0.0" iyz="1e-06" ixz="0.0"/>
   </inertial>
@@ -308,5 +308,5 @@
   <inertial>
     <origin xyz="0.0003495908132103466 -0.023268493362087077 -0.030853501915198367" rpy="0 0 0"/>
-    <mass value="0.20304073544640247"/>
+    <mass value="0.143723171211077"/>
     <inertia ixx="0.000176" iyy="0.00015" izz="6.2e-05" ixy="0.0" iyz="-2e-06" ixz="2e-06"/>
   </inertial>
@@ -328,5 +328,5 @@
   <inertial>
     <origin xyz="-0.020655130495365704 -0.023057637545579254 -0.017838420955394507" rpy="0 0 0"/>
-    <mass value="0.26345509510176346"/>
+    <mass value="0.151468601936124"/>
     <inertia ixx="0.000102" iyy="0.000212" izz="0.000173" ixy="-1e-06" iyz="-2e-06" ixz="-1.7e-05"/>
   </inertial>
@@ -348,5 +348,5 @@
   <inertial>
     <origin xyz="0.047641980853560625 -0.018107232571891542 -0.019782001520592507" rpy="0 0 0"/>
-    <mass value="0.37785469138016164"/>
+    <mass value="0.16613521684361"/>
     <inertia ixx="0.000247" iyy="0.000905" izz="0.001142" ixy="2.6e-05" iyz="-5e-06" ixz="1.4e-05"/>
   </inertial>
@@ -368,5 +368,5 @@
   <inertial>
     <origin xyz="0.00042714569282304837 -0.025390436050570106 -0.007100091033732914" rpy="0 0 0"/>
-    <mass value="0.42869731083494267"/>
+    <mass value="0.172653501389095"/>
     <inertia ixx="0.000136" iyy="0.000137" izz="0.000116" ixy="1e-06" iyz="-1.8e-05" ixz="4e-06"/>
   </inertial>
@@ -388,5 +388,5 @@
   <inertial>
     <origin xyz="-0.02068375587119517 -0.0008368909778958267 -0.05229697639295197" rpy="0 0 0"/>
-    <mass value="0.7365391814909177"/>
+    <mass value="0.212120407883451"/>
     <inertia ixx="0.000601" iyy="0.000616" izz="0.000236" ixy="-0.0" iyz="-1.3e-05" ixz="-9e-06"/>
   </inertial>

File: soccer_description/bez2_description/urdf/parameters.xacro (robot description, xacro)
@@ -12,18 +12,18 @@
     <xacro:property name="MX28_TORQUE" value="2.5"/>
     <xacro:property name="MX28_VELOCITY" value="5.76"/>
-    <xacro:property name="MX28_DAMPING" value="${JOINT_DAMPING}"/>
-    <xacro:property name="MX28_FRICTION" value="${JOINT_FRICTION}"/>
+    <xacro:property name="MX28_DAMPING" value="0.3"/>
+    <xacro:property name="MX28_FRICTION" value="0.83"/>
     <xacro:property name="MX64_TORQUE" value="6.0"/>
     <xacro:property name="MX64_VELOCITY" value="6.6"/>
-    <xacro:property name="MX64_DAMPING" value="${JOINT_DAMPING}"/>
-    <xacro:property name="MX64_FRICTION" value="${JOINT_FRICTION}"/>
+    <xacro:property name="MX64_DAMPING" value="0.66"/>
+    <xacro:property name="MX64_FRICTION" value="1.42"/>
     <xacro:property name="XM430_TORQUE" value="4.1"/>
     <xacro:property name="XM430_VELOCITY" value="4.82"/>
-    <xacro:property name="XM430_DAMPING" value="${JOINT_DAMPING}"/>
-    <xacro:property name="XM430_FRICTION" value="${JOINT_FRICTION}"/>
+    <xacro:property name="XM430_DAMPING" value="0.72"/>
+    <xacro:property name="XM430_FRICTION" value="0.72"/>
     <xacro:property name="XL430_TORQUE" value="1.5"/>
     <xacro:property name="XL430_VELOCITY" value="6.39"/>
-    <xacro:property name="XL430_DAMPING" value="${JOINT_DAMPING}"/>
-    <xacro:property name="XL430_FRICTION" value="${JOINT_FRICTION}"/>
+    <xacro:property name="XL430_DAMPING" value="0.16"/>
+    <xacro:property name="XL430_FRICTION" value="0.6"/>
     <xacro:property name="y_offset" value="0.21571129429326383"/>
     <xacro:property name="z_offset" value="0.05556097822952673"/>

Commit message: Attempt getup-back by vaulting forward

File: soccer_description/bez2_description/urdf/bez2.urdf (robot description, URDF)
Before this commit: robot bez2, 22 links, 21 joints
Links:
- link left_forearm: geometry collision box size=0.04800 0.05300 0.24838; visual mesh filename=package://bez2_description/meshes/Bez1_forearm_v7_1.stl scale=0.001 0.001 0.00133
- link right_forearm: geometry collision box size=0.04800 0.05300 0.24838; visual mesh filename=package://bez2_description/meshes/Bez1_forearm_v7_2.stl scale=0.001 0.001 0.00133
Joints:
- joint left_arm_motor_0: limit lower=-3.141592653589793 upper=3.9269908169872414 effort=4.1 velocity=4.82 -> effort=4.1 velocity=4.82
- joint right_arm_motor_0: limit lower=-3.141592653589793 upper=3.9269908169872414 effort=4.1 velocity=4.82 -> effort=4.1 velocity=4.82

Commit message: Getup backflip

File: soccer_description/bez2_description/urdf/bez2.urdf (robot description, URDF)
Before this commit: robot bez2, 22 links, 21 joints
Links:
- link left_forearm: geometry collision box size=0.04800 0.05300 0.18838; visual mesh filename=package://bez2_description/meshes/Bez1_forearm_v7_1.stl scale=0.001 0.001 0.001
- link right_forearm: geometry collision box size=0.04800 0.05300 0.18838; visual mesh filename=package://bez2_description/meshes/Bez1_forearm_v7_2.stl scale=0.001 0.001 0.001
Joints:
- joint left_arm_motor_0: limit effort=4.1 velocity=4.82 -> lower=-3.141592653589793 upper=3.9269908169872414 effort=4.1 velocity=4.82
- joint right_arm_motor_0: limit effort=4.1 velocity=4.82 -> lower=-3.141592653589793 upper=3.9269908169872414 effort=4.1 velocity=4.82

File: soccer_description/bez2_description/urdf/parameters.xacro (robot description, xacro)
@@ -7,23 +7,23 @@
     <xacro:property name="FOREARM_MU1" value="0.2"/>
     <xacro:property name="FOREARM_MU2" value="0.2"/>
-    <xacro:property name="JOINT_FRICTION" value="0.1"/>
-    <xacro:property name="JOINT_DAMPING" value="0.01"/>
+    <xacro:property name="JOINT_FRICTION" value="0"/>
+    <xacro:property name="JOINT_DAMPING" value="0"/>
 <!--TODO figure out why damping and friction mess with it so much-->
     <xacro:property name="MX28_TORQUE" value="2.5"/>
     <xacro:property name="MX28_VELOCITY" value="5.76"/>
-    <xacro:property name="MX28_DAMPING" value="0.3"/>
-    <xacro:property name="MX28_FRICTION" value="0.83"/>
+    <xacro:property name="MX28_DAMPING" value="0"/>
+    <xacro:property name="MX28_FRICTION" value="0"/>
     <xacro:property name="MX64_TORQUE" value="6.0"/>
     <xacro:property name="MX64_VELOCITY" value="6.6"/>
-    <xacro:property name="MX64_DAMPING" value="0.66"/>
-    <xacro:property name="MX64_FRICTION" value="1.42"/>
+    <xacro:property name="MX64_DAMPING" value="0"/>
+    <xacro:property name="MX64_FRICTION" value="0"/>
     <xacro:property name="XM430_TORQUE" value="4.1"/>
     <xacro:property name="XM430_VELOCITY" value="4.82"/>
-    <xacro:property name="XM430_DAMPING" value="0.72"/>
-    <xacro:property name="XM430_FRICTION" value="0.72"/>
+    <xacro:property name="XM430_DAMPING" value="0"/>
+    <xacro:property name="XM430_FRICTION" value="0"/>
     <xacro:property name="XL430_TORQUE" value="1.5"/>
     <xacro:property name="XL430_VELOCITY" value="6.39"/>
-    <xacro:property name="XL430_DAMPING" value="0.16"/>
-    <xacro:property name="XL430_FRICTION" value="0.6"/>
+    <xacro:property name="XL430_DAMPING" value="0"/>
+    <xacro:property name="XL430_FRICTION" value="0"/>
     <xacro:property name="y_offset" value="0.21571129429326383"/>
     <xacro:property name="z_offset" value="0.05556097822952673"/>

Commit message: eff

File: soccer_description/bez2_description/urdf/bez2.urdf (robot description, URDF)
Before this commit: robot bez2, 22 links, 21 joints
Links:
- added link torso_cylinder, mass 0.00001; collision cylinder length=0.08 radius=0.02; visual cylinder length=0.08 radius=0.02
Joints:
- added joint torso_cylinder_joint: type fixed, parent torso, child torso_cylinder, origin xyz=0.0 0 0.000 rpy=0 0 0, axis 0 0 0

File: soccer_description/bez2_description/urdf/bez2.xacro (robot description, xacro)
@@ -592,4 +592,30 @@
     </inertial>
   </link>
+<joint name="torso_cylinder_joint" type="fixed">
+  <parent link="torso"/>
+  <child link="torso_cylinder"/>
+  <origin rpy="0 0 0" xyz="0.0 0 0.000"/>
+  <axis xyz="0 0 0"/>
+</joint>
+<link name="torso_cylinder">
+  <inertial>
+    <origin xyz="-0.026300599945598205 0.02045796215352269 -0.07127075071519248" rpy="0 0 0"/>
+    <mass value="0.00001"/>
+    <inertia ixx="0.00001" iyy="0.00001" izz="0.00001" ixy="-0.0" iyz="-0.0" ixz="-0"/>
+  </inertial>
+  <visual>
+    <origin xyz="-0.14 0 -0.07" rpy="0 0 0"/>
+    <geometry>
+      <cylinder radius="0.02" length="0.08" />
+    </geometry>
+    <material name="plastic_matte_yellow"/>
+  </visual>
+  <collision>
+    <origin xyz="-0.14 0 -0.07" rpy="0 0 0"/>
+    <geometry>
+      <cylinder radius="0.02" length="0.08" />
+    </geometry>
+  </collision>
+</link>
   <joint name="torso_imu" type="fixed">
     <parent link="torso"/>

Commit message: Bez2 robocup (#845)
* Tested getup on Bez2 hw
- fw + fw interface modified to support 2 additional arm motors

* fixed getupfront

* work in progress getup back joanne

* getup/walk WIP

* update urdf/xacro with new torques

* improved model weights and physics

* Get up front updated - joanne

* Attempt getup-back by vaulting forward

* Getup backflip

* IMU fixes + full getup back trajectory

* eff

* eff

* latest stuff on nam's laptop

---------

Co-authored-by: nam <lkunelk@gmail.com>
Co-authored-by: JoanneT8 <joannetan121@gmail.com>
Co-authored-by: manx52 <jonathanspraggett@gmail.com>

File: soccer_description/bez2_description/urdf/bez2.urdf (robot description, URDF)
Before this commit: robot bez2, 22 links, 21 joints
Links:
- added link torso_cylinder, mass 0.00001; collision cylinder length=0.08 radius=0.02; visual cylinder length=0.08 radius=0.02
Joints:
- added joint torso_cylinder_joint: type fixed, parent torso, child torso_cylinder, origin xyz=0.0 0 0.000 rpy=0 0 0, axis 0 0 0

File: soccer_description/bez2_description/urdf/parameters.xacro (robot description, xacro)
@@ -12,18 +12,18 @@
     <xacro:property name="MX28_TORQUE" value="2.5"/>
     <xacro:property name="MX28_VELOCITY" value="5.76"/>
-    <xacro:property name="MX28_DAMPING" value="0.3"/>
-    <xacro:property name="MX28_FRICTION" value="0.83"/>
+    <xacro:property name="MX28_DAMPING" value="${JOINT_DAMPING}"/>
+    <xacro:property name="MX28_FRICTION" value="${JOINT_FRICTION}"/>
     <xacro:property name="MX64_TORQUE" value="6.0"/>
     <xacro:property name="MX64_VELOCITY" value="6.6"/>
-    <xacro:property name="MX64_DAMPING" value="0.66"/>
-    <xacro:property name="MX64_FRICTION" value="1.42"/>
+    <xacro:property name="MX64_DAMPING" value="${JOINT_DAMPING}"/>
+    <xacro:property name="MX64_FRICTION" value="${JOINT_FRICTION}"/>
     <xacro:property name="XM430_TORQUE" value="4.1"/>
     <xacro:property name="XM430_VELOCITY" value="4.82"/>
-    <xacro:property name="XM430_DAMPING" value="0.72"/>
-    <xacro:property name="XM430_FRICTION" value="0.72"/>
+    <xacro:property name="XM430_DAMPING" value="${JOINT_DAMPING}"/>
+    <xacro:property name="XM430_FRICTION" value="${JOINT_FRICTION}"/>
     <xacro:property name="XL430_TORQUE" value="1.5"/>
     <xacro:property name="XL430_VELOCITY" value="6.39"/>
-    <xacro:property name="XL430_DAMPING" value="0.16"/>
-    <xacro:property name="XL430_FRICTION" value="0.6"/>
+    <xacro:property name="XL430_DAMPING" value="${JOINT_DAMPING}"/>
+    <xacro:property name="XL430_FRICTION" value="${JOINT_FRICTION}"/>
     <xacro:property name="y_offset" value="0.21571129429326383"/>
     <xacro:property name="z_offset" value="0.05556097822952673"/>
