Commit message: added a rough draft of ros layer for placo and it works great out of the box

File: soccer_description/bez2_description/urdf/robot.urdf (robot description, URDF)
Before this commit: robot bez2, 22 links, 21 joints
Links:
- link head: geometry collision box size=0.07120 0.09400 0.07530; visual mesh filename=../meshes/Head_Pitch_Assembly_v4_1.stl scale=0.001 0.001 0.001
- link left_ankle: geometry collision box size=0.08910 0.05000 0.06398; visual mesh filename=../meshes/ankle_v2_1.stl scale=0.001 0.001 0.001
- link left_bicep: geometry collision box size=0.05000 0.04703 0.11202; visual mesh filename=../meshes/bicep_v1_1.stl scale=0.001 0.001 0.001
- link left_calve: geometry collision box size=0.04030 0.05350 0.10500; visual mesh filename=../meshes/calf_v1_1.stl scale=0.001 0.001 0.001
- link left_foot: geometry collision box size=0.17000 0.09000 0.03300; visual mesh filename=../meshes/left_foot_v2_1.stl scale=0.001 0.001 0.001
- link left_forearm: geometry collision box size=0.04800 0.05300 0.18838; visual mesh filename=../meshes/Bez1_forearm_v7_1.stl scale=0.001 0.001 0.001
- link left_hip_front: geometry collision box size=0.07402 0.04100 0.04650; visual mesh filename=../meshes/hip_v1_1.stl scale=0.001 0.001 0.001
- link left_hip_side: geometry collision box size=0.04100 0.02400 0.03050; visual mesh filename=../meshes/fr12_h101_v1_2.stl scale=0.001 0.001 0.001
- link left_shoulder: geometry collision box size=0.04360 0.04730 0.05100; visual mesh filename=../meshes/left_shoulder_v1_1.stl scale=0.001 0.001 0.001
- link left_thigh: geometry collision box size=0.03300 0.05100 0.12150; visual mesh filename=../meshes/thigh_v1_1.stl scale=0.001 0.001 0.001
- link neck: geometry collision box size=0.02200 0.05100 0.03800; visual mesh filename=../meshes/Head_Yaw_Assembly_v1_1.stl scale=0.001 0.001 0.001
- link right_ankle: geometry collision box size=0.08910 0.05000 0.06398; visual mesh filename=../meshes/ankle_v2_2.stl scale=0.001 0.001 0.001
- link right_bicep: geometry collision box size=0.05000 0.04703 0.11202; visual mesh filename=../meshes/bicep_v1_2.stl scale=0.001 0.001 0.001
- link right_calve: geometry collision box size=0.04030 0.05350 0.10500; visual mesh filename=../meshes/calf_v1_2.stl scale=0.001 0.001 0.001
- link right_foot: geometry collision box size=0.17000 0.09000 0.03300; visual mesh filename=../meshes/right_foot_v2_1.stl scale=0.001 0.001 0.001
- link right_forearm: geometry collision box size=0.04800 0.05300 0.18838; visual mesh filename=../meshes/Bez1_forearm_v7_2.stl scale=0.001 0.001 0.001
- link right_hip_front: geometry collision box size=0.07402 0.04100 0.04650; visual mesh filename=../meshes/hip_v1_2.stl scale=0.001 0.001 0.001
- link right_hip_side: geometry collision box size=0.04100 0.02400 0.03050; visual mesh filename=../meshes/fr12_h101_v1_1.stl scale=0.001 0.001 0.001
- link right_shoulder: geometry collision box size=0.04435 0.04730 0.05100; visual mesh filename=../meshes/right_shoulder_v2_1.stl scale=0.001 0.001 0.001
- link right_thigh: geometry collision box size=0.03300 0.05100 0.12150; visual mesh filename=../meshes/thigh_v1_2.stl scale=0.001 0.001 0.001
- link trunk: geometry collision box size=0.14440 0.20843 0.19912; visual mesh filename=../meshes/base_link.stl scale=0.001 0.001 0.001
