Commit message: Reorganized the mujoco mjcf files into there proper locations in soccer description. Removed bez2_description and renamed assembly into bez2. Tuned the walk engine for mujoco. removed pybullet and mujoco is now fully integrated, tests are still disorganized. Tested walking to goal. got trajectories to work in mujoco and organized the traj also added a unit test. modified the mjcf files to use attach so that we can have duplicate models and better integration for future 4v4 sim. added unit test for the ball relative pose, various types of walks. Had to modify the setting and getting pose in the world frame as it had to adapt for the ball and potentially more objects in the future. before they were connected and caused weird teleporations when either ball or robot were teleported. Not they are seperate objects and are fine for teleporataion. stopped using left foot as link for setting pose and switched for torso  as it was more aligned with stuff. had to calibrate and get the correct z positonf for all keyframs and add functionality for a custom pose.

File: soccer_description/bez2_description/urdf/materials.xacro (robot description, xacro)
@@ -4,9 +4,12 @@
   <color rgba="0.700 0.700 0.700 1.000"/>
 </material>
+<material name="aluminum_satin">
+  <color rgba="0.9607843137254902 0.9607843137254902 0.9647058823529412 1.0"/>
+</material>
 <material name="steel_satin">
   <color rgba="0.6274509803921569 0.6274509803921569 0.6274509803921569 1.0"/>
 </material>
-<material name="plastic_matte_yellow">
-  <color rgba="0.9098039215686274 0.6784313725490196 0.13725490196078433 1.0"/>
+<material name="abs_white">
+  <color rgba="0.36470588235294116 0.4392156862745098 0.5098039215686274 1.0"/>
 </material>
 </robot>

File: soccer_description/bez2_description/urdf/robot.urdf (robot description, URDF)
Before this commit: robot bez2, 22 links, 21 joints
Links:
- added link camera, mass 0.01
- link head: mass 0.5407373847724953 -> 0.26433915470596575; geometry collision mesh filename=../meshes/head_v4_1.stl scale=0.001 0.001 0.001; visual mesh filename=../meshes/head_v4_1.stl scale=0.001 0.001 0.001
- link left_ankle: mass 0.151468601936124 -> 0.2722002973016189; geometry collision mesh filename=../meshes/left_ankle_v7_1.stl scale=0.001 0.001 0.001; visual mesh filename=../meshes/left_ankle_v7_1.stl scale=0.001 0.001 0.001
- link left_bicep: mass 0.212120407883451 -> 0.18636400760544294; geometry collision mesh filename=../meshes/left_bicep_v6_1.stl scale=0.001 0.001 0.001; visual mesh filename=../meshes/left_bicep_v6_1.stl scale=0.001 0.001 0.001
- link left_calve: mass 0.143723171211077 -> 0.15898038946070936; geometry collision mesh filename=../meshes/left_calve_v5_1.stl scale=0.001 0.001 0.001; visual mesh filename=../meshes/left_calve_v5_1.stl scale=0.001 0.001 0.001
- link left_foot: mass 0.16613521684361 -> 0.03929273129474386; geometry collision mesh filename=../meshes/left_foot_v10_1.stl scale=0.001 0.001 0.001; visual mesh filename=../meshes/left_foot_v10_1.stl scale=0.001 0.001 0.001
- link left_forearm: mass 0.06415483406403591 -> 0.05984540204112203; geometry collision mesh filename=../meshes/left_forearm_v4_1.stl scale=0.001 0.001 0.001; visual mesh filename=../meshes/left_forearm_v4_1.stl scale=0.001 0.001 0.001
- link left_hip_front: mass 0.211645971103128 -> 0.2722002973016189; geometry collision mesh filename=../meshes/left_hip_front_v5_1.stl scale=0.001 0.001 0.001; visual mesh filename=../meshes/left_hip_front_v5_1.stl scale=0.001 0.001 0.001
- link left_hip_side: mass 0.120655957656288 -> 0.03929574358294283; geometry collision mesh filename=../meshes/left_hip_side_v5_1.stl scale=0.001 0.001 0.001; visual mesh filename=../meshes/left_hip_side_v5_1.stl scale=0.001 0.001 0.001
- link left_shoulder: mass 0.172653501389095 -> 0.010592862408759271; geometry collision mesh filename=../meshes/left_shoulder_v5_1.stl scale=0.001 0.001 0.001; visual mesh filename=../meshes/left_shoulder_v5_1.stl scale=0.001 0.001 0.001
- link left_thigh: mass 0.142301969468209 -> 0.02898284927838432; geometry collision mesh filename=../meshes/left_thigh_v1_1.stl scale=0.001 0.001 0.001; visual mesh filename=../meshes/left_thigh_v1_1.stl scale=0.001 0.001 0.001
- link neck: mass 0.015549664333897642 -> 0.004247113386163016; geometry collision mesh filename=../meshes/neck_v6_1.stl scale=0.001 0.001 0.001; visual mesh filename=../meshes/neck_v6_1.stl scale=0.001 0.001 0.001
- link right_ankle: mass 0.151468601936124 -> 0.2722002973016189; geometry collision mesh filename=../meshes/right_ankle_v2_1.stl scale=0.001 0.001 0.001; visual mesh filename=../meshes/right_ankle_v2_1.stl scale=0.001 0.001 0.001
- link right_bicep: mass 0.212120407883451 -> 0.18636400760544294; geometry collision mesh filename=../meshes/right_bicep_v2_1.stl scale=0.001 0.001 0.001; visual mesh filename=../meshes/right_bicep_v2_1.stl scale=0.001 0.001 0.001
- link right_calve: mass 0.143723171211077 -> 0.15898038946070936; geometry collision mesh filename=../meshes/right_calve_v1_1.stl scale=0.001 0.001 0.001; visual mesh filename=../meshes/right_calve_v1_1.stl scale=0.001 0.001 0.001
- link right_foot: mass 0.16613521684361 -> 0.03929273129474384; geometry collision mesh filename=../meshes/right_foot_v2_1.stl scale=0.001 0.001 0.001; visual mesh filename=../meshes/right_foot_v2_1.stl scale=0.001 0.001 0.001
- link right_forearm: mass 0.06415483406403591 -> 0.05984540204112203; geometry collision mesh filename=../meshes/right_forearm_v1_1.stl scale=0.001 0.001 0.001; visual mesh filename=../meshes/right_forearm_v1_1.stl scale=0.001 0.001 0.001
- link right_hip_front: mass 0.211645971103128 -> 0.2722002973016189; geometry collision mesh filename=../meshes/right_hip_front_v5_1.stl scale=0.001 0.001 0.001; visual mesh filename=../meshes/right_hip_front_v5_1.stl scale=0.001 0.001 0.001
- link right_hip_side: mass 0.120655957656288 -> 0.03929574358294283; geometry collision mesh filename=../meshes/right_hip_side_v1_1.stl scale=0.001 0.001 0.001; visual mesh filename=../meshes/right_hip_side_v1_1.stl scale=0.001 0.001 0.001
- link right_shoulder: mass 0.172653501389095 -> 0.010592862408759271; geometry collision mesh filename=../meshes/right_shoulder_v1_1.stl scale=0.001 0.001 0.001; visual mesh filename=../meshes/right_shoulder_v1_1.stl scale=0.001 0.001 0.001
- link right_thigh: mass 0.142301969468209 -> 0.02898284927838432; geometry collision mesh filename=../meshes/right_thigh_v1_1.stl scale=0.001 0.001 0.001; visual mesh filename=../meshes/right_thigh_v1_1.stl scale=0.001 0.001 0.001
- link trunk: mass 1.62191101903404 -> 1.4429325287174738; geometry collision mesh filename=../meshes/base_link.stl scale=0.001 0.001 0.001; visual mesh filename=../meshes/base_link.stl scale=0.001 0.001 0.001
Joints:
- added joint camera_frame: type fixed, parent head, child camera, origin xyz=0.015 0.00145 0.0474 rpy=0.0 0.0 0.0, axis 0.0 0.0 0.0, limit lower=0.0 upper=0.0 effort=0.0 velocity=0.0
- joint head_pitch: origin xyz=0.0 -0.0195 0.025 rpy=0 0 0 -> xyz=0.0 -0.0185 0.025 rpy=0 0 0
- joint head_yaw: axis 0.0 0.0 -1.0 -> -0.0 0.0 1.0; origin xyz=0.009539 0.002537 0.03138 rpy=0 0 0 -> xyz=0.0 0.00025 0.0725 rpy=0 0 0
- joint left_ankle_pitch: axis -0.0 -1.0 0.0 -> 0.0 -1.0 0.0; origin xyz=0.0013 0.0 -0.088 rpy=0 0 0 -> xyz=0.0 0.0 -0.088 rpy=0 0 0
- joint left_ankle_roll: axis 1.0 0.0 0.0 -> 1.0 -0.0 0.0; origin xyz=0 -0.025 0  rpy=0 0 0 -> xyz=-0.0663 -0.0235 -0.036 rpy=0 0 0
- joint left_elbow: limit lower=0 upper=3.141592653589793 effort=2.5 velocity=5.76 -> lower=0 upper=3.141592653589793 effort=4.1 velocity=4.82; origin xyz=-0.018688 0.021938 -0.08675 rpy=0 0 0 -> xyz=-0.020403 0.018801 -0.119141 rpy=0 0 0
- joint left_hip_pitch: limit lower=-0.7853981633974483 upper=2.356194490192345 effort=4.1 velocity=4.82 -> lower=-0.7853981633974483 upper=2.356194490192345 effort=6.0 velocity=6.6; origin xyz=0.020771 0.0203 0.0 rpy=0 0 0 -> xyz=0.066269 0.0235 -0.036 rpy=0 0 0
- joint left_hip_roll: axis 1.0 0.0 0.0 -> 1.0 -0.0 0.0; limit lower=-0.7853981633974483 upper=1.5707963267948966 effort=4.1 velocity=4.82 -> lower=-0.7853981633974483 upper=1.5707963267948966 effort=6.0 velocity=6.6; origin xyz=-0.0205 0.0 -0.028 rpy=0 0 0 -> xyz=-0.0707 0.0 -0.028 rpy=0 0 0
- joint left_hip_yaw: axis 0.0 0.0 -1.0 -> -0.0 -0.0 -1.0; origin xyz=0.018839 0.067737 -0.20662 rpy=0 0 0 -> xyz=0.016 0.04125 -0.1085 rpy=0 0 0
- joint left_knee: axis -0.0 -1.0 0.0 -> 0.0 -1.0 -0.0; origin xyz=0.0 0.005269 -0.116 rpy=0 0 0 -> xyz=0.0 0.0 -0.072 rpy=0 0 0
- joint left_shoulder_pitch: axis -0.0 -1.0 0.0 -> -0.0 -1.0 -0.0; origin xyz=0.006539 0.112237 -0.00062 rpy=0 0 0 -> xyz=0.003 0.084 0.04475 rpy=0 0 0
- joint left_shoulder_roll: limit lower=0 upper=1.5707963267948966 effort=2.5 velocity=5.76 -> lower=0 upper=1.5707963267948966 effort=4.1 velocity=4.82; origin xyz=0.0205 0.0295 -0.021 rpy=0 0 0 -> xyz=0.019 0.0303 0.0 rpy=0 0 0
- joint right_ankle_pitch: origin xyz=0.0013 0.0 -0.088 rpy=0 0 0 -> xyz=0.0 0.0 -0.088 rpy=0 0 0
- joint right_ankle_roll: axis -1.0 0.0 0.0 -> -1.0 -0.0 0.0; origin xyz=0 -0.025 0 rpy=0 0 0 -> xyz=-0.0663 0.0235 -0.036 rpy=0 0 0
- joint right_elbow: axis 0.0 -1.0 0.0 -> -0.0 -1.0 0.0; limit lower=0 upper=3.141592653589793 effort=2.5 velocity=5.76 -> lower=0 upper=3.141592653589793 effort=4.1 velocity=4.82; origin xyz=-0.021312 -0.021937 -0.08675 rpy=0 0 0 -> xyz=-0.019597 -0.020801 -0.119141 rpy=0 0 0
- joint right_hip_pitch: limit lower=-0.7853981633974483 upper=2.356194490192345 effort=4.1 velocity=4.82 -> lower=-0.7853981633974483 upper=2.356194490192345 effort=6.0 velocity=6.6; origin xyz=0.020771 0.0203 0.0 rpy=0 0 0 -> xyz=0.0663 -0.0235 -0.036 rpy=0 0 0
- joint right_hip_roll: axis -1.0 0.0 0.0 -> -1.0 -0.0 -0.0; limit lower=-0.7853981633974483 upper=1.5707963267948966 effort=4.1 velocity=4.82 -> lower=-0.7853981633974483 upper=1.5707963267948966 effort=6.0 velocity=6.6; origin xyz=-0.0205 0.0 -0.028 rpy=0 0 0 -> xyz=-0.0707 0.0 -0.028 rpy=0 0 0
- joint right_hip_yaw: axis -0.0 -0.0 1.0 -> -0.0 0.0 1.0; origin xyz=0.018839 -0.062663 -0.20662 rpy=0 0 0 -> xyz=0.016 -0.04125 -0.1085 rpy=0 0 0
- joint right_knee: axis -0.0 -1.0 0.0 -> 0.0 -1.0 -0.0; origin xyz=0.0 0.005269 -0.116 rpy=0 0 0 -> xyz=0.0 0.0 -0.072 rpy=0 0 0
- joint right_shoulder_pitch: axis 0.0 -1.0 -0.0 -> -0.0 -1.0 -0.0; origin xyz=0.006539 -0.107163 -0.00062 rpy=0 0 0 -> xyz=0.003 -0.084 0.04475 rpy=0 0 0
- joint right_shoulder_roll: axis -1.0 0.0 0.0 -> -1.0 0.0 -0.0; limit lower=0 upper=1.5707963267948966 effort=2.5 velocity=5.76 -> lower=0 upper=1.5707963267948966 effort=4.1 velocity=4.82; origin xyz=0.021 -0.0295 -0.021 rpy=0 0 0 -> xyz=0.019 -0.0303 0.0 rpy=0 0 0
