Commit message: bez3 URDF for placo
Rename things and add joint limits to make placo urdf happy

File: soccer_description/bez3_description/urdf/bez3.urdf (robot description, URDF)
Before this commit: robot bez3, 54 links, 53 joints
Links:
- removed link 25t-servo-hub_1
- removed link 25t-servo-hub_Mirror__1
- removed link Component32_1
- removed link JX_servo_v12_1
- removed link TX2_board_v2_1
- removed link camera-link_1
- removed link camera_1
- removed link custom_servo_support__lower_neck__v2_1
- removed link elbow-attach_1
- removed link elbow-attach_Mirror__1
- removed link elbow-bearing_1
- removed link elbow-bearing_Mirror__1
- removed link gobilda-servo_1
- removed link gobilda-servo_Mirror__1
- removed link head_1
- removed link imu-link_1
- removed link left_bicep_1
- removed link left_calve_1
- removed link left_foot_1
- removed link left_forearm_1
- removed link left_hip_front_1
- removed link left_hip_side_1
- removed link left_thigh_1
- removed link neck_1
- removed link right_ankle_1
- removed link right_bicep_1
- removed link right_calve_1
- removed link right_foot_1
- removed link right_forearm_1
- removed link right_hip_side_1
- removed link right_thigh_1
- removed link torso_1
- added link 25t-servo-hub, mass 0.005584850212079893; collision mesh filename=../meshes_simplified/25t-servo-hub_1.stl scale=0.001 0.001 0.001; visual mesh filename=../meshes_simplified/25t-servo-hub_1.stl scale=0.001 0.001 0.001
- added link 25t-servo-hub_Mirror_, mass 0.005584585205775494; collision mesh filename=../meshes_simplified/25t-servo-hub_Mirror__1.stl scale=0.001 0.001 0.001; visual mesh filename=../meshes_simplified/25t-servo-hub_Mirror__1.stl scale=0.001 0.001 0.001
- added link Component32, mass 0.31999527000000005; collision mesh filename=../meshes_simplified/Component32_1.stl scale=0.001 0.001 0.001; visual mesh filename=../meshes_simplified/Component32_1.stl scale=0.001 0.001 0.001
- added link JX_servo_v12, mass 0.19853540350189502; collision mesh filename=../meshes_simplified/JX_servo_v12_1.stl scale=0.001 0.001 0.001; visual mesh filename=../meshes_simplified/JX_servo_v12_1.stl scale=0.001 0.001 0.001
- added link TX2_board_v2, mass 0.2621637321081563; collision mesh filename=../meshes_simplified/TX2_board_v2_1.stl scale=0.001 0.001 0.001; visual mesh filename=../meshes_simplified/TX2_board_v2_1.stl scale=0.001 0.001 0.001
- added link camera, mass 0.094257141411043; collision mesh filename=../meshes_simplified/camera_1.stl scale=0.001 0.001 0.001; visual mesh filename=../meshes_simplified/camera_1.stl scale=0.001 0.001 0.001
- added link camera-link, mass 0.00019624999999999932; collision mesh filename=../meshes_simplified/camera-link_1.stl scale=0.001 0.001 0.001; visual mesh filename=../meshes_simplified/camera-link_1.stl scale=0.001 0.001 0.001
- added link custom_servo_support__lower_neck__v2, mass 0.003136252201459725; collision mesh filename=../meshes_simplified/custom_servo_support__lower_neck__v2_1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 scale=0.001 0.001 0.001; visual mesh filename=../meshes_simplified/custom_servo_support__lower_neck__v2_1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 scale=0.001 0.001 0.001
- added link elbow-attach, mass 0.005141835270301899; collision mesh filename=../meshes_simplified/elbow-attach_1.stl scale=0.001 0.001 0.001; visual mesh filename=../meshes_simplified/elbow-attach_1.stl scale=0.001 0.001 0.001
- added link elbow-attach_Mirror_, mass 0.005141835270301901; collision mesh filename=../meshes_simplified/elbow-attach_Mirror__1.stl scale=0.001 0.001 0.001; visual mesh filename=../meshes_simplified/elbow-attach_Mirror__1.stl scale=0.001 0.001 0.001
- added link elbow-bearing, mass 0.004941715818268227; collision mesh filename=../meshes_simplified/elbow-bearing_1.stl scale=0.001 0.001 0.001; visual mesh filename=../meshes_simplified/elbow-bearing_1.stl scale=0.001 0.001 0.001
- added link elbow-bearing_Mirror_, mass 0.004941715818268223; collision mesh filename=../meshes_simplified/elbow-bearing_Mirror__1.stl scale=0.001 0.001 0.001; visual mesh filename=../meshes_simplified/elbow-bearing_Mirror__1.stl scale=0.001 0.001 0.001
- added link gobilda-servo, mass 0.060587311248822606; collision mesh filename=../meshes_simplified/gobilda-servo_1.stl scale=0.001 0.001 0.001; visual mesh filename=../meshes_simplified/gobilda-servo_1.stl scale=0.001 0.001 0.001
- added link gobilda-servo_Mirror_, mass 0.06058731124882261; collision mesh filename=../meshes_simplified/gobilda-servo_Mirror__1.stl scale=0.001 0.001 0.001; visual mesh filename=../meshes_simplified/gobilda-servo_Mirror__1.stl scale=0.001 0.001 0.001
- added link head, mass 0.007653734054253099; collision mesh filename=../meshes_simplified/head_1.stl scale=0.001 0.001 0.001; visual mesh filename=../meshes_simplified/head_1.stl scale=0.001 0.001 0.001
- added link imu-link, mass 0.00019625; collision mesh filename=../meshes_simplified/imu-link_1.stl scale=0.001 0.001 0.001; visual mesh filename=../meshes_simplified/imu-link_1.stl scale=0.001 0.001 0.001
- added link left_bicep, mass 0.011455626340925264; collision mesh filename=../meshes_simplified/left_bicep_1.stl scale=0.001 0.001 0.001; visual mesh filename=../meshes_simplified/left_bicep_1.stl scale=0.001 0.001 0.001
- added link left_calve, mass 0.035688451730559324; collision mesh filename=../meshes_simplified/left_calve_1.stl scale=0.001 0.001 0.001; visual mesh filename=../meshes_simplified/left_calve_1.stl scale=0.001 0.001 0.001
- added link left_foot, mass 0.12353540058419325; collision mesh filename=../meshes_simplified/left_foot_1.stl scale=0.001 0.001 0.001; visual mesh filename=../meshes_simplified/left_foot_1.stl scale=0.001 0.001 0.001
- added link left_forearm, mass 0.027371737365874692; collision mesh filename=../meshes_simplified/left_forearm_1.stl scale=0.001 0.001 0.001; visual mesh filename=../meshes_simplified/left_forearm_1.stl scale=0.001 0.001 0.001
- added link left_hip_front, mass 0.025976181664280836; collision mesh filename=../meshes_simplified/left_hip_front_1.stl scale=0.001 0.001 0.001; visual mesh filename=../meshes_simplified/left_hip_front_1.stl scale=0.001 0.001 0.001
- added link left_hip_side, mass 0.018999817606213904; collision mesh filename=../meshes_simplified/left_hip_side_1.stl scale=0.001 0.001 0.001; visual mesh filename=../meshes_simplified/left_hip_side_1.stl scale=0.001 0.001 0.001
- added link left_thigh, mass 0.04698736144283967; collision mesh filename=../meshes_simplified/left_thigh_1.stl scale=0.001 0.001 0.001; visual mesh filename=../meshes_simplified/left_thigh_1.stl scale=0.001 0.001 0.001
- added link neck, mass 0.012940388012734224; collision mesh filename=../meshes_simplified/neck_1.stl scale=0.001 0.001 0.001; visual mesh filename=../meshes_simplified/neck_1.stl scale=0.001 0.001 0.001
- added link right_ankle, mass 0.025976181664280826; collision mesh filename=../meshes_simplified/right_ankle_1.stl scale=0.001 0.001 0.001; visual mesh filename=../meshes_simplified/right_ankle_1.stl scale=0.001 0.001 0.001
- added link right_bicep, mass 0.011455626340925269; collision mesh filename=../meshes_simplified/right_bicep_1.stl scale=0.001 0.001 0.001; visual mesh filename=../meshes_simplified/right_bicep_1.stl scale=0.001 0.001 0.001
- added link right_calve, mass 0.035688490814490284; collision mesh filename=../meshes_simplified/right_calve_1.stl scale=0.001 0.001 0.001; visual mesh filename=../meshes_simplified/right_calve_1.stl scale=0.001 0.001 0.001
- added link right_foot, mass 0.12353541624057736; collision mesh filename=../meshes_simplified/right_foot_1.stl scale=0.001 0.001 0.001; visual mesh filename=../meshes_simplified/right_foot_1.stl scale=0.001 0.001 0.001
- added link right_forearm, mass 0.027371737365874692; collision mesh filename=../meshes_simplified/right_forearm_1.stl scale=0.001 0.001 0.001; visual mesh filename=../meshes_simplified/right_forearm_1.stl scale=0.001 0.001 0.001
- added link right_hip_side, mass 0.018999817606213918; collision mesh filename=../meshes_simplified/right_hip_side_1.stl scale=0.001 0.001 0.001; visual mesh filename=../meshes_simplified/right_hip_side_1.stl scale=0.001 0.001 0.001
- added link right_thigh, mass 0.04698731628682583; collision mesh filename=../meshes_simplified/right_thigh_1.stl scale=0.001 0.001 0.001; visual mesh filename=../meshes_simplified/right_thigh_1.stl scale=0.001 0.001 0.001
- added link trunk, mass 0.2968069064800233; collision mesh filename=../meshes_simplified/torso_1.stl scale=0.001 0.001 0.001; visual mesh filename=../meshes_simplified/torso_1.stl scale=0.001 0.001 0.001
- link 25t-servo-hub_2: geometry collision mesh filename=../meshes_simplified/25t-servo-hub_2.stl scale=0.001 0.001 0.001; visual mesh filename=../meshes_simplified/25t-servo-hub_2.stl scale=0.001 0.001 0.001
- link 25t-servo-hub_3: geometry collision mesh filename=../meshes_simplified/25t-servo-hub_3.stl scale=0.001 0.001 0.001; visual mesh filename=../meshes_simplified/25t-servo-hub_3.stl scale=0.001 0.001 0.001
- link 25t-servo-hub_4: geometry collision mesh filename=../meshes_simplified/25t-servo-hub_4.stl scale=0.001 0.001 0.001; visual mesh filename=../meshes_simplified/25t-servo-hub_4.stl scale=0.001 0.001 0.001
- link 25t-servo-hub_Mirror__2: geometry collision mesh filename=../meshes_simplified/25t-servo-hub_Mirror__2.stl scale=0.001 0.001 0.001; visual mesh filename=../meshes_simplified/25t-servo-hub_Mirror__2.stl scale=0.001 0.001 0.001
- link JX_servo_v12_11: geometry collision mesh filename=../meshes_simplified/JX_servo_v12_11.stl scale=0.001 0.001 0.001; visual mesh filename=../meshes_simplified/JX_servo_v12_11.stl scale=0.001 0.001 0.001
- link JX_servo_v12_12: geometry collision mesh filename=../meshes_simplified/JX_servo_v12_12.stl scale=0.001 0.001 0.001; visual mesh filename=../meshes_simplified/JX_servo_v12_12.stl scale=0.001 0.001 0.001
- link JX_servo_v12_13: geometry collision mesh filename=../meshes_simplified/JX_servo_v12_13.stl scale=0.001 0.001 0.001; visual mesh filename=../meshes_simplified/JX_servo_v12_13.stl scale=0.001 0.001 0.001
- link JX_servo_v12_14: geometry collision mesh filename=../meshes_simplified/JX_servo_v12_14.stl scale=0.001 0.001 0.001; visual mesh filename=../meshes_simplified/JX_servo_v12_14.stl scale=0.001 0.001 0.001
- link JX_servo_v12_15: geometry collision mesh filename=../meshes_simplified/JX_servo_v12_15.stl scale=0.001 0.001 0.001; visual mesh filename=../meshes_simplified/JX_servo_v12_15.stl scale=0.001 0.001 0.001
- link JX_servo_v12_16: geometry collision mesh filename=../meshes_simplified/JX_servo_v12_16.stl scale=0.001 0.001 0.001; visual mesh filename=../meshes_simplified/JX_servo_v12_16.stl scale=0.001 0.001 0.001
- link JX_servo_v12_17: geometry collision mesh filename=../meshes_simplified/JX_servo_v12_17.stl scale=0.001 0.001 0.001; visual mesh filename=../meshes_simplified/JX_servo_v12_17.stl scale=0.001 0.001 0.001
- link JX_servo_v12_18: geometry collision mesh filename=../meshes_simplified/JX_servo_v12_18.stl scale=0.001 0.001 0.001; visual mesh filename=../meshes_simplified/JX_servo_v12_18.stl scale=0.001 0.001 0.001
- link JX_servo_v12_19: geometry collision mesh filename=../meshes_simplified/JX_servo_v12_19.stl scale=0.001 0.001 0.001; visual mesh filename=../meshes_simplified/JX_servo_v12_19.stl scale=0.001 0.001 0.001
- link JX_servo_v12_8: geometry collision mesh filename=../meshes_simplified/JX_servo_v12_8.stl scale=0.001 0.001 0.001; visual mesh filename=../meshes_simplified/JX_servo_v12_8.stl scale=0.001 0.001 0.001
- link JX_servo_v12_9: geometry collision mesh filename=../meshes_simplified/JX_servo_v12_9.stl scale=0.001 0.001 0.001; visual mesh filename=../meshes_simplified/JX_servo_v12_9.stl scale=0.001 0.001 0.001
- link base_link: geometry collision mesh filename=../meshes_simplified/base_link.stl scale=0.001 0.001 0.001; visual mesh filename=../meshes_simplified/base_link.stl scale=0.001 0.001 0.001
- link gobilda-servo_3: geometry collision mesh filename=../meshes_simplified/gobilda-servo_3.stl scale=0.001 0.001 0.001; visual mesh filename=../meshes_simplified/gobilda-servo_3.stl scale=0.001 0.001 0.001
- link gobilda-servo_4: geometry collision mesh filename=../meshes_simplified/gobilda-servo_4.stl scale=0.001 0.001 0.001; visual mesh filename=../meshes_simplified/gobilda-servo_4.stl scale=0.001 0.001 0.001
- link gobilda-servo_5: geometry collision mesh filename=../meshes_simplified/gobilda-servo_5.stl scale=0.001 0.001 0.001; visual mesh filename=../meshes_simplified/gobilda-servo_5.stl scale=0.001 0.001 0.001
- link gobilda-servo_Mirror__2: geometry collision mesh filename=../meshes_simplified/gobilda-servo_Mirror__2.stl scale=0.001 0.001 0.001; visual mesh filename=../meshes_simplified/gobilda-servo_Mirror__2.stl scale=0.001 0.001 0.001
- link left_hip_front_2: geometry collision mesh filename=../meshes_simplified/left_hip_front_2.stl scale=0.001 0.001 0.001; visual mesh filename=../meshes_simplified/left_hip_front_2.stl scale=0.001 0.001 0.001
- link right_ankle_2: geometry collision mesh filename=../meshes_simplified/right_ankle_2.stl scale=0.001 0.001 0.001; visual mesh filename=../meshes_simplified/right_ankle_2.stl scale=0.001 0.001 0.001
Joints:
- removed joint head_motor_0
- removed joint head_motor_1
- removed joint left_arm_motor_0
- removed joint left_arm_motor_1
- removed joint left_leg_motor_0
- removed joint left_leg_motor_1
- removed joint left_leg_motor_2
- removed joint left_leg_motor_3
- removed joint left_leg_motor_4
- removed joint left_leg_motor_5
- removed joint right_arm_motor_0
- removed joint right_arm_motor_1
- removed joint right_leg_motor_0
- removed joint right_leg_motor_1
- removed joint right_leg_motor_2
- removed joint right_leg_motor_3
- removed joint right_leg_motor_4
- removed joint right_leg_motor_5
- added joint head_pitch: type revolute, parent 25t-servo-hub_4, child gobilda-servo_5, origin xyz=0.0 0.002794 0.0 rpy=0 0 0, axis -0.0 1.0 -0.0, limit lower=-1.5707963267948966 upper=1.5707963267948966 effort=1.5 velocity=6.39
- added joint head_yaw: type revolute, parent gobilda-servo_4, child 25t-servo-hub_3, origin xyz=0.0075 0.0075 0.0369 rpy=0 0 0, axis 0.0 -0.0 1.0, limit lower=-1.5707963267948966 upper=1.5707963267948966 effort=1.5 velocity=6.39
- added joint left_ankle_pitch: type revolute, parent left_calve, child JX_servo_v12_12, origin xyz=-0.00855 0.028 -0.085005 rpy=0 0 0, axis 0.0 -1.0 0.0, limit lower=-1.5707963267948966 upper=1.5707963267948966 effort=1.5 velocity=6.39
- added joint left_ankle_roll: type revolute, parent JX_servo_v12_13, child left_foot, origin xyz=0.0264 0.0085 -0.0549 rpy=0 0 0, axis -1.0 -0.0 -0.0, limit lower=-1.5707963267948966 upper=1.5707963267948966 effort=1.5 velocity=6.39
- added joint left_elbow: type revolute, parent gobilda-servo_3, child 25t-servo-hub_2, origin xyz=0.0075 -0.0369 -0.0075 rpy=0 0 0, axis -0.0 1.0 -0.0, limit lower=-1.5707963267948966 upper=1.5707963267948966 effort=1.5 velocity=6.39
- added joint left_hip_pitch: type revolute, parent JX_servo_v12_9, child left_thigh, origin xyz=-0.0085 0.0225 0.0549 rpy=0 0 0, axis 0.0 -1.0 0.0, limit lower=-1.5707963267948966 upper=1.5707963267948966 effort=1.5 velocity=6.39
- added joint left_hip_roll: type revolute, parent left_hip_side, child JX_servo_v12_8, origin xyz=-0.03 0.0 -0.035336 rpy=0 0 0, axis -1.0 -0.0 -0.0, limit lower=-1.5707963267948966 upper=1.5707963267948966 effort=1.5 velocity=6.39
- added joint left_hip_yaw: type revolute, parent JX_servo_v12, child left_hip_side, origin xyz=0.018 0.0 -0.0264 rpy=0 0 0, axis 0.0 0.0 1.0, limit lower=-1.5707963267948966 upper=1.5707963267948966 effort=1.5 velocity=6.39
- added joint left_knee: type revolute, parent left_thigh, child JX_servo_v12_11, origin xyz=0.0 0.0 -0.124 rpy=0 0 0, axis 0.0 -1.0 0.0, limit lower=-1.5707963267948966 upper=1.5707963267948966 effort=1.5 velocity=6.39
- added joint left_shoulder_pitch: type revolute, parent 25t-servo-hub, child gobilda-servo, origin xyz=0.0 0.002794 0.0 rpy=0 0 0, axis 0.0 -1.0 0.0, limit lower=-1.5707963267948966 upper=1.5707963267948966 effort=1.5 velocity=6.39
- added joint right_ankle_pitch: type revolute, parent right_calve, child JX_servo_v12_18, origin xyz=-0.00855 -0.028 -0.085005 rpy=0 0 0, axis -0.0 -1.0 -0.0, limit lower=-1.5707963267948966 upper=1.5707963267948966 effort=1.5 velocity=6.39
- added joint right_ankle_roll: type revolute, parent JX_servo_v12_19, child right_foot, origin xyz=0.0264 -0.0085 -0.0549 rpy=0 0 0, axis -1.0 0.0 -0.0, limit lower=-1.5707963267948966 upper=1.5707963267948966 effort=1.5 velocity=6.39
- added joint right_elbow: type revolute, parent gobilda-servo_Mirror__2, child 25t-servo-hub_Mirror__2, origin xyz=0.0075 0.0369 -0.0075 rpy=0 0 0, axis -0.0 1.0 0.0, limit lower=-1.5707963267948966 upper=1.5707963267948966 effort=1.5 velocity=6.39
- added joint right_hip_pitch: type revolute, parent JX_servo_v12_16, child right_thigh, origin xyz=-0.0085 -0.0225 0.0549 rpy=0 0 0, axis 0.0 1.0 0.0, limit lower=-1.5707963267948966 upper=1.5707963267948966 effort=1.5 velocity=6.39
- added joint right_hip_roll: type revolute, parent right_hip_side, child JX_servo_v12_15, origin xyz=-0.03 0.0 -0.035336 rpy=0 0 0, axis 1.0 0.0 0.0, limit lower=-1.5707963267948966 upper=1.5707963267948966 effort=1.5 velocity=6.39
- added joint right_hip_yaw: type revolute, parent JX_servo_v12_14, child right_hip_side, origin xyz=0.018 0.0 -0.0264 rpy=0 0 0, axis -0.0 0.0 -1.0, limit lower=-1.5707963267948966 upper=1.5707963267948966 effort=1.5 velocity=6.39
- added joint right_knee: type revolute, parent right_thigh, child JX_servo_v12_17, origin xyz=0.0 0.0 -0.124 rpy=0 0 0, axis -0.0 -1.0 -0.0, limit lower=-1.5707963267948966 upper=1.5707963267948966 effort=1.5 velocity=6.39
- added joint right_shoulder_pitch: type revolute, parent 25t-servo-hub_Mirror_, child gobilda-servo_Mirror_, origin xyz=0.0 -0.002794 0.0 rpy=0 0 0, axis 0.0 -1.0 0.0, limit lower=-1.5707963267948966 upper=1.5707963267948966 effort=1.5 velocity=6.39
- joint Rigid1: child torso_1 -> trunk; limit (none) -> lower=-1.5707963267948966 upper=1.5707963267948966 effort=1.5 velocity=6.39
- joint Rigid11: limit (none) -> lower=-1.5707963267948966 upper=1.5707963267948966 effort=1.5 velocity=6.39
- joint Rigid12: limit (none) -> lower=-1.5707963267948966 upper=1.5707963267948966 effort=1.5 velocity=6.39
- joint Rigid14: limit (none) -> lower=-1.5707963267948966 upper=1.5707963267948966 effort=1.5 velocity=6.39; parent torso_1 -> trunk
- joint Rigid17: child right_ankle_1 -> right_ankle; limit (none) -> lower=-1.5707963267948966 upper=1.5707963267948966 effort=1.5 velocity=6.39
- joint Rigid18: limit (none) -> lower=-1.5707963267948966 upper=1.5707963267948966 effort=1.5 velocity=6.39; parent right_ankle_1 -> right_ankle
- joint Rigid2: child JX_servo_v12_1 -> JX_servo_v12; limit (none) -> lower=-1.5707963267948966 upper=1.5707963267948966 effort=1.5 velocity=6.39; parent torso_1 -> trunk
- joint Rigid21: child right_calve_1 -> right_calve; limit (none) -> lower=-1.5707963267948966 upper=1.5707963267948966 effort=1.5 velocity=6.39
- joint Rigid23: limit (none) -> lower=-1.5707963267948966 upper=1.5707963267948966 effort=1.5 velocity=6.39
- joint Rigid24: limit (none) -> lower=-1.5707963267948966 upper=1.5707963267948966 effort=1.5 velocity=6.39
- joint Rigid26: child 25t-servo-hub_1 -> 25t-servo-hub; limit (none) -> lower=-1.5707963267948966 upper=1.5707963267948966 effort=1.5 velocity=6.39; parent torso_1 -> trunk
- joint Rigid28: child left_bicep_1 -> left_bicep; limit (none) -> lower=-1.5707963267948966 upper=1.5707963267948966 effort=1.5 velocity=6.39; parent gobilda-servo_1 -> gobilda-servo
- joint Rigid29: limit (none) -> lower=-1.5707963267948966 upper=1.5707963267948966 effort=1.5 velocity=6.39; parent left_bicep_1 -> left_bicep
- joint Rigid31: child elbow-attach_1 -> elbow-attach; limit (none) -> lower=-1.5707963267948966 upper=1.5707963267948966 effort=1.5 velocity=6.39
- joint Rigid32: child left_forearm_1 -> left_forearm; limit (none) -> lower=-1.5707963267948966 upper=1.5707963267948966 effort=1.5 velocity=6.39; parent elbow-attach_1 -> elbow-attach
- joint Rigid33: child elbow-bearing_1 -> elbow-bearing; limit (none) -> lower=-1.5707963267948966 upper=1.5707963267948966 effort=1.5 velocity=6.39; parent left_forearm_1 -> left_forearm
- joint Rigid34: child 25t-servo-hub_Mirror__1 -> 25t-servo-hub_Mirror_; limit (none) -> lower=-1.5707963267948966 upper=1.5707963267948966 effort=1.5 velocity=6.39; parent torso_1 -> trunk
- joint Rigid36: child right_bicep_1 -> right_bicep; limit (none) -> lower=-1.5707963267948966 upper=1.5707963267948966 effort=1.5 velocity=6.39; parent gobilda-servo_Mirror__1 -> gobilda-servo_Mirror_
- joint Rigid37: limit (none) -> lower=-1.5707963267948966 upper=1.5707963267948966 effort=1.5 velocity=6.39; parent right_bicep_1 -> right_bicep
- joint Rigid39: child elbow-attach_Mirror__1 -> elbow-attach_Mirror_; limit (none) -> lower=-1.5707963267948966 upper=1.5707963267948966 effort=1.5 velocity=6.39
- joint Rigid40: child right_forearm_1 -> right_forearm; limit (none) -> lower=-1.5707963267948966 upper=1.5707963267948966 effort=1.5 velocity=6.39; parent elbow-attach_Mirror__1 -> elbow-attach_Mirror_
- joint Rigid41: child elbow-bearing_Mirror__1 -> elbow-bearing_Mirror_; limit (none) -> lower=-1.5707963267948966 upper=1.5707963267948966 effort=1.5 velocity=6.39; parent right_forearm_1 -> right_forearm
- joint Rigid42: child custom_servo_support__lower_neck__v2_1 -> custom_servo_support__lower_neck__v2; limit (none) -> lower=-1.5707963267948966 upper=1.5707963267948966 effort=1.5 velocity=6.39; parent torso_1 -> trunk
- joint Rigid43: limit (none) -> lower=-1.5707963267948966 upper=1.5707963267948966 effort=1.5 velocity=6.39; parent custom_servo_support__lower_neck__v2_1 -> custom_servo_support__lower_neck__v2
- joint Rigid45: child neck_1 -> neck; limit (none) -> lower=-1.5707963267948966 upper=1.5707963267948966 effort=1.5 velocity=6.39
- joint Rigid46: limit (none) -> lower=-1.5707963267948966 upper=1.5707963267948966 effort=1.5 velocity=6.39; parent neck_1 -> neck
- joint Rigid48: child head_1 -> head; limit (none) -> lower=-1.5707963267948966 upper=1.5707963267948966 effort=1.5 velocity=6.39
- joint Rigid49: child camera_1 -> camera; limit (none) -> lower=-1.5707963267948966 upper=1.5707963267948966 effort=1.5 velocity=6.39; parent head_1 -> head
- joint Rigid5: child left_hip_front_1 -> left_hip_front; limit (none) -> lower=-1.5707963267948966 upper=1.5707963267948966 effort=1.5 velocity=6.39
- joint Rigid52: child Component32_1 -> Component32; limit (none) -> lower=-1.5707963267948966 upper=1.5707963267948966 effort=1.5 velocity=6.39; parent torso_1 -> trunk
- joint Rigid53: child TX2_board_v2_1 -> TX2_board_v2; limit (none) -> lower=-1.5707963267948966 upper=1.5707963267948966 effort=1.5 velocity=6.39; parent Component32_1 -> Component32
- joint Rigid6: limit (none) -> lower=-1.5707963267948966 upper=1.5707963267948966 effort=1.5 velocity=6.39; parent left_hip_front_1 -> left_hip_front
- joint Rigid9: child left_calve_1 -> left_calve; limit (none) -> lower=-1.5707963267948966 upper=1.5707963267948966 effort=1.5 velocity=6.39
- joint camera_joint: child camera-link_1 -> camera-link; limit (none) -> lower=-1.5707963267948966 upper=1.5707963267948966 effort=1.5 velocity=6.39; parent camera_1 -> camera; type continuous -> revolute
- joint imu_joint: child imu-link_1 -> imu-link; limit (none) -> lower=-1.5707963267948966 upper=1.5707963267948966 effort=1.5 velocity=6.39; parent torso_1 -> trunk; type continuous -> revolute
