Commit message: Joint limits to make IK deterministic for placo
Knee joint limits needed to force the knees to bend the right way

File: soccer_description/bez3_description/urdf/bez3.urdf (robot description, URDF)
Before this commit: robot bez3, 54 links, 53 joints
Joints:
- joint left_knee: limit lower=-1.5707963267948966 upper=1.5707963267948966 effort=1.5 velocity=6.39 -> lower=-3.14 upper=0 effort=1.5 velocity=6.39
- joint right_knee: limit lower=-1.5707963267948966 upper=1.5707963267948966 effort=1.5 velocity=6.39 -> lower=-3.14 upper=0 effort=1.5 velocity=6.39

Commit message: Change bez3 foot position, start tuning

File: soccer_description/bez3_description/urdf/bez3.urdf (robot description, URDF)
Before this commit: robot bez3, 54 links, 53 joints
Joints:
- joint left_ankle_roll: origin xyz=0.0264 0.0085 -0.0549 rpy=0 0 0 -> xyz=0.0764 0.0085 -0.0549 rpy=0 0 0
- joint right_ankle_roll: origin xyz=0.0264 -0.0085 -0.0549 rpy=0 0 0 -> xyz=0.0764 -0.0085 -0.0549 rpy=0 0 0
