Commit message: got getupfront to work

File: soccer_description/assembly_description/urdf/robot.urdf (robot description, URDF)
Before this commit: robot assembly, 22 links, 21 joints
Joints:
- joint left_ankle_roll: origin xyz=0 -0.025 0  rpy=0 0 0 -> xyz=-0.0663 -0.0235 -0.036 rpy=0 0 0
- joint right_ankle_roll: origin xyz= 0 0.025 0  rpy=0 0 0 -> xyz=-0.0663 0.0235 -0.036 rpy=0 0 0
