Commit message: fixed the tf tree by editing the xacro to move properly. tuned the walking pid, tuned the trajectory and ready for video

File: soccer_description/assembly_description/urdf/assembly.xacro (robot description, xacro)
@@ -6,10 +6,10 @@
 <link name="base_link">
   <inertial>
-    <origin xyz="-0.02024929347181477 0.00329389202927954 -0.02671963219571571" rpy="0 0 0"/>
+    <origin xyz="-0.02024929347181477 0.00329389202927954 -0.02671963219571571" rpy="-1.57 0  0"/>
     <mass value="3.0429325287174738"/>
     <inertia ixx="0.009761" iyy="0.006663" izz="0.008082" ixy="7.9e-05" iyz="8.1e-05" ixz="-0.000195"/>
   </inertial>
   <visual>
-    <origin xyz="0 0 0" rpy="0 0 0"/>
+    <origin xyz="0 0 0" rpy="-1.57 0  0"/>
     <geometry>
       <mesh filename="package://assembly_description/meshes/simplified/base_link.stl" scale="0.001 0.001 0.001"/>
@@ -18,5 +18,5 @@
   </visual>
   <collision>
-    <origin xyz="0 0 0" rpy="0 0 0"/>
+    <origin xyz="0 0 0" rpy="-1.57 0  0"/>
     <geometry>
       <mesh filename="package://assembly_description/meshes/simplified/base_link.stl" scale="0.001 0.001 0.001"/>
@@ -24,12 +24,12 @@
   </collision>
 </link>
-<link name="left_hip_side_v5_1">
-  <inertial>
-    <origin xyz="-0.0176303342104258 -2.8796409701214998e-15 -0.007188418776152797" rpy="0 0 0"/>
+<link name="left_hip_side">
+  <inertial>
+    <origin xyz="-0.0176303342104258 -2.8796409701214998e-15 -0.007188418776152797" rpy="-1.57 0  0"/>
     <mass value="0.03929574358294283"/>
     <inertia ixx="7e-06" iyy="9.2e-05" izz="9e-05" ixy="0.0" iyz="0.0" ixz="4e-06"/>
   </inertial>
   <visual>
-    <origin xyz="-0.016 -0.04125 0.1085" rpy="0 0 0"/>
+    <origin xyz="-0.016 -0.04125 0.1085" rpy="-1.57 0  0"/>
     <geometry>
       <mesh filename="package://assembly_description/meshes/simplified/left_hip_side_v5_1.stl" scale="0.001 0.001 0.001"/>
@@ -38,5 +38,5 @@
   </visual>
   <collision>
-    <origin xyz="-0.016 -0.04125 0.1085" rpy="0 0 0"/>
+    <origin xyz="-0.016 -0.04125 0.1085" rpy="-1.57 0  0"/>
     <geometry>
       <mesh filename="package://assembly_description/meshes/simplified/left_hip_side_v5_1.stl" scale="0.001 0.001 0.001"/>
@@ -44,12 +44,12 @@
   </collision>
 </link>
-<link name="left_foot_v10_1">
-  <inertial>
-    <origin xyz="0.05312327716355333 0.01311710007932914 -0.017187548637288774" rpy="0 0 0"/>
+<link name="left_foot">
+  <inertial>
+    <origin xyz="0.05312327716355333 0.01311710007932914 -0.017187548637288774" rpy="-1.57 0  0"/>
     <mass value="0.03929273129474386"/>
     <inertia ixx="2.6e-05" iyy="0.000124" izz="0.000144" ixy="2e-06" iyz="2e-06" ixz="-3e-06"/>
   </inertial>
   <visual>
-    <origin xyz="0.054731 -0.04125 0.3685" rpy="0 0 0"/>
+    <origin xyz="0.054731 -0.04125 0.3685" rpy="-1.57 0  0"/>
     <geometry>
       <mesh filename="package://assembly_description/meshes/simplified/left_foot_v10_1.stl" scale="0.001 0.001 0.001"/>
@@ -58,5 +58,5 @@
   </visual>
   <collision>
-    <origin xyz="0.054731 -0.04125 0.3685" rpy="0 0 0"/>
+    <origin xyz="0.054731 -0.04125 0.3685" rpy="-1.57 0  0"/>
     <geometry>
       <mesh filename="package://assembly_description/meshes/simplified/left_foot_v10_1.stl" scale="0.001 0.001 0.001"/>
@@ -64,12 +64,12 @@
   </collision>
 </link>
-<link name="left_shoulder_v5_1">
-  <inertial>
-    <origin xyz="8.922688803092438e-11 0.007844026821939576 2.0192181260370035e-14" rpy="0 0 0"/>
+<link name="left_shoulder">
+  <inertial>
+    <origin xyz="8.922688803092438e-11 0.007844026821939576 2.0192181260370035e-14" rpy="-1.57 0  0"/>
     <mass value="0.010592862408759271"/>
     <inertia ixx="1e-06" iyy="3e-06" izz="3e-06" ixy="0.0" iyz="-0.0" ixz="0.0"/>
   </inertial>
   <visual>
-    <origin xyz="-0.003 -0.084 -0.04475" rpy="0 0 0"/>
+    <origin xyz="-0.003 -0.084 -0.04475" rpy="-1.57 0  0"/>
     <geometry>
       <mesh filename="package://assembly_description/meshes/simplified/left_shoulder_v5_1.stl" scale="0.001 0.001 0.001"/>
@@ -78,5 +78,5 @@
   </visual>
   <collision>
-    <origin xyz="-0.003 -0.084 -0.04475" rpy="0 0 0"/>
+    <origin xyz="-0.003 -0.084 -0.04475" rpy="-1.57 0  0"/>
     <geometry>
       <mesh filename="package://assembly_description/meshes/simplified/left_shoulder_v5_1.stl" scale="0.001 0.001 0.001"/>
@@ -84,12 +84,12 @@
   </collision>
 </link>
-<link name="left_bicep_v6_1">
-  <inertial>
-    <origin xyz="-0.019420473733666368 0.00010477857835172744 -0.06051458521988624" rpy="0 0 0"/>
+<link name="left_bicep">
+  <inertial>
+    <origin xyz="-0.019420473733666368 0.00010477857835172744 -0.06051458521988624" rpy="-1.57 0  0"/>
     <mass value="0.18636400760544294"/>
     <inertia ixx="0.000442" iyy="0.000444" izz="3.5e-05" ixy="0.0" iyz="3e-06" ixz="-1e-05"/>
   </inertial>
   <visual>
-    <origin xyz="-0.022 -0.1143 -0.04475" rpy="0 0 0"/>
+    <origin xyz="-0.022 -0.1143 -0.04475" rpy="-1.57 0  0"/>
     <geometry>
       <mesh filename="package://assembly_description/meshes/simplified/left_bicep_v6_1.stl" scale="0.001 0.001 0.001"/>
@@ -98,5 +98,5 @@
   </visual>
   <collision>
-    <origin xyz="-0.022 -0.1143 -0.04475" rpy="0 0 0"/>
+    <origin xyz="-0.022 -0.1143 -0.04475" rpy="-1.57 0  0"/>
     <geometry>
       <mesh filename="package://assembly_description/meshes/simplified/left_bicep_v6_1.stl" scale="0.001 0.001 0.001"/>
@@ -104,12 +104,12 @@
   </collision>
 </link>
-<link name="left_forearm_v4_1">
-  <inertial>
-    <origin xyz="0.0004904443113911659 -0.01970036030468776 -0.0814474917977369" rpy="0 0 0"/>
+<link name="left_forearm">
+  <inertial>
+    <origin xyz="0.0004904443113911659 -0.01970036030468776 -0.0814474917977369" rpy="-1.57 0  0"/>
     <mass value="0.05984540204112203"/>
     <inertia ixx="0.000124" iyy="0.000119" izz="2.1e-05" ixy="-0.0" iyz="-0.0" ixz="-0.0"/>
   </inertial>
   <visual>
-    <origin xyz="-0.001597 -0.133101 0.074391" rpy="0 0 0"/>
+    <origin xyz="-0.001597 -0.133101 0.074391" rpy="-1.57 0  0"/>
     <geometry>
       <mesh filename="package://assembly_description/meshes/simplified/left_forearm_v4_1.stl" scale="0.001 0.001 0.001"/>
@@ -118,5 +118,5 @@
   </visual>
   <collision>
-    <origin xyz="-0.001597 -0.133101 0.074391" rpy="0 0 0"/>
+    <origin xyz="-0.001597 -0.133101 0.074391" rpy="-1.57 0  0"/>
     <geometry>
       <mesh filename="package://assembly_description/meshes/simplified/left_forearm_v4_1.stl" scale="0.001 0.001 0.001"/>
@@ -124,12 +124,12 @@
   </collision>
 </link>
-<link name="neck_v6_1">
-  <inertial>
-    <origin xyz="8.936969206796164e-11 0.0012409815706136025 0.012040454865583" rpy="0 0 0"/>
+<link name="neck">
+  <inertial>
+    <origin xyz="8.936969206796164e-11 0.0012409815706136025 0.012040454865583" rpy="-1.57 0  0"/>
     <mass value="0.004247113386163016"/>
     <inertia ixx="2e-06" iyy="1e-06" izz="2e-06" ixy="-0.0" iyz="-0.0" ixz="0.0"/>
   </inertial>
   <visual>
-    <origin xyz="-0.0 -0.00025 -0.0725" rpy="0 0 0"/>
+    <origin xyz="-0.0 -0.00025 -0.0725" rpy="-1.57 0  0"/>
     <geometry>
       <mesh filename="package://assembly_description/meshes/simplified/neck_v6_1.stl" scale="0.001 0.001 0.001"/>
@@ -138,5 +138,5 @@
   </visual>
   <collision>
-    <origin xyz="-0.0 -0.00025 -0.0725" rpy="0 0 0"/>
+    <origin xyz="-0.0 -0.00025 -0.0725" rpy="-1.57 0  0"/>
     <geometry>
       <mesh filename="package://assembly_description/meshes/simplified/neck_v6_1.stl" scale="0.001 0.001 0.001"/>
@@ -144,12 +144,12 @@
   </collision>
 </link>
-<link name="head_v4_1">
-  <inertial>
-    <origin xyz="-0.0025761957912120003 0.01899177474904292 0.03300593624682499" rpy="0 0 0"/>
+<link name="head">
+  <inertial>
+    <origin xyz="-0.0025761957912120003 0.01899177474904292 0.03300593624682499" rpy="-1.57 0  0"/>
     <mass value="0.26433915470596575"/>
     <inertia ixx="0.000237" iyy="0.000239" izz="0.000166" ixy="-0.0" iyz="-2e-06" ixz="-5.6e-05"/>
   </inertial>
   <visual>
-    <origin xyz="-0.0 0.01825 -0.0975" rpy="0 0 0"/>
+    <origin xyz="-0.0 0.01825 -0.0975" rpy="-1.57 0  0"/>
     <geometry>
       <mesh filename="package://assembly_description/meshes/simplified/head_v4_1.stl" scale="0.001 0.001 0.001"/>
@@ -158,5 +158,5 @@
   </visual>
   <collision>
-    <origin xyz="-0.0 0.01825 -0.0975" rpy="0 0 0"/>
+    <origin xyz="-0.0 0.01825 -0.0975" rpy="-1.57 0  0"/>
     <geometry>
       <mesh filename="package://assembly_description/meshes/simplified/head_v4_1.stl" scale="0.001 0.001 0.001"/>
@@ -164,12 +164,12 @@
   </collision>
 </link>
-<link name="right_hip_side_v1_1">
-  <inertial>
-    <origin xyz="-0.017630334210425074 -2.7131075164277263e-15 -0.007188418776152866" rpy="0 0 0"/>
+<link name="right_hip_side">
+  <inertial>
+    <origin xyz="-0.017630334210425074 -2.7131075164277263e-15 -0.007188418776152866" rpy="-1.57 0  0"/>
     <mass value="0.03929574358294283"/>
     <inertia ixx="7e-06" iyy="9.2e-05" izz="9e-05" ixy="0.0" iyz="0.0" ixz="4e-06"/>
   </inertial>
   <visual>
-    <origin xyz="-0.016 0.04125 0.1085" rpy="0 0 0"/>
+    <origin xyz="-0.016 0.04125 0.1085" rpy="-1.57 0  0"/>
     <geometry>
       <mesh filename="package://assembly_description/meshes/simplified/right_hip_side_v1_1.stl" scale="0.001 0.001 0.001"/>
@@ -178,5 +178,5 @@
   </visual>
   <collision>
-    <origin xyz="-0.016 0.04125 0.1085" rpy="0 0 0"/>
+    <origin xyz="-0.016 0.04125 0.1085" rpy="-1.57 0  0"/>
     <geometry>
       <mesh filename="package://assembly_description/meshes/simplified/right_hip_side_v1_1.stl" scale="0.001 0.001 0.001"/>
@@ -184,12 +184,12 @@
   </collision>
 </link>
-<link name="right_ankle_v2_1">
-  <inertial>
-    <origin xyz="-0.019332548462524354 0.02355722240141854 -0.018170467896408804" rpy="0 0 0"/>
+<link name="right_ankle">
+  <inertial>
+    <origin xyz="-0.019332548462524354 0.02355722240141854 -0.018170467896408804" rpy="-1.57 0  0"/>
     <mass value="0.2722002973016189"/>
     <inertia ixx="0.000108" iyy="0.000229" izz="0.000189" ixy="-0.0" iyz="1e-06" ixz="-1.3e-05"/>
   </inertial>
   <visual>
-    <origin xyz="-0.0116 0.06475 0.3325" rpy="0 0 0"/>
+    <origin xyz="-0.0116 0.06475 0.3325" rpy="-1.57 0  0"/>
     <geometry>
       <mesh filename="package://assembly_description/meshes/simplified/right_ankle_v2_1.stl" scale="0.001 0.001 0.001"/>
@@ -198,5 +198,5 @@
   </visual>
   <collision>
-    <origin xyz="-0.0116 0.06475 0.3325" rpy="0 0 0"/>
+    <origin xyz="-0.0116 0.06475 0.3325" rpy="-1.57 0  0"/>
     <geometry>
       <mesh filename="package://assembly_description/meshes/simplified/right_ankle_v2_1.stl" scale="0.001 0.001 0.001"/>
@@ -204,12 +204,12 @@
   </collision>
 </link>
-<link name="right_foot_v2_1">
-  <inertial>
-    <origin xyz="0.053123527163554944 -0.01311710007932746 -0.017187548637289052" rpy="0 0 0"/>
+<link name="right_foot">
+  <inertial>
+    <origin xyz="0.053123527163554944 -0.01311710007932746 -0.017187548637289052" rpy="-1.57 0  0"/>
     <mass value="0.03929273129474384"/>
     <inertia ixx="2.6e-05" iyy="0.000124" izz="0.000144" ixy="-2e-06" iyz="-2e-06" ixz="-3e-06"/>
   </inertial>
   <visual>
-    <origin xyz="0.0547 0.04125 0.3685" rpy="0 0 0"/>
+    <origin xyz="0.0547 0.04125 0.3685" rpy="-1.57 0  0"/>
     <geometry>
       <mesh filename="package://assembly_description/meshes/simplified/right_foot_v2_1.stl" scale="0.001 0.001 0.001"/>
@@ -218,5 +218,5 @@
   </visual>
   <collision>
-    <origin xyz="0.0547 0.04125 0.3685" rpy="0 0 0"/>
+    <origin xyz="0.0547 0.04125 0.3685" rpy="-1.57 0  0"/>
     <geometry>
       <mesh filename="package://assembly_description/meshes/simplified/right_foot_v2_1.stl" scale="0.001 0.001 0.001"/>
@@ -224,12 +224,12 @@
   </collision>
 </link>
-<link name="right_shoulder_v1_1">
-  <inertial>
-    <origin xyz="8.958533047331851e-11 -0.007844026821937675 2.015054789694659e-14" rpy="0 0 0"/>
+<link name="right_shoulder">
+  <inertial>
+    <origin xyz="8.958533047331851e-11 -0.007844026821937675 2.015054789694659e-14" rpy="-1.57 0  0"/>
     <mass value="0.010592862408759271"/>
     <inertia ixx="1e-06" iyy="3e-06" izz="3e-06" ixy="0.0" iyz="0.0" ixz="-0.0"/>
   </inertial>
   <visual>
-    <origin xyz="-0.003 0.084 -0.04475" rpy="0 0 0"/>
+    <origin xyz="-0.003 0.084 -0.04475" rpy="-1.57 0  0"/>
     <geometry>
       <mesh filename="package://assembly_description/meshes/simplified/right_shoulder_v1_1.stl" scale="0.001 0.001 0.001"/>
@@ -238,5 +238,5 @@
   </visual>
   <collision>
-    <origin xyz="-0.003 0.084 -0.04475" rpy="0 0 0"/>
+    <origin xyz="-0.003 0.084 -0.04475" rpy="-1.57 0  0"/>
     <geometry>
       <mesh filename="package://assembly_description/meshes/simplified/right_shoulder_v1_1.stl" scale="0.001 0.001 0.001"/>
@@ -244,12 +244,12 @@
   </collision>
 </link>
-<link name="right_bicep_v2_1">
-  <inertial>
-    <origin xyz="-0.01907144993358056 -0.0012317079698353356 -0.06051458521988612" rpy="0 0 0"/>
+<link name="right_bicep">
+  <inertial>
+    <origin xyz="-0.01907144993358056 -0.0012317079698353356 -0.06051458521988612" rpy="-1.57 0  0"/>
     <mass value="0.18636400760544294"/>
     <inertia ixx="0.000443" iyy="0.000444" izz="3.5e-05" ixy="-0.0" iyz="-1.1e-05" ixz="-6e-06"/>
   </inertial>
   <visual>
-    <origin xyz="-0.022 0.1143 -0.04475" rpy="0 0 0"/>
+    <origin xyz="-0.022 0.1143 -0.04475" rpy="-1.57 0  0"/>
     <geometry>
       <mesh filename="package://assembly_description/meshes/simplified/right_bicep_v2_1.stl" scale="0.001 0.001 0.001"/>
@@ -258,5 +258,5 @@
   </visual>
   <collision>
-    <origin xyz="-0.022 0.1143 -0.04475" rpy="0 0 0"/>
+    <origin xyz="-0.022 0.1143 -0.04475" rpy="-1.57 0  0"/>
     <geometry>
       <mesh filename="package://assembly_description/meshes/simplified/right_bicep_v2_1.stl" scale="0.001 0.001 0.001"/>
@@ -264,12 +264,12 @@
   </collision>
 </link>
-<link name="right_forearm_v1_1">
-  <inertial>
-    <origin xyz="0.0004903254970113039 0.019700355234835765 -0.08144749179773612" rpy="0 0 0"/>
+<link name="right_forearm">
+  <inertial>
+    <origin xyz="0.0004903254970113039 0.019700355234835765 -0.08144749179773612" rpy="-1.57 0  0"/>
     <mass value="0.05984540204112203"/>
     <inertia ixx="0.000124" iyy="0.000119" izz="2.1e-05" ixy="-0.0" iyz="-0.0" ixz="-0.0"/>
   </inertial>
   <visual>
-    <origin xyz="-0.002403 0.135101 0.074391" rpy="0 0 0"/>
+    <origin xyz="-0.002403 0.135101 0.074391" rpy="-1.57 0  0"/>
     <geometry>
       <mesh filename="package://assembly_description/meshes/simplified/right_forearm_v1_1.stl" scale="0.001 0.001 0.001"/>
@@ -278,5 +278,5 @@
   </visual>
   <collision>
-    <origin xyz="-0.002403 0.135101 0.074391" rpy="0 0 0"/>
+    <origin xyz="-0.002403 0.135101 0.074391" rpy="-1.57 0  0"/>
     <geometry>
       <mesh filename="package://assembly_description/meshes/simplified/right_forearm_v1_1.stl" scale="0.001 0.001 0.001"/>
@@ -284,12 +284,12 @@
   </collision>
 </link>
-<link name="left_thigh_v1_1">
-  <inertial>
-    <origin xyz="-3.483251756527389e-07 -0.028961129249142487 -0.036619318233349435" rpy="0 0 0"/>
+<link name="left_thigh">
+  <inertial>
+    <origin xyz="-3.483251756527389e-07 -0.028961129249142487 -0.036619318233349435" rpy="-1.57 0  0"/>
     <mass value="0.02898284927838432"/>
     <inertia ixx="3.5e-05" iyy="2.1e-05" izz="1.7e-05" ixy="0.0" iyz="-0.0" ixz="0.0"/>
   </inertial>
   <visual>
-    <origin xyz="-0.011569 -0.06475 0.1725" rpy="0 0 0"/>
+    <origin xyz="-0.011569 -0.06475 0.1725" rpy="-1.57 0  0"/>
     <geometry>
       <mesh filename="package://assembly_description/meshes/simplified/left_thigh_v1_1.stl" scale="0.001 0.001 0.001"/>
@@ -298,5 +298,5 @@
   </visual>
   <collision>
-    <origin xyz="-0.011569 -0.06475 0.1725" rpy="0 0 0"/>
+    <origin xyz="-0.011569 -0.06475 0.1725" rpy="-1.57 0  0"/>
     <geometry>
       <mesh filename="package://assembly_description/meshes/simplified/left_thigh_v1_1.stl" scale="0.001 0.001 0.001"/>
@@ -304,12 +304,12 @@
   </collision>
 </link>
-<link name="right_thigh_v1_1">
-  <inertial>
-    <origin xyz="9.832517461512424e-08 0.028961129249143854 -0.03661931823334971" rpy="0 0 0"/>
+<link name="right_thigh">
+  <inertial>
+    <origin xyz="9.832517461512424e-08 0.028961129249143854 -0.03661931823334971" rpy="-1.57 0  0"/>
     <mass value="0.02898284927838432"/>
     <inertia ixx="3.5e-05" iyy="2.1e-05" izz="1.7e-05" ixy="0.0" iyz="0.0" ixz="-0.0"/>
   </inertial>
   <visual>
-    <origin xyz="-0.0116 0.06475 0.1725" rpy="0 0 0"/>
+    <origin xyz="-0.0116 0.06475 0.1725" rpy="-1.57 0  0"/>
     <geometry>
       <mesh filename="package://assembly_description/meshes/simplified/right_thigh_v1_1.stl" scale="0.001 0.001 0.001"/>
@@ -318,5 +318,5 @@
   </visual>
   <collision>
-    <origin xyz="-0.0116 0.06475 0.1725" rpy="0 0 0"/>
+    <origin xyz="-0.0116 0.06475 0.1725" rpy="-1.57 0  0"/>
     <geometry>
       <mesh filename="package://assembly_description/meshes/simplified/right_thigh_v1_1.stl" scale="0.001 0.001 0.001"/>
@@ -324,12 +324,12 @@
   </collision>
 </link>
-<link name="left_hip_front_v5_1">
-  <inertial>
-    <origin xyz="0.04719163872713075 0.0001729815107887056 -0.01748011628225432" rpy="0 0 0"/>
+<link name="left_hip_front">
+  <inertial>
+    <origin xyz="0.04719163872713075 0.0001729815107887056 -0.01748011628225432" rpy="-1.57 0  0"/>
     <mass value="0.2722002973016189"/>
     <inertia ixx="0.000107" iyy="0.000233" izz="0.000192" ixy="-1e-06" iyz="2e-06" ixz="1e-05"/>
   </inertial>
   <visual>
-    <origin xyz="0.0547 -0.04125 0.1365" rpy="0 0 0"/>
+    <origin xyz="0.0547 -0.04125 0.1365" rpy="-1.57 0  0"/>
     <geometry>
       <mesh filename="package://assembly_description/meshes/simplified/left_hip_front_v5_1.stl" scale="0.001 0.001 0.001"/>
@@ -338,5 +338,5 @@
   </visual>
   <collision>
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
File: soccer_description/bez2_description/urdf/bez2.xacro (robot description, xacro)
@@ -5,5 +5,5 @@
 <xacro:include filename="$(find bez2_description)/urdf/bez2.trans" />
 <xacro:include filename="$(find bez2_description)/urdf/bez2.gazebo" />
-<link name="trunk">
+<link name="torso">
   <inertial>
     <origin xyz="-2.6182166493521018e-05 0.0037391632790891283 -0.07310917852477573" rpy="0 0 0"/>
