Commit message: testing code for imu tf and replace stl with dae to speed up network.

File: soccer_description/assembly_description/urdf/assembly.xacro (robot description, xacro)
@@ -13,5 +13,5 @@
     <origin xyz="0 0 0" rpy="-1.57 0  0"/>
     <geometry>
-      <mesh filename="package://assembly_description/meshes/simplified/base_link.stl" scale="0.001 0.001 0.001"/>
+      <mesh filename="package://assembly_description/meshes/simplified/base_link.dae" scale="0.001 0.001 0.001"/>
     </geometry>
     <material name="silver_default"/>
@@ -20,5 +20,5 @@
     <origin xyz="0 0 0" rpy="-1.57 0  0"/>
     <geometry>
-      <mesh filename="package://assembly_description/meshes/simplified/base_link.stl" scale="0.001 0.001 0.001"/>
+      <mesh filename="package://assembly_description/meshes/simplified/base_link.dae" scale="0.001 0.001 0.001"/>
     </geometry>
   </collision>
@@ -33,5 +33,5 @@
     <origin xyz="-0.016 -0.04125 0.1085" rpy="-1.57 0  0"/>
     <geometry>
-      <mesh filename="package://assembly_description/meshes/simplified/left_hip_side_v5_1.stl" scale="0.001 0.001 0.001"/>
+      <mesh filename="package://assembly_description/meshes/simplified/left_hip_side_v5_1.dae" scale="0.001 0.001 0.001"/>
     </geometry>
     <material name="aluminum_satin"/>
@@ -40,5 +40,5 @@
     <origin xyz="-0.016 -0.04125 0.1085" rpy="-1.57 0  0"/>
     <geometry>
-      <mesh filename="package://assembly_description/meshes/simplified/left_hip_side_v5_1.stl" scale="0.001 0.001 0.001"/>
+      <mesh filename="package://assembly_description/meshes/simplified/left_hip_side_v5_1.dae" scale="0.001 0.001 0.001"/>
     </geometry>
   </collision>
@@ -53,5 +53,5 @@
     <origin xyz="0.054731 -0.04125 0.3685" rpy="-1.57 0  0"/>
     <geometry>
-      <mesh filename="package://assembly_description/meshes/simplified/left_foot_v10_1.stl" scale="0.001 0.001 0.001"/>
+      <mesh filename="package://assembly_description/meshes/simplified/left_foot_v10_1.dae" scale="0.001 0.001 0.001"/>
     </geometry>
     <material name="abs_white"/>
@@ -60,5 +60,5 @@
     <origin xyz="0.054731 -0.04125 0.3685" rpy="-1.57 0  0"/>
     <geometry>
-      <mesh filename="package://assembly_description/meshes/simplified/left_foot_v10_1.stl" scale="0.001 0.001 0.001"/>
+      <mesh filename="package://assembly_description/meshes/simplified/left_foot_v10_1.dae" scale="0.001 0.001 0.001"/>
     </geometry>
   </collision>
@@ -73,5 +73,5 @@
     <origin xyz="-0.003 -0.084 -0.04475" rpy="-1.57 0  0"/>
     <geometry>
-      <mesh filename="package://assembly_description/meshes/simplified/left_shoulder_v5_1.stl" scale="0.001 0.001 0.001"/>
+      <mesh filename="package://assembly_description/meshes/simplified/left_shoulder_v5_1.dae" scale="0.001 0.001 0.001"/>
     </geometry>
     <material name="aluminum_satin"/>
@@ -80,5 +80,5 @@
     <origin xyz="-0.003 -0.084 -0.04475" rpy="-1.57 0  0"/>
     <geometry>
-      <mesh filename="package://assembly_description/meshes/simplified/left_shoulder_v5_1.stl" scale="0.001 0.001 0.001"/>
+      <mesh filename="package://assembly_description/meshes/simplified/left_shoulder_v5_1.dae" scale="0.001 0.001 0.001"/>
     </geometry>
   </collision>
@@ -93,5 +93,5 @@
     <origin xyz="-0.022 -0.1143 -0.04475" rpy="-1.57 0  0"/>
     <geometry>
-      <mesh filename="package://assembly_description/meshes/simplified/left_bicep_v6_1.stl" scale="0.001 0.001 0.001"/>
+      <mesh filename="package://assembly_description/meshes/simplified/left_bicep_v6_1.dae" scale="0.001 0.001 0.001"/>
     </geometry>
     <material name="silver_default"/>
@@ -100,5 +100,5 @@
     <origin xyz="-0.022 -0.1143 -0.04475" rpy="-1.57 0  0"/>
     <geometry>
-      <mesh filename="package://assembly_description/meshes/simplified/left_bicep_v6_1.stl" scale="0.001 0.001 0.001"/>
+      <mesh filename="package://assembly_description/meshes/simplified/left_bicep_v6_1.dae" scale="0.001 0.001 0.001"/>
     </geometry>
   </collision>
@@ -113,5 +113,5 @@
     <origin xyz="-0.001597 -0.133101 0.074391" rpy="-1.57 0  0"/>
     <geometry>
-      <mesh filename="package://assembly_description/meshes/simplified/left_forearm_v4_1.stl" scale="0.001 0.001 0.001"/>
+      <mesh filename="package://assembly_description/meshes/simplified/left_forearm_v4_1.dae" scale="0.001 0.001 0.001"/>
     </geometry>
     <material name="abs_white"/>
@@ -120,5 +120,5 @@
     <origin xyz="-0.001597 -0.133101 0.074391" rpy="-1.57 0  0"/>
     <geometry>
-      <mesh filename="package://assembly_description/meshes/simplified/left_forearm_v4_1.stl" scale="0.001 0.001 0.001"/>
+      <mesh filename="package://assembly_description/meshes/simplified/left_forearm_v4_1.dae" scale="0.001 0.001 0.001"/>
     </geometry>
   </collision>
@@ -133,5 +133,5 @@
     <origin xyz="-0.0 -0.00025 -0.0725" rpy="-1.57 0  0"/>
     <geometry>
-      <mesh filename="package://assembly_description/meshes/simplified/neck_v6_1.stl" scale="0.001 0.001 0.001"/>
+      <mesh filename="package://assembly_description/meshes/simplified/neck_v6_1.dae" scale="0.001 0.001 0.001"/>
     </geometry>
     <material name="abs_white"/>
@@ -140,5 +140,5 @@
     <origin xyz="-0.0 -0.00025 -0.0725" rpy="-1.57 0  0"/>
     <geometry>
-      <mesh filename="package://assembly_description/meshes/simplified/neck_v6_1.stl" scale="0.001 0.001 0.001"/>
+      <mesh filename="package://assembly_description/meshes/simplified/neck_v6_1.dae" scale="0.001 0.001 0.001"/>
     </geometry>
   </collision>
@@ -153,5 +153,5 @@
     <origin xyz="-0.0 0.01825 -0.0975" rpy="-1.57 0  0"/>
     <geometry>
-      <mesh filename="package://assembly_description/meshes/simplified/head_v4_1.stl" scale="0.001 0.001 0.001"/>
+      <mesh filename="package://assembly_description/meshes/simplified/head_v4_1.dae" scale="0.001 0.001 0.001"/>
     </geometry>
     <material name="steel_satin"/>
@@ -160,5 +160,5 @@
     <origin xyz="-0.0 0.01825 -0.0975" rpy="-1.57 0  0"/>
     <geometry>
-      <mesh filename="package://assembly_description/meshes/simplified/head_v4_1.stl" scale="0.001 0.001 0.001"/>
+      <mesh filename="package://assembly_description/meshes/simplified/head_v4_1.dae" scale="0.001 0.001 0.001"/>
     </geometry>
   </collision>
@@ -173,5 +173,5 @@
     <origin xyz="-0.016 0.04125 0.1085" rpy="-1.57 0  0"/>
     <geometry>
-      <mesh filename="package://assembly_description/meshes/simplified/right_hip_side_v1_1.stl" scale="0.001 0.001 0.001"/>
+      <mesh filename="package://assembly_description/meshes/simplified/right_hip_side_v1_1.dae" scale="0.001 0.001 0.001"/>
     </geometry>
     <material name="aluminum_satin"/>
@@ -180,5 +180,5 @@
     <origin xyz="-0.016 0.04125 0.1085" rpy="-1.57 0  0"/>
     <geometry>
-      <mesh filename="package://assembly_description/meshes/simplified/right_hip_side_v1_1.stl" scale="0.001 0.001 0.001"/>
+      <mesh filename="package://assembly_description/meshes/simplified/right_hip_side_v1_1.dae" scale="0.001 0.001 0.001"/>
     </geometry>
   </collision>
@@ -193,5 +193,5 @@
     <origin xyz="-0.0116 0.06475 0.3325" rpy="-1.57 0  0"/>
     <geometry>
-      <mesh filename="package://assembly_description/meshes/simplified/right_ankle_v2_1.stl" scale="0.001 0.001 0.001"/>
+      <mesh filename="package://assembly_description/meshes/simplified/right_ankle_v2_1.dae" scale="0.001 0.001 0.001"/>
     </geometry>
     <material name="steel_satin"/>
@@ -200,5 +200,5 @@
     <origin xyz="-0.0116 0.06475 0.3325" rpy="-1.57 0  0"/>
     <geometry>
-      <mesh filename="package://assembly_description/meshes/simplified/right_ankle_v2_1.stl" scale="0.001 0.001 0.001"/>
+      <mesh filename="package://assembly_description/meshes/simplified/right_ankle_v2_1.dae" scale="0.001 0.001 0.001"/>
     </geometry>
   </collision>
@@ -213,5 +213,5 @@
     <origin xyz="0.0547 0.04125 0.3685" rpy="-1.57 0  0"/>
     <geometry>
-      <mesh filename="package://assembly_description/meshes/simplified/right_foot_v2_1.stl" scale="0.001 0.001 0.001"/>
+      <mesh filename="package://assembly_description/meshes/simplified/right_foot_v2_1.dae" scale="0.001 0.001 0.001"/>
     </geometry>
     <material name="abs_white"/>
@@ -220,5 +220,5 @@
     <origin xyz="0.0547 0.04125 0.3685" rpy="-1.57 0  0"/>
     <geometry>
-      <mesh filename="package://assembly_description/meshes/simplified/right_foot_v2_1.stl" scale="0.001 0.001 0.001"/>
+      <mesh filename="package://assembly_description/meshes/simplified/right_foot_v2_1.dae" scale="0.001 0.001 0.001"/>
     </geometry>
   </collision>
@@ -233,5 +233,5 @@
     <origin xyz="-0.003 0.084 -0.04475" rpy="-1.57 0  0"/>
     <geometry>
-      <mesh filename="package://assembly_description/meshes/simplified/right_shoulder_v1_1.stl" scale="0.001 0.001 0.001"/>
+      <mesh filename="package://assembly_description/meshes/simplified/right_shoulder_v1_1.dae" scale="0.001 0.001 0.001"/>
     </geometry>
     <material name="aluminum_satin"/>
@@ -240,5 +240,5 @@
     <origin xyz="-0.003 0.084 -0.04475" rpy="-1.57 0  0"/>
     <geometry>
-      <mesh filename="package://assembly_description/meshes/simplified/right_shoulder_v1_1.stl" scale="0.001 0.001 0.001"/>
+      <mesh filename="package://assembly_description/meshes/simplified/right_shoulder_v1_1.dae" scale="0.001 0.001 0.001"/>
     </geometry>
   </collision>
@@ -253,5 +253,5 @@
     <origin xyz="-0.022 0.1143 -0.04475" rpy="-1.57 0  0"/>
     <geometry>
-      <mesh filename="package://assembly_description/meshes/simplified/right_bicep_v2_1.stl" scale="0.001 0.001 0.001"/>
+      <mesh filename="package://assembly_description/meshes/simplified/right_bicep_v2_1.dae" scale="0.001 0.001 0.001"/>
     </geometry>
     <material name="silver_default"/>
@@ -260,5 +260,5 @@
     <origin xyz="-0.022 0.1143 -0.04475" rpy="-1.57 0  0"/>
     <geometry>
-      <mesh filename="package://assembly_description/meshes/simplified/right_bicep_v2_1.stl" scale="0.001 0.001 0.001"/>
+      <mesh filename="package://assembly_description/meshes/simplified/right_bicep_v2_1.dae" scale="0.001 0.001 0.001"/>
     </geometry>
   </collision>
@@ -273,5 +273,5 @@
     <origin xyz="-0.002403 0.135101 0.074391" rpy="-1.57 0  0"/>
     <geometry>
-      <mesh filename="package://assembly_description/meshes/simplified/right_forearm_v1_1.stl" scale="0.001 0.001 0.001"/>
+      <mesh filename="package://assembly_description/meshes/simplified/right_forearm_v1_1.dae" scale="0.001 0.001 0.001"/>
     </geometry>
     <material name="abs_white"/>
@@ -280,5 +280,5 @@
     <origin xyz="-0.002403 0.135101 0.074391" rpy="-1.57 0  0"/>
     <geometry>
-      <mesh filename="package://assembly_description/meshes/simplified/right_forearm_v1_1.stl" scale="0.001 0.001 0.001"/>
+      <mesh filename="package://assembly_description/meshes/simplified/right_forearm_v1_1.dae" scale="0.001 0.001 0.001"/>
     </geometry>
   </collision>
@@ -293,5 +293,5 @@
     <origin xyz="-0.011569 -0.06475 0.1725" rpy="-1.57 0  0"/>
     <geometry>
-      <mesh filename="package://assembly_description/meshes/simplified/left_thigh_v1_1.stl" scale="0.001 0.001 0.001"/>
+      <mesh filename="package://assembly_description/meshes/simplified/left_thigh_v1_1.dae" scale="0.001 0.001 0.001"/>
     </geometry>
     <material name="aluminum_satin"/>
@@ -300,5 +300,5 @@
     <origin xyz="-0.011569 -0.06475 0.1725" rpy="-1.57 0  0"/>
     <geometry>
-      <mesh filename="package://assembly_description/meshes/simplified/left_thigh_v1_1.stl" scale="0.001 0.001 0.001"/>
+      <mesh filename="package://assembly_description/meshes/simplified/left_thigh_v1_1.dae" scale="0.001 0.001 0.001"/>
     </geometry>
   </collision>
@@ -313,5 +313,5 @@
     <origin xyz="-0.0116 0.06475 0.1725" rpy="-1.57 0  0"/>
     <geometry>
-      <mesh filename="package://assembly_description/meshes/simplified/right_thigh_v1_1.stl" scale="0.001 0.001 0.001"/>
+      <mesh filename="package://assembly_description/meshes/simplified/right_thigh_v1_1.dae" scale="0.001 0.001 0.001"/>
     </geometry>
     <material name="aluminum_satin"/>
@@ -320,5 +320,5 @@
     <origin xyz="-0.0116 0.06475 0.1725" rpy="-1.57 0  0"/>
     <geometry>
-      <mesh filename="package://assembly_description/meshes/simplified/right_thigh_v1_1.stl" scale="0.001 0.001 0.001"/>
+      <mesh filename="package://assembly_description/meshes/simplified/right_thigh_v1_1.dae" scale="0.001 0.001 0.001"/>
     </geometry>
   </collision>
@@ -333,5 +333,5 @@
     <origin xyz="0.0547 -0.04125 0.1365" rpy="-1.57 0  0"/>
     <geometry>
-      <mesh filename="package://assembly_description/meshes/simplified/left_hip_front_v5_1.stl" scale="0.001 0.001 0.001"/>
+      <mesh filename="package://assembly_description/meshes/simplified/left_hip_front_v5_1.dae" scale="0.001 0.001 0.001"/>
     </geometry>
     <material name="aluminum_satin"/>
@@ -340,5 +340,5 @@
     <origin xyz="0.0547 -0.04125 0.1365" rpy="-1.57 0  0"/>
     <geometry>
-      <mesh filename="package://assembly_description/meshes/simplified/left_hip_front_v5_1.stl" scale="0.001 0.001 0.001"/>
+      <mesh filename="package://assembly_description/meshes/simplified/left_hip_front_v5_1.dae" scale="0.001 0.001 0.001"/>
     </geometry>
   </collision>
@@ -353,5 +353,5 @@
     <origin xyz="-0.011569 -0.06475 0.2445" rpy="-1.57 0  0"/>
     <geometry>
-      <mesh filename="package://assembly_description/meshes/simplified/left_calve_v5_1.stl" scale="0.001 0.001 0.001"/>
+      <mesh filename="package://assembly_description/meshes/simplified/left_calve_v5_1.dae" scale="0.001 0.001 0.001"/>
     </geometry>
     <material name="aluminum_satin"/>
@@ -360,5 +360,5 @@
     <origin xyz="-0.011569 -0.06475 0.2445" rpy="-1.57 0  0"/>
     <geometry>
-      <mesh filename="package://assembly_description/meshes/simplified/left_calve_v5_1.stl" scale="0.001 0.001 0.001"/>
+      <mesh filename="package://assembly_description/meshes/simplified/left_calve_v5_1.dae" scale="0.001 0.001 0.001"/>
     </geometry>
   </collision>
@@ -373,5 +373,5 @@
     <origin xyz="-0.011569 -0.06475 0.3325" rpy="-1.57 0  0"/>
     <geometry>
-      <mesh filename="package://assembly_description/meshes/simplified/left_ankle_v7_1.stl" scale="0.001 0.001 0.001"/>
+      <mesh filename="package://assembly_description/meshes/simplified/left_ankle_v7_1.dae" scale="0.001 0.001 0.001"/>
     </geometry>
     <material name="steel_satin"/>
@@ -380,5 +380,5 @@
     <origin xyz="-0.011569 -0.06475 0.3325" rpy="-1.57 0  0"/>
     <geometry>
-      <mesh filename="package://assembly_description/meshes/simplified/left_ankle_v7_1.stl" scale="0.001 0.001 0.001"/>
+      <mesh filename="package://assembly_description/meshes/simplified/left_ankle_v7_1.dae" scale="0.001 0.001 0.001"/>
     </geometry>
   </collision>
@@ -393,5 +393,5 @@
     <origin xyz="0.0547 0.04125 0.1365" rpy="-1.57 0  0"/>
     <geometry>
-      <mesh filename="package://assembly_description/meshes/simplified/right_hip_front_v5_1.stl" scale="0.001 0.001 0.001"/>
+      <mesh filename="package://assembly_description/meshes/simplified/right_hip_front_v5_1.dae" scale="0.001 0.001 0.001"/>
     </geometry>
     <material name="aluminum_satin"/>
@@ -400,5 +400,5 @@
     <origin xyz="0.0547 0.04125 0.1365" rpy="-1.57 0  0"/>
     <geometry>
-      <mesh filename="package://assembly_description/meshes/simplified/right_hip_front_v5_1.stl" scale="0.001 0.001 0.001"/>
+      <mesh filename="package://assembly_description/meshes/simplified/right_hip_front_v5_1.dae" scale="0.001 0.001 0.001"/>
     </geometry>
   </collision>
@@ -413,5 +413,5 @@
     <origin xyz="-0.0116 0.06475 0.2445" rpy="-1.57 0  0"/>
     <geometry>
-      <mesh filename="package://assembly_description/meshes/simplified/right_calve_v1_1.stl" scale="0.001 0.001 0.001"/>
+      <mesh filename="package://assembly_description/meshes/simplified/right_calve_v1_1.dae" scale="0.001 0.001 0.001"/>
     </geometry>
     <material name="aluminum_satin"/>
@@ -420,5 +420,5 @@
     <origin xyz="-0.0116 0.06475 0.2445" rpy="-1.57 0  0"/>
     <geometry>
-      <mesh filename="package://assembly_description/meshes/simplified/right_calve_v1_1.stl" scale="0.001 0.001 0.001"/>
+      <mesh filename="package://assembly_description/meshes/simplified/right_calve_v1_1.dae" scale="0.001 0.001 0.001"/>
     </geometry>
   </collision>
