Commit message: Js new (#912)
* added states to bez. fixed pybullet camera and tried to align with webots and reallife but needs more tuning. added a soccerball to pybullet world. added camera link to assembly placo urdf. minor edit to dae script. made the calculate_ball_from_bounding_boxes arg better arranged. disable cover horizon for now. added a new set of test that run object detection on pybullet camera images. Added both methods for object localization. starting to fill out strategy.

* moved ball to where bez is loaded. added a groundtruth get ball. speed up pybullet. properly enable head movement. tuned pid for nav on the new robot. created a new test that has nav without it owning the loops so we can add other operations.

* added camera joint to bez1 and new robot. created a new class for better handeling of the motors based on str or int inputs, dont know if i fully like it. fixed camera image from pybullet, had to use the motors for rpy of the camera because the angles get weird.  added a global and local ball ground truth. modified everywhere that interacted with motorcontrol. Got a ros version to work. swapped out pybullet setup with world and bez that control uses. no more duplicates. finished unit test for going to ball location based on yolov5.

* made a right kick and integrated vision into the walk loop for ros

* merged fron other branches

* finally finished getupfront

* made getupback faster and added an experiemntal kick planner

* getupback and rigth kick is finished

* finally walks

* aligned the transforms for getting the camera height to use the links on the real robot will be renamed to be in line with everything else. added some quality of life improvements from js_strat for enabling the tracking ball functionality. tuned ball tracking with head movements. Some merging with js_strat and akp_object. Fixed the camera fov settings to align with the actual spec of the camera, this helps the projection. To firmware interface,I Added a lock and got rid of the thread for the main loop so I can have more fine control over the loop frequency. a new test in ros walk where its a ros version of some placo test, but before we have camera as a node. Tuned the height and orientation of the camera, due to the xacro being wrong. Added a sync read function in the firmware, but im not sure about it, certain ports are stalling and I think it might be too a buffer overflow due to the frequency of messages, probably will go back, but it works okish for now. The robot can now trakc the ball with the camera.

* in firmware, I added a sync write function and this speeds up the loop by double, going from 120hz to 250hz for the imu and joint states. Experimented with 2mbs baud rate but was getting a lot more timedout errors. Added back non sync read, only 1 chain times out, still dont know how. Added a ball pixel so we can use a PID for the head to track the ball, added some checking so we dont work on init or  stale data. added some logic in nav ros so we have 3 modes, walk with a velocity, walk to the ball, walk in place. Tuned and pitch and role stabilization, needs some work for starting a walk, maybe more on placo side. It works in real life, it will detect the ball and walk towards it, we still need a sweep for the head and better kicking algorithim but the fundamentals work. Also added more lock nuts to the leg so it needs less maintence over time

* fixed the tf tree by editing the xacro to move properly. tuned the walking pid, tuned the trajectory and ready for video

* added some stuff to work

* fixed main unit test by going back to original head tracking

* refactoring

* wip

* converted msgs

* started full ros2 migration. finished migration of firmware interface. still need to be verfied on robot, but should work. Had to fix the param server. Started migrating soccer_traj with the structure.

* validated firmware interface

* Restore file contents that were previously in LFS

* changed workspace directory across codebase. finished soccer traj conversion. still need to verify it.

* migrated common and pycontrol. should work but unit test does not

* migrated description, minor changes

* current version with gamecontroller

* setup basic launch file and integrated imu complementary filter

* idk

* idk

* works

* removed pybullet running and added basic behavior for getting up and interruption

* latest version

* testing code for imu tf and replace stl with dae to speed up network.

* integrated obj dectection

* current version

* current version

File: soccer_description/assembly_description/urdf/assembly.xacro (robot description, xacro)
@@ -6,541 +6,609 @@
 <link name="base_link">
   <inertial>
-    <origin xyz="-0.02024929347181477 0.00329389202927954 -0.02671963219571571" rpy="0 0 0"/>
+    <origin xyz="-0.02024929347181477 0.00329389202927954 -0.02671963219571571" rpy="-1.57 0  0"/>
     <mass value="3.0429325287174738"/>
     <inertia ixx="0.009761" iyy="0.006663" izz="0.008082" ixy="7.9e-05" iyz="8.1e-05" ixz="-0.000195"/>
   </inertial>
   <visual>
-    <origin xyz="0 0 0" rpy="0 0 0"/>
-    <geometry>
-      <mesh filename="package://assembly_description/meshes/base_link.stl" scale="0.001 0.001 0.001"/>
+    <origin xyz="0 0 0" rpy="-1.57 0  0"/>
+    <geometry>
+      <mesh filename="package://assembly_description/meshes/simplified/base_link.dae" scale="0.001 0.001 0.001"/>
     </geometry>
     <material name="silver_default"/>
   </visual>
   <collision>
-    <origin xyz="0 0 0" rpy="0 0 0"/>
-    <geometry>
-      <mesh filename="package://assembly_description/meshes/base_link.stl" scale="0.001 0.001 0.001"/>
-    </geometry>
-  </collision>
-</link>
-<link name="left_hip_side_v5_1">
-  <inertial>
-    <origin xyz="-0.0176303342104258 -2.8796409701214998e-15 -0.007188418776152797" rpy="0 0 0"/>
+    <origin xyz="0 0 0" rpy="-1.57 0  0"/>
+    <geometry>
+      <mesh filename="package://assembly_description/meshes/simplified/base_link.dae" scale="0.001 0.001 0.001"/>
+    </geometry>
+  </collision>
+</link>
+<link name="left_hip_side">
+  <inertial>
+    <origin xyz="-0.0176303342104258 -2.8796409701214998e-15 -0.007188418776152797" rpy="-1.57 0  0"/>
     <mass value="0.03929574358294283"/>
     <inertia ixx="7e-06" iyy="9.2e-05" izz="9e-05" ixy="0.0" iyz="0.0" ixz="4e-06"/>
   </inertial>
   <visual>
-    <origin xyz="-0.016 -0.04125 0.1085" rpy="0 0 0"/>
-    <geometry>
-      <mesh filename="package://assembly_description/meshes/left_hip_side_v5_1.stl" scale="0.001 0.001 0.001"/>
-    </geometry>
-    <material name="aluminum_satin"/>
-  </visual>
-  <collision>
-    <origin xyz="-0.016 -0.04125 0.1085" rpy="0 0 0"/>
-    <geometry>
-      <mesh filename="package://assembly_description/meshes/left_hip_side_v5_1.stl" scale="0.001 0.001 0.001"/>
-    </geometry>
-  </collision>
-</link>
-<link name="left_foot_v10_1">
-  <inertial>
-    <origin xyz="0.05312327716355333 0.01311710007932914 -0.017187548637288774" rpy="0 0 0"/>
+    <origin xyz="-0.016 -0.04125 0.1085" rpy="-1.57 0  0"/>
+    <geometry>
+      <mesh filename="package://assembly_description/meshes/simplified/left_hip_side_v5_1.dae" scale="0.001 0.001 0.001"/>
+    </geometry>
+    <material name="aluminum_satin"/>
+  </visual>
+  <collision>
+    <origin xyz="-0.016 -0.04125 0.1085" rpy="-1.57 0  0"/>
+    <geometry>
+      <mesh filename="package://assembly_description/meshes/simplified/left_hip_side_v5_1.dae" scale="0.001 0.001 0.001"/>
+    </geometry>
+  </collision>
+</link>
+<link name="left_foot">
+  <inertial>
+    <origin xyz="0.05312327716355333 0.01311710007932914 -0.017187548637288774" rpy="-1.57 0  0"/>
     <mass value="0.03929273129474386"/>
     <inertia ixx="2.6e-05" iyy="0.000124" izz="0.000144" ixy="2e-06" iyz="2e-06" ixz="-3e-06"/>
   </inertial>
   <visual>
-    <origin xyz="0.054731 -0.04125 0.3685" rpy="0 0 0"/>
-    <geometry>
-      <mesh filename="package://assembly_description/meshes/left_foot_v10_1.stl" scale="0.001 0.001 0.001"/>
+    <origin xyz="0.054731 -0.04125 0.3685" rpy="-1.57 0  0"/>
+    <geometry>
+      <mesh filename="package://assembly_description/meshes/simplified/left_foot_v10_1.dae" scale="0.001 0.001 0.001"/>
     </geometry>
     <material name="abs_white"/>
   </visual>
   <collision>
-    <origin xyz="0.054731 -0.04125 0.3685" rpy="0 0 0"/>
-    <geometry>
-      <mesh filename="package://assembly_description/meshes/left_foot_v10_1.stl" scale="0.001 0.001 0.001"/>
-    </geometry>
-  </collision>
-</link>
-<link name="left_shoulder_v5_1">
-  <inertial>
-    <origin xyz="8.922688803092438e-11 0.007844026821939576 2.0192181260370035e-14" rpy="0 0 0"/>
+    <origin xyz="0.054731 -0.04125 0.3685" rpy="-1.57 0  0"/>
+    <geometry>
+      <mesh filename="package://assembly_description/meshes/simplified/left_foot_v10_1.dae" scale="0.001 0.001 0.001"/>
+    </geometry>
+  </collision>
+</link>
+<link name="left_shoulder">
+  <inertial>
+    <origin xyz="8.922688803092438e-11 0.007844026821939576 2.0192181260370035e-14" rpy="-1.57 0  0"/>
     <mass value="0.010592862408759271"/>
     <inertia ixx="1e-06" iyy="3e-06" izz="3e-06" ixy="0.0" iyz="-0.0" ixz="0.0"/>
   </inertial>
   <visual>
-    <origin xyz="-0.003 -0.084 -0.04475" rpy="0 0 0"/>
-    <geometry>
-      <mesh filename="package://assembly_description/meshes/left_shoulder_v5_1.stl" scale="0.001 0.001 0.001"/>
-    </geometry>
-    <material name="aluminum_satin"/>
-  </visual>
-  <collision>
-    <origin xyz="-0.003 -0.084 -0.04475" rpy="0 0 0"/>
-    <geometry>
-      <mesh filename="package://assembly_description/meshes/left_shoulder_v5_1.stl" scale="0.001 0.001 0.001"/>
-    </geometry>
-  </collision>
-</link>
-<link name="left_bicep_v6_1">
-  <inertial>
-    <origin xyz="-0.019420473733666368 0.00010477857835172744 -0.06051458521988624" rpy="0 0 0"/>
+    <origin xyz="-0.003 -0.084 -0.04475" rpy="-1.57 0  0"/>
+    <geometry>
+      <mesh filename="package://assembly_description/meshes/simplified/left_shoulder_v5_1.dae" scale="0.001 0.001 0.001"/>
+    </geometry>
+    <material name="aluminum_satin"/>
+  </visual>
+  <collision>
+    <origin xyz="-0.003 -0.084 -0.04475" rpy="-1.57 0  0"/>
+    <geometry>
+      <mesh filename="package://assembly_description/meshes/simplified/left_shoulder_v5_1.dae" scale="0.001 0.001 0.001"/>
+    </geometry>
+  </collision>
+</link>
+<link name="left_bicep">
+  <inertial>
+    <origin xyz="-0.019420473733666368 0.00010477857835172744 -0.06051458521988624" rpy="-1.57 0  0"/>
     <mass value="0.18636400760544294"/>
     <inertia ixx="0.000442" iyy="0.000444" izz="3.5e-05" ixy="0.0" iyz="3e-06" ixz="-1e-05"/>
   </inertial>
   <visual>
-    <origin xyz="-0.022 -0.1143 -0.04475" rpy="0 0 0"/>
-    <geometry>
-      <mesh filename="package://assembly_description/meshes/left_bicep_v6_1.stl" scale="0.001 0.001 0.001"/>
+    <origin xyz="-0.022 -0.1143 -0.04475" rpy="-1.57 0  0"/>
+    <geometry>
+      <mesh filename="package://assembly_description/meshes/simplified/left_bicep_v6_1.dae" scale="0.001 0.001 0.001"/>
     </geometry>
     <material name="silver_default"/>
   </visual>
   <collision>
-    <origin xyz="-0.022 -0.1143 -0.04475" rpy="0 0 0"/>
-    <geometry>
-      <mesh filename="package://assembly_description/meshes/left_bicep_v6_1.stl" scale="0.001 0.001 0.001"/>
-    </geometry>
-  </collision>
-</link>
-<link name="left_forearm_v4_1">
-  <inertial>
-    <origin xyz="0.0004904443113911659 -0.01970036030468776 -0.0814474917977369" rpy="0 0 0"/>
+    <origin xyz="-0.022 -0.1143 -0.04475" rpy="-1.57 0  0"/>
+    <geometry>
+      <mesh filename="package://assembly_description/meshes/simplified/left_bicep_v6_1.dae" scale="0.001 0.001 0.001"/>
+    </geometry>
+  </collision>
+</link>
+<link name="left_forearm">
+  <inertial>
+    <origin xyz="0.0004904443113911659 -0.01970036030468776 -0.0814474917977369" rpy="-1.57 0  0"/>
     <mass value="0.05984540204112203"/>
     <inertia ixx="0.000124" iyy="0.000119" izz="2.1e-05" ixy="-0.0" iyz="-0.0" ixz="-0.0"/>
   </inertial>
   <visual>
-    <origin xyz="-0.001597 -0.133101 0.074391" rpy="0 0 0"/>
-    <geometry>
-      <mesh filename="package://assembly_description/meshes/left_forearm_v4_1.stl" scale="0.001 0.001 0.001"/>
+    <origin xyz="-0.001597 -0.133101 0.074391" rpy="-1.57 0  0"/>
+    <geometry>
+      <mesh filename="package://assembly_description/meshes/simplified/left_forearm_v4_1.dae" scale="0.001 0.001 0.001"/>
     </geometry>
     <material name="abs_white"/>
   </visual>
   <collision>
-    <origin xyz="-0.001597 -0.133101 0.074391" rpy="0 0 0"/>
-    <geometry>
-      <mesh filename="package://assembly_description/meshes/left_forearm_v4_1.stl" scale="0.001 0.001 0.001"/>
-    </geometry>
-  </collision>
-</link>
-<link name="neck_v6_1">
-  <inertial>
-    <origin xyz="8.936969206796164e-11 0.0012409815706136025 0.012040454865583" rpy="0 0 0"/>
+    <origin xyz="-0.001597 -0.133101 0.074391" rpy="-1.57 0  0"/>
+    <geometry>
+      <mesh filename="package://assembly_description/meshes/simplified/left_forearm_v4_1.dae" scale="0.001 0.001 0.001"/>
+    </geometry>
+  </collision>
+</link>
+<link name="neck">
+  <inertial>
+    <origin xyz="8.936969206796164e-11 0.0012409815706136025 0.012040454865583" rpy="-1.57 0  0"/>
     <mass value="0.004247113386163016"/>
     <inertia ixx="2e-06" iyy="1e-06" izz="2e-06" ixy="-0.0" iyz="-0.0" ixz="0.0"/>
   </inertial>
   <visual>
-    <origin xyz="-0.0 -0.00025 -0.0725" rpy="0 0 0"/>
-    <geometry>
-      <mesh filename="package://assembly_description/meshes/neck_v6_1.stl" scale="0.001 0.001 0.001"/>
+    <origin xyz="-0.0 -0.00025 -0.0725" rpy="-1.57 0  0"/>
+    <geometry>
+      <mesh filename="package://assembly_description/meshes/simplified/neck_v6_1.dae" scale="0.001 0.001 0.001"/>
     </geometry>
     <material name="abs_white"/>
   </visual>
   <collision>
-    <origin xyz="-0.0 -0.00025 -0.0725" rpy="0 0 0"/>
-    <geometry>
-      <mesh filename="package://assembly_description/meshes/neck_v6_1.stl" scale="0.001 0.001 0.001"/>
-    </geometry>
-  </collision>
-</link>
-<link name="head_v4_1">
-  <inertial>
-    <origin xyz="-0.0025761957912120003 0.01899177474904292 0.03300593624682499" rpy="0 0 0"/>
+    <origin xyz="-0.0 -0.00025 -0.0725" rpy="-1.57 0  0"/>
+    <geometry>
+      <mesh filename="package://assembly_description/meshes/simplified/neck_v6_1.dae" scale="0.001 0.001 0.001"/>
+    </geometry>
+  </collision>
+</link>
+<link name="head">
+  <inertial>
+    <origin xyz="-0.0025761957912120003 0.01899177474904292 0.03300593624682499" rpy="-1.57 0  0"/>
     <mass value="0.26433915470596575"/>
     <inertia ixx="0.000237" iyy="0.000239" izz="0.000166" ixy="-0.0" iyz="-2e-06" ixz="-5.6e-05"/>
   </inertial>
   <visual>
-    <origin xyz="-0.0 0.01825 -0.0975" rpy="0 0 0"/>
-    <geometry>
-      <mesh filename="package://assembly_description/meshes/head_v4_1.stl" scale="0.001 0.001 0.001"/>
+    <origin xyz="-0.0 0.01825 -0.0975" rpy="-1.57 0  0"/>
+    <geometry>
+      <mesh filename="package://assembly_description/meshes/simplified/head_v4_1.dae" scale="0.001 0.001 0.001"/>
     </geometry>
     <material name="steel_satin"/>
   </visual>
   <collision>
-    <origin xyz="-0.0 0.01825 -0.0975" rpy="0 0 0"/>
-    <geometry>
-      <mesh filename="package://assembly_description/meshes/head_v4_1.stl" scale="0.001 0.001 0.001"/>
-    </geometry>
-  </collision>
-</link>
-<link name="right_hip_side_v1_1">
-  <inertial>
-    <origin xyz="-0.017630334210425074 -2.7131075164277263e-15 -0.007188418776152866" rpy="0 0 0"/>
+    <origin xyz="-0.0 0.01825 -0.0975" rpy="-1.57 0  0"/>
+    <geometry>
+      <mesh filename="package://assembly_description/meshes/simplified/head_v4_1.dae" scale="0.001 0.001 0.001"/>
+    </geometry>
+  </collision>
+</link>
+<link name="right_hip_side">
+  <inertial>
+    <origin xyz="-0.017630334210425074 -2.7131075164277263e-15 -0.007188418776152866" rpy="-1.57 0  0"/>
     <mass value="0.03929574358294283"/>
     <inertia ixx="7e-06" iyy="9.2e-05" izz="9e-05" ixy="0.0" iyz="0.0" ixz="4e-06"/>
   </inertial>
   <visual>
-    <origin xyz="-0.016 0.04125 0.1085" rpy="0 0 0"/>
-    <geometry>
-      <mesh filename="package://assembly_description/meshes/right_hip_side_v1_1.stl" scale="0.001 0.001 0.001"/>
-    </geometry>
-    <material name="aluminum_satin"/>
-  </visual>
-  <collision>
-    <origin xyz="-0.016 0.04125 0.1085" rpy="0 0 0"/>
-    <geometry>
-      <mesh filename="package://assembly_description/meshes/right_hip_side_v1_1.stl" scale="0.001 0.001 0.001"/>
-    </geometry>
-  </collision>
-</link>
-<link name="right_ankle_v2_1">
-  <inertial>
-    <origin xyz="-0.019332548462524354 0.02355722240141854 -0.018170467896408804" rpy="0 0 0"/>
+    <origin xyz="-0.016 0.04125 0.1085" rpy="-1.57 0  0"/>
+    <geometry>
+      <mesh filename="package://assembly_description/meshes/simplified/right_hip_side_v1_1.dae" scale="0.001 0.001 0.001"/>
+    </geometry>
+    <material name="aluminum_satin"/>
+  </visual>
+  <collision>
+    <origin xyz="-0.016 0.04125 0.1085" rpy="-1.57 0  0"/>
+    <geometry>
+      <mesh filename="package://assembly_description/meshes/simplified/right_hip_side_v1_1.dae" scale="0.001 0.001 0.001"/>
+    </geometry>
+  </collision>
+</link>
+<link name="right_ankle">
+  <inertial>
+    <origin xyz="-0.019332548462524354 0.02355722240141854 -0.018170467896408804" rpy="-1.57 0  0"/>
     <mass value="0.2722002973016189"/>
     <inertia ixx="0.000108" iyy="0.000229" izz="0.000189" ixy="-0.0" iyz="1e-06" ixz="-1.3e-05"/>
   </inertial>
   <visual>
-    <origin xyz="-0.0116 0.06475 0.3325" rpy="0 0 0"/>
-    <geometry>
-      <mesh filename="package://assembly_description/meshes/right_ankle_v2_1.stl" scale="0.001 0.001 0.001"/>
+    <origin xyz="-0.0116 0.06475 0.3325" rpy="-1.57 0  0"/>
+    <geometry>
+      <mesh filename="package://assembly_description/meshes/simplified/right_ankle_v2_1.dae" scale="0.001 0.001 0.001"/>
     </geometry>
     <material name="steel_satin"/>
   </visual>
   <collision>
-    <origin xyz="-0.0116 0.06475 0.3325" rpy="0 0 0"/>
-    <geometry>
-      <mesh filename="package://assembly_description/meshes/right_ankle_v2_1.stl" scale="0.001 0.001 0.001"/>
-    </geometry>
-  </collision>
-</link>
-<link name="right_foot_v2_1">
-  <inertial>
-    <origin xyz="0.053123527163554944 -0.01311710007932746 -0.017187548637289052" rpy="0 0 0"/>
+    <origin xyz="-0.0116 0.06475 0.3325" rpy="-1.57 0  0"/>
+    <geometry>
+      <mesh filename="package://assembly_description/meshes/simplified/right_ankle_v2_1.dae" scale="0.001 0.001 0.001"/>
+    </geometry>
+  </collision>
+</link>
+<link name="right_foot">
+  <inertial>
+    <origin xyz="0.053123527163554944 -0.01311710007932746 -0.017187548637289052" rpy="-1.57 0  0"/>
     <mass value="0.03929273129474384"/>
     <inertia ixx="2.6e-05" iyy="0.000124" izz="0.000144" ixy="-2e-06" iyz="-2e-06" ixz="-3e-06"/>
   </inertial>
   <visual>
-    <origin xyz="0.0547 0.04125 0.3685" rpy="0 0 0"/>
-    <geometry>
-      <mesh filename="package://assembly_description/meshes/right_foot_v2_1.stl" scale="0.001 0.001 0.001"/>
+    <origin xyz="0.0547 0.04125 0.3685" rpy="-1.57 0  0"/>
+    <geometry>
+      <mesh filename="package://assembly_description/meshes/simplified/right_foot_v2_1.dae" scale="0.001 0.001 0.001"/>
     </geometry>
     <material name="abs_white"/>
   </visual>
   <collision>
-    <origin xyz="0.0547 0.04125 0.3685" rpy="0 0 0"/>
-    <geometry>
-      <mesh filename="package://assembly_description/meshes/right_foot_v2_1.stl" scale="0.001 0.001 0.001"/>
-    </geometry>
-  </collision>
-</link>
-<link name="right_shoulder_v1_1">
-  <inertial>
-    <origin xyz="8.958533047331851e-11 -0.007844026821937675 2.015054789694659e-14" rpy="0 0 0"/>
+    <origin xyz="0.0547 0.04125 0.3685" rpy="-1.57 0  0"/>
+    <geometry>
+      <mesh filename="package://assembly_description/meshes/simplified/right_foot_v2_1.dae" scale="0.001 0.001 0.001"/>
+    </geometry>
+  </collision>
+</link>
+<link name="right_shoulder">
+  <inertial>
+    <origin xyz="8.958533047331851e-11 -0.007844026821937675 2.015054789694659e-14" rpy="-1.57 0  0"/>
     <mass value="0.010592862408759271"/>
     <inertia ixx="1e-06" iyy="3e-06" izz="3e-06" ixy="0.0" iyz="0.0" ixz="-0.0"/>
   </inertial>
   <visual>
-    <origin xyz="-0.003 0.084 -0.04475" rpy="0 0 0"/>
-    <geometry>
-      <mesh filename="package://assembly_description/meshes/right_shoulder_v1_1.stl" scale="0.001 0.001 0.001"/>
-    </geometry>
-    <material name="aluminum_satin"/>
-  </visual>
-  <collision>
-    <origin xyz="-0.003 0.084 -0.04475" rpy="0 0 0"/>
-    <geometry>
-      <mesh filename="package://assembly_description/meshes/right_shoulder_v1_1.stl" scale="0.001 0.001 0.001"/>
-    </geometry>
-  </collision>
-</link>
-<link name="right_bicep_v2_1">
-  <inertial>
-    <origin xyz="-0.01907144993358056 -0.0012317079698353356 -0.06051458521988612" rpy="0 0 0"/>
+    <origin xyz="-0.003 0.084 -0.04475" rpy="-1.57 0  0"/>
+    <geometry>
+      <mesh filename="package://assembly_description/meshes/simplified/right_shoulder_v1_1.dae" scale="0.001 0.001 0.001"/>
+    </geometry>
+    <material name="aluminum_satin"/>
+  </visual>
+  <collision>
+    <origin xyz="-0.003 0.084 -0.04475" rpy="-1.57 0  0"/>
+    <geometry>
+      <mesh filename="package://assembly_description/meshes/simplified/right_shoulder_v1_1.dae" scale="0.001 0.001 0.001"/>
+    </geometry>
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