Commit message: Fix initial rotation + meshdir

File: soccer_description/hip-rejoint_description/urdf/hip-rejoint.xacro (robot description, xacro)
@@ -20,5 +20,5 @@
   -->
   <mujoco>
-    <compiler meshdir="/home/q2/catkin_ws/src/hip-rejoint_description/meshes" balanceinertia="true" discardvisual="false"/>
+    <compiler meshdir="../meshes" balanceinertia="true" discardvisual="false"/>
   </mujoco>
 <xacro:include filename="$(find hip-rejoint_description)/urdf/materials.xacro" />
@@ -1086,6 +1086,6 @@
   </collision>
 </link>
-<joint name="rootfloat" type="floating">
-  <origin xyz="0 0 0" rpy="0 0 0" />
+<joint name="rootfloat" type="fixed">
+  <origin xyz="0 0 0" rpy="1.57 0 1.57" />
   <parent link="root" />
   <child link="torso" />

Commit message: Rename head joints manually + add further steps
Needs upstream model fix for renaming revolute head joints in placo
standard

File: soccer_description/hip-rejoint_description/urdf/hip-rejoint.xacro (robot description, xacro)
@@ -7,4 +7,6 @@
     - Rename `base_link` to `trunk` in the URDF to accomodate placo
     - Rejoint `trunk` to a new root link with a `floating` joint in URDF (i.e. `<link name="root" /><joint name="root-float" type="floating"><child link="trunk" /><parent link="root" /></joint>`
+    - Fix servo masses based on enclosure (masses currently include all optional enclosures)
+    - Fix necessary placo names (left_foot, right_foot, trunk) which have `_1` or some other digit appended by Fusion unique ID system
     - Generate URDF from xacro via:
       - `conda activate py2; rosrun xacro xacro '/path/to/model.xacro' > '/path/to/model.urdf';`
@@ -1561,5 +1563,5 @@
   <child link="25t-servo-hub_1"/>
 </joint>
-<joint name="Revolute 62" type="continuous">
+<joint name="head_yaw" type="continuous">
   <origin xyz="0.0 0.0 0.002794" rpy="0 0 0"/>
   <parent link="25t-servo-hub_1"/>
@@ -1567,5 +1569,5 @@
   <axis xyz="-0.0 0.0 1.0"/>
 </joint>
-<joint name="Revolute 63" type="continuous">
+<joint name="head_pitch" type="continuous">
   <origin xyz="0.0 0.026187 0.033817" rpy="0 0 0"/>
   <parent link="neck_1"/>
