Commit message: Remodel robot to orient in world frame + add head
Fusion 360 model changes to accomodate placo

File: soccer_description/hip-rejoint_description/urdf/hip-rejoint.urdf (robot description, URDF)
Before this commit: robot hip-rejoint, 54 links, 53 joints
Links:
- removed link root
- removed link torso
- added link 25t-servo-hub_1, mass 0.005584850212079893; collision mesh filename=package://hip-rejoint_description/meshes/25t-servo-hub_1.stl scale=0.001 0.001 0.001; visual mesh filename=package://hip-rejoint_description/meshes/25t-servo-hub_1.stl scale=0.001 0.001 0.001
- added link 25t-servo-hub_2, mass 0.005584850212079893; collision mesh filename=package://hip-rejoint_description/meshes/25t-servo-hub_2.stl scale=0.001 0.001 0.001; visual mesh filename=package://hip-rejoint_description/meshes/25t-servo-hub_2.stl scale=0.001 0.001 0.001
- added link base_link, mass 0.00106; collision mesh filename=package://hip-rejoint_description/meshes/base_link.stl scale=0.001 0.001 0.001; visual mesh filename=package://hip-rejoint_description/meshes/base_link.stl scale=0.001 0.001 0.001
- added link camera_1, mass 0.094257141411043; collision mesh filename=package://hip-rejoint_description/meshes/camera_1.stl scale=0.001 0.001 0.001; visual mesh filename=package://hip-rejoint_description/meshes/camera_1.stl scale=0.001 0.001 0.001
- added link custom_servo_support__lower_neck__v2_1, mass 0.0030444171650099846; collision mesh filename=package://hip-rejoint_description/meshes/custom_servo_suppo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 scale=0.001 0.001 0.001; visual mesh filename=package://hip-rejoint_description/meshes/custom_servo_suppo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 scale=0.001 0.001 0.001
- added link gobilda-servo_1, mass 0.06058731126055281; collision mesh filename=package://hip-rejoint_description/meshes/gobilda-servo_1.stl scale=0.001 0.001 0.001; visual mesh filename=package://hip-rejoint_description/meshes/gobilda-servo_1.stl scale=0.001 0.001 0.001
- added link gobilda-servo_2, mass 0.06058731126055281; collision mesh filename=package://hip-rejoint_description/meshes/gobilda-servo_2.stl scale=0.001 0.001 0.001; visual mesh filename=package://hip-rejoint_description/meshes/gobilda-servo_2.stl scale=0.001 0.001 0.001
- added link head_1, mass 0.007653734054253099; collision mesh filename=package://hip-rejoint_description/meshes/head_1.stl scale=0.001 0.001 0.001; visual mesh filename=package://hip-rejoint_description/meshes/head_1.stl scale=0.001 0.001 0.001
- added link neck_1, mass 0.015465374363363156; collision mesh filename=package://hip-rejoint_description/meshes/neck_1.stl scale=0.001 0.001 0.001; visual mesh filename=package://hip-rejoint_description/meshes/neck_1.stl scale=0.001 0.001 0.001
- added link trunk, mass 0.19337373769234342; collision mesh filename=package://hip-rejoint_description/meshes/trunk_1.stl scale=0.001 0.001 0.001; visual mesh filename=package://hip-rejoint_description/meshes/trunk_1.stl scale=0.001 0.001 0.001
- link Component66_1: mass 0.3199209891539212 -> 0.3199209891539211
- link JX_servo_v46_Mirror__1: mass 0.2114 -> 0.5886686504488787
- link JX_servo_v46_Mirror__10: mass 0.2114 -> 0.5886686504488787
- link JX_servo_v46_Mirror__11: mass 0.2114 -> 0.5886686504488787
- link JX_servo_v46_Mirror__12: mass 0.2114 -> 0.5886686504488787
- link JX_servo_v46_Mirror__13: mass 0.2114 -> 0.5886686504488787
- link JX_servo_v46_Mirror__2: mass 0.2114 -> 0.5886686504488787
- link JX_servo_v46_Mirror__3: mass 0.2114 -> 0.5886686504488787
- link JX_servo_v46_Mirror__7: mass 0.2114 -> 0.5886686504488787
- link JX_servo_v46_Mirror__8: mass 0.2114 -> 0.5886686504488787
- link JX_servo_v46_Mirror__9: mass 0.2114 -> 0.5886686504488787
- link JX_servo_v80_1: mass 0.2114 -> 2.2370303189525207
- link JX_servo_v80_2: mass 0.379197 -> 2.2370303189525207
- link JX_servo_v80_3: mass 0.2114 -> 2.2370303189525207
- link JX_servo_v80_4: mass 0.2114 -> 2.2370303189525207
- link JX_servo_v80_5: mass 0.2114 -> 2.2370303189525207
- link JX_servo_v80_7: mass 0.379197 -> 2.2370303189525207
- link left_foot: geometry collision mesh filename=package://hip-rejoint_description/meshes/left_foot_1.stl scale=0.001 0.001 0.001; visual mesh filename=package://hip-rejoint_description/meshes/left_foot_1.stl scale=0.001 0.001 0.001
- link right_foot: geometry collision mesh filename=package://hip-rejoint_description/meshes/right_foot_1.stl scale=0.001 0.001 0.001; visual mesh filename=package://hip-rejoint_description/meshes/right_foot_1.stl scale=0.001 0.001 0.001
Joints:
- removed joint left_shoulder
- removed joint right_shoulder
- removed joint rootfloat
- added joint Revolute 62: type continuous, parent 25t-servo-hub_1, child neck_1, origin xyz=0.0 0.0 0.002794 rpy=0 0 0, axis -0.0 0.0 1.0
- added joint Revolute 63: type continuous, parent neck_1, child 25t-servo-hub_2, origin xyz=0.0 0.026187 0.033817 rpy=0 0 0, axis -0.0 1.0 -0.0
- added joint Rigid 58: type fixed, parent base_link, child trunk, origin xyz=0.0 0.005 0.005 rpy=0 0 0
- added joint Rigid 59: type fixed, parent Component65_1, child custom_servo_support__lower_neck__v2_1, origin xyz=-0.057 -0.0052 0.0 rpy=0 0 0
- added joint Rigid 60: type fixed, parent custom_servo_support__lower_neck__v2_1, child gobilda-servo_1, origin xyz=0.02015 0.0 0.00298 rpy=0 0 0
- added joint Rigid 61: type fixed, parent gobilda-servo_1, child 25t-servo-hub_1, origin xyz=-0.0113 0.0 0.04092 rpy=0 0 0
- added joint Rigid 64: type fixed, parent 25t-servo-hub_2, child gobilda-servo_2, origin xyz=0.0 -0.002794 0.0 rpy=0 0 0
- added joint Rigid 65: type fixed, parent gobilda-servo_2, child head_1, origin xyz=-0.0113 -0.04092 0.0 rpy=0 0 0
- added joint Rigid 66: type fixed, parent head_1, child camera_1, origin xyz=0.0133 0.01802 0.021 rpy=0 0 0
- added joint left_shoulder_pitch: type continuous, parent Component65_1, child JX_servo_v46_Mirror__12, origin xyz=0.00015 0.0964 -0.03175 rpy=0 0 0, axis -0.0 1.0 0.0
- added joint right_shoulder_pitch: type continuous, parent Component65_1, child JX_servo_v46_Mirror__10, origin xyz=0.00015 -0.1068 -0.03175 rpy=0 0 0, axis 0.0 -1.0 -0.0
- joint Rigid 10: origin xyz=0.0 -0.02225 0.0 rpy=0 0 0 -> xyz=0.0 0.0 -0.022251 rpy=0 0 0
- joint Rigid 11: origin xyz=0.0 -0.033375 0.0 rpy=0 0 0 -> xyz=0.0 0.0 -0.033376 rpy=0 0 0
- joint Rigid 12: origin xyz=-7.6e-05 -0.04215 -0.03165 rpy=0 0 0 -> xyz=-0.03165 -7.6e-05 -0.04215 rpy=0 0 0
- joint Rigid 15: origin xyz=0.00835 -0.0556 -0.0125 rpy=0 0 0 -> xyz=-0.0125 0.00835 -0.0556 rpy=0 0 0
- joint Rigid 16: origin xyz=0.0 -0.000635 0.0 rpy=0 0 0 -> xyz=0.0 0.0 -0.000635 rpy=0 0 0
- joint Rigid 17: origin xyz=0.0 -0.005312 0.0 rpy=0 0 0 -> xyz=0.0 0.0 -0.005312 rpy=0 0 0
- joint Rigid 18: origin xyz=0.0 0.014682 0.0 rpy=0 0 0 -> xyz=0.0 0.0 0.014681 rpy=0 0 0
- joint Rigid 19: origin xyz=0.0 0.0001 0.0 rpy=0 0 0 -> xyz=0.0 0.0 0.0001 rpy=0 0 0
- joint Rigid 2: origin xyz=-0.117785 -0.019449 -0.021094 rpy=0 0 0 -> xyz=-0.025 0.0542 0.004763 rpy=0 0 0; parent torso -> trunk
- joint Rigid 20: origin xyz=0.00435 0.0 0.048601 rpy=0 0 0 -> xyz=0.048601 0.00435 0.0 rpy=0 0 0
- joint Rigid 21: origin xyz=0.0 -0.033375 0.0 rpy=0 0 0 -> xyz=0.0 0.0 -0.033376 rpy=0 0 0
- joint Rigid 22: origin xyz=0.0 -0.000635 0.0 rpy=0 0 0 -> xyz=0.0 0.0 -0.000635 rpy=0 0 0
- joint Rigid 23: origin xyz=0.0 -0.005312 0.0 rpy=0 0 0 -> xyz=0.0 0.0 -0.005312 rpy=0 0 0
- joint Rigid 24: origin xyz=-7.6e-05 -0.04215 -0.03165 rpy=0 0 0 -> xyz=-0.03165 -7.6e-05 -0.04215 rpy=0 0 0
- joint Rigid 26: origin xyz=0.00435 0.0 0.065601 rpy=0 0 0 -> xyz=0.065601 0.00435 0.0 rpy=0 0 0
- joint Rigid 27: origin xyz=0.00835 -0.0556 -0.0125 rpy=0 0 0 -> xyz=-0.0125 0.00835 -0.0556 rpy=0 0 0
- joint Rigid 28: origin xyz=0.0 -0.02225 0.0 rpy=0 0 0 -> xyz=0.0 0.0 -0.022251 rpy=0 0 0
- joint Rigid 29: origin xyz=0.0 0.010955 0.0 rpy=0 0 0 -> xyz=0.0 0.0 0.010954 rpy=0 0 0
- joint Rigid 3: origin xyz=-0.117785 -0.019449 -0.021094 rpy=0 0 0 -> xyz=-0.025 0.0542 0.004763 rpy=0 0 0; parent torso -> trunk
- joint Rigid 31: origin xyz=0.0 0.014682 0.0 rpy=0 0 0 -> xyz=0.0 0.0 0.014681 rpy=0 0 0
- joint Rigid 32: origin xyz=0.0 0.0001 0.0 rpy=0 0 0 -> xyz=0.0 0.0 0.0001 rpy=0 0 0
- joint Rigid 35: origin xyz=-0.0217 -0.0556 -0.0085 rpy=0 0 0 -> xyz=-0.0085 -0.0217 -0.0556 rpy=0 0 0
- joint Rigid 37: origin xyz=-0.0217 0.0556 0.0085 rpy=0 0 0 -> xyz=0.0085 -0.0217 0.0556 rpy=0 0 0
- joint Rigid 38: origin xyz=-0.0065 -0.0001 -0.067 rpy=0 0 0 -> xyz=-0.067 -0.0065 -0.0001 rpy=0 0 0
- joint Rigid 4: origin xyz=-0.226185 -0.019449 -0.021094 rpy=0 0 0 -> xyz=-0.025 -0.0542 0.004762 rpy=0 0 0; parent torso -> trunk
- joint Rigid 44: origin xyz=0.0217 -0.0556 -0.0085 rpy=0 0 0 -> xyz=-0.0085 0.0217 -0.0556 rpy=0 0 0
- joint Rigid 46: origin xyz=0.0217 0.0556 0.0085 rpy=0 0 0 -> xyz=0.0085 0.0217 0.0556 rpy=0 0 0
- joint Rigid 47: origin xyz=0.0235 -0.0752 -0.067 rpy=0 0 0 -> xyz=-0.067 0.0235 -0.0752 rpy=0 0 0
- joint Rigid 5: origin xyz=0.0 0.0 0.0 rpy=0 0 0 -> xyz=0.0 0.0 1e-06 rpy=0 0 0
- joint Rigid 50: origin xyz=0.0594 0.0671 -0.01515 rpy=0 0 0 -> xyz=-0.01515 0.0594 0.0671 rpy=0 0 0
- joint Rigid 51: origin xyz=-0.0052 0.0 -0.11415 rpy=0 0 0 -> xyz=-0.11415 -0.0052 0.0 rpy=0 0 0
- joint Rigid 53: origin xyz=-0.0576 -0.0557 -0.0085 rpy=0 0 0 -> xyz=-0.0085 -0.0576 -0.0557 rpy=0 0 0
- joint Rigid 55: origin xyz=0.0576 -0.0557 -0.0085 rpy=0 0 0 -> xyz=-0.0085 0.0576 -0.0557 rpy=0 0 0
- joint Rigid 6: origin xyz=-0.117785 -0.019449 -0.021094 rpy=0 0 0 -> xyz=-0.025 0.0542 0.004763 rpy=0 0 0; parent torso -> trunk
- joint Rigid 7: origin xyz=-0.226185 -0.019449 -0.021094 rpy=0 0 0 -> xyz=-0.025 -0.0542 0.004762 rpy=0 0 0; parent torso -> trunk
- joint Rigid 8: origin xyz=0.0 0.010955 0.0 rpy=0 0 0 -> xyz=0.0 0.0 0.010956 rpy=0 0 0
- joint left_ankle_pitch: axis 1.0 -0.0 -0.0 -> -0.0 1.0 -0.0; origin xyz=0.0224 -0.0836 0.0085 rpy=0 0 0 -> xyz=0.0085 0.0224 -0.0836 rpy=0 0 0
- joint left_ankle_roll: axis 0.0 -0.0 1.0 -> 1.0 0.0 -0.0; origin xyz=-0.0085 -0.0556 0.0256 rpy=0 0 0 -> xyz=0.0256 -0.0085 -0.0556 rpy=0 0 0
- joint left_elbow: axis 1.0 0.0 -0.0 -> -0.0 1.0 0.0; origin xyz=0.0217 -0.0556 0.0085 rpy=0 0 0 -> xyz=0.0085 0.0217 -0.0556 rpy=0 0 0
- joint left_hip_pitch: axis -1.0 0.0 -0.0 -> -0.0 -1.0 0.0; origin xyz=0.032475 0.0556 -0.00865 rpy=0 0 0 -> xyz=-0.00865 0.032475 0.0556 rpy=0 0 0
- joint left_hip_roll: axis 0.0 0.0 1.0 -> 1.0 0.0 0.0; origin xyz=0.0 0.0 -0.0127 rpy=0 0 0 -> xyz=-0.0127 0.0 0.0 rpy=0 0 0
- joint left_hip_yaw: axis -0.0 -1.0 0.0 -> 0.0 0.0 -1.0; origin xyz=0.0 0.000635 0.0 rpy=0 0 0 -> xyz=0.0 0.0 0.000636 rpy=0 0 0
- joint left_knee: axis 1.0 -0.0 -0.0 -> -0.0 1.0 -0.0; origin xyz=0.0 -0.16 0.0 rpy=0 0 0 -> xyz=0.0 0.0 -0.16 rpy=0 0 0
- joint right_ankle_pitch: axis 1.0 -0.0 -0.0 -> -0.0 1.0 -0.0; origin xyz=-0.0224 -0.0836 0.0085 rpy=0 0 0 -> xyz=0.0085 -0.0224 -0.0836 rpy=0 0 0
- joint right_ankle_roll: axis 0.0 -0.0 1.0 -> 1.0 0.0 -0.0; origin xyz=-0.0085 0.0196 0.0256 rpy=0 0 0 -> xyz=0.0256 -0.0085 0.0196 rpy=0 0 0
- joint right_elbow: axis -1.0 0.0 0.0 -> 0.0 -1.0 0.0; origin xyz=-0.0217 -0.0556 0.0085 rpy=0 0 0 -> xyz=0.0085 -0.0217 -0.0556 rpy=0 0 0
- joint right_hip_pitch: axis 1.0 -0.0 0.0 -> 0.0 1.0 -0.0; origin xyz=-0.057875 0.0556 0.00865 rpy=0 0 0 -> xyz=0.00865 -0.057875 0.0556 rpy=0 0 0
- joint right_hip_roll: axis 0.0 0.0 1.0 -> 1.0 0.0 0.0; origin xyz=0.0 0.0 -0.0127 rpy=0 0 0 -> xyz=-0.0127 0.0 0.0 rpy=0 0 0
- joint right_hip_yaw: axis -0.0 -1.0 0.0 -> 0.0 0.0 -1.0; origin xyz=0.0 0.000635 0.0 rpy=0 0 0 -> xyz=0.0 0.0 0.000635 rpy=0 0 0
- joint right_knee: axis 1.0 -0.0 0.0 -> 0.0 1.0 -0.0; origin xyz=0.0 -0.16 0.0 rpy=0 0 0 -> xyz=0.0 0.0 -0.16 rpy=0 0 0
