Commit message: Remodel robot to orient in world frame + add head
Fusion 360 model changes to accomodate placo

File: soccer_description/hip-rejoint_description/urdf/hip-rejoint.xacro (robot description, xacro)
@@ -4,9 +4,9 @@
     Steps to generate model:
     - Joint and export in Fusion
+    - Fix inertias in the URDF with `%s/i\(\w\)\1="\-*0.0"/i\1\1="1E-06"/g`
+    - Rename `base_link` to `trunk` in the URDF to accomodate placo
+    - Rejoint `trunk` to a new root link with a `floating` joint in URDF (i.e. `<link name="root" /><joint name="root-float" type="floating"><child link="trunk" /><parent link="root" /></joint>`
     - Generate URDF from xacro via:
       - `conda activate py2; rosrun xacro xacro '/path/to/model.xacro' > '/path/to/model.urdf';`
-    - Fix inertias in the URDF with `%s/i\(\w\)\1="\-*0.0"/i\1\1="1E-06"/g`
-    - Rename `base_link` to `torso` in the URDF to accomodate placo
-    - Rejoint `torso` to a new root link with a `floating` joint in URDF (i.e. `<link name="root" /><joint name="root-float" type="floating"><child link="torso" /><parent link="root" /></joint>`
     - Import to mujoco and save as XML
     - Ensure left and right foot links exist
@@ -25,10 +25,9 @@
 <xacro:include filename="$(find hip-rejoint_description)/urdf/hip-rejoint.trans" />
 <xacro:include filename="$(find hip-rejoint_description)/urdf/hip-rejoint.gazebo" />
-<link name="root" />
-<link name="torso">
-  <inertial>
-    <origin xyz="-0.17198470578696426 -0.024251867789563585 -0.021093953275271887" rpy="0 0 0"/>
-    <mass value="0.19337373769234342"/>
-    <inertia ixx="4.6e-05" iyy="0.000538" izz="0.000494" ixy="0.0" iyz="-0.0" ixz="0.0"/>
+<link name="base_link">
+  <inertial>
+    <origin xyz="0.005 0.005 0.005" rpy="0 0 0"/>
+    <mass value="0.00106"/>
+    <inertia ixx="1E-06" iyy="1E-06" izz="1E-06" ixy="0.0" iyz="0.0" ixz="0.0"/>
   </inertial>
   <visual>
@@ -37,5 +36,5 @@
       <mesh filename="package://hip-rejoint_description/meshes/base_link.stl" scale="0.001 0.001 0.001"/>
     </geometry>
-    <material name="acrylic_red"/>
+    <material name="abs_white"/>
   </visual>
   <collision>
@@ -48,10 +47,10 @@
 <link name="R8-2RS_Bearing_1">
   <inertial>
-    <origin xyz="2.942129484623246e-07 -0.003968361583188348 4.67247281074612e-08" rpy="0 0 0"/>
+    <origin xyz="4.85722573273506e-17 1.6393830737371218e-13 -0.003969249999999997" rpy="0 0 0"/>
     <mass value="0.03206594861680248"/>
-    <inertia ixx="2e-06" iyy="4e-06" izz="2e-06" ixy="-0.0" iyz="-0.0" ixz="0.0"/>
-  </inertial>
-  <visual>
-    <origin xyz="0.117785 0.019449 0.021094" rpy="0 0 0"/>
+    <inertia ixx="2e-06" iyy="2e-06" izz="4e-06" ixy="-0.0" iyz="-0.0" ixz="-0.0"/>
+  </inertial>
+  <visual>
+    <origin xyz="0.025 -0.0592 -0.009763" rpy="0 0 0"/>
     <geometry>
       <mesh filename="package://hip-rejoint_description/meshes/R8-2RS_Bearing_1.stl" scale="0.001 0.001 0.001"/>
@@ -60,5 +59,5 @@
   </visual>
   <collision>
-    <origin xyz="0.117785 0.019449 0.021094" rpy="0 0 0"/>
+    <origin xyz="0.025 -0.0592 -0.009763" rpy="0 0 0"/>
     <geometry>
       <mesh filename="package://hip-rejoint_description/meshes/R8-2RS_Bearing_1.stl" scale="0.001 0.001 0.001"/>
@@ -68,10 +67,10 @@
 <link name="R8-2RS_Bearing_2">
   <inertial>
-    <origin xyz="2.9421294850395796e-07 0.003969138416811653 4.672472811093065e-08" rpy="0 0 0"/>
+    <origin xyz="5.551115123125783e-17 1.6397300184323171e-13 0.003968250000000005" rpy="0 0 0"/>
     <mass value="0.03206594861680248"/>
-    <inertia ixx="2e-06" iyy="4e-06" izz="2e-06" ixy="-0.0" iyz="0.0" ixz="-0.0"/>
-  </inertial>
-  <visual>
-    <origin xyz="0.117785 0.019449 0.021094" rpy="0 0 0"/>
+    <inertia ixx="2e-06" iyy="2e-06" izz="4e-06" ixy="0.0" iyz="-0.0" ixz="0.0"/>
+  </inertial>
+  <visual>
+    <origin xyz="0.025 -0.0592 -0.009763" rpy="0 0 0"/>
     <geometry>
       <mesh filename="package://hip-rejoint_description/meshes/R8-2RS_Bearing_2.stl" scale="0.001 0.001 0.001"/>
@@ -80,5 +79,5 @@
   </visual>
   <collision>
-    <origin xyz="0.117785 0.019449 0.021094" rpy="0 0 0"/>
+    <origin xyz="0.025 -0.0592 -0.009763" rpy="0 0 0"/>
     <geometry>
       <mesh filename="package://hip-rejoint_description/meshes/R8-2RS_Bearing_2.stl" scale="0.001 0.001 0.001"/>
@@ -88,10 +87,10 @@
 <link name="R8-2RS_Bearing_3">
   <inertial>
-    <origin xyz="2.9421294739373494e-07 -0.0039683615831883345 4.6724728045011155e-08" rpy="0 0 0"/>
+    <origin xyz="-3.469446951953614e-18 1.6287665660641437e-13 -0.003968249999999989" rpy="0 0 0"/>
     <mass value="0.03206594861680248"/>
-    <inertia ixx="2e-06" iyy="4e-06" izz="2e-06" ixy="0.0" iyz="-0.0" ixz="0.0"/>
-  </inertial>
-  <visual>
-    <origin xyz="0.226185 0.019449 0.021094" rpy="0 0 0"/>
+    <inertia ixx="2e-06" iyy="2e-06" izz="4e-06" ixy="0.0" iyz="0.0" ixz="-0.0"/>
+  </inertial>
+  <visual>
+    <origin xyz="0.025 0.0492 -0.009762" rpy="0 0 0"/>
     <geometry>
       <mesh filename="package://hip-rejoint_description/meshes/R8-2RS_Bearing_3.stl" scale="0.001 0.001 0.001"/>
@@ -100,5 +99,5 @@
   </visual>
   <collision>
-    <origin xyz="0.226185 0.019449 0.021094" rpy="0 0 0"/>
+    <origin xyz="0.025 0.0492 -0.009762" rpy="0 0 0"/>
     <geometry>
       <mesh filename="package://hip-rejoint_description/meshes/R8-2RS_Bearing_3.stl" scale="0.001 0.001 0.001"/>
@@ -108,10 +107,10 @@
 <link name="R8-2RS_Bearing_4">
   <inertial>
-    <origin xyz="2.9421294750475724e-07 0.003969138416811662 4.6724728045011155e-08" rpy="0 0 0"/>
+    <origin xyz="-3.469446951953614e-18 1.6298074001497298e-13 0.00396825000000001" rpy="0 0 0"/>
     <mass value="0.03206594861680248"/>
-    <inertia ixx="2e-06" iyy="4e-06" izz="2e-06" ixy="0.0" iyz="-0.0" ixz="0.0"/>
-  </inertial>
-  <visual>
-    <origin xyz="0.226185 0.019449 0.021094" rpy="0 0 0"/>
+    <inertia ixx="2e-06" iyy="2e-06" izz="4e-06" ixy="0.0" iyz="-0.0" ixz="-0.0"/>
+  </inertial>
+  <visual>
+    <origin xyz="0.025 0.0492 -0.009763" rpy="0 0 0"/>
     <geometry>
       <mesh filename="package://hip-rejoint_description/meshes/R8-2RS_Bearing_4.stl" scale="0.001 0.001 0.001"/>
@@ -120,5 +119,5 @@
   </visual>
   <collision>
-    <origin xyz="0.226185 0.019449 0.021094" rpy="0 0 0"/>
+    <origin xyz="0.025 0.0492 -0.009763" rpy="0 0 0"/>
     <geometry>
       <mesh filename="package://hip-rejoint_description/meshes/R8-2RS_Bearing_4.stl" scale="0.001 0.001 0.001"/>
@@ -128,10 +127,10 @@
 <link name="Component2_2">
   <inertial>
-    <origin xyz="2.942126966776204e-07 0.006598864666209372 4.672472816297235e-08" rpy="0 0 0"/>
+    <origin xyz="9.020562075079397e-17 -8.781170235394598e-14 0.006597976249397723" rpy="0 0 0"/>
     <mass value="0.043046314847355716"/>
-    <inertia ixx="9e-06" iyy="1.6e-05" izz="9e-06" ixy="0.0" iyz="0.0" ixz="0.0"/>
-  </inertial>
-  <visual>
-    <origin xyz="0.117785 0.019449 0.021094" rpy="0 0 0"/>
+    <inertia ixx="9e-06" iyy="9e-06" izz="1.6e-05" ixy="0.0" iyz="0.0" ixz="0.0"/>
+  </inertial>
+  <visual>
+    <origin xyz="0.025 -0.0592 -0.009763" rpy="0 0 0"/>
     <geometry>
       <mesh filename="package://hip-rejoint_description/meshes/Component2_2.stl" scale="0.001 0.001 0.001"/>
@@ -140,5 +139,5 @@
   </visual>
   <collision>
-    <origin xyz="0.117785 0.019449 0.021094" rpy="0 0 0"/>
+    <origin xyz="0.025 -0.0592 -0.009763" rpy="0 0 0"/>
     <geometry>
       <mesh filename="package://hip-rejoint_description/meshes/Component2_2.stl" scale="0.001 0.001 0.001"/>
@@ -148,10 +147,10 @@
 <link name="Component2_1">
   <inertial>
-    <origin xyz="2.9421269573393083e-07 0.006598864666209387 4.672472808317507e-08" rpy="0 0 0"/>
+    <origin xyz="2.0816681711721685e-17 -8.87900863943969e-14 0.0065989762493977346" rpy="0 0 0"/>
     <mass value="0.043046314847355716"/>
-    <inertia ixx="9e-06" iyy="1.6e-05" izz="9e-06" ixy="0.0" iyz="0.0" ixz="0.0"/>
-  </inertial>
-  <visual>
-    <origin xyz="0.226185 0.019449 0.021094" rpy="0 0 0"/>
+    <inertia ixx="9e-06" iyy="9e-06" izz="1.6e-05" ixy="0.0" iyz="0.0" ixz="0.0"/>
+  </inertial>
+  <visual>
+    <origin xyz="0.025 0.0492 -0.009762" rpy="0 0 0"/>
     <geometry>
       <mesh filename="package://hip-rejoint_description/meshes/Component2_1.stl" scale="0.001 0.001 0.001"/>
@@ -160,5 +159,5 @@
   </visual>
   <collision>
-    <origin xyz="0.226185 0.019449 0.021094" rpy="0 0 0"/>
+    <origin xyz="0.025 0.0492 -0.009762" rpy="0 0 0"/>
     <geometry>
       <mesh filename="package://hip-rejoint_description/meshes/Component2_1.stl" scale="0.001 0.001 0.001"/>
@@ -168,10 +167,10 @@
 <link name="91590A121_External_Retaining_Ring_v1_2">
   <inertial>
-    <origin xyz="0.00028649178236625494 0.0003178884168116656 4.6724729946268084e-08" rpy="0 0 0"/>
+    <origin xyz="1.8943180357666733e-15 0.000286197569581724 0.0003170000000000117" rpy="0 0 0"/>
     <mass value="0.00024760918611349786"/>
-    <inertia ixx="1E-06" iyy="1E-06" izz="1E-06" ixy="-0.0" iyz="-0.0" ixz="0.0"/>
-  </inertial>
-  <visual>
-    <origin xyz="0.226185 0.008494 0.021094" rpy="0 0 0"/>
+    <inertia ixx="1E-06" iyy="1E-06" izz="1E-06" ixy="0.0" iyz="0.0" ixz="-0.0"/>
+  </inertial>
+  <visual>
+    <origin xyz="0.025 0.0492 -0.020718" rpy="0 0 0"/>
     <geometry>
       <mesh filename="package://hip-rejoint_description/meshes/91590A121_External_Retaining_Ring_v1_2.stl" scale="0.001 0.001 0.001"/>
@@ -180,5 +179,5 @@
   </visual>
   <collision>
-    <origin xyz="0.226185 0.008494 0.021094" rpy="0 0 0"/>
+    <origin xyz="0.025 0.0492 -0.020718" rpy="0 0 0"/>
     <geometry>
       <mesh filename="package://hip-rejoint_description/meshes/91590A121_External_Retaining_Ring_v1_2.stl" scale="0.001 0.001 0.001"/>
@@ -188,10 +187,10 @@
 <link name="2025K9_303_Stainless_Steel_Rotary_Shaft_with_Retaining_Ring_Grooves_v1_1">
   <inertial>
-    <origin xyz="2.9421339503565846e-07 -0.02344973289915206 4.672469118213729e-08" rpy="0 0 0"/>
+    <origin xyz="-3.686981275841106e-14 6.104977634535658e-13 -0.023450621315963708" rpy="0 0 0"/>
     <mass value="0.07269824555688346"/>
-    <inertia ixx="3.6e-05" iyy="1e-06" izz="3.6e-05" ixy="0.0" iyz="0.0" ixz="-0.0"/>
-  </inertial>
-  <visual>
-    <origin xyz="0.226185 0.007859 0.021094" rpy="0 0 0"/>
+    <inertia ixx="3.6e-05" iyy="3.6e-05" izz="1e-06" ixy="-0.0" iyz="0.0" ixz="0.0"/>
+  </inertial>
+  <visual>
+    <origin xyz="0.025 0.0492 -0.021353" rpy="0 0 0"/>
     <geometry>
       <mesh filename="package://hip-rejoint_description/meshes/2025K9_303_Stainless_Steel_Rotary_Shaft_with_Retaining_Ring_Grooves_v1_1.stl" scale="0.001 0.001 0.001"/>
@@ -200,5 +199,5 @@
   </visual>
   <collision>
-    <origin xyz="0.226185 0.007859 0.021094" rpy="0 0 0"/>
+    <origin xyz="0.025 0.0492 -0.021353" rpy="0 0 0"/>
     <geometry>
       <mesh filename="package://hip-rejoint_description/meshes/2025K9_303_Stainless_Steel_Rotary_Shaft_with_Retaining_Ring_Grooves_v1_1.stl" scale="0.001 0.001 0.001"/>
@@ -208,1162 +207,1384 @@
 <link name="91590A121_External_Retaining_Ring_v1_3">
   <inertial>
-    <origin xyz="-0.0002859033567979563 0.00031748841681164194 4.672472619232648e-08" rpy="0 0 0"/>
+    <origin xyz="-1.8561541192951836e-15 -0.00028619756958252196 0.00031759999999999026" rpy="0 0 0"/>
+    <mass value="0.00024760918611349786"/>
+    <inertia ixx="1E-06" iyy="1E-06" izz="1E-06" ixy="0.0" iyz="-0.0" ixz="-0.0"/>
+  </inertial>
+  <visual>
+    <origin xyz="0.025 0.0492 0.000898" rpy="0 0 0"/>
+    <geometry>
+      <mesh filename="package://hip-rejoint_description/meshes/91590A121_External_Retaining_Ring_v1_3.stl" scale="0.001 0.001 0.001"/>
+    </geometry>
+    <material name="steel_satin"/>
+  </visual>
+  <collision>
+    <origin xyz="0.025 0.0492 0.000898" rpy="0 0 0"/>
+    <geometry>
+      <mesh filename="package://hip-rejoint_description/meshes/91590A121_External_Retaining_Ring_v1_3.stl" scale="0.001 0.001 0.001"/>
+    </geometry>
+  </collision>
+</link>
+<link name="91590A121_External_Retaining_Ring_v1_1">
+  <inertial>
+    <origin xyz="-1.8561541192951836e-15 -0.000286197569582515 -0.0003176000000000255" rpy="0 0 0"/>
     <mass value="0.00024760918611349786"/>
     <inertia ixx="1E-06" iyy="1E-06" izz="1E-06" ixy="0.0" iyz="0.0" ixz="0.0"/>
   </inertial>
   <visual>
-    <origin xyz="0.226185 0.030109 0.021094" rpy="0 0 0"/>
-    <geometry>
-      <mesh filename="package://hip-rejoint_description/meshes/91590A121_External_Retaining_Ring_v1_3.stl" scale="0.001 0.001 0.001"/>
+    <origin xyz="0.025 0.0492 0.012023" rpy="0 0 0"/>
+    <geometry>
+      <mesh filename="package://hip-rejoint_description/meshes/91590A121_External_Retaining_Ring_v1_1.stl" scale="0.001 0.001 0.001"/>
     </geometry>
     <material name="steel_satin"/>
   </visual>
   <collision>
-    <origin xyz="0.226185 0.030109 0.021094" rpy="0 0 0"/>
-    <geometry>
-      <mesh filename="package://hip-rejoint_description/meshes/91590A121_External_Retaining_Ring_v1_3.stl" scale="0.001 0.001 0.001"/>
-    </geometry>
-  </collision>
-</link>
-<link name="91590A121_External_Retaining_Ring_v1_1">
-  <inertial>
-    <origin xyz="-0.0002859033567979563 -0.00031771158318838477 4.672472619232648e-08" rpy="0 0 0"/>
+    <origin xyz="0.025 0.0492 0.012023" rpy="0 0 0"/>
+    <geometry>
+      <mesh filename="package://hip-rejoint_description/meshes/91590A121_External_Retaining_Ring_v1_1.stl" scale="0.001 0.001 0.001"/>
+    </geometry>
+  </collision>
+</link>
+<link name="Component39_1">
+  <inertial>
+    <origin xyz="-0.004453658050594535 1.0708659631264439e-07 0.007256502814372477" rpy="0 0 0"/>
+    <mass value="0.015364690334044086"/>
+    <inertia ixx="2e-06" iyy="1e-06" izz="1e-06" ixy="-0.0" iyz="0.0" ixz="-0.0"/>
+  </inertial>
+  <visual>
+    <origin xyz="0.05665 0.049276 0.06012" rpy="0 0 0"/>
+    <geometry>
+      <mesh filename="package://hip-rejoint_description/meshes/Component39_1.stl" scale="0.001 0.001 0.001"/>
+    </geometry>
+    <material name="aluminum_satin"/>
+  </visual>
+  <collision>
+    <origin xyz="0.05665 0.049276 0.06012" rpy="0 0 0"/>
+    <geometry>
+      <mesh filename="package://hip-rejoint_description/meshes/Component39_1.stl" scale="0.001 0.001 0.001"/>
+    </geometry>
+  </collision>
+</link>
+<link name="JX_servo_v80_3">
+  <inertial>
+    <mass value="0.2114"/>
+    <origin xyz="-0.03281072928697727 -0.00014307061349972533 -0.016670466018917744" rpy="0 0 0"/>
+    <inertia ixx="0.001692" iyy="0.001903" izz="0.001012" ixy="-1e-06" iyz="-0.0" ixz="-4.9e-05"/>
+  </inertial>
+  <visual>
+    <origin xyz="0.06935 0.049276 0.06012" rpy="0 0 0"/>
+    <geometry>
+      <mesh filename="package://hip-rejoint_description/meshes/JX_servo_v80_3.stl" scale="0.001 0.001 0.001"/>
+    </geometry>
+    <material name="polystyrene"/>
+  </visual>
+  <collision>
+    <origin xyz="0.06935 0.049276 0.06012" rpy="0 0 0"/>
+    <geometry>
+      <mesh filename="package://hip-rejoint_description/meshes/JX_servo_v80_3.stl" scale="0.001 0.001 0.001"/>
+    </geometry>
+  </collision>
+</link>
+<link name="Component9__1__1">
+  <inertial>
+    <origin xyz="0.03333629681388652 -0.008439001260076934 -0.00027616991746298725" rpy="0 0 0"/>
+    <mass value="0.13759034791983457"/>
+    <inertia ixx="1e-05" iyy="5.4e-05" izz="6.2e-05" ixy="-0.0" iyz="0.0" ixz="0.0"/>
+  </inertial>
+  <visual>
+    <origin xyz="0.08185 0.040926 0.11572" rpy="0 0 0"/>
+    <geometry>
+      <mesh filename="package://hip-rejoint_description/meshes/Component9__1__1.stl" scale="0.001 0.001 0.001"/>
+    </geometry>
+    <material name="steel_satin"/>
+  </visual>
+  <collision>
+    <origin xyz="0.08185 0.040926 0.11572" rpy="0 0 0"/>
+    <geometry>
+      <mesh filename="package://hip-rejoint_description/meshes/Component9__1__1.stl" scale="0.001 0.001 0.001"/>
+    </geometry>
+  </collision>
+</link>
+<link name="Component4_1">
+  <inertial>
+    <origin xyz="4.5102810375396984e-17 -2.0160956237802452e-13 -0.0027446731476930067" rpy="0 0 0"/>
+    <mass value="0.011955695388392617"/>
+    <inertia ixx="1e-06" iyy="1e-06" izz="2e-06" ixy="0.0" iyz="0.0" ixz="0.0"/>
+  </inertial>
+  <visual>
+    <origin xyz="0.025 0.0492 0.012658" rpy="0 0 0"/>
+    <geometry>
+      <mesh filename="package://hip-rejoint_description/meshes/Component4_1.stl" scale="0.001 0.001 0.001"/>
+    </geometry>
+    <material name="aluminum_satin"/>
+  </visual>
+  <collision>
+    <origin xyz="0.025 0.0492 0.012658" rpy="0 0 0"/>
+    <geometry>
+      <mesh filename="package://hip-rejoint_description/meshes/Component4_1.stl" scale="0.001 0.001 0.001"/>
+    </geometry>
+  </collision>
+</link>
+<link name="Component32_1">
+  <inertial>
+    <origin xyz="0.0004621398104596615 -7.798356568446824e-05 -0.016749694753477054" rpy="0 0 0"/>
+    <mass value="0.11550269835963742"/>
+    <inertia ixx="4.9e-05" iyy="9.9e-05" izz="9.4e-05" ixy="-0.0" iyz="0.0" ixz="-0.0"/>
+  </inertial>
+  <visual>
+    <origin xyz="0.025 0.0492 0.01797" rpy="0 0 0"/>
+    <geometry>
+      <mesh filename="package://hip-rejoint_description/meshes/Component32_1.stl" scale="0.001 0.001 0.001"/>
+    </geometry>
+    <material name="aluminum_satin"/>
+  </visual>
+  <collision>
+    <origin xyz="0.025 0.0492 0.01797" rpy="0 0 0"/>
+    <geometry>
+      <mesh filename="package://hip-rejoint_description/meshes/Component32_1.stl" scale="0.001 0.001 0.001"/>
+    </geometry>
+  </collision>
+</link>
+<link name="15T-horn_v13_1">
+  <inertial>
+    <origin xyz="2.0469737016526324e-16 6.415796262119328e-05 -0.00120040750659281" rpy="0 0 0"/>
+    <mass value="0.004179712167666874"/>
+    <inertia ixx="1E-06" iyy="1E-06" izz="1E-06" ixy="-0.0" iyz="0.0" ixz="-0.0"/>
+  </inertial>
+  <visual>
+    <origin xyz="0.025 0.0492 -0.036034" rpy="0 0 0"/>
+    <geometry>
+      <mesh filename="package://hip-rejoint_description/meshes/15T-horn_v13_1.stl" scale="0.001 0.001 0.001"/>
+    </geometry>
+    <material name="aluminum_satin"/>
+  </visual>
+  <collision>
+    <origin xyz="0.025 0.0492 -0.036034" rpy="0 0 0"/>
+    <geometry>
+      <mesh filename="package://hip-rejoint_description/meshes/15T-horn_v13_1.stl" scale="0.001 0.001 0.001"/>
+    </geometry>
+  </collision>
+</link>
+<link name="JX_servo_v80_1">
+  <inertial>
+    <origin xyz="-0.0001431777001134303 0.01667036601891729 0.039010829286977536" rpy="0 0 0"/>
+    <mass value="0.2114"/>
+    <inertia ixx="0.001903" iyy="0.001012" izz="0.001692" ixy="0.0" iyz="-4.9e-05" ixz="1e-06"/>
+  </inertial>
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
File: soccer_description/hip-rejoint_description/urdf/materials.xacro (robot description, xacro)
@@ -25,3 +25,9 @@
   <color rgba="0.09803921568627451 0.09803921568627451 0.09803921568627451 1.0"/>
 </material>
+<material name="plastic_glossy_black">
+  <color rgba="0.09803921568627451 0.09803921568627451 0.09803921568627451 1.0"/>
+</material>
+<material name="plastic_glossy_grey">
+  <color rgba="0.2901960784313726 0.2901960784313726 0.2901960784313726 1.0"/>
+</material>
 </robot>

Commit message: Run xacro

File: soccer_description/hip-rejoint_description/urdf/hip-rejoint.urdf (robot description, URDF)
Before this commit: robot hip-rejoint, 62 links, 61 joints
Links:
- link JX_servo_v46_Mirror__1: mass 0.5886686504488787 -> 0.2114
- link JX_servo_v46_Mirror__10: mass 0.5886686504488787 -> 0.2114
- link JX_servo_v46_Mirror__11: mass 0.5886686504488787 -> 0.2114
- link JX_servo_v46_Mirror__12: mass 0.5886686504488787 -> 0.2114
- link JX_servo_v46_Mirror__13: mass 0.5886686504488787 -> 0.2114
- link JX_servo_v46_Mirror__2: mass 0.5886686504488787 -> 0.2114
- link JX_servo_v46_Mirror__3: mass 0.5886686504488787 -> 0.2114
- link JX_servo_v46_Mirror__7: mass 0.5886686504488787 -> 0.2114
- link JX_servo_v46_Mirror__8: mass 0.5886686504488787 -> 0.2114
- link JX_servo_v46_Mirror__9: mass 0.5886686504488787 -> 0.2114
- link JX_servo_v80_1: mass 2.2370303189525207 -> 0.2114
- link JX_servo_v80_2: mass 2.2370303189525207 -> 0.379197
- link JX_servo_v80_3: mass 2.2370303189525207 -> 0.2114
- link JX_servo_v80_4: mass 2.2370303189525207 -> 0.2114
- link JX_servo_v80_5: mass 2.2370303189525207 -> 0.2114
- link JX_servo_v80_7: mass 2.2370303189525207 -> 0.379197
Joints:
- removed joint Revolute 62
- removed joint Revolute 63
- added joint head_pitch: type continuous, parent neck_1, child 25t-servo-hub_2, origin xyz=0.0 0.026187 0.033817 rpy=0 0 0, axis -0.0 1.0 -0.0
- added joint head_yaw: type continuous, parent 25t-servo-hub_1, child neck_1, origin xyz=0.0 0.0 0.002794 rpy=0 0 0, axis -0.0 0.0 1.0
